File: raspbery-pi-headers-support.sch (KiCad schematic (older format))
At the start: 15 parts, among them J1 RasPi-CM3-Headers, J10 Micro_SD_Card, J11 HDMI-A-connector, U31 DMG1012T, U32 DMG1012T, U33 ESD7484, U34 ESD7484, U35 ESD5384, U36 AP2331X

Commit message: Finished first pass on power distro, annotated USB C controllers
Parts:
- renumbered C211 to C?, C212 to C?, C214 to C?, C213 to C?, J1 to J?, J10 to J?, J11 to J?, R124 to R?, R123 to R?, U35 to U?, U34 to U?, U33 to U?, U31 to U?, U36 to U?, U32 to U?
Changed lines of the file:
@@
 $EndDescr
 $Comp
-L RasPi-CM3-Headers J1
+L RasPi-CM3-Headers J?
 U 2 1 58ECDA7F
 P 1650 6000
-F 0 "J1" H 1350 5550 60  0000 C CNN
+F 0 "J?" H 1350 5550 60  0000 C CNN
 F 1 "RasPi-CM3-Headers" V 2250 6000 60  0000 C CNN
 F 2 "Sockets:Socket_SODIMM_DDR1-2_TE_1612618" H 1700 11100 60  0001 C CNN
@@
 $EndComp
 $Comp
-L RasPi-CM3-Headers J1
+L RasPi-CM3-Headers J?
 U 3 1 58ECDAC0
 P 9900 5250
-F 0 "J1" H 9700 4900 60  0000 C CNN
+F 0 "J?" H 9700 4900 60  0000 C CNN
 F 1 "RasPi-CM3-Headers" V 10200 5250 60  0000 C CNN
 F 2 "Sockets:Socket_SODIMM_DDR1-2_TE_1612618" H 9950 10350 60  0001 C CNN
@@
 $EndComp
 $Comp
-L RasPi-CM3-Headers J1
+L RasPi-CM3-Headers J?
 U 4 1 58ECDAF6
 P 9850 3300
-F 0 "J1" H 9750 2750 60  0000 C CNN
+F 0 "J?" H 9750 2750 60  0000 C CNN
 F 1 "RasPi-CM3-Headers" V 10150 3300 60  0000 C CNN
 F 2 "Sockets:Socket_SODIMM_DDR1-2_TE_1612618" H 9900 8400 60  0001 C CNN
@@
 $EndComp
 $Comp
-L RasPi-CM3-Headers J1
+L RasPi-CM3-Headers J?
 U 10 1 58ECDB2D
 P 10700 3300
-F 0 "J1" H 10600 2750 60  0000 C CNN
+F 0 "J?" H 10600 2750 60  0000 C CNN
 F 1 "RasPi-CM3-Headers" V 11000 3300 60  0000 C CNN
 F 2 "Sockets:Socket_SODIMM_DDR1-2_TE_1612618" H 10750 8400 60  0001 C CNN
@@
 $EndComp
 $Comp
-L RasPi-CM3-Headers J1
+L RasPi-CM3-Headers J?
 U 11 1 58ECDB78
 P 10700 5250
-F 0 "J1" H 10550 4900 60  0000 C CNN
+F 0 "J?" H 10550 4900 60  0000 C CNN
 F 1 "RasPi-CM3-Headers" V 11000 5250 60  0000 C CNN
 F 2 "Sockets:Socket_SODIMM_DDR1-2_TE_1612618" H 10750 10350 60  0001 C CNN
@@
 $EndComp
 $Comp
-L RasPi-CM3-Headers J1
+L RasPi-CM3-Headers J?
 U 12 1 58ECDBAE
 P 2100 2950
-F 0 "J1" H 1950 2250 60  0000 C CNN
+F 0 "J?" H 1950 2250 60  0000 C CNN
 F 1 "RasPi-CM3-Headers" V 2600 2950 60  0000 C CNN
 F 2 "Sockets:Socket_SODIMM_DDR1-2_TE_1612618" H 2150 8050 60  0001 C CNN
@@
 $EndComp
 $Comp
-L RasPi-CM3-Headers J1
+L RasPi-CM3-Headers J?
 U 14 1 58ECDBFE
 P 10700 4250
-F 0 "J1" H 10650 3950 60  0000 C CNN
+F 0 "J?" H 10650 3950 60  0000 C CNN
 F 1 "RasPi-CM3-Headers" V 11100 4250 60  0000 C CNN
 F 2 "Sockets:Socket_SODIMM_DDR1-2_TE_1612618" H 10750 9350 60  0001 C CNN
@@
 NoConn ~ 10400 4450
 $Comp
-L Micro_SD_Card J10
+L Micro_SD_Card J?
 U 1 1 591147C4
 P 4250 5950
-F 0 "J10" H 3600 6550 50  0000 C CNN
+F 0 "J?" H 3600 6550 50  0000 C CNN
 F 1 "Micro_SD_Card" H 4900 6550 50  0000 R CNN
 F 2 "" H 5400 6250 50  0001 C CNN
@@
 $EndComp
 $Comp
-L GNDREF #PWR0152
+L GNDREF #PWR?
 U 1 1 59114968
 P 3300 6850
-F 0 "#PWR0152" H 3300 6600 50  0001 C CNN
+F 0 "#PWR?" H 3300 6600 50  0001 C CNN
 F 1 "GNDREF" H 3300 6700 50  0000 C CNN
 F 2 "" H 3300 6850 50  0001 C CNN
@@
 $EndComp
 $Comp
-L +3V3 #PWR0153
+L +3V3 #PWR?
 U 1 1 59114A75
 P 3000 5500
-F 0 "#PWR0153" H 3000 5350 50  0001 C CNN
+F 0 "#PWR?" H 3000 5350 50  0001 C CNN
 F 1 "+3V3" H 3000 5640 50  0000 C CNN
 F 2 "" H 3000 5500 50  0001 C CNN
@@
 $EndComp
 $Comp
-L C_Small C211
+L C_Small C?
 U 1 1 5911519B
 P 2450 6600
-F 0 "C211" H 2460 6670 50  0000 L CNN
+F 0 "C?" H 2460 6670 50  0000 L CNN
 F 1 "4u7F" H 2460 6520 50  0000 L CNN
 F 2 "Capacitors_SMD:C_0603_HandSoldering" H 2450 6600 50  0001 C CNN
@@
 $EndComp
 $Comp
-L C_Small C212
+L C_Small C?
 U 1 1 5911521F
 P 2650 6600
-F 0 "C212" H 2660 6670 50  0000 L CNN
+F 0 "C?" H 2660 6670 50  0000 L CNN
 F 1 "4u7F" H 2660 6520 50  0000 L CNN
 F 2 "Capacitors_SMD:C_0603_HandSoldering" H 2650 6600 50  0001 C CNN
@@
 $EndComp
 $Comp
-L HDMI-A-connector J11
+L HDMI-A-connector J?
 U 1 1 5911658C
 P 5450 2950
-F 0 "J11" H 5050 3600 60  0000 C CNN
+F 0 "J?" H 5050 3600 60  0000 C CNN
 F 1 "HDMI-A-connector" H 5450 2300 60  0000 C CNN
 F 2 "" H 5450 2950 60  0001 C CNN
@@
 $EndComp
 $Comp
-L ESD5384 U35
+L ESD5384 U?
 U 1 1 591172E0
 P 5100 4150
-F 0 "U35" H 4950 4450 60  0000 C CNN
+F 0 "U?" H 4950 4450 60  0000 C CNN
 F 1 "ESD5384" H 5100 3850 60  0000 C CNN
 F 2 "" H 5100 4200 60  0001 C CNN
@@
 $EndComp
 $Comp
-L +5VD #PWR0154
+L +5VD #PWR?
 U 1 1 591176E4
 P 7100 4150
-F 0 "#PWR0154" H 7100 4000 50  0001 C CNN
+F 0 "#PWR?" H 7100 4000 50  0001 C CNN
 F 1 "+5VD" H 7100 4290 50  0000 C CNN
 F 2 "" H 7100 4150 50  0001 C CNN
@@
 Connection ~ 6200 2650
 $Comp
-L GNDREF #PWR0155
+L GNDREF #PWR?
 U 1 1 59117C76
 P 6500 3400
-F 0 "#PWR0155" H 6500 3150 50  0001 C CNN
+F 0 "#PWR?" H 6500 3150 50  0001 C CNN
 F 1 "GNDREF" H 6500 3250 50  0000 C CNN
 F 2 "" H 6500 3400 50  0001 C CNN
@@
 Connection ~ 6200 3350
 $Comp
-L GNDREF #PWR0156
+L GNDREF #PWR?
 U 1 1 59117D13
 P 5650 4450
-F 0 "#PWR0156" H 5650 4200 50  0001 C CNN
+F 0 "#PWR?" H 5650 4200 50  0001 C CNN
 F 1 "GNDREF" H 5650 4300 50  0000 C CNN
 F 2 "" H 5650 4450 50  0001 C CNN
@@
 Connection ~ 5650 4350
 $Comp
-L ESD7484 U34
+L ESD7484 U?
 U 1 1 5911871C
 P 3500 3950
-F 0 "U34" H 3200 3600 60  0000 C CNN
+F 0 "U?" H 3200 3600 60  0000 C CNN
 F 1 "ESD7484" H 3350 4200 60  0000 C CNN
 F 2 "" H 3500 3950 60  0001 C CNN
@@
 $EndComp
 $Comp
-L ESD7484 U33
+L ESD7484 U?
 U 1 1 591189BB
 P 3500 2200
-F 0 "U33" H 3200 1850 60  0000 C CNN
+F 0 "U?" H 3200 1850 60  0000 C CNN
 F 1 "ESD7484" H 3350 2450 60  0000 C CNN
 F 2 "" H 3500 2200 60  0001 C CNN
@@
 	4150 2350 4000 2350
 $Comp
-L DMG1012T U31
+L DMG1012T U?
 U 1 1 5911B6F8
 P 3150 1350
-F 0 "U31" H 2750 1600 60  0000 C CNN
+F 0 "U?" H 2750 1600 60  0000 C CNN
 F 1 "DMG1012T" V 3000 1350 60  0000 C CNN
 F 2 "" H 2750 1800 60  0001 C CNN
@@
 $EndComp
 $Comp
-L +1V8 #PWR0157
+L +1V8 #PWR?
 U 1 1 5911B770
 P 3400 700
-F 0 "#PWR0157" H 3400 550 50  0001 C CNN
+F 0 "#PWR?" H 3400 550 50  0001 C CNN
 F 1 "+1V8" H 3400 840 50  0000 C CNN
 F 2 "" H 3400 700 50  0001 C CNN
@@
 Connection ~ 4500 2400
 $Comp
-L R_Small R124
+L R_Small R?
 U 1 1 5911BA5B
 P 3400 900
-F 0 "R124" H 3430 920 50  0000 L CNN
+F 0 "R?" H 3430 920 50  0000 L CNN
 F 1 "100k 1%" H 3430 860 50  0000 L CNN
 F 2 "Capacitors_SMD:C_0603_HandSoldering" H 3400 900 50  0001 C CNN
@@
 	3400 1000 3400 1100
 $Comp
-L GNDREF #PWR0158
+L GNDREF #PWR?
 U 1 1 5911BCE1
 P 3400 1650
-F 0 "#PWR0158" H 3400 1400 50  0001 C CNN
+F 0 "#PWR?" H 3400 1400 50  0001 C CNN
 F 1 "GNDREF" H 3400 1500 50  0000 C CNN
 F 2 "" H 3400 1650 50  0001 C CNN
@@
 Connection ~ 3400 1050
 $Comp
-L AP2331X U36
+L AP2331X U?
 U 1 1 5911C05E
 P 6700 4150
-F 0 "U36" H 6550 4200 60  0000 C CNN
+F 0 "U?" H 6550 4200 60  0000 C CNN
 F 1 "AP2331X" H 6600 3800 60  0000 C CNN
 F 2 "TO_SOT_Packages_SMD:SOT-23" H 6800 5100 60  0001 C CNN
@@
 	6100 3950 6100 3450
 $Comp
-L C_Small C214
+L C_Small C?
 U 1 1 5911FC51
 P 7100 4300
-F 0 "C214" H 7110 4370 50  0000 L CNN
+F 0 "C?" H 7110 4370 50  0000 L CNN
 F 1 "100n" H 7110 4220 50  0000 L CNN
 F 2 "Capacitors_SMD:C_0603_HandSoldering" H 7100 4300 50  0001 C CNN
@@
 	7000 4400 7100 4400
 $Comp
-L GNDREF #PWR0159
+L GNDREF #PWR?
 U 1 1 5911FE33
 P 7100 4650
-F 0 "#PWR0159" H 7100 4400 50  0001 C CNN
+F 0 "#PWR?" H 7100 4400 50  0001 C CNN
 F 1 "GNDREF" H 7100 4500 50  0000 C CNN
 F 2 "" H 7100 4650 50  0001 C CNN
@@
 	5550 4050 5550 3950
 $Comp
-L C_Small C213
+L C_Small C?
 U 1 1 59120198
 P 6450 4450
-F 0 "C213" H 6460 4520 50  0000 L CNN
+F 0 "C?" H 6460 4520 50  0000 L CNN
 F 1 "100n" H 6460 4370 50  0000 L CNN
 F 2 "Capacitors_SMD:C_0603_HandSoldering" H 6450 4450 50  0001 C CNN
@@
 H5V
 $Comp
-L GNDREF #PWR0160
+L GNDREF #PWR?
 U 1 1 5912041E
 P 4000 4450
-F 0 "#PWR0160" H 4000 4200 50  0001 C CNN
+F 0 "#PWR?" H 4000 4200 50  0001 C CNN
 F 1 "GNDREF" H 4000 4300 50  0000 C CNN
 F 2 "" H 4000 4450 50  0001 C CNN
@@
 NoConn ~ 5500 4150
 $Comp
-L GNDREF #PWR0161
+L GNDREF #PWR?
 U 1 1 59120752
 P 4000 2700
-F 0 "#PWR0161" H 4000 2450 50  0001 C CNN
+F 0 "#PWR?" H 4000 2450 50  0001 C CNN
 F 1 "GNDREF" H 4000 2550 50  0000 C CNN
 F 2 "" H 4000 2700 50  0001 C CNN
@@
 Connection ~ 4000 2600
 $Comp
-L DMG1012T U32
+L DMG1012T U?
 U 1 1 591207FB
 P 3350 3550
-F 0 "U32" H 2950 3800 60  0000 C CNN
+F 0 "U?" H 2950 3800 60  0000 C CNN
 F 1 "DMG1012T" V 3200 3550 60  0000 C CNN
 F 2 "" H 2950 4000 60  0001 C CNN
@@
 Connection ~ 4450 3300
 $Comp
-L R_Small R123
+L R_Small R?
 U 1 1 591214D4
 P 2900 3100
-F 0 "R123" H 2930 3120 50  0000 L CNN
+F 0 "R?" H 2930 3120 50  0000 L CNN
 F 1 "27k 1%" H 2930 3060 50  0000 L CNN
 F 2 "Capacitors_SMD:C_0603_HandSoldering" H 2900 3100 50  0001 C CNN
@@
 Connection ~ 2900 3300
 $Comp
-L +3V3 #PWR0162
+L +3V3 #PWR?
 U 1 1 59121601
 P 2900 2850
-F 0 "#PWR0162" H 2900 2700 50  0001 C CNN
+F 0 "#PWR?" H 2900 2700 50  0001 C CNN
 F 1 "+3V3" H 2900 2990 50  0000 C CNN
 F 2 "" H 2900 2850 50  0001 C CNN

Commit message: Updated footprint assignments
Parts:
- C229, C230, C231, C232: renamed from C?; footprint Capacitors_SMD:C_0603_HandSoldering -> Capacitors_SMD:C_0603
- R122, R123: renamed from R?; footprint Capacitors_SMD:C_0603_HandSoldering -> Resistors_SMD:R_0603
- gave numbers to parts that had none: 9
Changed lines of the file:
@@
 $EndDescr
 $Comp
-L RasPi-CM3-Headers J?
+L RasPi-CM3-Headers J1
 U 2 1 58ECDA7F
 P 1650 6000
-F 0 "J?" H 1350 5550 60  0000 C CNN
+F 0 "J1" H 1350 5550 60  0000 C CNN
 F 1 "RasPi-CM3-Headers" V 2250 6000 60  0000 C CNN
 F 2 "Sockets:Socket_SODIMM_DDR1-2_TE_1612618" H 1700 11100 60  0001 C CNN
@@
 $EndComp
 $Comp
-L RasPi-CM3-Headers J?
+L RasPi-CM3-Headers J1
 U 3 1 58ECDAC0
 P 9900 5250
-F 0 "J?" H 9700 4900 60  0000 C CNN
+F 0 "J1" H 9700 4900 60  0000 C CNN
 F 1 "RasPi-CM3-Headers" V 10200 5250 60  0000 C CNN
 F 2 "Sockets:Socket_SODIMM_DDR1-2_TE_1612618" H 9950 10350 60  0001 C CNN
@@
 $EndComp
 $Comp
-L RasPi-CM3-Headers J?
+L RasPi-CM3-Headers J1
 U 4 1 58ECDAF6
 P 9850 3300
-F 0 "J?" H 9750 2750 60  0000 C CNN
+F 0 "J1" H 9750 2750 60  0000 C CNN
 F 1 "RasPi-CM3-Headers" V 10150 3300 60  0000 C CNN
 F 2 "Sockets:Socket_SODIMM_DDR1-2_TE_1612618" H 9900 8400 60  0001 C CNN
@@
 $EndComp
 $Comp
-L RasPi-CM3-Headers J?
+L RasPi-CM3-Headers J1
 U 10 1 58ECDB2D
 P 10700 3300
-F 0 "J?" H 10600 2750 60  0000 C CNN
+F 0 "J1" H 10600 2750 60  0000 C CNN
 F 1 "RasPi-CM3-Headers" V 11000 3300 60  0000 C CNN
 F 2 "Sockets:Socket_SODIMM_DDR1-2_TE_1612618" H 10750 8400 60  0001 C CNN
@@
 $EndComp
 $Comp
-L RasPi-CM3-Headers J?
+L RasPi-CM3-Headers J1
 U 11 1 58ECDB78
 P 10700 5250
-F 0 "J?" H 10550 4900 60  0000 C CNN
+F 0 "J1" H 10550 4900 60  0000 C CNN
 F 1 "RasPi-CM3-Headers" V 11000 5250 60  0000 C CNN
 F 2 "Sockets:Socket_SODIMM_DDR1-2_TE_1612618" H 10750 10350 60  0001 C CNN
@@
 $EndComp
 $Comp
-L RasPi-CM3-Headers J?
+L RasPi-CM3-Headers J1
 U 12 1 58ECDBAE
 P 2100 2950
-F 0 "J?" H 1950 2250 60  0000 C CNN
+F 0 "J1" H 1950 2250 60  0000 C CNN
 F 1 "RasPi-CM3-Headers" V 2600 2950 60  0000 C CNN
 F 2 "Sockets:Socket_SODIMM_DDR1-2_TE_1612618" H 2150 8050 60  0001 C CNN
@@
 $EndComp
 $Comp
-L RasPi-CM3-Headers J?
+L RasPi-CM3-Headers J1
 U 14 1 58ECDBFE
 P 10700 4250
-F 0 "J?" H 10650 3950 60  0000 C CNN
+F 0 "J1" H 10650 3950 60  0000 C CNN
 F 1 "RasPi-CM3-Headers" V 11100 4250 60  0000 C CNN
 F 2 "Sockets:Socket_SODIMM_DDR1-2_TE_1612618" H 10750 9350 60  0001 C CNN
@@
 NoConn ~ 10400 4450
 $Comp
-L Micro_SD_Card J?
+L Micro_SD_Card J10
 U 1 1 591147C4
 P 4250 5950
-F 0 "J?" H 3600 6550 50  0000 C CNN
+F 0 "J10" H 3600 6550 50  0000 C CNN
 F 1 "Micro_SD_Card" H 4900 6550 50  0000 R CNN
 F 2 "" H 5400 6250 50  0001 C CNN
@@
 $EndComp
 $Comp
-L GNDREF #PWR?
+L GNDREF #PWR0174
 U 1 1 59114968
 P 3300 6850
-F 0 "#PWR?" H 3300 6600 50  0001 C CNN
+F 0 "#PWR0174" H 3300 6600 50  0001 C CNN
 F 1 "GNDREF" H 3300 6700 50  0000 C CNN
 F 2 "" H 3300 6850 50  0001 C CNN
@@
 $EndComp
 $Comp
-L +3V3 #PWR?
+L +3V3 #PWR0175
 U 1 1 59114A75
 P 3000 5500
-F 0 "#PWR?" H 3000 5350 50  0001 C CNN
+F 0 "#PWR0175" H 3000 5350 50  0001 C CNN
 F 1 "+3V3" H 3000 5640 50  0000 C CNN
 F 2 "" H 3000 5500 50  0001 C CNN
@@
 $EndComp
 $Comp
-L C_Small C?
+L C_Small C229
 U 1 1 5911519B
 P 2450 6600
-F 0 "C?" H 2460 6670 50  0000 L CNN
+F 0 "C229" H 2460 6670 50  0000 L CNN
 F 1 "4u7F" H 2460 6520 50  0000 L CNN
-F 2 "Capacitors_SMD:C_0603_HandSoldering" H 2450 6600 50  0001 C CNN
+F 2 "Capacitors_SMD:C_0603" H 2450 6600 50  0001 C CNN
 F 3 "" H 2450 6600 50  0001 C CNN
 	1    2450 6600
@@
 $EndComp
 $Comp
-L C_Small C?
+L C_Small C230
 U 1 1 5911521F
 P 2650 6600
-F 0 "C?" H 2660 6670 50  0000 L CNN
+F 0 "C230" H 2660 6670 50  0000 L CNN
 F 1 "4u7F" H 2660 6520 50  0000 L CNN
-F 2 "Capacitors_SMD:C_0603_HandSoldering" H 2650 6600 50  0001 C CNN
+F 2 "Capacitors_SMD:C_0603" H 2650 6600 50  0001 C CNN
 F 3 "" H 2650 6600 50  0001 C CNN
 	1    2650 6600
@@
 $EndComp
 $Comp
-L HDMI-A-connector J?
+L HDMI-A-connector J11
 U 1 1 5911658C
 P 5450 2950
-F 0 "J?" H 5050 3600 60  0000 C CNN
+F 0 "J11" H 5050 3600 60  0000 C CNN
 F 1 "HDMI-A-connector" H 5450 2300 60  0000 C CNN
 F 2 "" H 5450 2950 60  0001 C CNN
@@
 $EndComp
 $Comp
-L ESD5384 U?
+L ESD5384 U42
 U 1 1 591172E0
 P 5100 4150
-F 0 "U?" H 4950 4450 60  0000 C CNN
+F 0 "U42" H 4950 4450 60  0000 C CNN
 F 1 "ESD5384" H 5100 3850 60  0000 C CNN
 F 2 "" H 5100 4200 60  0001 C CNN
@@
 $EndComp
 $Comp
-L +5VD #PWR?
+L +5VD #PWR0176
 U 1 1 591176E4
 P 7100 4150
-F 0 "#PWR?" H 7100 4000 50  0001 C CNN
+F 0 "#PWR0176" H 7100 4000 50  0001 C CNN
 F 1 "+5VD" H 7100 4290 50  0000 C CNN
 F 2 "" H 7100 4150 50  0001 C CNN
@@
 Connection ~ 6200 2650
 $Comp
-L GNDREF #PWR?
+L GNDREF #PWR0177
 U 1 1 59117C76
 P 6500 3400
-F 0 "#PWR?" H 6500 3150 50  0001 C CNN
+F 0 "#PWR0177" H 6500 3150 50  0001 C CNN
 F 1 "GNDREF" H 6500 3250 50  0000 C CNN
 F 2 "" H 6500 3400 50  0001 C CNN
@@
 Connection ~ 6200 3350
 $Comp
-L GNDREF #PWR?
+L GNDREF #PWR0178
 U 1 1 59117D13
 P 5650 4450
-F 0 "#PWR?" H 5650 4200 50  0001 C CNN
+F 0 "#PWR0178" H 5650 4200 50  0001 C CNN
 F 1 "GNDREF" H 5650 4300 50  0000 C CNN
 F 2 "" H 5650 4450 50  0001 C CNN
@@
 Connection ~ 5650 4350
 $Comp
-L ESD7484 U?
+L ESD7484 U41
 U 1 1 5911871C
 P 3500 3950
-F 0 "U?" H 3200 3600 60  0000 C CNN
+F 0 "U41" H 3200 3600 60  0000 C CNN
 F 1 "ESD7484" H 3350 4200 60  0000 C CNN
 F 2 "" H 3500 3950 60  0001 C CNN
@@
 $EndComp
 $Comp
-L ESD7484 U?
+L ESD7484 U40
 U 1 1 591189BB
 P 3500 2200
-F 0 "U?" H 3200 1850 60  0000 C CNN
+F 0 "U40" H 3200 1850 60  0000 C CNN
 F 1 "ESD7484" H 3350 2450 60  0000 C CNN
 F 2 "" H 3500 2200 60  0001 C CNN
@@
 	4150 2350 4000 2350
 $Comp
-L DMG1012T U?
+L DMG1012T U38
 U 1 1 5911B6F8
 P 3150 1350
-F 0 "U?" H 2750 1600 60  0000 C CNN
+F 0 "U38" H 2750 1600 60  0000 C CNN
 F 1 "DMG1012T" V 3000 1350 60  0000 C CNN
 F 2 "" H 2750 1800 60  0001 C CNN
@@
 $EndComp
 $Comp
-L +1V8 #PWR?
+L +1V8 #PWR0179
 U 1 1 5911B770
 P 3400 700
-F 0 "#PWR?" H 3400 550 50  0001 C CNN
+F 0 "#PWR0179" H 3400 550 50  0001 C CNN
 F 1 "+1V8" H 3400 840 50  0000 C CNN
 F 2 "" H 3400 700 50  0001 C CNN
@@
 Connection ~ 4500 2400
 $Comp
-L R_Small R?
+L R_Small R123
 U 1 1 5911BA5B
 P 3400 900
-F 0 "R?" H 3430 920 50  0000 L CNN
+F 0 "R123" H 3430 920 50  0000 L CNN
 F 1 "100k 1%" H 3430 860 50  0000 L CNN
-F 2 "Capacitors_SMD:C_0603_HandSoldering" H 3400 900 50  0001 C CNN
+F 2 "Resistors_SMD:R_0603" H 3400 900 50  0001 C CNN
 F 3 "" H 3400 900 50  0001 C CNN
 	1    3400 900
@@
 	3400 1000 3400 1100
 $Comp
-L GNDREF #PWR?
+L GNDREF #PWR0180
 U 1 1 5911BCE1
 P 3400 1650
-F 0 "#PWR?" H 3400 1400 50  0001 C CNN
+F 0 "#PWR0180" H 3400 1400 50  0001 C CNN
 F 1 "GNDREF" H 3400 1500 50  0000 C CNN
 F 2 "" H 3400 1650 50  0001 C CNN
@@
 Connection ~ 3400 1050
 $Comp
-L AP2331X U?
+L AP2331X U43
 U 1 1 5911C05E
 P 6700 4150
-F 0 "U?" H 6550 4200 60  0000 C CNN
+F 0 "U43" H 6550 4200 60  0000 C CNN
 F 1 "AP2331X" H 6600 3800 60  0000 C CNN
 F 2 "TO_SOT_Packages_SMD:SOT-23" H 6800 5100 60  0001 C CNN
@@
 	6100 3950 6100 3450
 $Comp
-L C_Small C?
+L C_Small C232
 U 1 1 5911FC51
 P 7100 4300
-F 0 "C?" H 7110 4370 50  0000 L CNN
+F 0 "C232" H 7110 4370 50  0000 L CNN
 F 1 "100n" H 7110 4220 50  0000 L CNN
-F 2 "Capacitors_SMD:C_0603_HandSoldering" H 7100 4300 50  0001 C CNN
+F 2 "Capacitors_SMD:C_0603" H 7100 4300 50  0001 C CNN
 F 3 "" H 7100 4300 50  0001 C CNN
 	1    7100 4300
@@
 	7000 4400 7100 4400
 $Comp
-L GNDREF #PWR?
+L GNDREF #PWR0181
 U 1 1 5911FE33
 P 7100 4650
-F 0 "#PWR?" H 7100 4400 50  0001 C CNN
+F 0 "#PWR0181" H 7100 4400 50  0001 C CNN
 F 1 "GNDREF" H 7100 4500 50  0000 C CNN
 F 2 "" H 7100 4650 50  0001 C CNN
@@
 	5550 4050 5550 3950
 $Comp
-L C_Small C?
+L C_Small C231
 U 1 1 59120198
 P 6450 4450
-F 0 "C?" H 6460 4520 50  0000 L CNN
+F 0 "C231" H 6460 4520 50  0000 L CNN
 F 1 "100n" H 6460 4370 50  0000 L CNN
-F 2 "Capacitors_SMD:C_0603_HandSoldering" H 6450 4450 50  0001 C CNN
+F 2 "Capacitors_SMD:C_0603" H 6450 4450 50  0001 C CNN
 F 3 "" H 6450 4450 50  0001 C CNN
 	1    6450 4450
@@
 H5V
 $Comp
-L GNDREF #PWR?
+L GNDREF #PWR0182
 U 1 1 5912041E
 P 4000 4450
-F 0 "#PWR?" H 4000 4200 50  0001 C CNN
+F 0 "#PWR0182" H 4000 4200 50  0001 C CNN
 F 1 "GNDREF" H 4000 4300 50  0000 C CNN
 F 2 "" H 4000 4450 50  0001 C CNN
@@
 NoConn ~ 5500 4150
 $Comp
-L GNDREF #PWR?
+L GNDREF #PWR0183
 U 1 1 59120752
 P 4000 2700
-F 0 "#PWR?" H 4000 2450 50  0001 C CNN
+F 0 "#PWR0183" H 4000 2450 50  0001 C CNN
 F 1 "GNDREF" H 4000 2550 50  0000 C CNN
 F 2 "" H 4000 2700 50  0001 C CNN
@@
 Connection ~ 4000 2600
 $Comp
-L DMG1012T U?
+L DMG1012T U39
 U 1 1 591207FB
 P 3350 3550
-F 0 "U?" H 2950 3800 60  0000 C CNN
+F 0 "U39" H 2950 3800 60  0000 C CNN
 F 1 "DMG1012T" V 3200 3550 60  0000 C CNN
 F 2 "" H 2950 4000 60  0001 C CNN
@@
 Connection ~ 4450 3300
 $Comp
-L R_Small R?
+L R_Small R122
 U 1 1 591214D4
 P 2900 3100
-F 0 "R?" H 2930 3120 50  0000 L CNN
+F 0 "R122" H 2930 3120 50  0000 L CNN
 F 1 "27k 1%" H 2930 3060 50  0000 L CNN
-F 2 "Capacitors_SMD:C_0603_HandSoldering" H 2900 3100 50  0001 C CNN
+F 2 "Resistors_SMD:R_0603" H 2900 3100 50  0001 C CNN
 F 3 "" H 2900 3100 50  0001 C CNN
 	1    2900 3100
@@
 Connection ~ 2900 3300
 $Comp
-L +3V3 #PWR?
+L +3V3 #PWR0184
 U 1 1 59121601
 P 2900 2850
-F 0 "#PWR?" H 2900 2700 50  0001 C CNN
+F 0 "#PWR0184" H 2900 2700 50  0001 C CNN
 F 1 "+3V3" H 2900 2990 50  0000 C CNN
 F 2 "" H 2900 2850 50  0001 C CNN

Commit message: Added all missing nonstandard footprints
Parts:
- J10: value Micro_SD_Card -> 500901-0801; footprint (none) -> SW-Molex:5009010801_sd; Description (none) -> MicroSD card holder, hinge type; Manufacturer (none) -> Molex; Pricing (none) -> 0.00@0
- J11: footprint (none) -> Pin_Headers:Pin_Header_Straight_2x10_Pitch1.27mm
- U38, U39: footprint (none) -> SW-Diodes:SOT523
- U40, U41: footprint (none) -> SW-On-Semi:WLCSP10-1.6x1.1mm
- U42: footprint (none) -> SW-On-Semi:WLCSP9-1.14x1.14mm
Changed lines of the file:
@@
 P 4250 5950
 F 0 "J10" H 3600 6550 50  0000 C CNN
-F 1 "Micro_SD_Card" H 4900 6550 50  0000 R CNN
-F 2 "" H 5400 6250 50  0001 C CNN
-F 3 "" H 4250 5950 50  0001 C CNN
+F 1 "500901-0801" H 4900 6550 50  0000 R CNN
+F 2 "SW-Molex:5009010801_sd" H 5400 6250 50  0001 C CNN
+F 3 "http://www.mouser.com/ds/2/276/5009010801_MEMORY_CARD_SOCKET-179079.pdf" H 4250 5950 50  0001 C CNN
+F 4 "Molex" H 4250 5950 60  0001 C CNN "Manufacturer"
+F 5 "MicroSD card holder, hinge type" H 4250 5950 60  0001 C CNN "Description"
+F 6 "0.00@0" H 4250 5950 60  0001 C CNN "Pricing"
 	1    4250 5950
 	1    0    0    -1
@@
 F 0 "J11" H 5050 3600 60  0000 C CNN
 F 1 "HDMI-A-connector" H 5450 2300 60  0000 C CNN
-F 2 "" H 5450 2950 60  0001 C CNN
+F 2 "Pin_Headers:Pin_Header_Straight_2x10_Pitch1.27mm" H 5450 2950 60  0001 C CNN
 F 3 "" H 5450 2950 60  0001 C CNN
 F 4 "0.00@0" H 5500 3850 60  0001 C CNN "Pricing"
@@
 F 0 "U42" H 4950 4450 60  0000 C CNN
 F 1 "ESD5384" H 5100 3850 60  0000 C CNN
-F 2 "" H 5100 4200 60  0001 C CNN
+F 2 "SW-On-Semi:WLCSP9-1.14x1.14mm" H 5100 4200 60  0001 C CNN
 F 3 "http://www.onsemi.com/pub/Collateral/ESD5384-D.PDF" H 5300 5000 60  0001 C CNN
 F 4 "0.00@0" H 5100 4700 60  0001 C CNN "Pricing"
@@
 F 0 "U41" H 3200 3600 60  0000 C CNN
 F 1 "ESD7484" H 3350 4200 60  0000 C CNN
-F 2 "" H 3500 3950 60  0001 C CNN
+F 2 "SW-On-Semi:WLCSP10-1.6x1.1mm" H 3500 3950 60  0001 C CNN
 F 3 "http://www.onsemi.com/pub/Collateral/ESD7484-D.PDF" H 4000 4700 60  0001 C CNN
 F 4 "0.00@0" H 3600 4850 60  0001 C CNN "Pricing"
@@
 F 0 "U40" H 3200 1850 60  0000 C CNN
 F 1 "ESD7484" H 3350 2450 60  0000 C CNN
-F 2 "" H 3500 2200 60  0001 C CNN
+F 2 "SW-On-Semi:WLCSP10-1.6x1.1mm" H 3500 2200 60  0001 C CNN
 F 3 "http://www.onsemi.com/pub/Collateral/ESD7484-D.PDF" H 4000 2950 60  0001 C CNN
 F 4 "0.00@0" H 3600 3100 60  0001 C CNN "Pricing"
@@
 F 0 "U38" H 2750 1600 60  0000 C CNN
 F 1 "DMG1012T" V 3000 1350 60  0000 C CNN
-F 2 "" H 2750 1800 60  0001 C CNN
+F 2 "SW-Diodes:SOT523" H 2750 1800 60  0001 C CNN
 F 3 "https://www.diodes.com/assets/Datasheets/ds31783.pdf" H 3150 2400 60  0001 C CNN
 F 4 "0.00@0" H 3150 2500 60  0001 C CNN "Pricing"
@@
 F 0 "U39" H 2950 3800 60  0000 C CNN
 F 1 "DMG1012T" V 3200 3550 60  0000 C CNN
-F 2 "" H 2950 4000 60  0001 C CNN
+F 2 "SW-Diodes:SOT523" H 2950 4000 60  0001 C CNN
 F 3 "https://www.diodes.com/assets/Datasheets/ds31783.pdf" H 3350 4600 60  0001 C CNN
 F 4 "0.00@0" H 3350 4700 60  0001 C CNN "Pricing"
