File: dev1-mux-conn.sch (KiCad schematic (older format))
At the start: 9 parts, among them J25 Device 1, U16 TS12A44514, U17 TS12A44514, U20 MAX4533, U50 74LS32, U51 LTC1391, U52 LTC1391, U53 LTC1391

Commit message: Updating power + libraries
- Reannotated all parts
- Migrated to new OR gate library
- Reorganized power sheet
Parts:
- removed U50: 74LS32, SMD_Packages:SSOP-14, symbol 74LS32
- added U19: 74LS32, symbol 74LS32
- renumbered C243 to C51, J25 to J27, U20 to U11, U51 to U33, U52 to U34, U53 to U35, U16 to U9, U17 to U9
Connections:
- wire segments 76 -> 77
Changed lines of the file:
@@
-EESchema Schematic File Version 2
+EESchema Schematic File Version 3
 LIBS:SW-Texas
 LIBS:power
@@
 $EndDescr
 $Comp
-L Conn_01x07 J25
+L Conn_01x07 J27
 U 1 1 58EA8BFC
 P 900 1150
-F 0 "J25" H 900 1600 50  0000 C CNN
+F 0 "J27" H 900 1600 50  0000 C CNN
 F 1 "Device 1" V 1000 1150 50  0000 C CNN
 F 2 "Pin_Headers:Pin_Header_Straight_1x07_Pitch2.54mm" H 900 1150 50  0001 C CNN
@@
 $EndComp
 $Comp
-L C_Small C243
+L C_Small C51
 U 1 1 58EA8C1B
 P 2500 1150
-F 0 "C243" H 2510 1220 50  0000 L CNN
+F 0 "C51" H 2510 1220 50  0000 L CNN
 F 1 "10u" H 2510 1070 50  0000 L CNN
 F 2 "Capacitors_SMD:C_0603" H 2500 1150 50  0001 C CNN
@@
 AUDIO-GROUND
 $Comp
-L LTC1391 U51
+L LTC1391 U33
 U 1 1 58EA8C2B
 P 6400 1400
-F 0 "U51" H 6150 1900 60  0000 C CNN
+F 0 "U33" H 6150 1900 60  0000 C CNN
 F 1 "LTC1391" H 6750 1850 60  0000 C CNN
 F 2 "Housings_SSOP:SSOP-16_3.9x4.9mm_Pitch0.635mm" H 6500 2650 60  0001 C CNN
@@
 DOUT
 $Comp
-L +5VD #PWR0199
+L +5VD #PWR066
 U 1 1 58EA8C36
 P 6400 700
-F 0 "#PWR0199" H 6400 550 50  0001 C CNN
+F 0 "#PWR066" H 6400 550 50  0001 C CNN
 F 1 "+5VD" H 6400 840 50  0000 C CNN
 F 2 "" H 6400 700 50  0001 C CNN
@@
 $EndComp
 $Comp
-L GNDREF #PWR0200
+L GNDREF #PWR067
 U 1 1 58EA8C3C
 P 6400 2000
-F 0 "#PWR0200" H 6400 1750 50  0001 C CNN
+F 0 "#PWR067" H 6400 1750 50  0001 C CNN
 F 1 "GNDREF" H 6400 1850 50  0000 C CNN
 F 2 "" H 6400 2000 50  0001 C CNN
@@
 PTT-7
 $Comp
-L LTC1391 U52
+L LTC1391 U34
 U 1 1 58EA8C79
 P 6400 3200
-F 0 "U52" H 6150 3700 60  0000 C CNN
+F 0 "U34" H 6150 3700 60  0000 C CNN
 F 1 "LTC1391" H 6750 3650 60  0000 C CNN
 F 2 "Housings_SSOP:SSOP-16_3.9x4.9mm_Pitch0.635mm" H 6500 4450 60  0001 C CNN
@@
 $EndComp
 $Comp
-L +5VD #PWR0201
+L +5VD #PWR068
 U 1 1 58EA8C80
 P 6400 2500
-F 0 "#PWR0201" H 6400 2350 50  0001 C CNN
+F 0 "#PWR068" H 6400 2350 50  0001 C CNN
 F 1 "+5VD" H 6400 2640 50  0000 C CNN
 F 2 "" H 6400 2500 50  0001 C CNN
@@
 $EndComp
 $Comp
-L GNDREF #PWR0202
+L GNDREF #PWR069
 U 1 1 58EA8C86
 P 6400 3800
-F 0 "#PWR0202" H 6400 3550 50  0001 C CNN
+F 0 "#PWR069" H 6400 3550 50  0001 C CNN
 F 1 "GNDREF" H 6400 3650 50  0000 C CNN
 F 2 "" H 6400 3800 50  0001 C CNN
@@
 $EndComp
 $Comp
-L LTC1391 U53
+L LTC1391 U35
 U 1 1 58EA8C90
 P 6400 4900
-F 0 "U53" H 6150 5400 60  0000 C CNN
+F 0 "U35" H 6150 5400 60  0000 C CNN
 F 1 "LTC1391" H 6750 5350 60  0000 C CNN
 F 2 "Housings_SSOP:SSOP-16_3.9x4.9mm_Pitch0.635mm" H 6500 6150 60  0001 C CNN
@@
 $EndComp
 $Comp
-L +5VD #PWR0203
+L +5VD #PWR070
 U 1 1 58EA8C97
 P 6400 4200
-F 0 "#PWR0203" H 6400 4050 50  0001 C CNN
+F 0 "#PWR070" H 6400 4050 50  0001 C CNN
 F 1 "+5VD" H 6400 4340 50  0000 C CNN
 F 2 "" H 6400 4200 50  0001 C CNN
@@
 $EndComp
 $Comp
-L GNDREF #PWR0204
+L GNDREF #PWR071
 U 1 1 58EA8C9D
 P 6400 5500
-F 0 "#PWR0204" H 6400 5250 50  0001 C CNN
+F 0 "#PWR071" H 6400 5250 50  0001 C CNN
 F 1 "GNDREF" H 6400 5350 50  0000 C CNN
 F 2 "" H 6400 5500 50  0001 C CNN
@@
 	2900 1800 2900 2850
 Wire Wire Line
-	4100 2750 4300 2750
-Wire Wire Line
-	4100 4450 4300 4450
+	3800 2750 4300 2750
+Wire Wire Line
+	3750 4450 4300 4450
 Wire Wire Line
 	2700 1500 3350 1500
 Connection ~ 3350 1500
 Wire Wire Line
-	2900 4550 2700 4550
+	2700 4550 3150 4550
 Wire Wire Line
 	2700 4550 2700 1700
@@
 	2050 2150 4050 2150
 Wire Wire Line
-	4100 2950 5950 2950
+	3800 2950 5950 2950
 Wire Wire Line
 	5650 3200 5950 3200
@@
 Connection ~ 6400 3800
 Wire Wire Line
-	4100 4650 5950 4650
+	3750 4650 5950 4650
 Wire Wire Line
 	3900 5100 5950 5100
@@
 	6850 5250 7150 5250
 $Comp
-L MAX4533 U20
+L MAX4533 U11
 U 2 1 58EA8E4A
 P 2350 1600
-F 0 "U20" H 2450 1800 60  0000 C CNN
+F 0 "U11" H 2450 1800 60  0000 C CNN
 F 1 "MAX4533" H 2000 1350 60  0000 C CNN
 F 2 "Housings_SSOP:SSOP-20_4.4x6.5mm_Pitch0.65mm" H 2450 2550 60  0001 C CNN
@@
 $EndComp
 $Comp
-L 74LS32 U50
-U 1 1 58EA8EE0
-P 3500 2850
-F 0 "U50" H 3500 2900 50  0000 C CNN
-F 1 "74LS32" H 3500 2800 50  0000 C CNN
-F 2 "SMD_Packages:SSOP-14" H 3500 2850 50  0001 C CNN
-F 3 "" H 3500 2850 50  0001 C CNN
-	1    3500 2850
-	-1   0    0    -1
-$EndComp
-$Comp
-L 74LS32 U50
-U 2 1 58EA8F3E
-P 3500 4550
-F 0 "U50" H 3500 4600 50  0000 C CNN
-F 1 "74LS32" H 3500 4500 50  0000 C CNN
-F 2 "SMD_Packages:SSOP-14" H 3500 4550 50  0001 C CNN
-F 3 "" H 3500 4550 50  0001 C CNN
-	2    3500 4550
-	-1   0    0    -1
-$EndComp
-$Comp
-L TS12A44514 U16
-U 2 1 58EA90C5
+L TS12A44514 U9
+U 3 1 58EA90C5
 P 1700 1450
-F 0 "U16" H 1550 1650 60  0000 C CNN
+F 0 "U9" H 1550 1650 60  0000 C CNN
 F 1 "TS12A44514" H 2000 1650 60  0000 C CNN
 F 2 "Housings_SSOP:TSSOP-14_4.4x5mm_Pitch0.65mm" H 2200 2750 60  0001 C CNN
@@
 F 7 "Texas Instruments" H 2100 2900 60  0001 C CNN "Manufacturer"
 F 8 "TSSOP14" H 2000 2650 60  0001 C CNN "Package ID"
-	2    1700 1450
-	1    0    0    -1
-$EndComp
-$Comp
-L TS12A44514 U17
-U 2 1 58EA913D
+	3    1700 1450
+	1    0    0    -1
+$EndComp
+$Comp
+L TS12A44514 U9
+U 4 1 58EA913D
 P 2950 1150
-F 0 "U17" H 2800 1350 60  0000 C CNN
+F 0 "U9" H 2800 1350 60  0000 C CNN
 F 1 "TS12A44514" H 3250 1350 60  0000 C CNN
 F 2 "Housings_SSOP:TSSOP-14_4.4x5mm_Pitch0.65mm" H 3450 2450 60  0001 C CNN
@@
 F 7 "Texas Instruments" H 3350 2600 60  0001 C CNN "Manufacturer"
 F 8 "TSSOP14" H 3250 2350 60  0001 C CNN "Package ID"
-	2    2950 1150
+	4    2950 1150
 	1    0    0    -1
 $EndComp
 Text Notes 800  3350 0    60   ~ 0
 1-Audio Ground\n2-L audio to MUX\n3-R audio to MUX\n4-Mic +\n5-Mic -\n6- PTT +\n7- PTT -
+$Comp
+L 74LS32 U19
+U 3 1 59D22D32
+P 3500 2850
+F 0 "U19" H 3500 2533 50  0000 C CNN
+F 1 "74LS32" H 3500 2624 50  0000 C CNN
+F 2 "" H 3500 2850 50  0001 C CNN
+F 3 "" H 3500 2850 50  0001 C CNN
+	3    3500 2850
+	-1   0    0    1
+$EndComp
+Wire Wire Line
+	2900 2850 3200 2850
+$Comp
+L 74LS32 U19
+U 4 1 59D22F35
+P 3450 4550
+F 0 "U19" H 3450 4233 50  0000 C CNN
+F 1 "74LS32" H 3450 4324 50  0000 C CNN
+F 2 "" H 3450 4550 50  0001 C CNN
+F 3 "" H 3450 4550 50  0001 C CNN
+	4    3450 4550
+	-1   0    0    1
+$EndComp
 $EndSCHEMATC

Commit message: Updates during pcb layout
Added more net labels
moved switches and OR gates to +5V instead of +5VD
Parts:
- J27: footprint Pin_Headers:Pin_Header_Straight_1x07_Pitch2.54mm -> SW-TEConn:3-794681-8
- U19: footprint (none) -> Housings_SSOP:SSOP-14_5.3x6.2mm_Pitch0.65mm
Connections:
- net +5VD renamed +5V
Changed lines of the file:
@@
 LIBS:SW-Diodes-Inc
 LIBS:interface
+LIBS:SW-gElectroMech
 LIBS:edc-mux-board-cache
 EELAYER 26 0
@@
 F 0 "J27" H 900 1600 50  0000 C CNN
 F 1 "Device 1" V 1000 1150 50  0000 C CNN
-F 2 "Pin_Headers:Pin_Header_Straight_1x07_Pitch2.54mm" H 900 1150 50  0001 C CNN
+F 2 "SW-TEConn:3-794681-8" H 900 1150 50  0001 C CNN
 F 3 "" H 900 1150 50  0001 C CNN
 F 4 "0.00@0" H 900 1150 60  0001 C CNN "Pricing"
@@
 Text HLabel 3900 5100 0    60   Output ~ 0
 DOUT
-$Comp
-L +5VD #PWR066
-U 1 1 58EA8C36
-P 6400 700
-F 0 "#PWR066" H 6400 550 50  0001 C CNN
-F 1 "+5VD" H 6400 840 50  0000 C CNN
-F 2 "" H 6400 700 50  0001 C CNN
-F 3 "" H 6400 700 50  0001 C CNN
-	1    6400 700
-	1    0    0    -1
-$EndComp
 $Comp
 L GNDREF #PWR067
@@
 $EndComp
 $Comp
-L +5VD #PWR068
-U 1 1 58EA8C80
-P 6400 2500
-F 0 "#PWR068" H 6400 2350 50  0001 C CNN
-F 1 "+5VD" H 6400 2640 50  0000 C CNN
-F 2 "" H 6400 2500 50  0001 C CNN
-F 3 "" H 6400 2500 50  0001 C CNN
-	1    6400 2500
-	1    0    0    -1
-$EndComp
-$Comp
 L GNDREF #PWR069
 U 1 1 58EA8C86
@@
 $EndComp
 $Comp
-L +5VD #PWR070
-U 1 1 58EA8C97
-P 6400 4200
-F 0 "#PWR070" H 6400 4050 50  0001 C CNN
-F 1 "+5VD" H 6400 4340 50  0000 C CNN
-F 2 "" H 6400 4200 50  0001 C CNN
-F 3 "" H 6400 4200 50  0001 C CNN
-	1    6400 4200
-	1    0    0    -1
-$EndComp
-$Comp
 L GNDREF #PWR071
 U 1 1 58EA8C9D
@@
 $EndComp
 Wire Wire Line
-	1300 850  1300 1750
+	1300 850  1300 1250
+Wire Wire Line
+	1300 1250 1300 1750
 Wire Wire Line
 	1100 850  1300 850
@@
 	3900 1500 5950 1500
 Wire Wire Line
-	3900 1400 5950 1400
-Wire Wire Line
-	3900 1300 5950 1300
+	3900 1400 5650 1400
+Wire Wire Line
+	5650 1400 5950 1400
+Wire Wire Line
+	3900 1300 5750 1300
+Wire Wire Line
+	5750 1300 5950 1300
 Wire Wire Line
 	6400 700  6400 800
 Wire Wire Line
-	6350 2000 6450 2000
+	6350 2000 6400 2000
+Wire Wire Line
+	6400 2000 6450 2000
 Wire Wire Line
 	6400 2000 6400 2000
 Connection ~ 6400 2000
 Wire Wire Line
-	3350 1300 3350 1800
+	3350 1300 3350 1500
+Wire Wire Line
+	3350 1500 3350 1800
 Wire Wire Line
 	3350 1800 2900 1800
@@
 	6400 2500 6400 2600
 Wire Wire Line
-	6350 3800 6450 3800
+	6350 3800 6400 3800
+Wire Wire Line
+	6400 3800 6450 3800
 Wire Wire Line
 	6400 3800 6400 3800
@@
 	6400 4200 6400 4300
 Wire Wire Line
-	6350 5500 6450 5500
+	6350 5500 6400 5500
+Wire Wire Line
+	6400 5500 6450 5500
 Wire Wire Line
 	6400 5500 6400 5500
 Connection ~ 6400 5500
 Wire Wire Line
-	5750 1300 5750 4800
+	5750 1300 5750 3100
+Wire Wire Line
+	5750 3100 5750 4800
 Connection ~ 5750 3100
 Connection ~ 5750 1300
 Wire Wire Line
-	5650 1400 5650 4900
+	5650 1400 5650 3200
+Wire Wire Line
+	5650 3200 5650 4900
 Connection ~ 5650 3200
 Connection ~ 5650 1400
@@
 F 0 "U19" H 3500 2533 50  0000 C CNN
 F 1 "74LS32" H 3500 2624 50  0000 C CNN
-F 2 "" H 3500 2850 50  0001 C CNN
+F 2 "Housings_SSOP:SSOP-14_5.3x6.2mm_Pitch0.65mm" H 3500 2850 50  0001 C CNN
 F 3 "" H 3500 2850 50  0001 C CNN
 	3    3500 2850
@@
 F 0 "U19" H 3450 4233 50  0000 C CNN
 F 1 "74LS32" H 3450 4324 50  0000 C CNN
-F 2 "" H 3450 4550 50  0001 C CNN
+F 2 "Housings_SSOP:SSOP-14_5.3x6.2mm_Pitch0.65mm" H 3450 4550 50  0001 C CNN
 F 3 "" H 3450 4550 50  0001 C CNN
 	4    3450 4550
 	-1   0    0    1
 $EndComp
+$Comp
+L +5V #PWR?
+U 1 1 59D232E2
+P 6400 700
+F 0 "#PWR?" H 6400 550 50  0001 C CNN
+F 1 "+5V" H 6415 873 50  0000 C CNN
+F 2 "" H 6400 700 50  0001 C CNN
+F 3 "" H 6400 700 50  0001 C CNN
+	1    6400 700
+	1    0    0    -1
+$EndComp
+$Comp
+L +5V #PWR?
+U 1 1 59D23330
+P 6400 2500
+F 0 "#PWR?" H 6400 2350 50  0001 C CNN
+F 1 "+5V" H 6415 2673 50  0000 C CNN
+F 2 "" H 6400 2500 50  0001 C CNN
+F 3 "" H 6400 2500 50  0001 C CNN
+	1    6400 2500
+	1    0    0    -1
+$EndComp
+$Comp
+L +5V #PWR?
+U 1 1 59D2340E
+P 6400 4200
+F 0 "#PWR?" H 6400 4050 50  0001 C CNN
+F 1 "+5V" H 6415 4373 50  0000 C CNN
+F 2 "" H 6400 4200 50  0001 C CNN
+F 3 "" H 6400 4200 50  0001 C CNN
+	1    6400 4200
+	1    0    0    -1
+$EndComp
 $EndSCHEMATC

Commit message: Lots of progress on PCB
Changed lines of the file:
@@
 $EndComp
 Wire Wire Line
-	1300 850  1300 1250
-Wire Wire Line
-	1300 1250 1300 1750
+	1300 850  1300 1750
 Wire Wire Line
 	1100 850  1300 850
@@
 	3900 1500 5950 1500
 Wire Wire Line
-	3900 1400 5650 1400
-Wire Wire Line
-	5650 1400 5950 1400
-Wire Wire Line
-	3900 1300 5750 1300
-Wire Wire Line
-	5750 1300 5950 1300
+	3900 1400 5950 1400
+Wire Wire Line
+	3900 1300 5950 1300
 Wire Wire Line
 	6400 700  6400 800
 Wire Wire Line
-	6350 2000 6400 2000
-Wire Wire Line
-	6400 2000 6450 2000
+	6350 2000 6450 2000
 Wire Wire Line
 	6400 2000 6400 2000
 Connection ~ 6400 2000
 Wire Wire Line
-	3350 1300 3350 1500
-Wire Wire Line
-	3350 1500 3350 1800
+	3350 1300 3350 1800
 Wire Wire Line
 	3350 1800 2900 1800
@@
 	6400 2500 6400 2600
 Wire Wire Line
-	6350 3800 6400 3800
-Wire Wire Line
-	6400 3800 6450 3800
+	6350 3800 6450 3800
 Wire Wire Line
 	6400 3800 6400 3800
@@
 	6400 4200 6400 4300
 Wire Wire Line
-	6350 5500 6400 5500
-Wire Wire Line
-	6400 5500 6450 5500
+	6350 5500 6450 5500
 Wire Wire Line
 	6400 5500 6400 5500
 Connection ~ 6400 5500
 Wire Wire Line
-	5750 1300 5750 3100
-Wire Wire Line
-	5750 3100 5750 4800
+	5750 1300 5750 4800
 Connection ~ 5750 3100
 Connection ~ 5750 1300
 Wire Wire Line
-	5650 1400 5650 3200
-Wire Wire Line
-	5650 3200 5650 4900
+	5650 1400 5650 4900
 Connection ~ 5650 3200
 Connection ~ 5650 1400
@@
 $EndComp
 $Comp
-L +5V #PWR?
+L +5V #PWR066
 U 1 1 59D232E2
 P 6400 700
-F 0 "#PWR?" H 6400 550 50  0001 C CNN
+F 0 "#PWR066" H 6400 550 50  0001 C CNN
 F 1 "+5V" H 6415 873 50  0000 C CNN
 F 2 "" H 6400 700 50  0001 C CNN
@@
 $EndComp
 $Comp
-L +5V #PWR?
+L +5V #PWR068
 U 1 1 59D23330
 P 6400 2500
-F 0 "#PWR?" H 6400 2350 50  0001 C CNN
+F 0 "#PWR068" H 6400 2350 50  0001 C CNN
 F 1 "+5V" H 6415 2673 50  0000 C CNN
 F 2 "" H 6400 2500 50  0001 C CNN
@@
 $EndComp
 $Comp
-L +5V #PWR?
+L +5V #PWR070
 U 1 1 59D2340E
 P 6400 4200
-F 0 "#PWR?" H 6400 4050 50  0001 C CNN
+F 0 "#PWR070" H 6400 4050 50  0001 C CNN
 F 1 "+5V" H 6415 4373 50  0000 C CNN
 F 2 "" H 6400 4200 50  0001 C CNN

Commit message: Re arranging pins and component names
to make pcb layout saner
Parts:
- U14, U16: renamed from U19; Pricing (none) -> 0.00@0
- renumbered U9 to U7
Connections:
- net MIC-MUTE-Pi: now also U14.5; no longer U14.10
- net PTT-Pi: now also U16.5; no longer U16.13
- net at J27.6 (Pin_6): now also U9.4 (COM2); no longer U9.9 (COM3)
- net at J27.7 (Pin_7): now also U9.3 (NO2); no longer U9.8 (NO3)
- net at C51.1: now also U7.3 (NO2); no longer U7.11 (NO4)
- net at U33.15 (D): now also U7.4 (COM2); no longer U7.10 (COM4)
- net at U34.15 (D): now also U14.4; no longer U14.9
- net at U35.15 (D): now also U16.4; no longer U16.12
- net at U11.7 (NC2): now also U16.6; no longer U16.11
- net at U11.8 (COM2): now also U9.5 (IN2); no longer U9.6 (IN3)
- new net: U11.9 (NO2), U14.6, U7.5 (IN2)
Changed lines of the file:
@@
 $Comp
 L TS12A44514 U9
-U 3 1 58EA90C5
+U 2 1 58EA90C5
 P 1700 1450
 F 0 "U9" H 1550 1650 60  0000 C CNN
@@
 F 2 "Housings_SSOP:TSSOP-14_4.4x5mm_Pitch0.65mm" H 2200 2750 60  0001 C CNN
 F 3 "" H 1850 1400 60  0001 C CNN
-F 4 "0.00@0" H 1750 2450 60  0001 C CNN "Pricing"
-F 5 "2-V to 12-V Single-Supply Operation• Specified ON-State Resistance:– 15-Ω Maximum With 12-V Supply– 20-Ω Maximum With 5-V Supply– 50-Ω Maximum With 3.3-V Supply• ΔRON Matching– 2.5-Ω (Max) at 12 V– 3-Ω(Max)at5V– 3.5-Ω (Max) at 3.3 V" H 2050 3000 60  0001 C CNN "Characteristics"
+F 4 "2-V to 12-V Single-Supply Operation• Specified ON-State Resistance:– 15-Ω Maximum With 12-V Supply– 20-Ω Maximum With 5-V Supply– 50-Ω Maximum With 3.3-V Supply• ΔRON Matching– 2.5-Ω (Max) at 12 V– 3-Ω(Max)at5V– 3.5-Ω (Max) at 3.3 V" H 2050 3000 60  0001 C CNN "Characteristics"
+F 5 "Texas Instruments" H 2100 2900 60  0001 C CNN "Manufacturer"
 F 6 "Low ON-State Resistance 4-Channel SPST CMOS AnalogSwitch" H 2000 2550 60  0001 C CNN "Description"
-F 7 "Texas Instruments" H 2100 2900 60  0001 C CNN "Manufacturer"
-F 8 "TSSOP14" H 2000 2650 60  0001 C CNN "Package ID"
-	3    1700 1450
+F 7 "TSSOP14" H 2000 2650 60  0001 C CNN "Package ID"
+F 8 "0.00@0" H 1750 2450 60  0001 C CNN "Pricing"
+	2    1700 1450
 	1    0    0    -1
 $EndComp
 $Comp
-L TS12A44514 U9
-U 4 1 58EA913D
+L TS12A44514 U7
+U 2 1 58EA913D
 P 2950 1150
-F 0 "U9" H 2800 1350 60  0000 C CNN
+F 0 "U7" H 2800 1350 60  0000 C CNN
 F 1 "TS12A44514" H 3250 1350 60  0000 C CNN
 F 2 "Housings_SSOP:TSSOP-14_4.4x5mm_Pitch0.65mm" H 3450 2450 60  0001 C CNN
 F 3 "" H 3100 1100 60  0001 C CNN
-F 4 "0.00@0" H 3000 2150 60  0001 C CNN "Pricing"
-F 5 "2-V to 12-V Single-Supply Operation• Specified ON-State Resistance:– 15-Ω Maximum With 12-V Supply– 20-Ω Maximum With 5-V Supply– 50-Ω Maximum With 3.3-V Supply• ΔRON Matching– 2.5-Ω (Max) at 12 V– 3-Ω(Max)at5V– 3.5-Ω (Max) at 3.3 V" H 3300 2700 60  0001 C CNN "Characteristics"
+F 4 "2-V to 12-V Single-Supply Operation• Specified ON-State Resistance:– 15-Ω Maximum With 12-V Supply– 20-Ω Maximum With 5-V Supply– 50-Ω Maximum With 3.3-V Supply• ΔRON Matching– 2.5-Ω (Max) at 12 V– 3-Ω(Max)at5V– 3.5-Ω (Max) at 3.3 V" H 3300 2700 60  0001 C CNN "Characteristics"
+F 5 "Texas Instruments" H 3350 2600 60  0001 C CNN "Manufacturer"
 F 6 "Low ON-State Resistance 4-Channel SPST CMOS AnalogSwitch" H 3250 2250 60  0001 C CNN "Description"
-F 7 "Texas Instruments" H 3350 2600 60  0001 C CNN "Manufacturer"
-F 8 "TSSOP14" H 3250 2350 60  0001 C CNN "Package ID"
-	4    2950 1150
+F 7 "TSSOP14" H 3250 2350 60  0001 C CNN "Package ID"
+F 8 "0.00@0" H 3000 2150 60  0001 C CNN "Pricing"
+	2    2950 1150
 	1    0    0    -1
 $EndComp
@@
 1-Audio Ground\n2-L audio to MUX\n3-R audio to MUX\n4-Mic +\n5-Mic -\n6- PTT +\n7- PTT -
 $Comp
-L 74LS32 U19
-U 3 1 59D22D32
+L 74LS32 U14
+U 2 1 59D22D32
 P 3500 2850
-F 0 "U19" H 3500 2533 50  0000 C CNN
+F 0 "U14" H 3500 2533 50  0000 C CNN
 F 1 "74LS32" H 3500 2624 50  0000 C CNN
 F 2 "Housings_SSOP:SSOP-14_5.3x6.2mm_Pitch0.65mm" H 3500 2850 50  0001 C CNN
 F 3 "" H 3500 2850 50  0001 C CNN
-	3    3500 2850
+F 4 "0.00@0" H 3500 2850 60  0001 C CNN "Pricing"
+	2    3500 2850
 	-1   0    0    1
 $EndComp
@@
 	2900 2850 3200 2850
 $Comp
-L 74LS32 U19
-U 4 1 59D22F35
+L 74LS32 U16
+U 2 1 59D22F35
 P 3450 4550
-F 0 "U19" H 3450 4233 50  0000 C CNN
+F 0 "U16" H 3450 4233 50  0000 C CNN
 F 1 "74LS32" H 3450 4324 50  0000 C CNN
 F 2 "Housings_SSOP:SSOP-14_5.3x6.2mm_Pitch0.65mm" H 3450 4550 50  0001 C CNN
 F 3 "" H 3450 4550 50  0001 C CNN
-	4    3450 4550
+F 4 "0.00@0" H 3450 4550 60  0001 C CNN "Pricing"
+	2    3450 4550
 	-1   0    0    1
 $EndComp

Commit message: Adding libraries and Notes
Other:
- note added: "Device power provided by\nexternal connection"
Changed lines of the file:
@@
 LIBS:interface
 LIBS:SW-gElectroMech
+LIBS:SW-Analog
+LIBS:SW-Semtech
 LIBS:edc-mux-board-cache
 EELAYER 26 0
@@
 $Descr USLetter 11000 8500
 encoding utf-8
-Sheet 6 14
+Sheet 5 14
 Title ""
 Date ""
@@
 	1    0    0    -1
 $EndComp
+Text Notes -700 1150 0    60   ~ 0
+Device power provided by\nexternal connection
 $EndSCHEMATC
