File: rpi-audio-io.sch (KiCad schematic (older format))
At the start: 18 parts

Commit message: Continuing with rpi audio interface
Parts:
- added C? (x4): 2.2uF, symbol C_Small
- added C? (x3): 10uF, symbol C_Small
- added C? (x4): 10uF, symbol CP1_Small
- added C? (x4): 0.1uF, symbol C_Small
- U?: value PCM510xA -> PCM5102A
Connections:
- net GNDREF: now also U?.10 (DEMP), U?.11 (FLT), U?.12 (DGND), U?.16 (FMT), U?.19 (DGND), U?.25 (ADR), U?.26 (MD0), U?.3 (CPGND), U?.7 (AGND), U?.~ (AGND), C?.1, C?.1, C?.2, C?.2, C?.2, C?.2, C?.2, C?.2, C?.2, C?.2, C?.2, C?.2
- net LIN: now also C?.1
- net LOUT: now also U?.6 (OUTL)
- net RIN: now also C?.1
- net ROUT: now also U?.7 (OUTR)
- net BCLK: now reaches J?.63 (GPIO18)
- net BCLK: now also U?.13 (BCLK), U?.17 (BCLK)
- net LRCLK: now reaches J?.65 (GPIO19)
- net LRCLK: now also U?.15 (LRCLK), U?.16 (LRCLK)
- net ADC>RPI: now reaches J?.69 (GPIO20)
- net ADC>RPI: now also U?.18 (DOUT)
- net RPI>DAC: now reaches J?.71 (GPIO21)
- net RPI>DAC: now also U?.14 (DIN)
- net at J?.75 (GPIO22): now also U?.17 (XSMT)
- net at J?.77 (GPIO23): now also U?.19 (GPIO_3)
- net LDOADC: now reaches U?.11 (LDO)
- net LDOADC: now also C?.1
- net +3V3: now reaches U?.13 (DVDD)
- net +3V3: now also U?.1 (CPVDD), U?.14 (IOVDD), U?.20 (DVDD), U?.8 (AVDD), U?.8 (AVDD), C?.1, C?.1, C?.1, C?.1, C?.1, C?.1, C?.2
- net 24MHz-CLK: now reaches U?.15 (SCLKI)
- net SDA3v3: now reaches U?.23 (SDA)
- net SCL3v3: now reaches U?.24 (SCL)
- net at U?.3 (VINL1): now also C?.2
- net at U?.4 (VINR1): now also C?.2
- net at U?.6 (VREF): now also C?.1
- net LDODAC: now reaches U?.18 (LDO)
- net LDODAC: now also C?.1, C?.1
- net at U?.2 (CAPP): now also C?.1
- net at U?.4 (CAPM): now also C?.2
- net at U?.5 (VNEG): now also C?.2
- no-connect marks 0 -> 13
Other:
- note added: "24MHz-CLK feeds ADC clock source\nfrom LAN9514 clock output"
- note added: "Address: 1001010"
- note added: "FMT low = i2s audio\nFLT low = normal latency filter\nDEMP low = de-emphasis control for 44.1kHz off\n"
- note added: "additional audio inputs available"
- moved on the sheet: J?G
