File: audio-mux-control.sch (KiCad schematic (older format))
At the start: 124 parts, among them J11 RasPi-CM3-Headers, J15 Outputs to Mixer, J16 Mixer_Power_CTL, J17 Light 0, J18 Light 1, J19 Headset 0, J20 Headset 1, J21 Headset 2, J22 Headset 3, J23 Headset 4, J24 Headset 5, J25 Headset 6, J26 Headset 7

Commit message: Continued working on final audio connections between headset and devices
Parts:
- removed C? (x7): 10u, Capacitors_SMD:C_0603, symbol C_Small
- removed C? (x3): 0.1uF, symbol C_Small
- removed J?: Device 1, SW-TEConn:3-794681-8, symbol Conn_01x07
- removed J?: Device 0, SW-TEConn:3-794681-8, symbol Conn_01x07
- removed J?: Device 2, SW-TEConn:3-794681-8, symbol Conn_01x07
- removed J?: Device 3, SW-TEConn:3-794681-8, symbol Conn_01x07
- removed J?: Device 4, SW-TEConn:3-794681-8, symbol Conn_01x07
- removed J?: Device 5, SW-TEConn:3-794681-8, symbol Conn_01x07
- removed J?: Device 6, SW-TEConn:3-794681-8, symbol Conn_01x07
- removed J?: Device 7, SW-TEConn:3-794681-8, symbol Conn_01x07
- removed U? (x7): TS12A44514, Housings_SSOP:TSSOP-14_4.4x5mm_Pitch0.65mm, symbol TS12A44514
- removed U? (x6): 74LS32, Housings_SSOP:SSOP-14_5.3x6.2mm_Pitch0.65mm, symbol 74LS32
- removed U? (x2): ADG708, Housings_SSOP:TSSOP-16_4.4x5mm_Pitch0.65mm, symbol ADG708
- added C? (x24): 0.1uF, symbol C_Small
- added C? (x7): 10u, Capacitors_SMD:C_0603, symbol C_Small
- added D? (x16): 0582BQ, symbol 0582BQ
- added D? (x8): TPD1E10B06, symbol TPD1E10B06
- added J?: Device 0, SW-TEConn:3-794681-8, symbol Conn_01x08
- added J?: Device 1, SW-TEConn:3-794681-8, symbol Conn_01x08
- added J?: Device 2, SW-TEConn:3-794681-8, symbol Conn_01x08
- added J?: Device 3, SW-TEConn:3-794681-8, symbol Conn_01x08
- added J?: Device 4, SW-TEConn:3-794681-8, symbol Conn_01x08
- added J?: Device 5, SW-TEConn:3-794681-8, symbol Conn_01x08
- added J?: Device 6, SW-TEConn:3-794681-8, symbol Conn_01x08
- added J?: Device 7, SW-TEConn:3-794681-8, symbol Conn_01x08
- added U? (x8): ADG715, Housings_SSOP:TSSOP-24_4.4x7.8mm_Pitch0.65mm, symbol ADG715
- added U? (x16): ADG708, Housings_SSOP:TSSOP-16_4.4x5mm_Pitch0.65mm, symbol ADG708
- added U? (x16): ADG734, Housings_SSOP:TSSOP-20_4.4x6.5mm_Pitch0.65mm, symbol ADG734
- added U? (x7): TS12A44514, Housings_SSOP:TSSOP-14_4.4x5mm_Pitch0.65mm, symbol TS12A44514
- added U? (x7): 74LS32, Housings_SSOP:SSOP-14_5.3x6.2mm_Pitch0.65mm, symbol 74LS32
- J19: Pricing (none) -> 0.00@0
Connections:
- net labels added: AMP-MIC-IN-0, AMP-MIC-IN-1, AMP-MIC-IN-2, AMP-MIC-IN-3, AMP-MIC-IN-4, AMP-MIC-IN-5, AMP-MIC-IN-6, AMP-MIC-IN-7
- net labels removed: AUDIO-GROUND, LEFT-OUT, PTT-Pi, RIGHT-OUT
- wire segments 727 -> 1321
Other:
- note added: "1-Ground\n2-L audio to MUX\n3-R audio to MUX\n4-Mic +\n5-Mic -\n6-+5V for active cables\n7- PTT +\n8- PTT -"
- note added: "Address lines for MUXes (2 different voltage levels)\nPTT from IO expander (5v)\ntwo SPDT switches from IO expander (2.5v)"
- note added: "Connect to Stereo Distro amp\nfrom RPi audio out"
- note added: "L/R RPi\nAudio"
- note added: "RPi audio/\nMic audio"
- note added: "out 1 goes to L_In/R_in bus\nout 2 goes to Mixer"
- note added: "out 1 goes to Mixer\nout 2 goes to L_In/R_in bus"
- note removed: "1-Audio Ground\n2-L audio to MUX\n3-R audio to MUX\n4-Mic +\n5-Mic -\n6- PTT +\n7- PTT -"
- moved on the sheet: C?, J15, U?A, U?C

Commit message: Finished audio and control busses on device side
Parts:
- added C? (x5): 0.1uF, symbol C_Small
- added R? (x5): 10kΩ, symbol R_Small
- added U? (x5): TCA9555, Housings_SSOP:TSSOP-24_4.4x7.8mm_Pitch0.65mm, symbol TCA9555
Connections:
- net labels added: AMP-MIC-IN-0-0, AMP-MIC-IN-0-1, AMP-MIC-IN-0-2, AMP-MIC-IN-0-3, AMP-MIC-IN-0-4, AMP-MIC-IN-0-5, AMP-MIC-IN-0-6, AMP-MIC-IN-0-7, AMP-MIC-IN-1-0, AMP-MIC-IN-1-1, AMP-MIC-IN-1-2, AMP-MIC-IN-1-3, AMP-MIC-IN-1-4, AMP-MIC-IN-1-5, AMP-MIC-IN-1-6, AMP-MIC-IN-1-7, AMP-MIC-IN-2-0, AMP-MIC-IN-2-1, AMP-MIC-IN-2-2, AMP-MIC-IN-2-3, AMP-MIC-IN-2-4, AMP-MIC-IN-2-5, AMP-MIC-IN-2-6, AMP-MIC-IN-2-7, AMP-MIC-IN-3-0, AMP-MIC-IN-3-1, AMP-MIC-IN-3-2, AMP-MIC-IN-3-3, AMP-MIC-IN-3-4, AMP-MIC-IN-3-5, AMP-MIC-IN-3-6, AMP-MIC-IN-3-7, AMP-MIC-IN-4-0, AMP-MIC-IN-4-1, AMP-MIC-IN-4-2, AMP-MIC-IN-4-3, AMP-MIC-IN-4-4, AMP-MIC-IN-4-5, AMP-MIC-IN-4-6, AMP-MIC-IN-4-7, AMP-MIC-IN-5-0, AMP-MIC-IN-5-1, AMP-MIC-IN-5-2, AMP-MIC-IN-5-3, AMP-MIC-IN-5-4, AMP-MIC-IN-5-5, AMP-MIC-IN-5-6, AMP-MIC-IN-5-7, AMP-MIC-IN-6-0, AMP-MIC-IN-6-1, AMP-MIC-IN-6-2, AMP-MIC-IN-6-3, AMP-MIC-IN-6-4, AMP-MIC-IN-6-5, AMP-MIC-IN-6-6, AMP-MIC-IN-6-7, AMP-MIC-IN-7-0, AMP-MIC-IN-7-1, AMP-MIC-IN-7-2, AMP-MIC-IN-7-3, AMP-MIC-IN-7-4, AMP-MIC-IN-7-5, AMP-MIC-IN-7-6, AMP-MIC-IN-7-7, DEV-MIC-IN-XBAR-CTL0, DEV-MIC-IN-XBAR-CTL1, DEV-MIC-IN-XBAR-CTL10, DEV-MIC-IN-XBAR-CTL11, DEV-MIC-IN-XBAR-CTL12, DEV-MIC-IN-XBAR-CTL13, DEV-MIC-IN-XBAR-CTL14, DEV-MIC-IN-XBAR-CTL15, DEV-MIC-IN-XBAR-CTL16, DEV-MIC-IN-XBAR-CTL17, DEV-MIC-IN-XBAR-CTL18, DEV-MIC-IN-XBAR-CTL19, DEV-MIC-IN-XBAR-CTL2, DEV-MIC-IN-XBAR-CTL20, DEV-MIC-IN-XBAR-CTL21, DEV-MIC-IN-XBAR-CTL22, DEV-MIC-IN-XBAR-CTL23, DEV-MIC-IN-XBAR-CTL3, DEV-MIC-IN-XBAR-CTL4, DEV-MIC-IN-XBAR-CTL5, DEV-MIC-IN-XBAR-CTL6, DEV-MIC-IN-XBAR-CTL7, DEV-MIC-IN-XBAR-CTL8, DEV-MIC-IN-XBAR-CTL9, DEV-MIC-IN-XBAR-CTL[0..23], DEV-PTT-XBAR-CTL0, DEV-PTT-XBAR-CTL1, DEV-PTT-XBAR-CTL10, DEV-PTT-XBAR-CTL11, DEV-PTT-XBAR-CTL12, DEV-PTT-XBAR-CTL13, DEV-PTT-XBAR-CTL14, DEV-PTT-XBAR-CTL15, DEV-PTT-XBAR-CTL16, DEV-PTT-XBAR-CTL17, DEV-PTT-XBAR-CTL18, DEV-PTT-XBAR-CTL19, DEV-PTT-XBAR-CTL2, DEV-PTT-XBAR-CTL20, DEV-PTT-XBAR-CTL21, DEV-PTT-XBAR-CTL22, DEV-PTT-XBAR-CTL23, DEV-PTT-XBAR-CTL3, DEV-PTT-XBAR-CTL4, DEV-PTT-XBAR-CTL5, DEV-PTT-XBAR-CTL6, DEV-PTT-XBAR-CTL7, DEV-PTT-XBAR-CTL8, DEV-PTT-XBAR-CTL9, DEV-PTT-XBAR-CTL[0..23], HEADSET-AUDIO-SOURCE-L-0, HEADSET-AUDIO-SOURCE-L-1, HEADSET-AUDIO-SOURCE-L-2, HEADSET-AUDIO-SOURCE-L-3, HEADSET-AUDIO-SOURCE-L-4, HEADSET-AUDIO-SOURCE-L-5, HEADSET-AUDIO-SOURCE-L-6, HEADSET-AUDIO-SOURCE-L-7, HEADSET-AUDIO-SOURCE-L-[0..7], HEADSET-AUDIO-SOURCE-R-0, HEADSET-AUDIO-SOURCE-R-1, HEADSET-AUDIO-SOURCE-R-2, HEADSET-AUDIO-SOURCE-R-3, HEADSET-AUDIO-SOURCE-R-4, HEADSET-AUDIO-SOURCE-R-5, HEADSET-AUDIO-SOURCE-R-6, HEADSET-AUDIO-SOURCE-R-7, HEADSET-AUDIO-SOURCE-R-[0..7], MIXER-OUT-L-0, MIXER-OUT-L-1, MIXER-OUT-L-2, MIXER-OUT-L-3, MIXER-OUT-L-4, MIXER-OUT-L-5, MIXER-OUT-L-6, MIXER-OUT-L-7, MIXER-OUT-L-[0..7], MIXER-OUT-R-0, MIXER-OUT-R-1, MIXER-OUT-R-2, MIXER-OUT-R-3, MIXER-OUT-R-4, MIXER-OUT-R-5, MIXER-OUT-R-6, MIXER-OUT-R-7, MIXER-OUT-R-[0..7], RPI-LR-0, RPI-LR-1, RPI-LR-2, RPI-LR-3, RPI-LR-4, RPI-LR-5, RPI-LR-6, RPI-LR-7, RPI-LR-[0..7], RPI-PTT-0, RPI-PTT-1, RPI-PTT-2, RPI-PTT-3, RPI-PTT-4, RPI-PTT-5, RPI-PTT-6, RPI-PTT-7, RPI-PTT-[0..7], RPI/MIC-0, RPI/MIC-1, RPI/MIC-2, RPI/MIC-3, RPI/MIC-4, RPI/MIC-5, RPI/MIC-6, RPI/MIC-7, RPI/MIC-[0..7]
- net labels removed: AMP-MIC-IN-0, AMP-MIC-IN-1, AMP-MIC-IN-2, AMP-MIC-IN-3, AMP-MIC-IN-4, AMP-MIC-IN-5, AMP-MIC-IN-6, AMP-MIC-IN-7
Other:
- note added: "ADDR: 0100001"
- note added: "ADDR: 0100010"
- note added: "ADDR: 0100011"
- moved on the sheet: F14, J16

Commit message: Finished audio distro on main sheet. Started RPi Audio Interface
Parts:
- removed unit 7 of J11
Connections:
- net RPI-OUT-L0: now reaches U?.7 (NC2)
- net RPI-OUT-R0: now reaches U?.9 (NO2)
- net RPI-OUT-L1: now reaches U?.17 (NC4)
- net RPI-OUT-R1: now reaches U?.19 (NO4)
- net RPI-OUT-L2: now reaches U?.7 (NC2)
- net RPI-OUT-R2: now reaches U?.9 (NO2)
- net RPI-OUT-L3: now reaches U?.17 (NC4)
- net RPI-OUT-R3: now reaches U?.19 (NO4)
- net RPI-OUT-L4: now reaches U?.7 (NC2)
- net RPI-OUT-R4: now reaches U?.9 (NO2)
- net RPI-OUT-L5: now reaches U?.17 (NC4)
- net RPI-OUT-R5: now reaches U?.19 (NO4)
- net RPI-OUT-L6: now reaches U?.7 (NC2)
- net RPI-OUT-R6: now reaches U?.9 (NO2)
- net RPI-OUT-L7: now reaches U?.17 (NC4)
- net RPI-OUT-R7: now reaches U?.19 (NO4)
- net CE0: no longer names the net of J11.27 (GPIO8)
- net CE1: no longer names the net of J11.23 (GPIO7)
- net MISO: no longer names the net of J11.29 (GPIO9)
- net MOSI: no longer names the net of J11.33 (GPIO10)
- net SCLK: no longer names the net of J11.35 (GPIO11)
- no-connect marks 10 -> 13
Other:
- note added: "i2c pins (I2C 0) GPIO 0,1 alt0\ni2c pins (I2C 1) GPIO 2,3 alt0\n"
- note removed: "GPIO 18-21 are PCM/i2s data"
- note removed: "i2c pins (I2C 1) GPIO 2,3 alt0\nspi pins (SPI 0) GPIO 7,8,9,10,11 alt0"

Commit message: Continuing with rpi audio interface
Other:
- note added: "GPIO Pins 4,5,6,7 are\nused to monitor PiUPS"
- note removed: "GPIO Pins 4,5,6,12 are\nused to monitor PiUPS"
Changed lines of the file:
@@
 Standard Android headset controls can be accomodated\nwith an external converter that measures the resistances\non the mic line and transforms those into a pulse code on\nthe mic mute line that the raspberry pi is monitoring for.
 Text Notes 22550 13750 0    60   ~ 0
-GPIO Pins 4,5,6,12 are\nused to monitor PiUPS
+GPIO Pins 4,5,6,7 are\nused to monitor PiUPS
 $Comp
 L TCA9548A U?
@@
 	8850 2100 8850 35200
 Wire Bus Line
-	27500 35200 8850 35200
+	8850 35200 27500 35200
 Wire Bus Line
-	27500 31450 27500 35200
+	27500 35200 27500 31450
 Wire Bus Line
 	9000 1900 9000 35050
@@
 F5 "RPI-R-IN[0..7]" I L 23250 31550 60
 $EndSheet
-NoConn ~ 21800 14000
 NoConn ~ 21800 14100
 NoConn ~ 21800 14350
@@
 	27200 31650 26850 31650
 Wire Bus Line
-	26850 31450 27500 31450
+	27500 31450 26850 31450
+NoConn ~ 21800 14650
 $EndSCHEMATC

Commit message: Removing and archiving raspberry pi stuff
Parts:
- removed J11: RasPi-CM3-Headers, Sockets:Socket_SODIMM_DDR1-2_TE_1612618, symbol RasPi-CM3-Headers
Connections:
- no-connect marks 13 -> 1
Other:
- note removed: "GPIO Pins 4,5,6,7 are\nused to monitor PiUPS"
Changed lines of the file:
@@
 $Descr User 30000 40000
 encoding utf-8
-Sheet 4 50
+Sheet 4 47
 Title ""
 Date ""
@@
 Text Label 26250 1050 2    60   ~ 0
 MIC-IN-0
-$Comp
-L RasPi-CM3-Headers J11
-U 5 1 59349764
-P 22150 13700
-F 0 "J11" H 22050 13200 60  0000 C CNN
-F 1 "RasPi-CM3-Headers" V 22400 13700 60  0000 C CNN
-F 2 "Sockets:Socket_SODIMM_DDR1-2_TE_1612618" H 22200 18800 60  0001 C CNN
-F 3 "https://www.raspberrypi.org/documentation/hardware/computemodule/RPI-CM-DATASHEET-V1_0.pdf" H 22200 18500 60  0001 C CNN
-F 4 "0.00@0" H 22150 18400 60  0001 C CNN "Pricing"
-F 5 "Raspberry Pi Compute Module 3 Connector Pinout" H 22150 18700 60  0001 C CNN "Description"
-F 6 "Raspberry Pi Foundation" H 22150 18600 60  0001 C CNN "Manufacturer"
-	5    22150 13700
-	1    0    0    -1
-$EndComp
-$Comp
-L RasPi-CM3-Headers J11
-U 6 1 5934A1A4
-P 22150 14750
-F 0 "J11" H 22100 14250 60  0000 C CNN
-F 1 "RasPi-CM3-Headers" V 22400 14750 60  0000 C CNN
-F 2 "Sockets:Socket_SODIMM_DDR1-2_TE_1612618" H 22200 19850 60  0001 C CNN
-F 3 "https://www.raspberrypi.org/documentation/hardware/computemodule/RPI-CM-DATASHEET-V1_0.pdf" H 22200 19550 60  0001 C CNN
-F 4 "0.00@0" H 22150 19450 60  0001 C CNN "Pricing"
-F 5 "Raspberry Pi Compute Module 3 Connector Pinout" H 22150 19750 60  0001 C CNN "Description"
-F 6 "Raspberry Pi Foundation" H 22150 19650 60  0001 C CNN "Manufacturer"
-	6    22150 14750
-	1    0    0    -1
-$EndComp
 Text Label 26250 1450 2    60   ~ 0
 MIC-MUTE-0
@@
 Text Notes 19850 10650 0    60   ~ 0
 Verify IO voltage levels for\nswitch inputs.
-Text Label 21550 13500 2    60   ~ 0
-SDA
-Text Label 21550 13600 2    60   ~ 0
-SCL
-NoConn ~ 21800 13300
-NoConn ~ 21800 13400
-NoConn ~ 21800 14750
-NoConn ~ 21800 14850
-NoConn ~ 21800 14950
-NoConn ~ 21800 15050
-NoConn ~ 21800 15150
 Text Label 25600 13250 2    60   ~ 0
 SDA
@@
 Text Notes 25000 150  0    60   ~ 0
 Standard Android headset controls can be accomodated\nwith an external converter that measures the resistances\non the mic line and transforms those into a pulse code on\nthe mic mute line that the raspberry pi is monitoring for.
-Text Notes 22550 13750 0    60   ~ 0
-GPIO Pins 4,5,6,7 are\nused to monitor PiUPS
 $Comp
 L TCA9548A U?
@@
 	26250 8350 26900 8350
 Wire Wire Line
-	21800 13500 21550 13500
-Wire Wire Line
-	21550 13600 21800 13600
-Wire Wire Line
 	25600 13250 26400 13250
 Wire Wire Line
@@
 Text Label 15950 35200 0    60   ~ 0
 RPI-OUT-L[0..7]
-$Sheet
-S 23250 30900 3600 2300
-U 5A632C9B
-F0 "RPI Audio IO" 60
-F1 "rpi-audio-io.sch" 60
-F2 "RPI-L-OUT[0..7]" O R 26850 31450 60
-F3 "RPI-R-OUT[0..7]" O R 26850 31650 60
-F4 "RPI-L-IN[0..7]" I L 23250 31350 60
-F5 "RPI-R-IN[0..7]" I L 23250 31550 60
-$EndSheet
-NoConn ~ 21800 14100
-NoConn ~ 21800 14350
-NoConn ~ 21800 14450
-NoConn ~ 21800 14550
 Wire Wire Line
 	21900 1450 22050 1450
@@
 Wire Bus Line
 	27500 31450 26850 31450
-NoConn ~ 21800 14650
 $EndSCHEMATC

Commit message: Raspberry Pi removal cleanup and simplification
Parts:
- removed C?: 0.1uF, symbol C_Small
- removed R?: 10kΩ, symbol R_Small
- removed U?: TCA9555, Housings_SSOP:TSSOP-24_4.4x7.8mm_Pitch0.65mm, symbol TCA9555
- removed U? (x16): ADG734, Housings_SSOP:TSSOP-20_4.4x6.5mm_Pitch0.65mm, symbol ADG734
Connections:
- net at U?.6 (D1): now also U?.8 (D)
- net at U?.8 (D2): now also U?.8 (D)
- net at U?.10 (D3): now also U?.8 (D)
- net at U?.12 (D4): now also U?.8 (D)
- net at U?.13 (D5): now also U?.8 (D)
- net at U?.15 (D6): now also U?.8 (D)
- net at U?.17 (D7): now also U?.8 (D)
- net at U?.19 (D8): now also U?.8 (D)
- net RPI/MIC-0: no longer names the net of U?.4 (P00)
- net RPI/MIC-1: no longer names the net of U?.5 (P01)
- net RPI/MIC-2: no longer names the net of U?.6 (P02)
- net RPI/MIC-3: no longer names the net of U?.7 (P03)
- net RPI/MIC-4: no longer names the net of U?.8 (P04)
- net RPI/MIC-5: no longer names the net of U?.9 (P05)
- net RPI/MIC-6: no longer names the net of U?.10 (P06)
- net RPI/MIC-7: no longer names the net of U?.11 (P07)
Other:
- note removed: "Address lines for MUXes (2 different voltage levels)\nPTT from IO expander (5v)\ntwo SPDT switches from IO expander (2.5v)"
- note removed: "Connect to Stereo Distro amp\nfrom RPi audio out"
- note removed: "L/R RPi\nAudio"
- note removed: "RPi audio/\nMic audio"

Commit message: Removed flashlight and headset power and control connectors
Parts:
- removed F12, F13: 2A, SW-Littelfuse:NANO-0154-OMNI-BLOK-Fuse-Holder, symbol Fuse_Small
- removed F14: 600mA, SW-Littelfuse:NANO-0154-OMNI-BLOK-Fuse-Holder, symbol Fuse_Small
- removed J16: Mixer_Power_CTL, SW-TEConn:3-794681-8, symbol Conn_01x08
- removed J17: Light 0, Pin_Headers:Pin_Header_Straight_1x04_Pitch2.54mm, symbol Conn_01x04
- removed J18: Light 1, Pin_Headers:Pin_Header_Straight_1x04_Pitch2.54mm, symbol Conn_01x04
- added J?: Mixer Audio In, symbol Conn_01x03
Connections:
- net GNDREF: now also J?.3 (Pin_3)
- net Headset LR audio out Mux and Source Selection/MIXER_L_IN: now also J?.1 (Pin_1)
- net Headset LR audio out Mux and Source Selection/MIXER_R_IN: now also J?.2 (Pin_2)
Other:
- note added: "1=Left=Tip\n2=Right=Ring\n3=GND=Sleeve\n"
- note removed: "1=Left=Tip\n2=Right=Ring\n3=GNDA=Sleeve\n4=SDA\n5=SCL\n6=+12V\n7=GND\n8=GND"
- note removed: "Flashlight/headlamp connectors\n12V+, GND, SDA, SCL"
- note removed: "Verify IO voltage levels for\nswitch inputs."
- note removed: "i2c pins (I2C 0) GPIO 0,1 alt0\ni2c pins (I2C 1) GPIO 2,3 alt0\n"

Commit message: Starting reworking of power supply w/ dual rails
Connections:
- net GNDA is gone; now on net GNDREF: J19.1 (Pin_1), J19.5 (Pin_5), J20.1 (Pin_1), J20.5 (Pin_5), J21.1 (Pin_1), J21.5 (Pin_5), J22.1 (Pin_1), J22.5 (Pin_5), J23.1 (Pin_1), J23.5 (Pin_5), J24.1 (Pin_1), J24.5 (Pin_5), J25.1 (Pin_1), J25.5 (Pin_5), J26.1 (Pin_1), J26.5 (Pin_5)
Other:
- note removed: "TCA9534 addresses all start with 0100 (32-39),\nTCA9534A variant starts with 0111 (56-63)"
- moved on the sheet: C43, C44, C45, C46, C47, C48, C49, C50, C?, D?, J19, J20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
