File: 1-8-stereo-buffer-amp.sch (KiCad schematic (older format))
At the start: 69 parts

Commit message: Adding sheet for arduino nano ethernet connections
Parts:
- gave numbers to parts that had none: 51

Commit message: Finished schematic layout, starting to assign footprints
Parts:
- renumbered C178 to C182, C179 to C183, C173 to C184, C177 to C185, C172 to C186, C176 to C187, C170 to C188, C174 to C189, C171 to C190, C175 to C191, R94 to R106, R78 to R107, R77 to R108, R95 to R109, R74 to R110, R79 to R111, R96 to R112, R76 to R113, R80 to R114, R75 to R115, R97 to R116, R81 to R117, R98 to R118, R82 to R119, R99 to R120, R83 to R121, R100 to R122, R84 to R123, R101 to R124, R85 to R125, R102 to R126, R86 to R127, R103 to R128, R87 to R129, R104 to R130, R88 to R131, R105 to R132, R89 to R133, R106 to R134, R90 to R135, R107 to R136, R91 to R137, R108 to R138, R92 to R139, R109 to R140, R93 to R141, U75 to U77, U78 to U77, U74 to U78, U76 to U79, U77 to U79, U77 to U80, U75 to U80, U78 to U81, U76 to U81

Commit message: Finalized footprint assignment. ready for pcb time
Parts:
- C182, C183, C184, C185, C186, C187, C188, C189, C190, C191: footprint (none) -> Capacitor_SMD:C_0805_2012Metric_Pad1.15x1.50mm_HandSolder
- R106, R107, R108, R109, R110, R111, R112, R113, R114, R115, R116, R117, R118, R119, R120, R121, R122, R123, R124, R125, R126, R127, R128, R129, R130, R131, R132, R133, R134, R135, R136, R137, R138, R139, R140, R141: footprint (none) -> Resistor_SMD:R_0603_1608Metric_Pad0.84x1.00mm_HandSolder
- U77, U79, U80, U81: footprint (none) -> Package_SOIC:SOIC-14_3.9x8.7mm_P1.27mm
- U78: footprint (none) -> Package_SOIC:SOIC-8_3.9x4.9mm_P1.27mm

Commit message: Finished fixing power supply and starting pcb layout
Parts:
- C182, C183, C184, C185, C186, C187, C188, C189, C190, C191: Characteristics (none) -> 10% -55ºC + 125ºC X7R; Manufacturer (none) -> TDK; Manufacturer Part Number (none) -> CGA4J2X7R1H104K125AE
- R106, R107, R108, R109, R110, R111, R112, R113, R114, R115, R116, R117, R118, R119, R120, R121, R122, R123, R124, R125, R126, R127, R128, R129, R130, R131, R132, R133, R134, R135, R136, R137, R138, R139, R140, R141: value 100k -> 100kΩ; Characteristics (none) -> 0.5% -55ºC +125ºC 100mW; Description (none) -> Thin Film Resistor; Manufacturer (none) -> Vishay; Manufacturer Part Number (none) -> MCT06030D1003DP500; Package ID (none) -> 1608 metric
- U77, U79, U80, U81: footprint Package_SOIC:SOIC-14_3.9x8.7mm_P1.27mm -> Package_SSOP:TSSOP-14_4.4x5mm_P0.65mm; Manufacturer Part Number (none) -> OPA1604AIPWR
- U78: Manufacturer Part Number (none) -> OPA1602AIDGKR

Commit message: Fixed 1:8 buffer amp unit mixup, placed more components
Connections:
- net GNDREF: now also U77.10 (C+), U77.12 (D+), U79.10 (C+), U79.12 (D+), U80.10 (C+), U80.12 (D+), U81.10 (C+), U81.12 (D+); no longer U77.10 (C+), U77.12 (D+), U79.10 (C+), U79.12 (D+), U80.10 (C+), U80.12 (D+), U81.10 (C+), U81.12 (D+)
- net L_OUT1: now also U77.14 (D); no longer U77.8 (C)
- net L_OUT3: now also U79.14 (D); no longer U79.8 (C)
- net L_OUT5: now also U80.14 (D); no longer U80.8 (C)
- net L_OUT7: now also U81.14 (D); no longer U81.8 (C)
- net R_OUT1: now also U77.8 (C); no longer U77.14 (D)
- net R_OUT3: now also U79.8 (C); no longer U79.14 (D)
- net R_OUT5: now also U80.8 (C); no longer U80.14 (D)
- net R_OUT7: now also U81.8 (C); no longer U81.14 (D)
- net at R112.2, R114.1: now also U77.13 (D-); no longer U77.9 (C-)
- net at R116.2, R117.1: now also U77.9 (C-); no longer U77.13 (D-)
- net at R122.2, R123.1: now also U79.13 (D-); no longer U79.9 (C-)
- net at R124.2, R125.1: now also U79.9 (C-); no longer U79.13 (D-)
- net at R130.2, R131.1: now also U80.13 (D-); no longer U80.9 (C-)
- net at R132.2, R133.1: now also U80.9 (C-); no longer U80.13 (D-)
- net at R138.2, R139.1: now also U81.13 (D-); no longer U81.9 (C-)
- net at R140.2, R141.1: now also U81.9 (C-); no longer U81.13 (D-)
