File: headset-audio-out-mux-switching.sch (KiCad schematic (older format))
At the start: 76 parts

Commit message: Adding sheet for arduino nano ethernet connections
Parts:
- gave numbers to parts that had none: 64

Commit message: Finished schematic layout, starting to assign footprints
Parts:
- renumbered C142 to C146, C159 to C147, C134 to C148, C151 to C149, C143 to C150, C160 to C151, C135 to C152, C152 to C153, C144 to C154, C161 to C155, C136 to C156, C153 to C157, C145 to C158, C162 to C159, C137 to C160, C154 to C161, C146 to C162, C138 to C164, C155 to C165, C147 to C166, C164 to C167, C139 to C168, C156 to C169, C148 to C170, C165 to C171, C140 to C172, C157 to C173, C149 to C174, C166 to C175, C141 to C176, C158 to C177, C167 to C178, C168 to C179, C150 to C180, C169 to C181, R71 to R102, R72 to R103, R70 to R104, R73 to R105, U12 to U13, U13 to U14, U14 to U16, U54 to U57, U63 to U58, U55 to U59, U64 to U60, U56 to U61, U65 to U62, U57 to U63, U66 to U64, U58 to U65, U67 to U66, U59 to U67, U60 to U69, U69 to U70, U61 to U71, U70 to U72, U71 to U73, U72 to U74, U62 to U75, U73 to U76
Connections:
- net GNDREF: now also C147.2, C149.1, U58.14 (GND)

Commit message: Finalized footprint assignment. ready for pcb time
Parts:
- C146, C147, C148, C149, C150, C151, C152, C153, C154, C155, C156, C157, C158, C159, C160, C161, C162, C163, C164, C165, C166, C167, C168, C169, C170, C171, C172, C173, C174, C175, C176, C177, C178, C179, C180, C181: footprint (none) -> Capacitor_SMD:C_0805_2012Metric_Pad1.15x1.50mm_HandSolder
- R102, R103, R104, R105: footprint (none) -> Resistor_SMD:R_0603_1608Metric_Pad0.84x1.00mm_HandSolder
- U11, U13, U14, U16: footprint Housings_SSOP:TSSOP-20_4.4x6.5mm_Pitch0.65mm -> Package_SSOP:TSSOP-20_4.4x6.5mm_P0.65mm
- U57, U58, U59, U60, U61, U62, U63, U64, U65, U66, U67, U68, U69, U70, U71, U72: footprint Housings_SSOP:TSSOP-16_4.4x5mm_Pitch0.65mm -> Package_SSOP:TSSOP-16_4.4x5mm_P0.65mm
- U73, U74, U75, U76: footprint Housings_SSOP:TSSOP-24_4.4x7.8mm_Pitch0.65mm -> Package_SSOP:TSSOP-24_4.4x7.8mm_P0.65mm

Commit message: Fix non printing characters in descriptions
Parts:
- U11, U13, U14, U16: Description CMOS, 2.5 Low Voltage, Quad SPDT Switch -> CMOS, 2.5 Low Voltage, Quad SPDT Switch
Changed lines of the file:
@@
 F 4 "0.00@0" H 9850 16000 60  0001 C CNN "Pricing"
 F 5 "Analog Devices" H 9900 16300 60  0001 C CNN "Manufacturer"
-F 6 "CMOS, 2.5 Low Voltage, Quad SPDT Switch" H 9800 16100 60  0001 C CNN "Description"
+F 6 "CMOS, 2.5 Low Voltage, Quad SPDT Switch" H 9800 16100 60  0001 C CNN "Description"
 F 7 "TSSOP20" H 9850 16200 60  0001 C CNN "Package ID"
 	1    9850 15550
@@
 F 4 "0.00@0" H 9850 16450 60  0001 C CNN "Pricing"
 F 5 "Analog Devices" H 9900 16750 60  0001 C CNN "Manufacturer"
-F 6 "CMOS, 2.5 Low Voltage, Quad SPDT Switch" H 9800 16550 60  0001 C CNN "Description"
+F 6 "CMOS, 2.5 Low Voltage, Quad SPDT Switch" H 9800 16550 60  0001 C CNN "Description"
 F 7 "TSSOP20" H 9850 16650 60  0001 C CNN "Package ID"
 	2    9850 16000
@@
 F 4 "0.00@0" H 9850 17350 60  0001 C CNN "Pricing"
 F 5 "Analog Devices" H 9900 17650 60  0001 C CNN "Manufacturer"
-F 6 "CMOS, 2.5 Low Voltage, Quad SPDT Switch" H 9800 17450 60  0001 C CNN "Description"
+F 6 "CMOS, 2.5 Low Voltage, Quad SPDT Switch" H 9800 17450 60  0001 C CNN "Description"
 F 7 "TSSOP20" H 9850 17550 60  0001 C CNN "Package ID"
 	3    9850 16900
@@
 F 4 "0.00@0" H 9850 17800 60  0001 C CNN "Pricing"
 F 5 "Analog Devices" H 9900 18100 60  0001 C CNN "Manufacturer"
-F 6 "CMOS, 2.5 Low Voltage, Quad SPDT Switch" H 9800 17900 60  0001 C CNN "Description"
+F 6 "CMOS, 2.5 Low Voltage, Quad SPDT Switch" H 9800 17900 60  0001 C CNN "Description"
 F 7 "TSSOP20" H 9850 18000 60  0001 C CNN "Package ID"
 	4    9850 17350
@@
 F 4 "0.00@0" H 9850 18700 60  0001 C CNN "Pricing"
 F 5 "Analog Devices" H 9900 19000 60  0001 C CNN "Manufacturer"
-F 6 "CMOS, 2.5 Low Voltage, Quad SPDT Switch" H 9800 18800 60  0001 C CNN "Description"
+F 6 "CMOS, 2.5 Low Voltage, Quad SPDT Switch" H 9800 18800 60  0001 C CNN "Description"
 F 7 "TSSOP20" H 9850 18900 60  0001 C CNN "Package ID"
 	1    9850 18250
@@
 F 4 "0.00@0" H 9850 19150 60  0001 C CNN "Pricing"
 F 5 "Analog Devices" H 9900 19450 60  0001 C CNN "Manufacturer"
-F 6 "CMOS, 2.5 Low Voltage, Quad SPDT Switch" H 9800 19250 60  0001 C CNN "Description"
+F 6 "CMOS, 2.5 Low Voltage, Quad SPDT Switch" H 9800 19250 60  0001 C CNN "Description"
 F 7 "TSSOP20" H 9850 19350 60  0001 C CNN "Package ID"
 	2    9850 18700
@@
 F 4 "0.00@0" H 9850 20050 60  0001 C CNN "Pricing"
 F 5 "Analog Devices" H 9900 20350 60  0001 C CNN "Manufacturer"
-F 6 "CMOS, 2.5 Low Voltage, Quad SPDT Switch" H 9800 20150 60  0001 C CNN "Description"
+F 6 "CMOS, 2.5 Low Voltage, Quad SPDT Switch" H 9800 20150 60  0001 C CNN "Description"
 F 7 "TSSOP20" H 9850 20250 60  0001 C CNN "Package ID"
 	3    9850 19600
@@
 F 4 "0.00@0" H 9850 20500 60  0001 C CNN "Pricing"
 F 5 "Analog Devices" H 9900 20800 60  0001 C CNN "Manufacturer"
-F 6 "CMOS, 2.5 Low Voltage, Quad SPDT Switch" H 9800 20600 60  0001 C CNN "Description"
+F 6 "CMOS, 2.5 Low Voltage, Quad SPDT Switch" H 9800 20600 60  0001 C CNN "Description"
 F 7 "TSSOP20" H 9850 20700 60  0001 C CNN "Package ID"
 	4    9850 20050
@@
 F 4 "0.00@0" H 9850 21400 60  0001 C CNN "Pricing"
 F 5 "Analog Devices" H 9900 21700 60  0001 C CNN "Manufacturer"
-F 6 "CMOS, 2.5 Low Voltage, Quad SPDT Switch" H 9800 21500 60  0001 C CNN "Description"
+F 6 "CMOS, 2.5 Low Voltage, Quad SPDT Switch" H 9800 21500 60  0001 C CNN "Description"
 F 7 "TSSOP20" H 9850 21600 60  0001 C CNN "Package ID"
 	1    9850 20950
@@
 F 4 "0.00@0" H 9850 21850 60  0001 C CNN "Pricing"
 F 5 "Analog Devices" H 9900 22150 60  0001 C CNN "Manufacturer"
-F 6 "CMOS, 2.5 Low Voltage, Quad SPDT Switch" H 9800 21950 60  0001 C CNN "Description"
+F 6 "CMOS, 2.5 Low Voltage, Quad SPDT Switch" H 9800 21950 60  0001 C CNN "Description"
 F 7 "TSSOP20" H 9850 22050 60  0001 C CNN "Package ID"
 	2    9850 21400
@@
 F 4 "0.00@0" H 9850 22750 60  0001 C CNN "Pricing"
 F 5 "Analog Devices" H 9900 23050 60  0001 C CNN "Manufacturer"
-F 6 "CMOS, 2.5 Low Voltage, Quad SPDT Switch" H 9800 22850 60  0001 C CNN "Description"
+F 6 "CMOS, 2.5 Low Voltage, Quad SPDT Switch" H 9800 22850 60  0001 C CNN "Description"
 F 7 "TSSOP20" H 9850 22950 60  0001 C CNN "Package ID"
 	3    9850 22300
@@
 F 4 "0.00@0" H 9850 23200 60  0001 C CNN "Pricing"
 F 5 "Analog Devices" H 9900 23500 60  0001 C CNN "Manufacturer"
-F 6 "CMOS, 2.5 Low Voltage, Quad SPDT Switch" H 9800 23300 60  0001 C CNN "Description"
+F 6 "CMOS, 2.5 Low Voltage, Quad SPDT Switch" H 9800 23300 60  0001 C CNN "Description"
 F 7 "TSSOP20" H 9850 23400 60  0001 C CNN "Package ID"
 	4    9850 22750
@@
 F 4 "0.00@0" H 9850 24100 60  0001 C CNN "Pricing"
 F 5 "Analog Devices" H 9900 24400 60  0001 C CNN "Manufacturer"
-F 6 "CMOS, 2.5 Low Voltage, Quad SPDT Switch" H 9800 24200 60  0001 C CNN "Description"
+F 6 "CMOS, 2.5 Low Voltage, Quad SPDT Switch" H 9800 24200 60  0001 C CNN "Description"
 F 7 "TSSOP20" H 9850 24300 60  0001 C CNN "Package ID"
 	1    9850 23650
@@
 F 4 "0.00@0" H 9850 24550 60  0001 C CNN "Pricing"
 F 5 "Analog Devices" H 9900 24850 60  0001 C CNN "Manufacturer"
-F 6 "CMOS, 2.5 Low Voltage, Quad SPDT Switch" H 9800 24650 60  0001 C CNN "Description"
+F 6 "CMOS, 2.5 Low Voltage, Quad SPDT Switch" H 9800 24650 60  0001 C CNN "Description"
 F 7 "TSSOP20" H 9850 24750 60  0001 C CNN "Package ID"
 	2    9850 24100
@@
 F 4 "0.00@0" H 9850 25450 60  0001 C CNN "Pricing"
 F 5 "Analog Devices" H 9900 25750 60  0001 C CNN "Manufacturer"
-F 6 "CMOS, 2.5 Low Voltage, Quad SPDT Switch" H 9800 25550 60  0001 C CNN "Description"
+F 6 "CMOS, 2.5 Low Voltage, Quad SPDT Switch" H 9800 25550 60  0001 C CNN "Description"
 F 7 "TSSOP20" H 9850 25650 60  0001 C CNN "Package ID"
 	3    9850 25000
@@
 F 4 "0.00@0" H 9850 25900 60  0001 C CNN "Pricing"
 F 5 "Analog Devices" H 9900 26200 60  0001 C CNN "Manufacturer"
-F 6 "CMOS, 2.5 Low Voltage, Quad SPDT Switch" H 9800 26000 60  0001 C CNN "Description"
+F 6 "CMOS, 2.5 Low Voltage, Quad SPDT Switch" H 9800 26000 60  0001 C CNN "Description"
 F 7 "TSSOP20" H 9850 26100 60  0001 C CNN "Package ID"
 	4    9850 25450

Commit message: Finished fixing power supply and starting pcb layout
Parts:
- C146, C147, C148, C149, C150, C151, C152, C153, C154, C155, C156, C157, C158, C159, C160, C161, C162, C163, C164, C165, C166, C167, C168, C169, C170, C171, C172, C173, C174, C175, C176, C177, C178, C179, C180, C181: Characteristics (none) -> 10% -55ºC + 125ºC X7R; Manufacturer (none) -> TDK; Manufacturer Part Number (none) -> CGA4J2X7R1H104K125AE
- R102, R103, R104, R105: Characteristics (none) -> 0.5% -55ºC +155ºC 100mW; Manufacturer (none) -> Vishay; Manufacturer Part Number (none) -> MCT06030D1002DP500; Package ID (none) -> 1608 metric
- U11, U13, U14, U16: Manufacturer Part Number (none) -> ADG734BRUZ
- U57, U58, U59, U60, U61, U62, U63, U64, U65, U66, U67, U68, U69, U70, U71, U72: Manufacturer Part Number (none) -> ADG708BRUZ
- U73, U74, U75, U76: Manufacturer Part Number (none) -> TCA9555PWR

Commit message: Updating to new library structure
Parts:
- C146, C147, C148, C149, C150, C151, C152, C153, C154, C155, C156, C157, C158, C159, C160, C161, C162, C163, C164, C165, C166, C167, C168, C169, C170, C171, C172, C173, C174, C175, C176, C177, C178, C179, C180, C181: symbol C_Small -> Device:C_Small
- R102, R103, R104, R105: symbol R_Small -> Device:R_Small
- U11, U13, U14, U16: symbol ADG734 -> SW-Analog:ADG734
- U57, U58, U59, U60, U61, U62, U63, U64, U65, U66, U67, U68, U69, U70, U71, U72: symbol ADG708 -> SW-Analog:ADG708
- U73, U74, U75, U76: symbol TCA9555 -> SW-Texas:TCA9555
