File: headphone-mux/audio-mux-control.sch (KiCad schematic (older format))
At the start: 197 parts, among them J10 Headset 2, J11 Headset 3, J12 Headset 4, J13 Headset 5, J14 Device 5, J15 Headset 6, J16 Headset 7, J17 Device 6, J18 5V-I2C-2, J19 5V-I2C-3, J2 Device 0, J20 5V-I2C-4, J21 5V-I2C-5, J22 5V-I2C-6, J23 Extra GPIO, J24 Device 7, J25 Outputs to Mixer, J3 Device 1, J4 Device 2, J5 Mixer Audio In, J6 Device 3, J7 Headset 0, J8 Headset 1, J9 Device 4, U17 74ACT32, U18 ADG708, U19 ADG708, U2 ADG715, U20 ADG708, U21 ADG708, U22 ADG708, U23 ADG708, U24 ADG708, U25 ADG708, U26 74ACT32, U27 ADG708, U28 ADG708, U29 ADG708, U30 ADG708, U31 TCA9555, U32 TCA9548A, U33 ADG708, U34 ADG708, U35 TCA9555, U36 TCA9555, U37 ADG708, U38 TCA9555, U39 TCA9555, U4 ADG715, U40 ADG708, U7 TS12A44514, U8 TS12A44514, U9 ADG715

Commit message: Started working on headphone-mux
Parts:
- removed C20, C24, C28, C32, C35, C36, C37, C39, C40, C41, C42, C43, C44, C45, C46, C47, C48, C51, C52, C53, C55, C56, C57, C58, C59, C60, C61, C62, C63, C64, C69, C76: 1uF, SW-Kemet:Kemet_CAP_2220_5750Metric, symbol Device:C_Small
- removed C21, C22, C23, C25, C26, C27, C29, C30, C31, C33, C34, C38, C49, C50, C54, C65, C66, C67, C68, C71, C72, C74: 0.1uF, Capacitor_SMD:C_0805_2012Metric_Pad1.15x1.50mm_HandSolder, symbol Device:C_Small
- removed D1, D10, D14, D17, D19, D23, D26, D29, D32, D34, D37, D4, D41, D43, D7: TPD1E10B06, SW-Texas:DPY_(R-PX1SON-N2), symbol SW-Texas:TPD1E10B06
- removed D11, D12, D13, D15, D16, D18, D2, D20, D21, D22, D24, D25, D27, D28, D3, D30, D31, D33, D35, D36, D38, D39, D40, D42, D44, D45, D5, D6, D8, D9: 0582BQ, SW-Semtech:SC-75_3L, symbol SW-Semtech:0582BQ
- removed J10: Headset 2, SW-TEConn:3-794681-8, symbol Connector_Generic:Conn_01x08
- removed J11: Headset 3, SW-TEConn:3-794681-8, symbol Connector_Generic:Conn_01x08
- removed J12: Headset 4, SW-TEConn:3-794681-8, symbol Connector_Generic:Conn_01x08
- removed J13: Headset 5, SW-TEConn:3-794681-8, symbol Connector_Generic:Conn_01x08
- removed J14: Device 5, SW-TEConn:3-794681-8, symbol Connector_Generic:Conn_01x08
- removed J15: Headset 6, SW-TEConn:3-794681-8, symbol Connector_Generic:Conn_01x08
- removed J16: Headset 7, SW-TEConn:3-794681-8, symbol Connector_Generic:Conn_01x08
- removed J17: Device 6, SW-TEConn:3-794681-8, symbol Connector_Generic:Conn_01x08
- removed J2: Device 0, SW-TEConn:3-794681-8, symbol Connector_Generic:Conn_01x08
- removed J24: Device 7, SW-TEConn:3-794681-8, symbol Connector_Generic:Conn_01x08
- removed J3: Device 1, SW-TEConn:3-794681-8, symbol Connector_Generic:Conn_01x08
- removed J4: Device 2, SW-TEConn:3-794681-8, symbol Connector_Generic:Conn_01x08
- removed J6: Device 3, SW-TEConn:3-794681-8, symbol Connector_Generic:Conn_01x08
- removed J7: Headset 0, SW-TEConn:3-794681-8, symbol Connector_Generic:Conn_01x08
- removed J8: Headset 1, SW-TEConn:3-794681-8, symbol Connector_Generic:Conn_01x08
- removed J9: Device 4, SW-TEConn:3-794681-8, symbol Connector_Generic:Conn_01x08
- removed R14: 10kΩ, Resistor_SMD:R_0603_1608Metric_Pad0.84x1.00mm_HandSolder, symbol Device:R_Small
- removed RN1: 4818P-T02-202LF, SW-Bournes:SOM-18, symbol SW-Passives:R_Network17
- removed U17: 74ACT32, Package_SSOP:TSSOP-14_4.4x5mm_P0.65mm, symbol Logic_74xx:74LS32
- removed U18, U19, U20, U21, U22, U23, U24, U25, U27, U28, U29, U30, U33, U34: ADG708, Package_SSOP:TSSOP-16_4.4x5mm_P0.65mm, symbol SW-Analog:ADG708
- removed unit 3 of U2
- removed unit 4 of U2
- removed unit 5 of U2
- removed unit 6 of U2
- removed unit 7 of U2
- removed unit 8 of U2
- removed unit 9 of U2
- removed unit 10 of U2
- removed unit 2 of U26
- removed unit 3 of U26
- removed unit 4 of U26
- removed U31: TCA9555, Package_SSOP:TSSOP-24_4.4x7.8mm_P0.65mm, symbol SW-Texas:TCA9555
- removed U7: TS12A44514, Package_SSOP:TSSOP-14_4.4x5mm_P0.65mm, symbol SW-Texas:TS12A44514
- removed unit 2 of U8
- removed unit 1 of U8
- removed unit 4 of U8
Connections:
- net labels removed: AMP-MIC-IN-0-0, AMP-MIC-IN-0-1, AMP-MIC-IN-0-2, AMP-MIC-IN-0-3, AMP-MIC-IN-0-4, AMP-MIC-IN-0-5, AMP-MIC-IN-0-6, AMP-MIC-IN-1-0, AMP-MIC-IN-1-1, AMP-MIC-IN-1-2, AMP-MIC-IN-1-3, AMP-MIC-IN-1-4, AMP-MIC-IN-1-5, AMP-MIC-IN-1-6, AMP-MIC-IN-2-0, AMP-MIC-IN-2-1, AMP-MIC-IN-2-2, AMP-MIC-IN-2-3, AMP-MIC-IN-2-4, AMP-MIC-IN-2-5, AMP-MIC-IN-2-6, AMP-MIC-IN-3-0, AMP-MIC-IN-3-1, AMP-MIC-IN-3-2, AMP-MIC-IN-3-3, AMP-MIC-IN-3-4, AMP-MIC-IN-3-5, AMP-MIC-IN-3-6, AMP-MIC-IN-4-0, AMP-MIC-IN-4-1, AMP-MIC-IN-4-2, AMP-MIC-IN-4-3, AMP-MIC-IN-4-4, AMP-MIC-IN-4-5, AMP-MIC-IN-4-6, AMP-MIC-IN-5-0, AMP-MIC-IN-5-1, AMP-MIC-IN-5-2, AMP-MIC-IN-5-3, AMP-MIC-IN-5-4, AMP-MIC-IN-5-5, AMP-MIC-IN-5-6, AMP-MIC-IN-6-0, AMP-MIC-IN-6-1, AMP-MIC-IN-6-2, AMP-MIC-IN-6-3, AMP-MIC-IN-6-4, AMP-MIC-IN-6-5, AMP-MIC-IN-6-6, AMP-MIC-IN-7-0, AMP-MIC-IN-7-1, AMP-MIC-IN-7-2, AMP-MIC-IN-7-3, AMP-MIC-IN-7-4, AMP-MIC-IN-7-5, AMP-MIC-IN-7-6, HEADSET-AUDIO-SOURCE-L-0, HEADSET-AUDIO-SOURCE-L-1, HEADSET-AUDIO-SOURCE-L-2, HEADSET-AUDIO-SOURCE-L-3, HEADSET-AUDIO-SOURCE-L-4, HEADSET-AUDIO-SOURCE-L-5, HEADSET-AUDIO-SOURCE-L-6, HEADSET-AUDIO-SOURCE-R-0, HEADSET-AUDIO-SOURCE-R-1, HEADSET-AUDIO-SOURCE-R-2, HEADSET-AUDIO-SOURCE-R-3, HEADSET-AUDIO-SOURCE-R-4, HEADSET-AUDIO-SOURCE-R-5, HEADSET-AUDIO-SOURCE-R-6, MIC-IN-0, MIC-IN-1, MIC-IN-2, MIC-IN-3, MIC-IN-4, MIC-IN-5, MIC-IN-6, MIC-IN-7, MIC-MUTE-0, MIC-MUTE-1, MIC-MUTE-2, MIC-MUTE-3, MIC-MUTE-4, MIC-MUTE-5, MIC-MUTE-6, MIC-MUTE-7, PTT/MM-~INT
- wire segments 1773 -> 560
- no-connect marks 1 -> 0
Other:
- note removed: "1-Ground\n2-L audio to MUX\n3-R audio to MUX\n4-Mic +\n5-Mic -\n6-+5V for active cables\n7- PTT +\n8- PTT -"
- note removed: "Device power provided by\nexternal connection"
- note removed: "For 2 wire mic connection (separate ground, baofeng)\nConnect +,- mic to +,- mic in cable\nFor 1 wire mic connection (same ground, iphone)\nconnect +,- mic to +,ground in cable."
- note removed: "PTT for each device is an electronic switch closure. \nThis can be controlled via a digital signal from RPi\nor from other ptt inputs"
- note removed: "Standard Android headset controls can be accomodated\nwith an external converter that measures the resistances\non the mic line and transforms those into a pulse code on\nthe mic mute line that the raspberry pi is monitoring for."
- note removed: "cap to block dc bias from devices"
- note removed: "out 1 goes to L_In/R_in bus\nout 2 goes to Mixer"
- note removed: "out 1 goes to Mixer\nout 2 goes to L_In/R_in bus"
