File: headphone-mux/headset-audio-out-mux-switching.sch (KiCad schematic (older format))
At the start: 64 parts, among them U11 ADG734, U13 ADG734, U14 ADG734, U16 ADG734, U57 ADG708, U58 ADG708, U59 ADG708, U60 ADG708, U61 ADG708, U62 ADG708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

Commit message: Remove unnecessary parts of schematic to convert to daughterboard
commit before importing netlist
Parts:
- renumbered C148 to C13, C152 to C14, C156 to C15, C160 to C16, C164 to C17, C168 to C18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
