File: headphone-mux/headphone-mux.sch (KiCad schematic (older format))
At the start: 5 parts

Commit message: Started working on headphone-mux
Connections:
- wire segments 23 -> 8
Changed lines of the file:
@@
 EESchema Schematic File Version 4
-LIBS:edc-mux-board-cache
 EELAYER 26 0
 EELAYER END
 $Descr USLetter 11000 8500
 encoding utf-8
-Sheet 1 38
+Sheet 1 13
 Title ""
 Date ""
@@
 F6 "SPST_~RST" I R 5450 1800 60
 $EndSheet
-$Sheet
-S 950  3100 1900 1450
-U 5A6B6560
-F0 "Arduino Nano Header Connections + Ethernet connection" 60
-F1 "ard-nano-hdr-ethernet.sch" 60
-F2 "5V-SDA" B R 2850 3650 60
-F3 "5V-SCL" O R 2850 3550 60
-F4 "D2_SPST" O R 2850 3800 60
-F5 "D3_I2C" O R 2850 3900 60
-F6 "D5_INT" I R 2850 4000 60
-$EndSheet
 Text Notes 6950 6200 0    60   ~ 0
 All signal directions are indicated from the\nperspective of the MUX box\n\n8x connectors with stereo audio out, mono mic in, \nPTT in, Mic Mute in, +5V bias out\nEach connector can be used for one or more functions.\nThese connectors are for speakermics, headsets and ptt switches.\nConnector model is Amphenol LTW circular connector 8 pin\n\n8x connectors with stereo audio in, mono mic out, PTT out\nEach connector can be used for one or more functions.\nThese connectors are for smartphones and radios.\nConnector model is Amphenol LTW circular connector 8pin\n\n1x DB25 connector to connect to mixer\n1x TRS connector for output from mixer to MUX\n\n
-Wire Wire Line
-	5450 2050 5550 2050
-Wire Wire Line
-	5550 2050 5550 3550
-Wire Wire Line
-	5550 3550 2850 3550
-Wire Wire Line
-	5450 1950 5650 1950
-Wire Wire Line
-	5650 1950 5650 3650
-Wire Wire Line
-	5650 3650 2850 3650
-Wire Wire Line
-	5450 1800 5750 1800
-Wire Wire Line
-	5750 1800 5750 3800
-Wire Wire Line
-	5750 3800 2850 3800
-Wire Wire Line
-	5450 1700 5850 1700
-Wire Wire Line
-	5850 1700 5850 3900
-Wire Wire Line
-	5850 3900 2850 3900
-Wire Wire Line
-	5450 1600 5950 1600
-Wire Wire Line
-	5950 1600 5950 4000
-Wire Wire Line
-	5950 4000 2850 4000
 $Comp
 L Mechanical:Mounting_Hole_PAD MK1

Commit message: Remove unnecessary parts of schematic to convert to daughterboard
commit before importing netlist
Parts:
- removed MK5: Mounting_Hole_PAD, MountingHole:MountingHole_4.3mm_M4_Pad_Via, symbol Mechanical:Mounting_Hole_PAD
- added C1, C10, C11, C12, C2, C3, C4, C5, C6, C7, C8, C9: 0.1uF, Capacitor_SMD:C_0805_2012Metric_Pad1.15x1.50mm_HandSolder, symbol Device:C_Small
- added D1: 0582BQ, SW-Semtech:SC-75_3L, symbol SW-Semtech:0582BQ
- added J1: Audio-Input, SW-Hirose:DF11-16DS-2DSA, symbol Connector_Generic:Conn_02x08_Odd_Even
- added J2: Mixer Audio In, SW-Hirose:DF11-4DP-2DSA, symbol Connector_Generic:Conn_02x02_Odd_Even
- added J3: Power Input, SW-Hirose:DF11-8DS-2DSA, symbol Connector_Generic:Conn_02x04_Odd_Even
- added J4: Audio Output, SW-Hirose:DF11-16DS-2DSA, symbol Connector_Generic:Conn_02x08_Odd_Even
- added J5: I2C and Reset, SW-Hirose:DF11-8DS-2DSA, symbol Connector_Generic:Conn_02x04_Odd_Even
- added U1, U2: ADG715, Package_SSOP:TSSOP-24_4.4x7.8mm_P0.65mm, symbol SW-Analog:ADG715
- added U3, U4, U5, U6: ADG734, Package_SSOP:TSSOP-20_4.4x6.5mm_P0.65mm, symbol SW-Analog:ADG734
- renumbered MK3 to MK2, MK2 to MK3
Connections:
- net labels added: +12VA, +2V5, -12VA, -2.5V, 2v5-SCL-0, 2v5-SDA-0, HEADSET-AUDIO-SOURCE-L-0, HEADSET-AUDIO-SOURCE-L-1, HEADSET-AUDIO-SOURCE-L-2, HEADSET-AUDIO-SOURCE-L-3, HEADSET-AUDIO-SOURCE-L-4, HEADSET-AUDIO-SOURCE-L-5, HEADSET-AUDIO-SOURCE-L-6, HEADSET-AUDIO-SOURCE-L-7, HEADSET-AUDIO-SOURCE-L-[0..7], HEADSET-AUDIO-SOURCE-R-0, HEADSET-AUDIO-SOURCE-R-1, HEADSET-AUDIO-SOURCE-R-2, HEADSET-AUDIO-SOURCE-R-3, HEADSET-AUDIO-SOURCE-R-4, HEADSET-AUDIO-SOURCE-R-5, HEADSET-AUDIO-SOURCE-R-6, HEADSET-AUDIO-SOURCE-R-7, HEADSET-AUDIO-SOURCE-R-[0..7], L_OUT0, L_OUT1, L_OUT2, L_OUT3, L_OUT4, L_OUT5, L_OUT6, L_OUT7, L_OUT[0..7], R_OUT0, R_OUT1, R_OUT2, R_OUT3, R_OUT4, R_OUT5, R_OUT6, R_OUT7, R_OUT[0..7], SPST_~RST
- wire segments 8 -> 204
Other:
- note added: "+12V is regulated +12V@5A DC supply. \n\n+12VA is positive supply for op amps used as audio amplifiers\n-12VA is negative supply for op amps used as audio amplifiers\n+2.5V is positive supply for audio switch chips and io \nexpanders at that logic level\n-2.5V is positive supply for audio switch chips and io \nexpanders at that logic level\n\n\n"
- note added: "1=Left=Tip\n2=Right=Ring\n3=GND=Sleeve\n"
- note added: "Audio signal switch chips will use \n+2.5VA as positive rail\n-2.5VA as negative rail\n\nOp amps use \n+12VA as analog positive rail\n-12VA as analog negative rail\n\nfor each chip voltage level, i2c lines are pulled to \nthe individual vdd of the chip.\n\n"
- note added: "Power connections for Headphone MUX"
- note added: "Power for ADG715 and ADG734\nanalog switches"
- note removed: "All signal directions are indicated from the\nperspective of the MUX box\n\n8x connectors with stereo audio out, mono mic in, \nPTT in, Mic Mute in, +5V bias out\nEach connector can be used for one or more functions.\nThese connectors are for speakermics, headsets and ptt switches.\nConnector model is Amphenol LTW circular connector 8 pin\n\n8x connectors with stereo audio in, mono mic out, PTT o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"

Commit message: Fixing more annotation errors and starting initial reroute
Other:
- note added: "+12VA is positive supply for op amps used as audio amplifiers\n-12VA is negative supply for op amps used as audio amplifiers\n+2.5V is positive supply for audio switch chips and io \nexpanders at that logic level\n-2.5V is positive supply for audio switch chips and io \nexpanders at that logic level\n\n\n"
- note removed: "+12V is regulated +12V@5A DC supply. \n\n+12VA is positive supply for op amps used as audio amplifiers\n-12VA is negative supply for op amps used as audio amplifiers\n+2.5V is positive supply for audio switch chips and io \nexpanders at that logic level\n-2.5V is positive supply for audio switch chips and io \nexpanders at that logic level\n\n\n"
Changed lines of the file:
@@
 Power connections for Headphone MUX
 Text Notes 7150 8000 0    60   ~ 0
-+12V is regulated +12V@5A DC supply. \n\n+12VA is positive supply for op amps used as audio amplifiers\n-12VA is negative supply for op amps used as audio amplifiers\n+2.5V is positive supply for audio switch chips and io \nexpanders at that logic level\n-2.5V is positive supply for audio switch chips and io \nexpanders at that logic level\n\n\n
++12VA is positive supply for op amps used as audio amplifiers\n-12VA is negative supply for op amps used as audio amplifiers\n+2.5V is positive supply for audio switch chips and io \nexpanders at that logic level\n-2.5V is positive supply for audio switch chips and io \nexpanders at that logic level\n\n\n
 Text Notes 7750 7000 0    60   ~ 0
 Audio signal switch chips will use \n+2.5VA as positive rail\n-2.5VA as negative rail\n\nOp amps use \n+12VA as analog positive rail\n-12VA as analog negative rail\n\nfor each chip voltage level, i2c lines are pulled to \nthe individual vdd of the chip.\n\n

Commit message: Finished routing board for now.
Finalized positions of connectors and mouting holes, as well as board
edge locations. DRC checks still need to be run
Changed lines of the file:
@@
 L Connector_Generic:Conn_02x08_Odd_Even J4
 U 1 1 5C025B93
-P 12450 1450
-F 0 "J4" H 12500 1967 50  0000 C CNN
-F 1 "Audio Output" H 12500 1876 50  0000 C CNN
-F 2 "SW-Hirose:DF11-16DS-2DSA" H 12450 1450 50  0001 C CNN
-F 3 "~" H 12450 1450 50  0001 C CNN
-	1    12450 1450
-	1    0    0    -1
+P 12550 1450
+F 0 "J4" H 12600 1967 50  0000 C CNN
+F 1 "Audio Output" H 12600 1876 50  0000 C CNN
+F 2 "SW-Hirose:DF11-16DS-2DSA" H 12550 1450 50  0001 C CNN
+F 3 "~" H 12550 1450 50  0001 C CNN
+	1    12550 1450
+	-1   0    0    -1
 $EndComp
 Text Label 2800 1350 0    50   ~ 0

Commit message: Reworked IO connections due to footprint mistakes
Other:
- note added: "Changed 4-7 for nicer PCB layout"
Changed lines of the file:
@@
 Text Label 2800 1650 0    50   ~ 0
 HEADSET-AUDIO-SOURCE-L-3
+Text Label 2800 2050 0    50   ~ 0
+HEADSET-AUDIO-SOURCE-L-4
+Text Label 2800 1950 0    50   ~ 0
+HEADSET-AUDIO-SOURCE-L-5
+Text Label 2800 1850 0    50   ~ 0
+HEADSET-AUDIO-SOURCE-L-6
 Text Label 2800 1750 0    50   ~ 0
-HEADSET-AUDIO-SOURCE-L-4
-Text Label 2800 1850 0    50   ~ 0
-HEADSET-AUDIO-SOURCE-L-5
-Text Label 2800 1950 0    50   ~ 0
-HEADSET-AUDIO-SOURCE-L-6
-Text Label 2800 2050 0    50   ~ 0
 HEADSET-AUDIO-SOURCE-L-7
 Text Label 2100 1350 2    50   ~ 0
@@
 Text Label 2100 1650 2    50   ~ 0
 HEADSET-AUDIO-SOURCE-R-3
+Text Label 2100 2050 2    50   ~ 0
+HEADSET-AUDIO-SOURCE-R-4
+Text Label 2100 1950 2    50   ~ 0
+HEADSET-AUDIO-SOURCE-R-5
+Text Label 2100 1850 2    50   ~ 0
+HEADSET-AUDIO-SOURCE-R-6
 Text Label 2100 1750 2    50   ~ 0
-HEADSET-AUDIO-SOURCE-R-4
-Text Label 2100 1850 2    50   ~ 0
-HEADSET-AUDIO-SOURCE-R-5
-Text Label 2100 1950 2    50   ~ 0
-HEADSET-AUDIO-SOURCE-R-6
-Text Label 2100 2050 2    50   ~ 0
 HEADSET-AUDIO-SOURCE-R-7
 Wire Wire Line
@@
 Wire Bus Line
 	14700 1250 14700 2800
+Text Notes 1800 2250 0    50   ~ 0
+Changed 4-7 for nicer PCB layout
 $EndSCHEMATC
