File: mic-mux/power_handling.sch (KiCad schematic (older format))
At the start: 68 parts, among them J1 Power In, U1 LM27762, U11 ADG734, U12 LM1085-5V, U13 ADG734, U14 ADG734, U15 LM27762, U16 ADG734, U17 74ACT32, U2 ADG715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

Commit message: Starting work on separating mic mux
Parts:
- removed C1, C15, C17, C4: 2u2F, Capacitor_SMD:C_0805_2012Metric_Pad1.15x1.50mm_HandSolder, symbol Device:C_Small
- removed C10, C11, C12, C9: 22uF, Capacitor_SMD:C_1206_3216Metric_Pad1.24x1.80mm_HandSolder, symbol Device:C_Small
- removed C13, C14, C7, C8: 10uF, Capacitor_SMD:C_1206_3216Metric_Pad1.24x1.80mm_HandSolder, symbol Device:C_Small
- removed C16, C2: 0.47uF, Capacitor_SMD:C_0805_2012Metric_Pad1.15x1.50mm_HandSolder, symbol Device:C_Small
- removed C18, C19, C5, C6: 4u7F, Capacitor_SMD:C_0805_2012Metric_Pad1.15x1.50mm_HandSolder, symbol Device:C_Small
- removed C3: 15uF, Capacitor_SMD:C_0805_2012Metric_Pad1.15x1.50mm_HandSolder, symbol Device:C_Small
- removed F1: 5A, SW-Littelfuse:NANO-0154-OMNI-BLOK-Fuse-Holder, symbol Device:Fuse_Small
- removed J1: Power In, SW-Molex:43255-0121, symbol Connector_Specialized:Barrel_Jack
- removed R10, R13: 220kΩ, Resistor_SMD:R_0603_1608Metric_Pad0.84x1.00mm_HandSolder, symbol Device:R_Small
- removed R11, R12, R3, R4: 68kΩ, Resistor_SMD:R_0603_1608Metric_Pad0.84x1.00mm_HandSolder, symbol Device:R_Small
- removed R2, R6: 75kΩ, Resistor_SMD:R_0603_1608Metric_Pad0.84x1.00mm_HandSolder, symbol Device:R_Small
- removed R5: 174kΩ, Resistor_SMD:R_0603_1608Metric_Pad0.84x1.00mm_HandSolder, symbol Device:R_Small
- removed R7: 22.6kΩ, Resistor_SMD:R_0603_1608Metric_Pad0.84x1.00mm_HandSolder, symbol Device:R_Small
- removed R702, R703: 1.3Ω, Resistor_SMD:R_0603_1608Metric_Pad0.84x1.00mm_HandSolder, symbol Device:R_Small
- removed R8: 143kΩ, Resistor_SMD:R_0603_1608Metric_Pad0.84x1.00mm_HandSolder, symbol Device:R_Small
- removed U1, U15: LM27762, Package_SON:WSON-12-1EP_3x2mm_P0.5mm, symbol SW-Texas:LM27762
- removed U12: LM1085-5V, Package_TO_SOT_SMD:TO-263-3_TabPin4, symbol SW-Texas:LM1085
- removed U3: LMZ34002, SW-Texas:RKG_(S-PB1QFN-N41), symbol SW-Texas:LMZ34002
- removed U6: LM1085-12V, Package_TO_SOT_SMD:TO-263-3_TabPin4, symbol SW-Texas:LM1085
Connections:
- net labels removed: +12V, +12V-F, +12VA, +5VA, -12VA, -5VA, VIN+
- wire segments 294 -> 82
- no-connect marks 3 -> 0
Other:
- note removed: "88uF total capacitance"
- note removed: "Main +12V supply\n3A max supply\n"
- note removed: "Main Power Supplies"
- note removed: "Provides -12V supply for op amps"
- note removed: "Provides ±2.5 supply for\naudio muxes, switches\nand related IO expanders\nIout = 250mA max \nAssume Iin = 500mA max"
- note removed: "Provides ±5VA supply for\ndigital potentiometers\nIout = 250mA max \nAssume Iin = 500mA max"
- note removed: "Vout = 1.2V * (R1+R2)/R2\n2.52 ~~= 1.2V * (75k + 68k)/68k \nusing E24 values\n\ncaps need low ESR\nuse X7R or X5R\nceramic SMD caps\n"
- note removed: "Vout = 1.2V * (R1+R2)/R2\n5.08 ~~= 1.2V * (220k + 68k)/68k \nusing E24 values\n\ncaps need low ESR\nuse X7R or X5R\nceramic SMD caps\n"
