File: mic-mux/stereo-amp.sch (KiCad schematic (older format))
At the start: 18 parts, among them U41 OPA1604, U42 DS1882

Commit message: Re annotating entire schematic. This time properly
Parts:
- renumbered C82 to C21, C83 to C22, C84 to C23, C85 to C24, C86 to C25, C87 to C26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
