File: mic-mux/mic-mux-control.sch (KiCad schematic (older format))
At the start: 32 parts, among them J23 Extra GPIO, U18 ADG708, U2 ADG715, U20 ADG708, U22 ADG708, U24 ADG708, U27 ADG708, U29 ADG708, U33 ADG708, U35 TCA9555, U37 ADG708, U38 TCA9555

Commit message: Final schematic edits, moving on to pcb
Parts:
- U2: footprint Housings_SSOP:TSSOP-24_4.4x7.8mm_Pitch0.65mm -> Package_SSOP:TSSOP-24_4.4x7.8mm_P0.65mm
Connections:
- net labels added: MIC-IN-[0..7]
- wire segments 441 -> 465
Changed lines of the file:
@@
 EESchema Schematic File Version 4
+LIBS:mic-mux-cache
 EELAYER 26 0
 EELAYER END
@@
 F 0 "U2" H 5300 1959 60  0000 C CNN
 F 1 "ADG715" H 5300 1853 60  0000 C CNN
-F 2 "Housings_SSOP:TSSOP-24_4.4x7.8mm_Pitch0.65mm" H 5550 3050 60  0001 C CNN
+F 2 "Package_SSOP:TSSOP-24_4.4x7.8mm_P0.65mm" H 5550 3050 60  0001 C CNN
 F 3 "http://www.analog.com/media/en/technical-documentation/data-sheets/ADG714_715.pdf" H 5550 3150 60  0001 C CNN
 F 4 "i2c, 2.7 -5V single supply, +-2.5V dual supply, 2.5Ω On Resistance, 0.6Ω  On Resistance Flatness, 100 pA Leakage Currents" H 5400 3250 60  0001 C CNN "Characteristics"
@@
 F 0 "U2" H 5300 3359 60  0000 C CNN
 F 1 "ADG715" H 5300 3253 60  0000 C CNN
-F 2 "Housings_SSOP:TSSOP-24_4.4x7.8mm_Pitch0.65mm" H 5550 4450 60  0001 C CNN
+F 2 "Package_SSOP:TSSOP-24_4.4x7.8mm_P0.65mm" H 5550 4450 60  0001 C CNN
 F 3 "http://www.analog.com/media/en/technical-documentation/data-sheets/ADG714_715.pdf" H 5550 4550 60  0001 C CNN
 F 4 "i2c, 2.7 -5V single supply, +-2.5V dual supply, 2.5Ω On Resistance, 0.6Ω  On Resistance Flatness, 100 pA Leakage Currents" H 5400 4650 60  0001 C CNN "Characteristics"
@@
 F 0 "U2" H 5300 4759 60  0000 C CNN
 F 1 "ADG715" H 5300 4653 60  0000 C CNN
-F 2 "Housings_SSOP:TSSOP-24_4.4x7.8mm_Pitch0.65mm" H 5550 5850 60  0001 C CNN
+F 2 "Package_SSOP:TSSOP-24_4.4x7.8mm_P0.65mm" H 5550 5850 60  0001 C CNN
 F 3 "http://www.analog.com/media/en/technical-documentation/data-sheets/ADG714_715.pdf" H 5550 5950 60  0001 C CNN
 F 4 "i2c, 2.7 -5V single supply, +-2.5V dual supply, 2.5Ω On Resistance, 0.6Ω  On Resistance Flatness, 100 pA Leakage Currents" H 5400 6050 60  0001 C CNN "Characteristics"
@@
 F 0 "U2" H 5300 6159 60  0000 C CNN
 F 1 "ADG715" H 5300 6053 60  0000 C CNN
-F 2 "Housings_SSOP:TSSOP-24_4.4x7.8mm_Pitch0.65mm" H 5550 7250 60  0001 C CNN
+F 2 "Package_SSOP:TSSOP-24_4.4x7.8mm_P0.65mm" H 5550 7250 60  0001 C CNN
 F 3 "http://www.analog.com/media/en/technical-documentation/data-sheets/ADG714_715.pdf" H 5550 7350 60  0001 C CNN
 F 4 "i2c, 2.7 -5V single supply, +-2.5V dual supply, 2.5Ω On Resistance, 0.6Ω  On Resistance Flatness, 100 pA Leakage Currents" H 5400 7450 60  0001 C CNN "Characteristics"
@@
 F 0 "U2" H 5300 7559 60  0000 C CNN
 F 1 "ADG715" H 5300 7453 60  0000 C CNN
-F 2 "Housings_SSOP:TSSOP-24_4.4x7.8mm_Pitch0.65mm" H 5550 8650 60  0001 C CNN
+F 2 "Package_SSOP:TSSOP-24_4.4x7.8mm_P0.65mm" H 5550 8650 60  0001 C CNN
 F 3 "http://www.analog.com/media/en/technical-documentation/data-sheets/ADG714_715.pdf" H 5550 8750 60  0001 C CNN
 F 4 "i2c, 2.7 -5V single supply, +-2.5V dual supply, 2.5Ω On Resistance, 0.6Ω  On Resistance Flatness, 100 pA Leakage Currents" H 5400 8850 60  0001 C CNN "Characteristics"
@@
 F 0 "U2" H 5300 8959 60  0000 C CNN
 F 1 "ADG715" H 5300 8853 60  0000 C CNN
-F 2 "Housings_SSOP:TSSOP-24_4.4x7.8mm_Pitch0.65mm" H 5550 10050 60  0001 C CNN
+F 2 "Package_SSOP:TSSOP-24_4.4x7.8mm_P0.65mm" H 5550 10050 60  0001 C CNN
 F 3 "http://www.analog.com/media/en/technical-documentation/data-sheets/ADG714_715.pdf" H 5550 10150 60  0001 C CNN
 F 4 "i2c, 2.7 -5V single supply, +-2.5V dual supply, 2.5Ω On Resistance, 0.6Ω  On Resistance Flatness, 100 pA Leakage Currents" H 5400 10250 60  0001 C CNN "Characteristics"
@@
 F 0 "U2" H 5300 10359 60  0000 C CNN
 F 1 "ADG715" H 5300 10253 60  0000 C CNN
-F 2 "Housings_SSOP:TSSOP-24_4.4x7.8mm_Pitch0.65mm" H 5550 11450 60  0001 C CNN
+F 2 "Package_SSOP:TSSOP-24_4.4x7.8mm_P0.65mm" H 5550 11450 60  0001 C CNN
 F 3 "http://www.analog.com/media/en/technical-documentation/data-sheets/ADG714_715.pdf" H 5550 11550 60  0001 C CNN
 F 4 "i2c, 2.7 -5V single supply, +-2.5V dual supply, 2.5Ω On Resistance, 0.6Ω  On Resistance Flatness, 100 pA Leakage Currents" H 5400 11650 60  0001 C CNN "Characteristics"
@@
 F 0 "U2" H 5300 11759 60  0000 C CNN
 F 1 "ADG715" H 5300 11653 60  0000 C CNN
-F 2 "Housings_SSOP:TSSOP-24_4.4x7.8mm_Pitch0.65mm" H 5550 12850 60  0001 C CNN
+F 2 "Package_SSOP:TSSOP-24_4.4x7.8mm_P0.65mm" H 5550 12850 60  0001 C CNN
 F 3 "http://www.analog.com/media/en/technical-documentation/data-sheets/ADG714_715.pdf" H 5550 12950 60  0001 C CNN
 F 4 "i2c, 2.7 -5V single supply, +-2.5V dual supply, 2.5Ω On Resistance, 0.6Ω  On Resistance Flatness, 100 pA Leakage Currents" H 5400 13050 60  0001 C CNN "Characteristics"
@@
 MIC-OUT[0..7]
 Wire Wire Line
-	7000 2600 7350 2600
-Wire Wire Line
-	7000 4000 7350 4000
-Wire Wire Line
-	7000 5400 7350 5400
-Wire Wire Line
-	7000 6800 7350 6800
-Wire Wire Line
-	7000 8200 7350 8200
-Wire Wire Line
-	7000 9600 7350 9600
-Wire Wire Line
-	7000 11000 7350 11000
-Wire Wire Line
-	7000 12400 7350 12400
-Wire Wire Line
-	5800 2400 7550 2400
-Wire Wire Line
-	5800 3800 7550 3800
-Wire Wire Line
-	5800 5200 7550 5200
-Wire Wire Line
-	5800 6600 7550 6600
-Wire Wire Line
-	5800 8000 7550 8000
-Wire Wire Line
-	5800 9400 7550 9400
-Wire Wire Line
-	5800 10800 7550 10800
-Wire Wire Line
-	5800 12200 7550 12200
+	7000 2600 7200 2600
+Wire Wire Line
+	7000 4000 7200 4000
+Wire Wire Line
+	7000 5400 7200 5400
+Wire Wire Line
+	7000 6800 7200 6800
+Wire Wire Line
+	7000 8200 7200 8200
+Wire Wire Line
+	7000 9600 7200 9600
+Wire Wire Line
+	7000 11000 7200 11000
+Wire Wire Line
+	7000 12400 7200 12400
+Wire Wire Line
+	5800 2400 7000 2400
+Wire Wire Line
+	5800 3800 7000 3800
+Wire Wire Line
+	5800 5200 7000 5200
+Wire Wire Line
+	5800 6600 7000 6600
+Wire Wire Line
+	5800 8000 7000 8000
+Wire Wire Line
+	5800 9400 7000 9400
+Wire Wire Line
+	5800 10800 7000 10800
+Wire Wire Line
+	5800 12200 7000 12200
 Text HLabel 9650 12450 0    50   Input ~ 0
 2v5-SCL-0
@@
 Wire Wire Line
 	17350 10200 18050 10200
-Wire Bus Line
-	4400 2200 4400 14100
+Text HLabel 16750 12300 0    50   Input ~ 0
+MIC-IN[0..7]
+Text Label 17350 12300 0    50   ~ 0
+MIC-IN-[0..7]
+Connection ~ 7000 2400
+Wire Wire Line
+	7000 2400 7200 2400
+Connection ~ 7200 2400
+Wire Wire Line
+	7200 2400 7550 2400
+Connection ~ 7200 2600
+Wire Wire Line
+	7200 2600 7350 2600
+Connection ~ 7000 3800
+Wire Wire Line
+	7000 3800 7200 3800
+Connection ~ 7200 3800
+Wire Wire Line
+	7200 3800 7550 3800
+Connection ~ 7200 4000
+Wire Wire Line
+	7200 4000 7350 4000
+Connection ~ 7000 5200
+Wire Wire Line
+	7000 5200 7200 5200
+Connection ~ 7200 5200
+Wire Wire Line
+	7200 5200 7550 5200
+Connection ~ 7200 5400
+Wire Wire Line
+	7200 5400 7350 5400
+Connection ~ 7000 6600
+Wire Wire Line
+	7000 6600 7200 6600
+Connection ~ 7200 6600
+Wire Wire Line
+	7200 6600 7550 6600
+Connection ~ 7200 6800
+Wire Wire Line
+	7200 6800 7350 6800
+Connection ~ 7000 8000
+Wire Wire Line
+	7000 8000 7200 8000
+Connection ~ 7200 8000
+Wire Wire Line
+	7200 8000 7550 8000
+Connection ~ 7200 8200
+Wire Wire Line
+	7200 8200 7350 8200
+Connection ~ 7000 9400
+Wire Wire Line
+	7000 9400 7200 9400
+Connection ~ 7200 9400
+Wire Wire Line
+	7200 9400 7550 9400
+Connection ~ 7200 9600
+Wire Wire Line
+	7200 9600 7350 9600
+Connection ~ 7000 10800
+Wire Wire Line
+	7000 10800 7200 10800
+Connection ~ 7200 10800
+Wire Wire Line
+	7200 10800 7550 10800
+Connection ~ 7200 11000
+Wire Wire Line
+	7200 11000 7350 11000
+Connection ~ 7000 12200
+Wire Wire Line
+	7000 12200 7200 12200
+Connection ~ 7200 12200
+Wire Wire Line
+	7200 12200 7550 12200
+Connection ~ 7200 12400
+Wire Wire Line
+	7200 12400 7350 12400
 Wire Bus Line
 	18150 2100 18150 12300
@@
 Wire Bus Line
 	4300 15600 13300 15600
-Text HLabel 16750 12300 0    50   Input ~ 0
-MIC-IN[0..7]
-Text Label 17350 12300 0    50   ~ 0
-MIC-IN[0..7]
+Wire Bus Line
+	4400 2200 4400 14100
 $EndSCHEMATC

Commit message: Re annotating entire schematic. This time properly
Parts:
- renumbered C34 to C10, C49 to C11, C50 to C12, C65 to C13, C66 to C14, C71 to C15, C72 to C16, C79 to C17, C80 to C18, C73 to C19, C77 to C20, C21 to C3, C22 to C4, C25 to C5, C26 to C6, C29 to C7, C30 to C8, C33 to C9, J23 to J12, R34 to R1, R36 to R2, U2 to U1, U35 to U10, U38 to U11, U18 to U2, U20 to U3, U22 to U4, U24 to U5, U27 to U6, U29 to U7, U33 to U8, U37 to U9

Commit message: positioning connectors and mounting holes
Parts:
- J12: footprint Connector_PinHeader_2.54mm:PinHeader_2x06_P2.54mm_Vertical -> SW-Hirose:DF11-12DP-2DS
Changed lines of the file:
@@
 F 0 "J12" H 9330 15092 50  0000 L CNN
 F 1 "Extra GPIO" H 9330 15001 50  0000 L CNN
-F 2 "Connector_PinHeader_2.54mm:PinHeader_2x06_P2.54mm_Vertical" H 9250 15100 50  0001 C CNN
+F 2 "SW-Hirose:DF11-12DP-2DS" H 9250 15100 50  0001 C CNN
 F 3 "" H 9250 15100 50  0001 C CNN
 F 4 "0.00@0" H 9250 15100 60  0001 C CNN "Pricing"
