File: motherboard/power_handling.sch (KiCad schematic (older format))
At the start: 68 parts, among them J1 Power In, U1 LM27762, U11 ADG734, U12 LM1085-5V, U13 ADG734, U14 ADG734, U15 LM27762, U16 ADG734, U17 74ACT32, U2 ADG715, U26 74ACT32, U3 LMZ34002, U4 ADG715, U6 LM1085-12V, U7 TS12A44514, U8 TS12A44514, U9 ADG715

Commit message: All initial schematic edits made, removing headphone and mic mux
Parts:
- removed C376, C377, C378, C381, C383, C384, C385, C387, C388, C389, C390, C391, C392, C393: 0.1uF, Capacitor_SMD:C_0805_2012Metric_Pad1.15x1.50mm_HandSolder, symbol Device:C_Small
- removed J1: Power In, SW-Molex:43255-0121, symbol Connector_Specialized:Barrel_Jack
- removed U11, U13, U14, U16: ADG734, Package_SSOP:TSSOP-20_4.4x6.5mm_P0.65mm, symbol SW-Analog:ADG734
- removed U2, U4, U9: ADG715, Package_SSOP:TSSOP-24_4.4x7.8mm_P0.65mm, symbol SW-Analog:ADG715
- added J1: Power In (Male-top), SW-Hirose:DF11-4DP-2DSA, symbol Connector_Generic:Conn_02x02_Odd_Even
- added J23: GND (Male-top), SW-Hirose:DF11-8DP-2DSA, symbol Connector_Generic:Conn_02x04_Odd_Even
- added J5: Power Out (Male-top), SW-Hirose:DF11-8DP-2DSA, symbol Connector_Generic:Conn_02x04_Odd_Even
Connections:
- wire segments 294 -> 277
- no-connect marks 3 -> 2
Other:
- note removed: "Power for ADG715 and ADG734\nanalog switches"

Commit message: after initial trace cleanup from reimport + reannotating schematic
Parts:
- renumbered C8 to C10, C382 to C11, C386 to C12, C9 to C13, C10 to C14, C11 to C15, C12 to C16, C13 to C17, C14 to C18, C15 to C19, C16 to C20, C17 to C21, C18 to C22, C19 to C23, C379 to C5, C5 to C6, C6 to C7, C380 to C8, C7 to C9, J5 to J2, J23 to J3, R2 to R1, R3 to R2, R4 to R3, R5 to R4, R6 to R5, R7 to R6, R702 to R7, R703 to R9, U17 to U2, U7 to U3, U3 to U4, U6 to U5, U8 to U6, U26 to U7, U12 to U8, U15 to U9

Commit message: Fixing db25 connector and routing headphone distribution connections
Connections:
- wire segments 277 -> 276
Changed lines of the file:
@@
 Wire Wire Line
 	7550 2750 7550 2800
-Connection ~ 7350 2750
 Wire Wire Line
 	7350 2600 7350 2750
@@
 	8550 2750 8550 2600
 Wire Wire Line
-	7150 2750 7350 2750
-Wire Wire Line
 	7500 2200 7500 2400
 Wire Wire Line
@@
 	2150 2000 2150 2300
 Wire Wire Line
-	7500 1700 7500 2000
+	7500 1700 7500 1800
 Wire Wire Line
 	13150 1700 13400 1700
@@
 $EndComp
 Wire Wire Line
-	7150 1800 7100 1800
-Wire Wire Line
-	7150 1800 7150 2750
-Wire Wire Line
 	7100 1700 7500 1700
 $Comp
@@
 Wire Wire Line
 	6550 1800 6550 1700
+Wire Wire Line
+	7100 1800 7500 1800
+Connection ~ 7500 1800
+Wire Wire Line
+	7500 1800 7500 2000
 $EndSCHEMATC
