File: motherboard/motherboard.kicad_pcb (KiCad board)
At the start: 4 copper layers, 507 parts, among them J1 Power In (Male-top), J10 Headset 1, J11 Device 1, J12 Headset 2, J13 Headset 3, J14 Headset 4, J15 Device 2, J16 Headset 5, J17 Headset 6, J18 Device 3, J19 Headset 7, J2 Power Out (Male-top), J20 I2C and RESET (Male-top), J21 Device 4, J22 Device 5, J23 Device 6, J24 5V-I2C-2, J25 5V-I2C-3, J26 5V-I2C-4, J27 5V-I2C-5, J28 5V-I2C-6, J29 Device 7, J3 GND (Male-top), J30 Outputs to Mixer, J4 MIC-IN (Male-top), J5 Headphone Audio Out (Male-top), J6 Headphone Audio In (Male-top), J7 MIC-OUT (Male-top), J8 Device 0, J9 Headset 0, U1 LM27762, U10 ADG708, U11 ADG708, U12 ADG708, U13 ADG708, U14 TCA9555, U15 ADG708, U16 ADG708, U17 TCA9548A, U18 ADG708, U19 TCA9555, U2 74ACT32, U20 ADG708, U21 TCA9555, U22 OPA1604, U23 DS1882, U24 OPA1604, U25 DS1882, U26 OPA1604, U27 DS1882, U28 OPA1604, U29 DS1882, U3 TS12A44514, U30 OPA1604, U31 DS1882, U32 OPA1604, U33 DS1882, U34 OPA1604, U35 DS1882, U36 OPA1604, U37 DS1882, U38 OPA1602, U39 OPA1604, U4 LMZ34002, U40 OPA1602, U41 OPA1604, U42 OPA1602, U43 OPA1604, U44 OPA1602, U45 OPA1604, U46 OPA1602, U47 OPA1604, U48 OPA1602, U49 OPA1604, U5 LM1085-12V, U50 OPA1602, U51 OPA1604, U52 OPA1602, U53 OPA1604, U6 TS12A44514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

Commit message: More updates, finalizing schematic and starting layout
Parts:
- moved J2 330.5 mm to (126.7, 378.1)
- moved R14 322.4 mm to (230.5, 418.0)
- moved C57 322.4 mm to (237.4, 426.0)
- moved D50 254.0 mm to (292.6, 369.6)
- moved D51 254.0 mm to (292.6, 357.1)
- moved D53 254.0 mm to (292.6, 361.3)
- moved D54 254.0 mm to (292.6, 378.0)
- moved D56 254.0 mm to (292.6, 382.2)
- moved J30 254.0 mm to (296.7, 369.0)
- moved D49 254.0 mm to (292.6, 353.0)
- moved D52 254.0 mm to (292.6, 373.8)
- moved D55 254.0 mm to (292.6, 365.5)
- moved C77 238.8 mm to (377.6, 170.6)
- moved C79 238.8 mm to (366.0, 157.0)
- moved C81 238.8 mm to (362.2, 157.9)
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Connections:
- C62 pad 2: (no net) -> Net-(C62-Pad2)
- J11 pad 2: /Audio Mux and Control/Device LR Distro Amplifier 1/L_IN -> GNDREF
- J11 pad 4: Net-(C32-Pad2) -> +5V
- J11 pad 5: GNDREF -> /Audio Mux and Control/Device LR Distro Amplifier 1/L_IN
- J11 pad 6: +5V -> Net-(D12-Pad2)
- J11 pad 7: Net-(D12-Pad2) -> Net-(C32-Pad2)
- J15 pad 2: /Audio Mux and Control/Device LR Distro Amplifier 2/L_IN -> GNDREF
- J15 pad 4: Net-(C43-Pad2) -> +5V
- J15 pad 5: GNDREF -> /Audio Mux and Control/Device LR Distro Amplifier 2/L_IN
- J15 pad 6: +5V -> Net-(D24-Pad2)
- J15 pad 7: Net-(D24-Pad2) -> Net-(C43-Pad2)
- J18 pad 2: /Audio Mux and Control/Device LR Distro Amplifier 3/L_IN -> GNDREF
- J18 pad 4: Net-(C52-Pad2) -> +5V
- J18 pad 5: GNDREF -> /Audio Mux and Control/Device LR Distro Amplifier 3/L_IN
- J18 pad 6: +5V -> Net-(D35-Pad2)
- J18 pad 7: Net-(D35-Pad2) -> Net-(C52-Pad2)
- J21 pad 2: /Audio Mux and Control/Device LR Distro Amplifier 4/L_IN -> GNDREF
- J21 pad 4: Net-(C56-Pad2) -> +5V
- J21 pad 5: GNDREF -> /Audio Mux and Control/Device LR Distro Amplifier 4/L_IN
- J21 pad 6: +5V -> Net-(D39-Pad2)
- J21 pad 7: Net-(D39-Pad2) -> Net-(C56-Pad2)
- J22 pad 2: /Audio Mux and Control/Device LR Distro Amplifier 5/L_IN -> GNDREF
- J22 pad 4: Net-(C59-Pad2) -> +5V
- J22 pad 5: GNDREF -> /Audio Mux and Control/Device LR Distro Amplifier 5/L_IN
- J22 pad 6: +5V -> Net-(D42-Pad2)
- J22 pad 7: Net-(D42-Pad2) -> Net-(C59-Pad2)
- J23 pad 2: /Audio Mux and Control/Device LR Distro Amplifier 6/L_IN -> GNDREF
- J23 pad 4: Net-(C62-Pad2) -> +5V
- J23 pad 5: GNDREF -> /Audio Mux and Control/Device LR Distro Amplifier 6/L_IN
- J23 pad 6: +5V -> Net-(D45-Pad2)
- J23 pad 7: Net-(D45-Pad2) -> Net-(C62-Pad2)
- J29 pad 2: /Audio Mux and Control/Device LR Distro Amplifier 7/L_IN -> GNDREF
- J29 pad 4: Net-(C65-Pad2) -> +5V
- J29 pad 5: GNDREF -> /Audio Mux and Control/Device LR Distro Amplifier 7/L_IN
- J29 pad 6: +5V -> Net-(D48-Pad2)
- J29 pad 7: Net-(D48-Pad2) -> Net-(C65-Pad2)
- J6 pad 1: /Audio Mux and Control/L_OUT0 -> /Audio Mux and Control/R_OUT0
- J6 pad 10: /Audio Mux and Control/R_OUT4 -> /Audio Mux and Control/L_OUT4
- J6 pad 11: /Audio Mux and Control/L_OUT5 -> /Audio Mux and Control/R_OUT5
- J6 pad 12: /Audio Mux and Control/R_OUT5 -> /Audio Mux and Control/L_OUT5
- J6 pad 13: /Audio Mux and Control/L_OUT6 -> /Audio Mux and Control/R_OUT6
- J6 pad 14: /Audio Mux and Control/R_OUT6 -> /Audio Mux and Control/L_OUT6
- J6 pad 15: /Audio Mux and Control/L_OUT7 -> /Audio Mux and Control/R_OUT7
- J6 pad 16: /Audio Mux and Control/R_OUT7 -> /Audio Mux and Control/L_OUT7
- J6 pad 2: /Audio Mux and Control/R_OUT0 -> /Audio Mux and Control/L_OUT0
- J6 pad 3: /Audio Mux and Control/L_OUT1 -> /Audio Mux and Control/R_OUT1
- J6 pad 4: /Audio Mux and Control/R_OUT1 -> /Audio Mux and Control/L_OUT1
- J6 pad 5: /Audio Mux and Control/L_OUT2 -> /Audio Mux and Control/R_OUT2
- J6 pad 6: /Audio Mux and Control/R_OUT2 -> /Audio Mux and Control/L_OUT2
- J6 pad 7: /Audio Mux and Control/L_OUT3 -> /Audio Mux and Control/R_OUT3
- J6 pad 8: /Audio Mux and Control/R_OUT3 -> /Audio Mux and Control/L_OUT3
- J6 pad 9: /Audio Mux and Control/L_OUT4 -> /Audio Mux and Control/R_OUT4
- J8 pad 2: /Audio Mux and Control/Device LR Distro Amplifier 0/L_IN -> GNDREF
- J8 pad 4: Net-(C24-Pad2) -> +5V
- J8 pad 5: GNDREF -> /Audio Mux and Control/Device LR Distro Amplifier 0/L_IN
- J8 pad 6: +5V -> Net-(D3-Pad2)
- J8 pad 7: Net-(D3-Pad2) -> Net-(C24-Pad2)
Routing:
- net /Audio Mux and Control/MIXER-OUT-R-7: track 179.2 -> 24.8 mm
- net /Audio Mux and Control/MIXER-OUT-L-7: track 168.5 -> 17.7 mm
- net /Audio Mux and Control/MIXER-OUT-R-6: track 160.1 -> 21.7 mm
- net /Audio Mux and Control/MIXER-OUT-L-6: track 153.6 -> 15.6 mm
- net /Audio Mux and Control/MIXER-OUT-R-5: track 134.7 -> 11.1 mm
- net /Audio Mux and Control/MIXER-OUT-L-5: track 132.4 -> 11.7 mm
- net /Audio Mux and Control/MIXER-OUT-L-4: track 114.9 -> 8.24 mm
- net /Audio Mux and Control/MIXER-OUT-R-4: track 127.6 -> 21.2 mm
- net /Audio Mux and Control/MIXER-OUT-R-3: track 117.3 -> 25.8 mm
- net /Audio Mux and Control/MIXER-OUT-L-3: track 98.5 -> 7.08 mm
- net /Audio Mux and Control/MIXER-OUT-R-2: track 96.4 -> 21.1 mm
- net /Audio Mux and Control/MIXER-OUT-L-2: track 83.1 -> 10.2 mm
- net /Audio Mux and Control/MIXER-OUT-R-1: track 86.6 -> 26.7 mm
- net /Audio Mux and Control/MIXER-OUT-L-1: track 69.2 -> 10.1 mm
- net /Audio Mux and Control/MIXER-OUT-R-0: track 65.4 -> 21.9 mm
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- added copper zone on F.Cu, net Net-(U4-Pad21)
- removed copper zone on In1.Cu, net +12V
- removed copper zone on F.Cu, net Net-(U3-Pad21)

Commit message: Fixing db25 connector and routing headphone distribution connections
Parts:
- J30: value Outputs to Mixer -> Output to Mixer; moved to F.Cu
- moved J9 517.5 mm to (-38.8, 291.7), turned to 0 degrees
- moved J10 513.4 mm to (-38.8, 279.9), turned to 0 degrees
- moved J19 511.7 mm to (-38.8, 209.5), turned to 0 degrees
- moved J12 510.5 mm to (-38.8, 268.2), turned to 0 degrees
- moved J17 509.3 mm to (-38.8, 221.3), turned to 0 degrees
- moved J13 508.6 mm to (-38.8, 256.5), turned to 0 degrees
- moved J16 508.0 mm to (-38.8, 233.0), turned to 0 degrees
- moved J14 507.7 mm to (-38.8, 244.7), turned to 0 degrees
- moved D4 502.4 mm to (-32.0, 286.9), turned to 180 degrees
- moved D6 500.6 mm to (-29.1, 296.5), turned to 0 degrees
- moved D33 500.0 mm to (-32.2, 204.7), turned to 180 degrees
- moved D7 498.9 mm to (-32.2, 274.7), turned to 180 degrees
- moved D28 496.9 mm to (-32.2, 216.9), turned to 180 degrees
- moved D10 496.0 mm to (-29.2, 284.3), turned to 0 degrees
- moved D13 496.0 mm to (-32.0, 262.5), turned to 180 degrees
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Connections:
- net Net-(D12-Pad1) renamed /Audio Mux and Control/PTT-DEV1
- net Net-(D12-Pad2) renamed /Audio Mux and Control/PTT+DEV1
- net Net-(D24-Pad1) renamed /Audio Mux and Control/PTT-DEV2
- net Net-(D24-Pad2) renamed /Audio Mux and Control/PTT+DEV2
- net Net-(D3-Pad1) renamed /Audio Mux and Control/PTT-DEV0
- net Net-(D3-Pad2) renamed /Audio Mux and Control/PTT+DEV0
- net Net-(D35-Pad1) renamed /Audio Mux and Control/PTT-DEV3
- net Net-(D35-Pad2) renamed /Audio Mux and Control/PTT+DEV3
- net Net-(D39-Pad1) renamed /Audio Mux and Control/PTT-DEV4
- net Net-(D39-Pad2) renamed /Audio Mux and Control/PTT+DEV4
- net Net-(D42-Pad1) renamed /Audio Mux and Control/PTT-DEV5
- net Net-(D42-Pad2) renamed /Audio Mux and Control/PTT+DEV5
- net Net-(D45-Pad1) renamed /Audio Mux and Control/PTT-DEV6
- net Net-(D45-Pad2) renamed /Audio Mux and Control/PTT+DEV6
- net Net-(D48-Pad1) renamed /Audio Mux and Control/PTT-DEV7
- net Net-(D48-Pad2) renamed /Audio Mux and Control/PTT+DEV7
- net Net-(U10-Pad8) renamed /Audio Mux and Control/MUX->OR-0
- net Net-(U11-Pad8) renamed /Audio Mux and Control/MUX->OR-1
- net Net-(U12-Pad8) renamed /Audio Mux and Control/MUX->OR-2
- net Net-(U13-Pad8) renamed /Audio Mux and Control/MUX->OR-3
- net Net-(U15-Pad8) renamed /Audio Mux and Control/MUX->OR-4
- net Net-(U16-Pad8) renamed /Audio Mux and Control/MUX->OR-5
- net Net-(U18-Pad8) renamed /Audio Mux and Control/MUX->OR-6
- net Net-(U2-Pad11) renamed /Audio Mux and Control/DEV-PTT-TRGR-2
- net Net-(U2-Pad3) renamed /Audio Mux and Control/DEV-PTT-TRGR-3
- net Net-(U2-Pad6) renamed /Audio Mux and Control/DEV-PTT-TRGR-0
- net Net-(U2-Pad8) renamed /Audio Mux and Control/DEV-PTT-TRGR-1
- net Net-(U20-Pad8) renamed /Audio Mux and Control/MUX->OR-7
- net Net-(U6-Pad12) renamed /Audio Mux and Control/DEV-PTT-TRGR-6
- net Net-(U6-Pad13) renamed /Audio Mux and Control/DEV-PTT-TRGR-5
- net Net-(U6-Pad5) renamed /Audio Mux and Control/DEV-PTT-TRGR-4
- net Net-(U6-Pad6) renamed /Audio Mux and Control/DEV-PTT-TRGR-7
- D11 pad 1: /Audio Mux and Control/Device LR Distro Amplifier 1/L_IN -> /Audio Mux and Control/Device LR Distro Amplifier 1/R_IN
- D11 pad 2: /Audio Mux and Control/Device LR Distro Amplifier 1/R_IN -> /Audio Mux and Control/Device LR Distro Amplifier 1/L_IN
- D2 pad 1: /Audio Mux and Control/Device LR Distro Amplifier 0/L_IN -> /Audio Mux and Control/Device LR Distro Amplifier 0/R_IN
- D2 pad 2: /Audio Mux and Control/Device LR Distro Amplifier 0/R_IN -> /Audio Mux and Control/Device LR Distro Amplifier 0/L_IN
- D22 pad 1: /Audio Mux and Control/Device LR Distro Amplifier 2/L_IN -> /Audio Mux and Control/Device LR Distro Amplifier 2/R_IN
- D22 pad 2: /Audio Mux and Control/Device LR Distro Amplifier 2/R_IN -> /Audio Mux and Control/Device LR Distro Amplifier 2/L_IN
- D32 pad 1: /Audio Mux and Control/Device LR Distro Amplifier 3/L_IN -> /Audio Mux and Control/Device LR Distro Amplifier 3/R_IN
- D32 pad 2: /Audio Mux and Control/Device LR Distro Amplifier 3/R_IN -> /Audio Mux and Control/Device LR Distro Amplifier 3/L_IN
- D38 pad 1: /Audio Mux and Control/Device LR Distro Amplifier 4/L_IN -> /Audio Mux and Control/Device LR Distro Amplifier 4/R_IN
- D38 pad 2: /Audio Mux and Control/Device LR Distro Amplifier 4/R_IN -> /Audio Mux and Control/Device LR Distro Amplifier 4/L_IN
- D41 pad 1: /Audio Mux and Control/Device LR Distro Amplifier 5/L_IN -> /Audio Mux and Control/Device LR Distro Amplifier 5/R_IN
- D41 pad 2: /Audio Mux and Control/Device LR Distro Amplifier 5/R_IN -> /Audio Mux and Control/Device LR Distro Amplifier 5/L_IN
- D44 pad 1: /Audio Mux and Control/Device LR Distro Amplifier 6/L_IN -> /Audio Mux and Control/Device LR Distro Amplifier 6/R_IN
- D44 pad 2: /Audio Mux and Control/Device LR Distro Amplifier 6/R_IN -> /Audio Mux and Control/Device LR Distro Amplifier 6/L_IN
- D47 pad 1: /Audio Mux and Control/Device LR Distro Amplifier 7/L_IN -> /Audio Mux and Control/Device LR Distro Amplifier 7/R_IN
- D47 pad 2: /Audio Mux and Control/Device LR Distro Amplifier 7/R_IN -> /Audio Mux and Control/Device LR Distro Amplifier 7/L_IN
- D50 pad 1: /Audio Mux and Control/MIXER-OUT-R-4 -> /Audio Mux and Control/MIXER-OUT-L-1
- D50 pad 2: /Audio Mux and Control/MIXER-OUT-L-4 -> /Audio Mux and Control/MIXER-OUT-R-1
- D51 pad 1: /Audio Mux and Control/MIXER-OUT-R-1 -> /Audio Mux and Control/MIXER-OUT-R-2
- D51 pad 2: /Audio Mux and Control/MIXER-OUT-L-1 -> /Audio Mux and Control/MIXER-OUT-L-2
- D52 pad 1: /Audio Mux and Control/MIXER-OUT-L-5 -> /Audio Mux and Control/MIXER-OUT-L-3
- D52 pad 2: /Audio Mux and Control/MIXER-OUT-R-5 -> /Audio Mux and Control/MIXER-OUT-R-3
- D53 pad 1: /Audio Mux and Control/MIXER-OUT-R-2 -> /Audio Mux and Control/MIXER-OUT-R-4
- D53 pad 2: /Audio Mux and Control/MIXER-OUT-L-2 -> /Audio Mux and Control/MIXER-OUT-L-4
- D54 pad 1: /Audio Mux and Control/MIXER-OUT-R-6 -> /Audio Mux and Control/MIXER-OUT-L-5
- D54 pad 2: /Audio Mux and Control/MIXER-OUT-L-6 -> /Audio Mux and Control/MIXER-OUT-R-5
- D55 pad 1: /Audio Mux and Control/MIXER-OUT-R-3 -> /Audio Mux and Control/MIXER-OUT-R-6
- D55 pad 2: /Audio Mux and Control/MIXER-OUT-L-3 -> /Audio Mux and Control/MIXER-OUT-L-6
- D56 pad 1: /Audio Mux and Control/MIXER-OUT-R-7 -> /Audio Mux and Control/MIXER-OUT-L-7
- D56 pad 2: /Audio Mux and Control/MIXER-OUT-L-7 -> /Audio Mux and Control/MIXER-OUT-R-7
- J1 pad 4: GNDREF -> /Power Handling/VIN+
- J30 pad 1: /Audio Mux and Control/MIXER-OUT-R-0 -> GNDREF
- J30 pad 10: /Audio Mux and Control/MIXER-OUT-R-6 -> /Audio Mux and Control/MIXER-OUT-R-2
- J30 pad 11: GNDREF -> /Audio Mux and Control/MIXER-OUT-R-3
- J30 pad 12: /Audio Mux and Control/MIXER-OUT-L-7 -> GNDREF
- J30 pad 14: /Audio Mux and Control/MIXER-OUT-L-0 -> /Audio Mux and Control/MIXER-OUT-L-4
- J30 pad 15: /Audio Mux and Control/MIXER-OUT-R-1 -> /Audio Mux and Control/MIXER-OUT-L-5
- J30 pad 16: GNDREF -> /Audio Mux and Control/MIXER-OUT-R-4
- J30 pad 17: /Audio Mux and Control/MIXER-OUT-L-2 -> /Audio Mux and Control/MIXER-OUT-R-5
- J30 pad 18: /Audio Mux and Control/MIXER-OUT-R-3 -> GNDREF
- J30 pad 2: GNDREF -> /Audio Mux and Control/MIXER-OUT-L-0
- J30 pad 20: /Audio Mux and Control/MIXER-OUT-L-4 -> /Audio Mux and Control/MIXER-OUT-L-6
- J30 pad 21: /Audio Mux and Control/MIXER-OUT-R-5 -> /Audio Mux and Control/MIXER-OUT-L-7
- J30 pad 22: GNDREF -> /Audio Mux and Control/MIXER-OUT-R-6
- J30 pad 23: /Audio Mux and Control/MIXER-OUT-L-6 -> /Audio Mux and Control/MIXER-OUT-R-7
- J30 pad 24: /Audio Mux and Control/MIXER-OUT-R-7 -> GNDREF
- J30 pad 4: /Audio Mux and Control/MIXER-OUT-R-2 -> /Audio Mux and Control/MIXER-OUT-R-0
- J30 pad 5: GNDREF -> /Audio Mux and Control/MIXER-OUT-R-1
- J30 pad 6: /Audio Mux and Control/MIXER-OUT-L-3 -> GNDREF
- J30 pad 7: /Audio Mux and Control/MIXER-OUT-R-4 -> GNDREF
- J30 pad 8: GNDREF -> /Audio Mux and Control/MIXER-OUT-L-2
- J30 pad 9: /Audio Mux and Control/MIXER-OUT-L-5 -> /Audio Mux and Control/MIXER-OUT-L-3
Routing:
- net GNDREF: track 576.9 -> 416.2 mm, vias 535 -> 454
- net /Audio Mux and Control/HEADSET-AUDIO-SOURCE-R-7: track 9.68 -> 161.2 mm
- net /Audio Mux and Control/HEADSET-AUDIO-SOURCE-L-7: track 11.4 -> 155.7 mm
- net /Audio Mux and Control/HEADSET-AUDIO-SOURCE-R-6: track 7.67 -> 146.5 mm
- net /Audio Mux and Control/HEADSET-AUDIO-SOURCE-L-6: track 15.0 -> 141.1 mm
- net /Audio Mux and Control/HEADSET-AUDIO-SOURCE-R-5: track 9.57 -> 131.8 mm
- net /Audio Mux and Control/HEADSET-AUDIO-SOURCE-L-5: track 15.6 -> 126.2 mm
- net /Audio Mux and Control/HEADSET-AUDIO-SOURCE-R-4: track 8.78 -> 117.0 mm
- net /Audio Mux and Control/HEADSET-AUDIO-SOURCE-L-4: track 13.3 -> 111.6 mm
- net /Audio Mux and Control/HEADSET-AUDIO-SOURCE-L-3: track 2.60 -> 96.8 mm
- net /Audio Mux and Control/HEADSET-AUDIO-SOURCE-R-3: track 12.0 -> 102.3 mm
- net /Audio Mux and Control/HEADSET-AUDIO-SOURCE-R-2: track 2.81 -> 87.7 mm
- net /Audio Mux and Control/HEADSET-AUDIO-SOURCE-L-2: track 3.26 -> 82.1 mm
- net /Audio Mux and Control/MIC-OUT7: track 0.00 -> 78.5 mm, vias 0 -> 1
- net /Audio Mux and Control/MIC-OUT6: track 1.18 -> 67.8 mm, vias 0 -> 1
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- removed copper zone on In1.Cu, net -12VA
Other:
- board outline added: 142.2 x 203.2 mm
- net class 2A: clearance 0.127 -> 0.254; trace_width 0.508 -> 0.254
- net class 3A: clearance 0.127 -> 0.254
- net class GND: clearance 0.127 -> 0.254; trace_width 0.127 -> 0.254; via_dia 0.4572 -> 0.508

Commit message: Almost done with initial motherboard layout
Parts:
- C24, C25, C26, C27, C29, C30, C31, C32, C33, C34, C35, C36, C37, C39, C40, C41, C42, C43, C44, C45, C46, C48, C49, C50, C51, C52, C53, C54, C56, C59, C62, C65: footprint SW-Kemet:Kemet_CAP_2220_5750Metric -> SW-Kemet:Kemet_CAP_2220_5750Metric_D
- moved C125 313.3 mm to (97.0, 219.2), turned to 0 degrees
- moved R93 312.6 mm to (97.0, 217.1), turned to 180 degrees
- moved R94 310.3 mm to (99.8, 221.4), turned to 90 degrees
- moved R92 308.6 mm to (99.8, 216.9), turned to 270 degrees
- moved C131 308.2 mm to (98.3, 211.0), turned to 0 degrees
- moved C130 307.6 mm to (98.3, 208.9), turned to 0 degrees
- moved U36 302.9 mm to (104.7, 219.2), turned to 0 degrees
- moved R96 302.4 mm to (103.7, 214.1), turned to 90 degrees
- moved S1 301.1 mm to (192.0, 177.8), turned to 180 degrees
- moved R99 299.2 mm to (105.9, 214.1), turned to 90 degrees
- moved U37 299.2 mm to (104.7, 209.0), turned to 0 degrees
- moved R98 297.2 mm to (109.5, 221.4), turned to 90 degrees
- moved C66 296.7 mm to (60.2, 157.2), turned to 90 degrees
- moved R95 295.6 mm to (109.5, 216.9), turned to 270 degrees
- moved C124 292.6 mm to (112.3, 219.2), turned to 180 degrees
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Connections:
- RN1 pad 1: /Audio Mux and Control/MIC-MUTE-7 -> /Audio Mux and Control/MIC-MUTE-4
- RN1 pad 10: /Audio Mux and Control/PTT-7 -> /Audio Mux and Control/PTT-0
- RN1 pad 11: /Audio Mux and Control/PTT-6 -> /Audio Mux and Control/PTT-1
- RN1 pad 12: /Audio Mux and Control/PTT-5 -> /Audio Mux and Control/PTT-2
- RN1 pad 13: /Audio Mux and Control/PTT-4 -> /Audio Mux and Control/PTT-3
- RN1 pad 14: /Audio Mux and Control/PTT-3 -> /Audio Mux and Control/PTT-4
- RN1 pad 15: /Audio Mux and Control/PTT-2 -> /Audio Mux and Control/PTT-5
- RN1 pad 16: /Audio Mux and Control/PTT-1 -> /Audio Mux and Control/PTT-6
- RN1 pad 17: /Audio Mux and Control/PTT-0 -> /Audio Mux and Control/PTT-7
- RN1 pad 2: /Audio Mux and Control/MIC-MUTE-6 -> /Audio Mux and Control/MIC-MUTE-5
- RN1 pad 3: /Audio Mux and Control/MIC-MUTE-5 -> /Audio Mux and Control/MIC-MUTE-6
- RN1 pad 4: /Audio Mux and Control/MIC-MUTE-4 -> /Audio Mux and Control/MIC-MUTE-7
- U14 pad 10: /Audio Mux and Control/PTT-6 -> /Audio Mux and Control/PTT-1
- U14 pad 11: /Audio Mux and Control/PTT-7 -> /Audio Mux and Control/PTT-0
- U14 pad 17: /Audio Mux and Control/MIC-MUTE-4 -> /Audio Mux and Control/MIC-MUTE-7
- U14 pad 18: /Audio Mux and Control/MIC-MUTE-5 -> /Audio Mux and Control/MIC-MUTE-6
- U14 pad 19: /Audio Mux and Control/MIC-MUTE-6 -> /Audio Mux and Control/MIC-MUTE-5
- U14 pad 20: /Audio Mux and Control/MIC-MUTE-7 -> /Audio Mux and Control/MIC-MUTE-4
- U14 pad 4: /Audio Mux and Control/PTT-0 -> /Audio Mux and Control/PTT-7
- U14 pad 5: /Audio Mux and Control/PTT-1 -> /Audio Mux and Control/PTT-6
- U14 pad 6: /Audio Mux and Control/PTT-2 -> /Audio Mux and Control/PTT-5
- U14 pad 7: /Audio Mux and Control/PTT-3 -> /Audio Mux and Control/PTT-4
- U14 pad 8: /Audio Mux and Control/PTT-4 -> /Audio Mux and Control/PTT-3
- U14 pad 9: /Audio Mux and Control/PTT-5 -> /Audio Mux and Control/PTT-2
Routing:
- net /Audio Mux and Control/5V-SCL-0: track 42.4 -> 370.1 mm, vias 0 -> 12
- net /Audio Mux and Control/5V-SDA-0: track 41.3 -> 363.7 mm, vias 0 -> 12
- net +5V: track 169.2 -> 438.9 mm, vias 36 -> 123
- net GNDREF: track 416.2 -> 146.7 mm, vias 454 -> 412
- net +5VA: track 61.8 -> 323.2 mm, vias 8 -> 10
- net -12VA: track 94.4 -> 347.3 mm, vias 24 -> 48
- net -5VA: track 53.8 -> 305.2 mm, vias 8 -> 9
- net +12V: track 83.8 -> 329.1 mm, vias 24 -> 101
- net /Arduino Nano Header Connections + Ethernet connection/D5_INT: track 0.00 -> 241.0 mm, vias 0 -> 1
- net /Arduino Nano Header Connections + Ethernet connection/D2_SPST: track 0.00 -> 215.8 mm
- net /Audio Mux and Control/L_OUT3: track 0.00 -> 189.9 mm, vias 0 -> 1
- net /Audio Mux and Control/R_OUT4: track 0.00 -> 184.9 mm, vias 0 -> 1
- net /Audio Mux and Control/L_OUT4: track 0.00 -> 168.8 mm, vias 0 -> 1
- net /Audio Mux and Control/R_OUT3: track 0.00 -> 168.7 mm, vias 0 -> 1
- net /Audio Mux and Control/L_OUT2: track 0.00 -> 167.2 mm, vias 0 -> 1
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- added copper zone on B.Cu, net +12V
- added copper zone on In1.Cu, net +12V
- added copper zone on B.Cu, net -12VA
- added copper zone on In1.Cu, net -12VA
- added copper zone on F.Cu, net /Power Handling/VIN+
Other:
- board size 142.2 x 203.2 mm -> 142.2 x 209.6 mm
