File: motherboard/motherboard.sch (KiCad schematic (older format))
At the start: 5 parts

Commit message: All initial schematic edits made, removing headphone and mic mux
Parts:
- removed MK5: Mounting_Hole_PAD, MountingHole:MountingHole_4.3mm_M4_Pad_Via, symbol Mechanical:Mounting_Hole_PAD
Connections:
- wire segments 23 -> 22
Changed lines of the file:
@@
 EESchema Schematic File Version 4
-LIBS:edc-mux-board-cache
+LIBS:motherboard-cache
 EELAYER 26 0
 EELAYER END
 $Descr USLetter 11000 8500
 encoding utf-8
-Sheet 1 38
+Sheet 1 20
 Title ""
 Date ""
@@
 Wire Wire Line
 	7000 1400 7000 1600
-$Comp
-L Mechanical:Mounting_Hole_PAD MK5
-U 1 1 5AADA511
-P 8600 1400
-F 0 "MK5" V 8554 1550 50  0000 L CNN
-F 1 "Mounting_Hole_PAD" V 8645 1550 50  0000 L CNN
-F 2 "MountingHole:MountingHole_4.3mm_M4_Pad_Via" H 8600 1400 50  0001 C CNN
-F 3 "" H 8600 1400 50  0001 C CNN
-	1    8600 1400
-	0    1    1    0
-$EndComp
-Wire Wire Line
-	8500 1400 8200 1400
 $EndSCHEMATC

Commit message: Fixed clearance issues with ethernet shield
added cutout guides for mic mux board above
Parts:
- added MK5, MK6, MK7, MK8: Mounting_Hole_PAD, MountingHole:MountingHole_2.7mm_M2.5_Pad_Via, symbol Mechanical:Mounting_Hole_PAD
Connections:
- wire segments 22 -> 29
Other:
- note added: "Board Mounting Holes"
Changed lines of the file:
@@
 Wire Wire Line
 	7000 1400 7000 1600
+Wire Notes Line
+	6900 1950 8700 1950
+Wire Notes Line
+	8700 800  6900 800
+Text Notes 7400 950  0    50   ~ 0
+Board Mounting Holes
+$Comp
+L Mechanical:Mounting_Hole_PAD MK5
+U 1 1 5AB64D36
+P 7300 2300
+F 0 "MK5" H 7400 2400 50  0000 L CNN
+F 1 "Mounting_Hole_PAD" H 7400 2300 50  0000 L CNN
+F 2 "MountingHole:MountingHole_2.7mm_M2.5_Pad_Via" H 7300 2300 50  0001 C CNN
+F 3 "" H 7300 2300 50  0001 C CNN
+F 4 "0.00@0" H 7300 2300 50  0001 C CNN "Pricing"
+	1    7300 2300
+	1    0    0    -1
+$EndComp
+$Comp
+L Mechanical:Mounting_Hole_PAD MK6
+U 1 1 5AB64E31
+P 8100 2300
+F 0 "MK6" H 8200 2400 50  0000 L CNN
+F 1 "Mounting_Hole_PAD" H 8200 2300 50  0000 L CNN
+F 2 "MountingHole:MountingHole_2.7mm_M2.5_Pad_Via" H 8100 2300 50  0001 C CNN
+F 3 "" H 8100 2300 50  0001 C CNN
+F 4 "0.00@0" H 8100 2300 50  0001 C CNN "Pricing"
+	1    8100 2300
+	1    0    0    -1
+$EndComp
+$Comp
+L Mechanical:Mounting_Hole_PAD MK7
+U 1 1 5AB64E5E
+P 7300 2700
+F 0 "MK7" H 7200 2650 50  0000 R CNN
+F 1 "Mounting_Hole_PAD" H 7200 2750 50  0000 R CNN
+F 2 "MountingHole:MountingHole_2.7mm_M2.5_Pad_Via" H 7300 2700 50  0001 C CNN
+F 3 "" H 7300 2700 50  0001 C CNN
+F 4 "0.00@0" H 7300 2700 50  0001 C CNN "Pricing"
+	1    7300 2700
+	-1   0    0    1
+$EndComp
+$Comp
+L Mechanical:Mounting_Hole_PAD MK8
+U 1 1 5AB64E91
+P 8100 2700
+F 0 "MK8" H 8000 2650 50  0000 R CNN
+F 1 "Mounting_Hole_PAD" H 8000 2750 50  0000 R CNN
+F 2 "MountingHole:MountingHole_2.7mm_M2.5_Pad_Via" H 8100 2700 50  0001 C CNN
+F 3 "" H 8100 2700 50  0001 C CNN
+F 4 "0.00@0" H 8100 2700 50  0001 C CNN "Pricing"
+	1    8100 2700
+	-1   0    0    1
+$EndComp
+$Comp
+L power:GNDREF #PWR0269
+U 1 1 5AB6567B
+P 7000 2800
+F 0 "#PWR0269" H 7000 2550 50  0001 C CNN
+F 1 "GNDREF" H 7005 2627 50  0000 C CNN
+F 2 "" H 7000 2800 50  0001 C CNN
+F 3 "" H 7000 2800 50  0001 C CNN
+	1    7000 2800
+	1    0    0    -1
+$EndComp
+Wire Wire Line
+	7000 2800 7000 2500
+Wire Wire Line
+	7000 2500 7300 2500
+Wire Wire Line
+	8100 2500 8100 2400
+Wire Wire Line
+	8100 2600 8100 2500
+Connection ~ 8100 2500
+Wire Wire Line
+	7300 2600 7300 2500
+Connection ~ 7300 2500
+Wire Wire Line
+	7300 2500 8100 2500
+Wire Wire Line
+	7300 2500 7300 2400
+Wire Notes Line
+	6900 3050 8700 3050
+Wire Notes Line
+	8700 800  8700 3050
+Wire Notes Line
+	6900 800  6900 3050
 $EndSCHEMATC
