File: motherboard/audio-mux-control.sch (KiCad schematic (older format))
At the start: 197 parts, among them J10 Headset 2, J11 Headset 3, J12 Headset 4, J13 Headset 5, J14 Device 5, J15 Headset 6, J16 Headset 7, J17 Device 6, J18 5V-I2C-2, J19 5V-I2C-3, J2 Device 0, J20 5V-I2C-4, J21 5V-I2C-5, J22 5V-I2C-6, J23 Extra GPIO, J24 Device 7, J25 Outputs to Mixer, J3 Device 1, J4 Device 2, J5 Mixer Audio In, J6 Device 3, J7 Headset 0, J8 Headset 1, J9 Device 4, U17 74ACT32, U18 ADG708, U19 ADG708, U2 ADG715, U20 ADG708, U21 ADG708, U22 ADG708, U23 ADG708, U24 ADG708, U25 ADG708, U26 74ACT32, U27 ADG708, U28 ADG708, U29 ADG708, U30 ADG708, U31 TCA9555, U32 TCA9548A, U33 ADG708, U34 ADG708, U35 TCA9555, U36 TCA9555, U37 ADG708, U38 TCA9555, U39 TCA9555, U4 ADG715, U40 ADG708, U7 TS12A44514, U8 TS12A44514, U9 ADG715

Commit message: All initial schematic edits made, removing headphone and mic mux
Parts:
- removed C21, C22, C25, C26, C29, C30, C33, C34, C49, C50, C65, C66, C71, C72, C73, C77, C79, C80: 0.1uF, Capacitor_SMD:C_0805_2012Metric_Pad1.15x1.50mm_HandSolder, symbol Device:C_Small
- removed D57: 0582BQ, SW-Semtech:SC-75_3L, symbol SW-Semtech:0582BQ
- removed J23: Extra GPIO, Connector_PinHeader_2.54mm:PinHeader_2x06_P2.54mm_Vertical, symbol Connector_Generic:Conn_01x12
- removed J5: Mixer Audio In, Connector_PinHeader_2.54mm:PinHeader_1x03_P2.54mm_Vertical, symbol Connector_Generic:Conn_01x03
- removed R34, R36: 10kΩ, Resistor_SMD:R_0603_1608Metric_Pad0.84x1.00mm_HandSolder, symbol Device:R_Small
- removed U18, U20, U22, U24, U27, U29, U33, U37: ADG708, Package_SSOP:TSSOP-16_4.4x5mm_P0.65mm, symbol SW-Analog:ADG708
- removed U2, U4, U9: ADG715, Package_SSOP:TSSOP-24_4.4x7.8mm_P0.65mm, symbol SW-Analog:ADG715
- removed U35, U38: TCA9555, Package_SSOP:TSSOP-24_4.4x7.8mm_P0.65mm, symbol SW-Texas:TCA9555
- added J26: MIC-IN (Male-top), SW-Hirose:DF11-8DP-2DSA, symbol Connector_Generic:Conn_02x04_Odd_Even
- added J27: Headphone Audio Out (Male-top), SW-Hirose:DF11-16DP-2DSA, symbol Connector_Generic:Conn_02x08_Odd_Even
- added J28: Headphone Audio In (Male-top), SW-Hirose:DF11-16DP-2DSA, symbol Connector_Generic:Conn_02x08_Odd_Even
- added J29: MIC-OUT (Male-top), SW-Hirose:DF11-8DP-2DSA, symbol Connector_Generic:Conn_02x04_Odd_Even
- added J30: I2C and RESET (Male-top), SW-Hirose:DF11-8DP-2DSA, symbol Connector_Generic:Conn_02x04_Odd_Even
- J10, J11, J12, J13, J14, J15, J16, J17, J2, J24, J3, J4, J6, J7, J8, J9: footprint SW-TEConn:3-794681-8 -> SW-Hirose:DF11-8DP-2DSA
- J25: footprint SW-AmphenolLTW:SDB-25PFFP-SR8001 -> SW-Hirose:DF11-24DP-2DSA
Connections:
- net labels added: MIC-IN0, MIC-IN1, MIC-IN2, MIC-IN3, MIC-IN4, MIC-IN5, MIC-IN6, MIC-IN7, MIC-IN[0..7], MIC-OUT0, MIC-OUT1, MIC-OUT2, MIC-OUT3, MIC-OUT4, MIC-OUT5, MIC-OUT6, MIC-OUT7, MIC-OUT[0..7]
- net labels removed: -2.5V, AMP-MIC-IN-0-0, AMP-MIC-IN-0-1, AMP-MIC-IN-0-2, AMP-MIC-IN-0-3, AMP-MIC-IN-0-4, AMP-MIC-IN-0-5, AMP-MIC-IN-0-6, AMP-MIC-IN-0-7, AMP-MIC-IN-1-0, AMP-MIC-IN-1-1, AMP-MIC-IN-1-2, AMP-MIC-IN-1-3, AMP-MIC-IN-1-4, AMP-MIC-IN-1-5, AMP-MIC-IN-1-6, AMP-MIC-IN-1-7, AMP-MIC-IN-2-0, AMP-MIC-IN-2-1, AMP-MIC-IN-2-2, AMP-MIC-IN-2-3, AMP-MIC-IN-2-4, AMP-MIC-IN-2-5, AMP-MIC-IN-2-6, AMP-MIC-IN-2-7, AMP-MIC-IN-3-0, AMP-MIC-IN-3-1, AMP-MIC-IN-3-2, AMP-MIC-IN-3-3, AMP-MIC-IN-3-4, AMP-MIC-IN-3-5, AMP-MIC-IN-3-6, AMP-MIC-IN-3-7, AMP-MIC-IN-4-0, AMP-MIC-IN-4-1, AMP-MIC-IN-4-2, AMP-MIC-IN-4-3, AMP-MIC-IN-4-4, AMP-MIC-IN-4-5, AMP-MIC-IN-4-6, AMP-MIC-IN-4-7, AMP-MIC-IN-5-0, AMP-MIC-IN-5-1, AMP-MIC-IN-5-2, AMP-MIC-IN-5-3, AMP-MIC-IN-5-4, AMP-MIC-IN-5-5, AMP-MIC-IN-5-6, AMP-MIC-IN-5-7, AMP-MIC-IN-6-0, AMP-MIC-IN-6-1, AMP-MIC-IN-6-2, AMP-MIC-IN-6-3, AMP-MIC-IN-6-4, AMP-MIC-IN-6-5, AMP-MIC-IN-6-6, AMP-MIC-IN-6-7, AMP-MIC-IN-7-0, AMP-MIC-IN-7-1, AMP-MIC-IN-7-2, AMP-MIC-IN-7-3, AMP-MIC-IN-7-4, AMP-MIC-IN-7-5, AMP-MIC-IN-7-6, AMP-MIC-IN-7-7, DEV-MIC-IN-XBAR-CTL0, DEV-MIC-IN-XBAR-CTL1, DEV-MIC-IN-XBAR-CTL10, DEV-MIC-IN-XBAR-CTL11, DEV-MIC-IN-XBAR-CTL12, DEV-MIC-IN-XBAR-CTL13, DEV-MIC-IN-XBAR-CTL14, DEV-MIC-IN-XBAR-CTL15, DEV-MIC-IN-XBAR-CTL16, DEV-MIC-IN-XBAR-CTL17, DEV-MIC-IN-XBAR-CTL18, DEV-MIC-IN-XBAR-CTL19, DEV-MIC-IN-XBAR-CTL2, DEV-MIC-IN-XBAR-CTL20, DEV-MIC-IN-XBAR-CTL21, DEV-MIC-IN-XBAR-CTL22, DEV-MIC-IN-XBAR-CTL23, DEV-MIC-IN-XBAR-CTL3, DEV-MIC-IN-XBAR-CTL4, DEV-MIC-IN-XBAR-CTL5, DEV-MIC-IN-XBAR-CTL6, DEV-MIC-IN-XBAR-CTL7, DEV-MIC-IN-XBAR-CTL8, DEV-MIC-IN-XBAR-CTL9, DEV-MIC-IN-XBAR-CTL[0..23], MIC-IN-0, MIC-IN-1, MIC-IN-2, MIC-IN-3, MIC-IN-4, MIC-IN-5, MIC-IN-6, MIC-IN-7
- wire segments 1773 -> 1318
- no-connect marks 1 -> 2
Other:
- note added: "Connector directions are\nWRT motherboard"
- note added: "PTT for each device is an electronic switch closure. \nThis can be controlled via a digital signal from Nano\nor from other ptt inputs"
- note added: "connected via 24 pin header"
- note removed: "1=Left=Tip\n2=Right=Ring\n3=GND=Sleeve\n"
- note removed: "ADDR: 0100100"
- note removed: "ADDR: 0100101"
- note removed: "PTT for each device is an electronic switch closure. \nThis can be controlled via a digital signal from RPi\nor from other ptt inputs"

Commit message: after initial trace cleanup from reimport + reannotating schematic
Parts:
- renumbered C20 to C24, C35 to C25, C36 to C26, C37 to C27, C23 to C28, C39 to C29, C40 to C30, C41 to C31, C24 to C32, C43 to C33, C44 to C34, C45 to C35, C46 to C36, C47 to C37, C27 to C38, C48 to C39, C51 to C40, C52 to C41, C53 to C42, C28 to C43, C55 to C44, C56 to C45, C57 to C46, C31 to C47, C59 to C48, C60 to C49, C61 to C50, C62 to C51, C32 to C52, C63 to C53, C64 to C54, C38 to C55, C42 to C56, C67 to C57, C54 to C58, C58 to C59, C70 to C60, C68 to C61, C69 to C62, C75 to C63, C74 to C64, C76 to C65, C78 to C66, C81 to C67, D18 to D10, D5 to D11, D6 to D12, D22 to D13, D23 to D14, D24 to D15, D25 to D16, D26 to D17, D27 to D18, D28 to D19, D29 to D20, D7 to D21, D8 to D22, D30 to D23, D9 to D24, D31 to D25, D32 to D26, D33 to D27, D36 to D28, D37 to D29, D39 to D30, D10 to D31, D11 to D32, D40 to D33, D41 to D34, D12 to D35, D42 to D36, D19 to D37, D20 to D38, D21 to D39, D13 to D4, D34 to D40, D35 to D41, D38 to D42, D14 to D5, D15 to D6, D16 to D7, D17 to D8, D4 to D9, J8 to J10, J3 to J11, J10 to J12, J11 to J13, J12 to J14, J4 to J15, J13 to J16, J15 to J17, J6 to J18, J16 to J19, J30 to J20, J9 to J21, J14 to J22, J17 to J23, J18 to J24, J19 to J25, J20 to J26, J21 to J27, J22 to J28, J24 to J29, J25 to J30, J26 to J4, J27 to J5, J28 to J6, J29 to J7, J2 to J8, J7 to J9, R35 to R34, R37 to R35, U19 to U10, U21 to U11, U23 to U12, U25 to U13, U31 to U14, U28 to U15, U30 to U16, U32 to U17, U34 to U18, U36 to U19, U17 to U2, U40 to U20, U39 to U21, U7 to U3, U8 to U6, U26 to U7

Commit message: Changing layout of Device connectors for optimum pcb layout
Connections:
- wire segments 1318 -> 1316
Other:
- note added: "1-Ground\n2-Mic -\n3-R audio to MUX\n4-+5V for active cables\n5-L audio to MUX\n6-PTT +\n7- Mic +\n8- PTT -"
- note removed: "1-Ground\n2-L audio to MUX\n3-R audio to MUX\n4-Mic +\n5-Mic -\n6-+5V for active cables\n7- PTT +\n8- PTT -"

Commit message: More updates, finalizing schematic and starting layout
Changed lines of the file:
@@
 L Connector_Generic:Conn_02x08_Odd_Even J6
 U 1 1 635E0E6F
-P 16150 1400
-F 0 "J6" H 16200 1950 50  0000 C CNN
-F 1 "Headphone Audio In (Male-top)" H 16200 1850 50  0000 C CNN
-F 2 "SW-Hirose:DF11-16DP-2DSA" H 16150 1400 50  0001 C CNN
-F 3 "~" H 16150 1400 50  0001 C CNN
-	1    16150 1400
-	1    0    0    -1
+P 16250 1400
+F 0 "J6" H 16300 1950 50  0000 C CNN
+F 1 "Headphone Audio In (Male-top)" H 16300 1850 50  0000 C CNN
+F 2 "SW-Hirose:DF11-16DP-2DSA" H 16250 1400 50  0001 C CNN
+F 3 "~" H 16250 1400 50  0001 C CNN
+	1    16250 1400
+	-1   0    0    -1
 $EndComp
 $Comp
@@
 Connection ~ 4850 22550
 Wire Bus Line
+	6600 1400 6600 1800
+Wire Bus Line
+	8500 1400 8500 1800
+Wire Bus Line
+	17350 1400 17350 2100
+Wire Bus Line
 	19100 1400 19100 2100
 Wire Bus Line
-	17350 1400 17350 2100
-Wire Bus Line
-	8500 1400 8500 1800
-Wire Bus Line
-	6600 1400 6600 1800
+	17050 1200 17050 3400
+Wire Bus Line
+	15350 1200 15350 3250
+Wire Bus Line
+	15150 1200 15150 2400
+Wire Bus Line
+	11600 1200 11600 2300
+Wire Bus Line
+	3800 4000 3800 25850
+Wire Bus Line
+	12400 3400 12400 11350
+Wire Bus Line
+	12100 3250 12100 11200
+Wire Bus Line
+	10900 22900 13200 22900
+Wire Bus Line
+	10800 22750 13050 22750
+Wire Bus Line
+	15100 20850 15100 25850
+Wire Bus Line
+	11200 2400 11200 22500
+Wire Bus Line
+	11050 2300 11050 22600
+Wire Bus Line
+	11350 2900 11350 22550
+Wire Bus Line
+	11500 2800 11500 22450
 Wire Bus Line
 	6200 1800 6200 22350
 Wire Bus Line
-	11500 2800 11500 22450
-Wire Bus Line
-	11350 2900 11350 22550
-Wire Bus Line
-	11050 2300 11050 22600
-Wire Bus Line
-	11200 2400 11200 22500
-Wire Bus Line
-	15100 20850 15100 25850
-Wire Bus Line
-	10800 22750 13050 22750
-Wire Bus Line
-	10900 22900 13200 22900
-Wire Bus Line
-	12100 3250 12100 11200
-Wire Bus Line
-	12400 3400 12400 11350
-Wire Bus Line
-	3800 4000 3800 25850
-Wire Bus Line
-	11600 1200 11600 2300
-Wire Bus Line
-	15150 1200 15150 2400
-Wire Bus Line
-	15350 1200 15350 3250
-Wire Bus Line
-	17050 1200 17050 3400
-Wire Bus Line
 	4450 4100 4450 25450

Commit message: Fixing db25 connector and routing headphone distribution connections
Parts:
- removed J30: Outputs to Mixer, SW-Hirose:DF11-24DP-2DSA, symbol Connector_Specialized:DB25_Female
- added J30: Output to Mixer, SW-Hirose:DF11-24DP-2DSA, symbol Connector_Generic:Conn_02x12_Odd_Even
Connections:
- net labels added: DEV-PTT-TRGR-0, DEV-PTT-TRGR-1, DEV-PTT-TRGR-2, DEV-PTT-TRGR-3, DEV-PTT-TRGR-4, DEV-PTT-TRGR-5, DEV-PTT-TRGR-6, DEV-PTT-TRGR-7, MUX->OR-0, MUX->OR-1, MUX->OR-2, MUX->OR-3, MUX->OR-4, MUX->OR-5, MUX->OR-6, MUX->OR-7, PTT+DEV0, PTT+DEV1, PTT+DEV2, PTT+DEV3, PTT+DEV4, PTT+DEV5, PTT+DEV6, PTT+DEV7, PTT-DEV0, PTT-DEV1, PTT-DEV2, PTT-DEV3, PTT-DEV4, PTT-DEV5, PTT-DEV6, PTT-DEV7
- wire segments 1316 -> 1337
- no-connect marks 2 -> 1

Commit message: Almost done with initial motherboard layout
Parts:
- C24, C25, C26, C27, C29, C30, C31, C32, C33, C34, C35, C36, C37, C39, C40, C41, C42, C43, C44, C45, C46, C48, C49, C50, C51, C52, C53, C54, C56, C59, C62, C65: footprint SW-Kemet:Kemet_CAP_2220_5750Metric -> SW-Kemet:Kemet_CAP_2220_5750Metric_D

Commit message: Finished routing on mic mux and motherboard after cutting mic-mux
Changed lines of the file:
@@
 Text Label 19700 13900 2    60   ~ 0
 PTT-7
+Text Label 19700 15500 2    60   ~ 0
+MIC-MUTE-0
+Text Label 19700 15400 2    60   ~ 0
+MIC-MUTE-1
+Text Label 19700 15300 2    60   ~ 0
+MIC-MUTE-2
+Text Label 19700 15200 2    60   ~ 0
+MIC-MUTE-3
+Text Label 19700 15100 2    60   ~ 0
+MIC-MUTE-4
+Text Label 19700 15000 2    60   ~ 0
+MIC-MUTE-5
+Text Label 19700 14900 2    60   ~ 0
+MIC-MUTE-6
 Text Label 19700 14800 2    60   ~ 0
-MIC-MUTE-0
-Text Label 19700 14900 2    60   ~ 0
-MIC-MUTE-1
-Text Label 19700 15000 2    60   ~ 0
-MIC-MUTE-2
-Text Label 19700 15100 2    60   ~ 0
-MIC-MUTE-3
-Text Label 19700 15500 2    60   ~ 0
-MIC-MUTE-4
-Text Label 19700 15400 2    60   ~ 0
-MIC-MUTE-5
-Text Label 19700 15300 2    60   ~ 0
-MIC-MUTE-6
-Text Label 19700 15200 2    60   ~ 0
 MIC-MUTE-7
 Text Notes 19550 23300 0    60   ~ 0

Commit message: updating part
Parts:
- C24: Pricing (none) -> 0.00@0
Changed lines of the file:
@@
 F 3 "https://www.mouser.com/ds/2/212/KEM_F3078_LDE-1103670.pdf" H 5350 3200 50  0001 C CNN
 F 4 "10% -55ºC + 125ºC" H 5121 3300 50  0001 C CNN "Characteristics"
-F 5 "Film Capacitor" H 5121 3300 50  0001 C CNN "Description"
-F 6 "LDEDD4100KA0N00" H 5121 3300 50  0001 C CNN "Manufacturer Part Number"
-F 7 "Kemet" H 5121 3300 50  0001 C CNN "Manufacturer"
+F 5 "Kemet" H 5121 3300 50  0001 C CNN "Manufacturer"
+F 6 "Film Capacitor" H 5121 3300 50  0001 C CNN "Description"
+F 7 "0.00@0" H 5350 3200 50  0001 C CNN "Pricing"
+F 8 "LDEDD4100KA0N00" H 5121 3300 50  0001 C CNN "Manufacturer Part Number"
 	1    5350 3200
 	0    1    1    0
