File: edc-mux-board-fpga/conn15.sch (KiCad schematic (older format))
At the start: 38 parts, among them J17 Device 15, U52 MAX4910, U53 TLV320AIC3206, U54 P82B96

Commit message: changed from film to ceramic 1uF caps and updated fields of other caps
Parts:
- C304, C305, C309, C310, C311, C312, C313, C314, C315, C316, C321, C323, F16: Package ID (none) -> 0603in/1608mm
- C306, C318: Package ID 0603in/1608mm -> 1206in/3216mm
- C307, C308, C319, C320: footprint SW-WIMA:2220_film_cap -> Capacitor_SMD:C_0805_2012Metric; Manufacturer Wima -> Kemet; Manufacturers Part Number SMDTC04100QB00KP00 -> C0805X105J3RACAUTO; Package ID (none) -> 0805in/2012mm
- C317, C322: Manufacturer (none) -> TDK; Manufacturers Part Number (none) -> CGA3E1X7R1E105K080AC; Package ID (none) -> 0603in/1608mm
- D97: Package ID (none) -> SMA Diode
- FB81: Package ID 0603 -> 0603in/1608mm
Changed lines of the file:
@@
 F 2 "Capacitor_SMD:C_0603_1608Metric" H 6150 2700 50  0001 C CNN
 F 3 "~" H 6150 2700 50  0001 C CNN
+F 4 "0603in/1608mm" H 0   0   50  0001 C CNN "Package ID"
 	1    6150 2700
 	0    1    1    0
@@
 F 2 "Capacitor_SMD:C_0603_1608Metric" H 7000 4800 50  0001 C CNN
 F 3 "~" H 7000 4800 50  0001 C CNN
+F 4 "0603in/1608mm" H 0   0   50  0001 C CNN "Package ID"
 	1    7000 4800
 	-1   0    0    1
@@
 F 2 "Capacitor_SMD:C_0603_1608Metric" H 5350 4800 50  0001 C CNN
 F 3 "~" H 5350 4800 50  0001 C CNN
+F 4 "TDK" H 0   0   50  0001 C CNN "Manufacturer"
+F 5 "CGA3E1X7R1E105K080AC" H 0   0   50  0001 C CNN "Manufacturers Part Number"
+F 6 "0603in/1608mm" H 0   0   50  0001 C CNN "Package ID"
 	1    5350 4800
 	-1   0    0    1
@@
 F 0 "C308" V 3350 3100 50  0000 C CNN
 F 1 "1uF" V 3450 3100 50  0000 C CNN
-F 2 "SW-WIMA:2220_film_cap" H 3200 3100 50  0001 C CNN
+F 2 "Capacitor_SMD:C_0805_2012Metric" H 3200 3100 50  0001 C CNN
 F 3 "~" H 3200 3100 50  0001 C CNN
-F 4 "Wima" H 3200 3100 50  0001 C CNN "Manufacturer"
-F 5 "SMDTC04100QB00KP00" H 3200 3100 50  0001 C CNN "Manufacturers Part Number"
+F 4 "Kemet" H 3200 3100 50  0001 C CNN "Manufacturer"
+F 5 "C0805X105J3RACAUTO" H 3200 3100 50  0001 C CNN "Manufacturers Part Number"
+F 6 "0805in/2012mm" H 0   0   50  0001 C CNN "Package ID"
 	1    3200 3100
 	0    1    1    0
@@
 F 2 "Capacitor_SMD:C_0603_1608Metric" H 4900 3600 50  0001 C CNN
 F 3 "~" H 4900 3600 50  0001 C CNN
+F 4 "0603in/1608mm" H 0   0   50  0001 C CNN "Package ID"
 	1    4900 3600
 	-1   0    0    1
@@
 F 2 "Capacitor_SMD:C_0603_1608Metric" H 5100 3600 50  0001 C CNN
 F 3 "~" H 5100 3600 50  0001 C CNN
+F 4 "0603in/1608mm" H 0   0   50  0001 C CNN "Package ID"
 	1    5100 3600
 	-1   0    0    1
@@
 F 3 "https://product.tdk.com/info/en/catalog/datasheets/beads_commercial_power_mpz1608_en.pdf" H 7500 4700 50  0001 C CNN
 F 4 "TDK" H 7500 4700 50  0001 C CNN "Manufacturer"
-F 5 "0603" H 7500 4700 50  0001 C CNN "Package ID"
+F 5 "0603in/1608mm" H 7500 4700 50  0001 C CNN "Package ID"
 F 6 "MPZ1608S221A" H 7500 4700 50  0001 C CNN "Manufacturers Part Number"
 	1    7500 4700
@@
 F 2 "Capacitor_SMD:C_0603_1608Metric" H 4500 3300 50  0001 C CNN
 F 3 "~" H 4500 3300 50  0001 C CNN
+F 4 "0603in/1608mm" H 0   0   50  0001 C CNN "Package ID"
 	1    4500 3300
 	-1   0    0    1
@@
 F 2 "Capacitor_SMD:C_0603_1608Metric" H 4700 3300 50  0001 C CNN
 F 3 "~" H 4700 3300 50  0001 C CNN
+F 4 "0603in/1608mm" H 0   0   50  0001 C CNN "Package ID"
 	1    4700 3300
 	-1   0    0    1
@@
 F 2 "Capacitor_SMD:C_0603_1608Metric" H 7700 3750 50  0001 C CNN
 F 3 "~" H 7700 3750 50  0001 C CNN
+F 4 "TDK" H 0   0   50  0001 C CNN "Manufacturer"
+F 5 "CGA3E1X7R1E105K080AC" H 0   0   50  0001 C CNN "Manufacturers Part Number"
+F 6 "0603in/1608mm" H 0   0   50  0001 C CNN "Package ID"
 	1    7700 3750
 	-1   0    0    1
@@
 F 3 "~" H 7850 3750 50  0001 C CNN
 F 4 "Kemet" H 8000 2900 50  0001 C CNN "Manufacturer"
-F 5 "0603in/1608mm" H 8000 2900 50  0001 C CNN "Package ID"
+F 5 "1206in/3216mm" H 8000 2900 50  0001 C CNN "Package ID"
 F 6 "C1206C106J3RACAUTO" H 8000 2900 50  0001 C CNN "Manufacturers Part Number"
 	1    7850 3750
@@
 F 2 "Capacitor_SMD:C_0603_1608Metric" H 7450 3750 50  0001 C CNN
 F 3 "~" H 7450 3750 50  0001 C CNN
+F 4 "0603in/1608mm" H 0   0   50  0001 C CNN "Package ID"
 	1    7450 3750
 	-1   0    0    1
@@
 F 2 "Capacitor_SMD:C_0603_1608Metric" H 8000 2700 50  0001 C CNN
 F 3 "~" H 8000 2700 50  0001 C CNN
+F 4 "0603in/1608mm" H 0   0   50  0001 C CNN "Package ID"
 	1    8000 2700
 	0    1    1    0
@@
 F 3 "~" H 8000 2900 50  0001 C CNN
 F 4 "Kemet" H 8000 2900 50  0001 C CNN "Manufacturer"
-F 5 "0603in/1608mm" H 8000 2900 50  0001 C CNN "Package ID"
+F 5 "1206in/3216mm" H 8000 2900 50  0001 C CNN "Package ID"
 F 6 "C1206C106J3RACAUTO" H 8000 2900 50  0001 C CNN "Manufacturers Part Number"
 	1    8000 2900
@@
 F 2 "Capacitor_SMD:C_0603_1608Metric" H 8000 3100 50  0001 C CNN
 F 3 "~" H 8000 3100 50  0001 C CNN
+F 4 "0603in/1608mm" H 0   0   50  0001 C CNN "Package ID"
 	1    8000 3100
 	0    1    1    0
@@
 F 2 "Capacitor_SMD:C_0603_1608Metric" H 8000 3300 50  0001 C CNN
 F 3 "~" H 8000 3300 50  0001 C CNN
+F 4 "0603in/1608mm" H 0   0   50  0001 C CNN "Package ID"
 	1    8000 3300
 	0    1    1    0
@@
 F 2 "Capacitor_SMD:C_0603_1608Metric" H 8950 3150 50  0001 C CNN
 F 3 "~" H 8950 3150 50  0001 C CNN
+F 4 "0603in/1608mm" H 0   0   50  0001 C CNN "Package ID"
 	1    8950 3150
 	0    -1   -1   0
@@
 F 0 "C307" V 2750 3000 50  0000 C CNN
 F 1 "1uF" V 2850 3000 50  0000 C CNN
-F 2 "SW-WIMA:2220_film_cap" H 3000 3000 50  0001 C CNN
+F 2 "Capacitor_SMD:C_0805_2012Metric" H 3000 3000 50  0001 C CNN
 F 3 "~" H 3000 3000 50  0001 C CNN
-F 4 "SMDTC04100QB00KP00" H 3000 3000 50  0001 C CNN "Manufacturers Part Number"
-F 5 "Wima" H 3000 3000 50  0001 C CNN "Manufacturer"
+F 4 "C0805X105J3RACAUTO" H 3000 3000 50  0001 C CNN "Manufacturers Part Number"
+F 5 "Kemet" H 3000 3000 50  0001 C CNN "Manufacturer"
+F 6 "0805in/2012mm" H 0   0   50  0001 C CNN "Package ID"
 	1    3000 3000
 	0    1    1    0
@@
 F 2 "Capacitor_SMD:C_0603_1608Metric" H 4650 4550 50  0001 C CNN
 F 3 "~" H 4650 4550 50  0001 C CNN
+F 4 "0603in/1608mm" H 0   0   50  0001 C CNN "Package ID"
 	1    4650 4550
 	0    -1   -1   0
@@
 F 2 "Fuse:Fuse_0603_1608Metric" H 2250 3800 50  0001 L CNN
 F 3 "~" H 2200 4000 50  0001 C CNN
+F 4 "0603in/1608mm" H 0   0   50  0001 C CNN "Package ID"
 	1    2200 4000
 	0    1    1    0
@@
 F 5 "Transient Voltage Suppresion Diode" H 2000 4250 50  0001 C CNN "Description"
 F 6 "SMAJ12CA" H 2000 4250 50  0001 C CNN "Manufacturers Part Number"
+F 7 "SMA Diode" H 0   0   50  0001 C CNN "Package ID"
 	1    2000 4250
 	0    1    1    0
@@
 F 0 "C319" V 7250 4150 50  0000 C CNN
 F 1 "1uF" V 7350 4150 50  0000 C CNN
-F 2 "SW-WIMA:2220_film_cap" H 7100 4150 50  0001 C CNN
+F 2 "Capacitor_SMD:C_0805_2012Metric" H 7100 4150 50  0001 C CNN
 F 3 "~" H 7100 4150 50  0001 C CNN
-F 4 "Wima" H 7100 4150 50  0001 C CNN "Manufacturer"
-F 5 "SMDTC04100QB00KP00" H 7100 4150 50  0001 C CNN "Manufacturers Part Number"
+F 4 "Kemet" H 7100 4150 50  0001 C CNN "Manufacturer"
+F 5 "C0805X105J3RACAUTO" H 7100 4150 50  0001 C CNN "Manufacturers Part Number"
+F 6 "0805in/2012mm" H 0   0   50  0001 C CNN "Package ID"
 	1    7100 4150
 	0    1    1    0
@@
 F 0 "C320" V 7500 4250 50  0000 C CNN
 F 1 "1uF" V 7600 4250 50  0000 C CNN
-F 2 "SW-WIMA:2220_film_cap" H 7350 4250 50  0001 C CNN
+F 2 "Capacitor_SMD:C_0805_2012Metric" H 7350 4250 50  0001 C CNN
 F 3 "~" H 7350 4250 50  0001 C CNN
-F 4 "Wima" H 7350 4250 50  0001 C CNN "Manufacturer"
-F 5 "SMDTC04100QB00KP00" H 7350 4250 50  0001 C CNN "Manufacturers Part Number"
+F 4 "Kemet" H 7350 4250 50  0001 C CNN "Manufacturer"
+F 5 "C0805X105J3RACAUTO" H 7350 4250 50  0001 C CNN "Manufacturers Part Number"
+F 6 "0805in/2012mm" H 0   0   50  0001 C CNN "Package ID"
 	1    7350 4250
 	0    1    1    0
