File: edc-mux-board-fpga/conn3.sch (KiCad schematic (older format))
At the start: 24 parts

Commit message: Finished FPGA and MCU interconnections.
Finished up interrupt wiring
Fixed a few missing connections
Annotated Schematic
Parts:
- removed C? (x2): 1uF, Capacitor_SMD:C_0805_2012Metric, symbol Device:C_Small
- removed C? (x2): 2.2uF X7R, Capacitor_SMD:C_0603_1608Metric, symbol Device:C_Small
- removed C? (x2): 1uF, Capacitor_SMD:C_0603_1608Metric, symbol Device:C_Small
- removed C? (x8): 100nF, Capacitor_SMD:C_0603_1608Metric, symbol Device:C_Small
- removed C? (x2): 33pF, Capacitor_SMD:C_0603_1608Metric, symbol Device:C_Small
- removed C?: 10uF, Capacitor_SMD:C_1206_3216Metric, symbol Device:C_Small
- removed R? (x2): 750Ω, Resistor_SMD:R_0603_1608Metric, symbol Device:R_Small_US
- removed U?: TLV320AIC3206, Package_DFN_QFN:UQFN-40-1EP_5x5mm_P0.4mm_EP3.8x3.8mm_ThermalVias, symbol SW-Texas:TLV320AIC3206
- removed U?: MAX4910, Package_DFN_QFN:TQFN-16-1EP_3x3mm_P0.5mm_EP1.23x1.23mm, symbol SW-dallas-semi-maxim:MAX4910
- removed U?: P82B96, Package_SO:TSSOP-8_3x3mm_P0.65mm, symbol Interface_Expansion:P82B96
- added C59, C76: 2.2uF X7R, Capacitor_SMD:C_0603_1608Metric, symbol Device:C_Small
- added C60, C62, C63, C66, C67, C68, C69, C74: 100nF, Capacitor_SMD:C_0603_1608Metric, symbol Device:C_Small
- added C64, C65: 33pF, Capacitor_SMD:C_0603_1608Metric, symbol Device:C_Small
- added C70, C75: 1uF, Capacitor_SMD:C_0603_1608Metric, symbol Device:C_Small
- added C71: 10uF, Capacitor_SMD:C_1206_3216Metric, symbol Device:C_Small
- added C72, C73: 1uF, Capacitor_SMD:C_0805_2012Metric, symbol Device:C_Small
- added R21, R22: 750Ω, Resistor_SMD:R_0603_1608Metric, symbol Device:R_Small_US
- added U13: MAX4910, Package_DFN_QFN:TQFN-16-1EP_3x3mm_P0.5mm_EP1.23x1.23mm, symbol SW-dallas-semi-maxim:MAX4910
- added U14: TLV320AIC3206, Package_DFN_QFN:UQFN-40-1EP_5x5mm_P0.4mm_EP3.8x3.8mm_ThermalVias, symbol SW-Texas:TLV320AIC3206
- added U15: P82B96, Package_SO:TSSOP-8_3x3mm_P0.65mm, symbol Interface_Expansion:P82B96
- gave numbers to parts that had none: 2
Connections:
- net +12V: now also C74.1, R21.1, R22.1, U15.8 (VCC)
- net +1V8: now also C62.2, C66.2, U14.30 (VSYS), U14.40 (DVDD)
- net +1V8A: now also C69.2, C70.2, C71.2, U14.29 (AVDD), U14.32 (DRVDD_HP), U14.39 (DVDD_CP)
- net +3V3: now also C60.2, C63.2, U13.14 (VCC), U14.10 (IOVDD)
- net AUD_GND: now also U13.4 (COM2)
- net BCLK: now also U14.6 (BCLK)
- net DIN: now also U14.8 (DIN)
- net DOUT: now also U14.9 (DOUT)
- net GND: now also C60.1, C62.1, C63.1, C64.1, C65.1, C66.1, C67.1, C68.1, C69.1, C70.1, C71.1, C74.2, C75.1, C76.1, U13.17 (PAD), U13.5 (NC2), U13.6 (GND), U14.1 (DVSS), U14.11 (IOVSS), U14.16 (SPI_SELECT), U14.2 (DVSS), U14.21 (AVSS), U14.37 (DVSS_CP), U14.41 (PAD), U15.4 (GND)
- net HP_~LINE~_SEL: now also U13.10 (CB2), U13.2 (CB1), U14.4 (INT2_OUT)
- net L_IN: now also C64.2, U14.17 (IN1_L)
- net L_OUT: now also U13.16 (COM1)
- net MCLK: now also U14.5 (MCLK)
- net R_IN: now also C65.2, U14.18 (IN1_R)
- net R_OUT: now also U13.8 (COM3)
- net SCL: now also U14.13 (SCL), U15.7 (SCL)
- net SCL_HV: now also R22.2, U15.5 (TXD-SCL), U15.6 (RXD-SCL)
- net SDA: now also U14.14 (SDA), U15.1 (SDA)
- net SDA_HV: now also R21.2, U15.2 (RXD-SDA), U15.3 (TXD-SDA)
- net WCLK: now also U14.7 (WCLK)
- net ~RESET: now also U14.3 (~RESET)
- net at FB6.1: now also U13.3 (NO2), U14.28 (GND_SENSE)
- new net: C72.1, U13.1 (NC1)
- new net: C72.2, U14.26 (LINE_OUT_L)
- new net: C73.1, U13.9 (NC3)
- new net: C73.2, U14.27 (LINE_OUT_R)
- new net: C67.2, U14.19 (IN2_L), U14.20 (IN2_R)
- new net: C75.2, U14.22 (REF)
- new net: C68.2, U14.24 (IN3_L), U14.25 (IN3_R)
- new net: U13.15 (NO1), U14.31 (HPL)
- new net: U13.7 (NO3), U14.33 (HPR)
- new net: C76.2, U14.35 (VNEG)
- new net: C59.1, U14.36 (FLY_N)
- new net: C59.2, U14.38 (FLY_P)
Changed lines of the file:
@@
 $EndDescr
 $Comp
-L SW-Texas:TLV320AIC3206 U?
-U 1 1 5CE6F2E7
+L SW-Texas:TLV320AIC3206 U14
+U 1 1 5DAC04B8
 P 5200 3400
-F 0 "U?" H 5650 2350 50  0000 C CNN
+F 0 "U14" H 5650 2350 50  0000 C CNN
 F 1 "TLV320AIC3206" H 4700 4450 50  0000 C CNN
 F 2 "Package_DFN_QFN:UQFN-40-1EP_5x5mm_P0.4mm_EP3.8x3.8mm_ThermalVias" H 5250 4800 50  0001 C CNN
@@
 $EndComp
 $Comp
-L Device:C_Small C?
-U 1 1 5CE6F309
+L Device:C_Small C59
+U 1 1 5DAC04C0
 P 5200 2150
-F 0 "C?" V 4950 2150 50  0000 C CNN
+F 0 "C59" V 4950 2150 50  0000 C CNN
 F 1 "2.2uF X7R" V 5050 2150 50  0000 C CNN
 F 2 "Capacitor_SMD:C_0603_1608Metric" H 5200 2150 50  0001 C CNN
@@
 	5300 2250 5300 2150
 $Comp
-L Device:C_Small C?
-U 1 1 5CE6F311
+L Device:C_Small C76
+U 1 1 5DAC04D8
 P 6050 4250
-F 0 "C?" V 5800 4250 50  0000 C CNN
+F 0 "C76" V 5800 4250 50  0000 C CNN
 F 1 "2.2uF X7R" V 5900 4250 50  0000 C CNN
 F 2 "Capacitor_SMD:C_0603_1608Metric" H 6050 4250 50  0001 C CNN
@@
 	6050 4100 6050 4150
 $Comp
-L power:GND #PWR?
-U 1 1 5CE6F323
+L power:GND #PWR055
+U 1 1 5DAC04DC
 P 5750 4750
-F 0 "#PWR?" H 5750 4500 50  0001 C CNN
+F 0 "#PWR055" H 5750 4500 50  0001 C CNN
 F 1 "GND" H 5750 4600 50  0000 C CNN
 F 2 "" H 5750 4750 50  0001 C CNN
@@
 	5450 4650 5750 4650
 $Comp
-L Device:C_Small C?
-U 1 1 5CE6F329
+L Device:C_Small C75
+U 1 1 5DAC04F4
 P 4400 4250
-F 0 "C?" H 4500 4200 50  0000 L CNN
+F 0 "C75" H 4500 4200 50  0000 L CNN
 F 1 "1uF" H 4500 4250 50  0000 L CNN
 F 2 "Capacitor_SMD:C_0603_1608Metric" H 4400 4250 50  0001 C CNN
@@
 Connection ~ 4950 4650
 $Comp
-L Device:C_Small C?
-U 1 1 5CE6F348
+L Device:C_Small C67
+U 1 1 5DAC0501
 P 3950 3050
-F 0 "C?" H 4050 3000 50  0000 L CNN
+F 0 "C67" H 4050 3000 50  0000 L CNN
 F 1 "100nF" H 4050 3050 50  0000 L CNN
 F 2 "Capacitor_SMD:C_0603_1608Metric" H 3950 3050 50  0001 C CNN
@@
 $EndComp
 $Comp
-L Device:C_Small C?
-U 1 1 5CE6F363
+L Device:C_Small C68
+U 1 1 5DAC0513
 P 4150 3050
-F 0 "C?" H 4050 3000 50  0000 R CNN
+F 0 "C68" H 4050 3000 50  0000 R CNN
 F 1 "100nF" H 4050 3050 50  0000 R CNN
 F 2 "Capacitor_SMD:C_0603_1608Metric" H 4150 3050 50  0001 C CNN
@@
 Connection ~ 4400 2950
 $Comp
-L power:GND #PWR?
-U 1 1 5CE6F368
+L power:GND #PWR050
+U 1 1 5DAC0517
 P 3550 3250
-F 0 "#PWR?" H 3550 3000 50  0001 C CNN
+F 0 "#PWR050" H 3550 3000 50  0001 C CNN
 F 1 "GND" H 3550 3100 50  0000 C CNN
 F 2 "" H 3550 3250 50  0001 C CNN
@@
 	8650 3300 8850 3300
 $Comp
-L SW-dallas-semi-maxim:MAX4910 U?
-U 1 1 5CE6F375
+L SW-dallas-semi-maxim:MAX4910 U13
+U 1 1 5DAC0529
 P 8300 3350
-F 0 "U?" H 8500 2800 50  0000 C CNN
+F 0 "U13" H 8500 2800 50  0000 C CNN
 F 1 "MAX4910" H 7950 3350 50  0000 C CNN
 F 2 "Package_DFN_QFN:TQFN-16-1EP_3x3mm_P0.5mm_EP1.23x1.23mm" H 9950 4500 50  0001 C CNN
@@
 	7750 3450 7750 4250
 $Comp
-L power:GND #PWR?
-U 1 1 5CE6F387
+L power:GND #PWR054
+U 1 1 5DAC053F
 P 7750 4400
-F 0 "#PWR?" H 7750 4150 50  0001 C CNN
+F 0 "#PWR054" H 7750 4150 50  0001 C CNN
 F 1 "GND" H 7750 4250 50  0000 C CNN
 F 2 "" H 7750 4400 50  0001 C CNN
@@
 	8650 3500 8850 3500
 $Comp
-L Device:Ferrite_Bead_Small FB?
+L Device:Ferrite_Bead_Small FB6
 U 1 1 5CE6F39A
 P 6550 4150
-F 0 "FB?" H 6625 4200 50  0000 L CNN
+F 0 "FB6" H 6625 4200 50  0000 L CNN
 F 1 "220Ω/2A" H 6625 4100 50  0000 L CNN
 F 2 "Resistor_SMD:R_0603_1608Metric" V 6480 4150 50  0001 C CNN
@@
 	3750 2600 4450 2600
 $Comp
-L Device:C_Small C?
-U 1 1 5CE6F3AC
+L Device:C_Small C64
+U 1 1 5DAC055C
 P 3550 2750
-F 0 "C?" H 3650 2700 50  0000 L CNN
+F 0 "C64" H 3650 2700 50  0000 L CNN
 F 1 "33pF" H 3650 2750 50  0000 L CNN
 F 2 "Capacitor_SMD:C_0603_1608Metric" H 3550 2750 50  0001 C CNN
@@
 	3200 2550 3750 2550
 $Comp
-L Device:C_Small C?
-U 1 1 5CE6F3B7
+L Device:C_Small C65
+U 1 1 5DAC0567
 P 3750 2750
-F 0 "C?" H 3650 2700 50  0000 R CNN
+F 0 "C65" H 3650 2700 50  0000 R CNN
 F 1 "33pF" H 3650 2750 50  0000 R CNN
 F 2 "Capacitor_SMD:C_0603_1608Metric" H 3750 2750 50  0001 C CNN
@@
 	5950 3000 6500 3000
 $Comp
-L SW-power:+1V8A #+1V8A?
-U 1 1 5CE6F3C8
+L SW-power:+1V8A #+1V8A05
+U 1 1 5DAC0573
 P 6750 2100
-F 0 "#+1V8A?" H 7500 1800 60  0001 C CNN
+F 0 "#+1V8A05" H 7500 1800 60  0001 C CNN
 F 1 "+1V8A" H 6750 2300 50  0000 C CNN
 F 2 "" H 6750 2100 60  0001 C CNN
@@
 $EndComp
 $Comp
-L power:+1V8 #PWR?
-U 1 1 5CE6F3D1
+L power:+1V8 #PWR048
+U 1 1 5DAC0582
 P 6500 2100
-F 0 "#PWR?" H 6500 1950 50  0001 C CNN
+F 0 "#PWR048" H 6500 1950 50  0001 C CNN
 F 1 "+1V8" H 6500 2240 50  0000 C CNN
 F 2 "" H 6500 2100 50  0001 C CNN
@@
 	6750 2800 6750 2900
 $Comp
-L power:+3V3 #PWR?
-U 1 1 5CE6F3E5
+L power:+3V3 #PWR047
+U 1 1 5DAC0595
 P 6250 2100
-F 0 "#PWR?" H 6250 1950 50  0001 C CNN
+F 0 "#PWR047" H 6250 1950 50  0001 C CNN
 F 1 "+3V3" H 6250 2240 50  0000 C CNN
 F 2 "" H 6250 2100 50  0001 C CNN
@@
 	6250 2600 6250 2350
 $Comp
-L Device:C_Small C?
-U 1 1 5CE6F3F4
+L Device:C_Small C70
+U 1 1 5DAC059D
 P 6750 3200
-F 0 "C?" H 6850 3100 50  0000 R CNN
+F 0 "C70" H 6850 3100 50  0000 R CNN
 F 1 "1uF" H 6900 3300 50  0000 R CNN
 F 2 "Capacitor_SMD:C_0603_1608Metric" H 6750 3200 50  0001 C CNN
@@
 $EndComp
 $Comp
-L power:GND #PWR?
-U 1 1 5CE6F403
+L power:GND #PWR051
+U 1 1 5DAC05B7
 P 6650 3400
-F 0 "#PWR?" H 6650 3150 50  0001 C CNN
+F 0 "#PWR051" H 6650 3150 50  0001 C CNN
 F 1 "GND" H 6650 3250 50  0000 C CNN
 F 2 "" H 6650 3400 50  0001 C CNN
@@
 $EndComp
 $Comp
-L Device:C_Small C?
-U 1 1 5CE6F40F
+L Device:C_Small C71
+U 1 1 5DAC05C6
 P 6900 3200
-F 0 "C?" H 6800 3150 50  0000 R CNN
+F 0 "C71" H 6800 3150 50  0000 R CNN
 F 1 "10uF" H 6800 3200 50  0000 R CNN
 F 2 "Capacitor_SMD:C_1206_3216Metric" H 6900 3200 50  0001 C CNN
@@
 $EndComp
 $Comp
-L Device:C_Small C?
-U 1 1 5CE6F425
+L Device:C_Small C69
+U 1 1 5DAC05D3
 P 6500 3200
-F 0 "C?" H 6650 3100 50  0000 R CNN
+F 0 "C69" H 6650 3100 50  0000 R CNN
 F 1 "100nF" V 6600 3400 50  0000 R CNN
 F 2 "Capacitor_SMD:C_0603_1608Metric" H 6500 3200 50  0001 C CNN
@@
 	6650 3350 6750 3350
 $Comp
-L Device:C_Small C?
-U 1 1 5CE6F42F
+L Device:C_Small C60
+U 1 1 5DAC05DD
 P 7050 2150
-F 0 "C?" H 7200 2050 50  0000 R CNN
+F 0 "C60" H 7200 2050 50  0000 R CNN
 F 1 "100nF" V 7150 2350 50  0000 R CNN
 F 2 "Capacitor_SMD:C_0603_1608Metric" H 7050 2150 50  0001 C CNN
@@
 $EndComp
 $Comp
-L Device:C_Small C?
+L Device:C_Small C61
 U 1 1 5CE6F439
 P 7050 2350
-F 0 "C?" H 6950 2450 50  0000 C CNN
+F 0 "C61" H 6950 2450 50  0000 C CNN
 F 1 "10uF" V 6950 2300 50  0000 C CNN
 F 2 "Capacitor_SMD:C_1206_3216Metric" H 7050 2350 50  0001 C CNN
@@
 	6250 2150 6250 2100
 $Comp
-L Device:C_Small C?
-U 1 1 5CE6F451
+L Device:C_Small C62
+U 1 1 5DAC05FC
 P 7050 2550
-F 0 "C?" H 7200 2450 50  0000 R CNN
+F 0 "C62" H 7200 2450 50  0000 R CNN
 F 1 "100nF" V 7150 2750 50  0000 R CNN
 F 2 "Capacitor_SMD:C_0603_1608Metric" H 7050 2550 50  0001 C CNN
@@
 	6500 2550 6500 2500
 $Comp
-L Device:C_Small C?
-U 1 1 5CE6F456
+L Device:C_Small C66
+U 1 1 5DAC060E
 P 7050 2750
-F 0 "C?" H 7200 2650 50  0000 R CNN
+F 0 "C66" H 7200 2650 50  0000 R CNN
 F 1 "100nF" V 7150 2950 50  0000 R CNN
 F 2 "Capacitor_SMD:C_0603_1608Metric" H 7050 2750 50  0001 C CNN
@@
 NoConn ~ 8650 3750
 $Comp
-L Device:C_Small C?
-U 1 1 5CE6F46F
+L Device:C_Small C63
+U 1 1 5DAC061F
 P 8000 2600
-F 0 "C?" H 8150 2500 50  0000 R CNN
+F 0 "C63" H 8150 2500 50  0000 R CNN
 F 1 "100nF" V 8100 2800 50  0000 R CNN
 F 2 "Capacitor_SMD:C_0603_1608Metric" H 8000 2600 50  0001 C CNN
@@
 $EndComp
 $Comp
-L power:+3V3 #PWR?
-U 1 1 5CE6F47E
+L power:+3V3 #PWR049
+U 1 1 5DAC0626
 P 8300 2350
-F 0 "#PWR?" H 8300 2200 50  0001 C CNN
+F 0 "#PWR049" H 8300 2200 50  0001 C CNN
 F 1 "+3V3" H 8300 2490 50  0000 C CNN
 F 2 "" H 8300 2350 50  0001 C CNN
@@
 	8250 4250 8350 4250
 $Comp
-L Interface_Expansion:P82B96 U?
-U 1 1 5CE6F489
+L Interface_Expansion:P82B96 U15
+U 1 1 5DAC0641
 P 2600 4300
-F 0 "U?" H 2100 4800 50  0000 L CNN
+F 0 "U15" H 2100 4800 50  0000 L CNN
 F 1 "P82B96" H 2800 4800 50  0000 L CNN
 F 2 "Package_SO:TSSOP-8_3x3mm_P0.65mm" H 2600 4300 50  0001 C CNN
@@
 $EndComp
 $Comp
-L power:+12V #PWR?
+L power:+12V #PWR052
 U 1 1 5CE6F490
 P 1550 3550
-F 0 "#PWR?" H 1550 3400 50  0001 C CNN
+F 0 "#PWR052" H 1550 3400 50  0001 C CNN
 F 1 "+12V" H 1550 3690 50  0000 C CNN
 F 2 "" H 1550 3550 50  0001 C CNN
@@
 	1900 4100 1900 4200
 $Comp
-L Device:R_Small_US R?
-U 1 1 5CE6F4C1
+L Device:R_Small_US R21
+U 1 1 5DAC0655
 P 1700 3900
-F 0 "R?" H 1800 3950 50  0000 L CNN
+F 0 "R21" H 1800 3950 50  0000 L CNN
 F 1 "750Ω" H 1800 3900 50  0000 L CNN
 F 2 "Resistor_SMD:R_0603_1608Metric" H 1700 3900 50  0001 C CNN
@@
 $EndComp
 $Comp
-L Device:R_Small_US R?
-U 1 1 5CE6F4D0
+L Device:R_Small_US R22
+U 1 1 5DAC066A
 P 1550 4300
-F 0 "R?" H 1650 4350 50  0000 L CNN
+F 0 "R22" H 1650 4350 50  0000 L CNN
 F 1 "750Ω" H 1650 4300 50  0000 L CNN
 F 2 "Resistor_SMD:R_0603_1608Metric" H 1550 4300 50  0001 C CNN
@@
 	1700 4100 1900 4100
 $Comp
-L power:+12V #PWR?
-U 1 1 5CE6F4E1
+L power:+12V #PWR053
+U 1 1 5DAC067A
 P 3250 3750
-F 0 "#PWR?" H 3250 3600 50  0001 C CNN
+F 0 "#PWR053" H 3250 3600 50  0001 C CNN
 F 1 "+12V" H 3250 3890 50  0000 C CNN
 F 2 "" H 3250 3750 50  0001 C CNN
@@
 	3200 4400 3400 4400
 $Comp
-L Device:C_Small C?
-U 1 1 5CE6F4F3
+L Device:C_Small C74
+U 1 1 5DAC0682
 P 3700 4000
-F 0 "C?" V 3550 4000 50  0000 C CNN
+F 0 "C74" V 3550 4000 50  0000 C CNN
 F 1 "100nF" V 3450 4000 50  0000 C CNN
 F 2 "Capacitor_SMD:C_0603_1608Metric" H 3700 4000 50  0001 C CNN
@@
 	1450 4500 1550 4500
 $Comp
-L Device:C_Small C?
-U 1 1 5CE6F2C0
+L Device:C_Small C72
+U 1 1 5DAC0493
 P 6150 3600
-F 0 "C?" V 6300 3600 50  0000 C CNN
+F 0 "C72" V 6300 3600 50  0000 C CNN
 F 1 "1uF" V 6400 3600 50  0000 C CNN
 F 2 "Capacitor_SMD:C_0805_2012Metric" H 6150 3600 50  0001 C CNN
@@
 $EndComp
 $Comp
-L Device:C_Small C?
-U 1 1 5CE6F2D4
+L Device:C_Small C73
+U 1 1 5DAC04AC
 P 6400 3700
-F 0 "C?" V 6550 3700 50  0000 C CNN
+F 0 "C73" V 6550 3700 50  0000 C CNN
 F 1 "1uF" V 6650 3700 50  0000 C CNN
 F 2 "Capacitor_SMD:C_0805_2012Metric" H 6400 3700 50  0001 C CNN

Commit message: assigned more footprints
Parts:
- C61, C71: value 10uF -> 10uF X7R
- C70, C75: value 1uF -> 1uF X7R
- C72, C73: value 1uF -> 1uF X7R flex
Changed lines of the file:
@@
 P 4400 4250
 F 0 "C75" H 4500 4200 50  0000 L CNN
-F 1 "1uF" H 4500 4250 50  0000 L CNN
+F 1 "1uF X7R" H 4500 4250 50  0000 L CNN
 F 2 "Capacitor_SMD:C_0603_1608Metric" H 4400 4250 50  0001 C CNN
 F 3 "~" H 4400 4250 50  0001 C CNN
@@
 P 6750 3200
 F 0 "C70" H 6850 3100 50  0000 R CNN
-F 1 "1uF" H 6900 3300 50  0000 R CNN
+F 1 "1uF X7R" H 6900 3300 50  0000 R CNN
 F 2 "Capacitor_SMD:C_0603_1608Metric" H 6750 3200 50  0001 C CNN
 F 3 "~" H 6750 3200 50  0001 C CNN
@@
 P 6900 3200
 F 0 "C71" H 6800 3150 50  0000 R CNN
-F 1 "10uF" H 6800 3200 50  0000 R CNN
+F 1 "10uF X7R" H 6800 3200 50  0000 R CNN
 F 2 "Capacitor_SMD:C_1206_3216Metric" H 6900 3200 50  0001 C CNN
 F 3 "~" H 6900 3200 50  0001 C CNN
@@
 P 7050 2350
 F 0 "C61" H 6950 2450 50  0000 C CNN
-F 1 "10uF" V 6950 2300 50  0000 C CNN
+F 1 "10uF X7R" V 6950 2300 50  0000 C CNN
 F 2 "Capacitor_SMD:C_1206_3216Metric" H 7050 2350 50  0001 C CNN
 F 3 "~" H 7050 2350 50  0001 C CNN
@@
 P 6150 3600
 F 0 "C72" V 6300 3600 50  0000 C CNN
-F 1 "1uF" V 6400 3600 50  0000 C CNN
+F 1 "1uF X7R flex" V 6400 3600 50  0000 C CNN
 F 2 "Capacitor_SMD:C_0805_2012Metric" H 6150 3600 50  0001 C CNN
 F 3 "~" H 6150 3600 50  0001 C CNN
@@
 P 6400 3700
 F 0 "C73" V 6550 3700 50  0000 C CNN
-F 1 "1uF" V 6650 3700 50  0000 C CNN
+F 1 "1uF X7R flex" V 6650 3700 50  0000 C CNN
 F 2 "Capacitor_SMD:C_0805_2012Metric" H 6400 3700 50  0001 C CNN
 F 3 "~" H 6400 3700 50  0001 C CNN

Commit message: re-annotating after adding power ICs and decoupling capacitors.
Also verified most footprints, and updated schematic field data.
Parts:
- C171: renamed from C74; value 100nF -> 100nF X7R
- C173: renamed from C67; value 100nF -> 100nF X7R
- C174: renamed from C68; value 100nF -> 100nF X7R
- C180: renamed from C69; value 100nF -> 100nF X7R
- C183: renamed from C60; value 100nF -> 100nF X7R
- C185: renamed from C62; value 100nF -> 100nF X7R
- C186: renamed from C66; value 100nF -> 100nF X7R
- C187: renamed from C63; value 100nF -> 100nF X7R
- R21: renamed from R22; Package ID (none) -> 0402in/1005mm
- R22: renamed from R21; Package ID (none) -> 0402in/1005mm
- renumbered C64 to C170, C65 to C172, C75 to C175, C59 to C176, C76 to C177, C72 to C178, C73 to C179, C70 to C181, C71 to C182, C61 to C184, FB6 to FB7, U15 to U18, U14 to U19, U13 to U20

Commit message: Reannotating and adding more fields to components
Parts:
- C170, C172: value 33pF -> 33pF NP0; footprint Capacitor_SMD:C_0603_1608Metric -> Capacitor_SMD:C_0402_1005Metric; Characteristics (none) -> CAP CER 33PF 25V NP0 0402; Description (none) -> MLCC Capacitor; Manufacturer (none) -> AVX; Manufacturers Part Number (none) -> 04023A330FAT2A; Package ID 0603in/1608mm -> 0402in/1005mm
- C171, C173, C174, C180, C183, C185, C186, C187: Characteristics (none) -> CAP CER 0.1UF 25V X7R 0603; Description (none) -> MLCC Capacitor; Manufacturer (none) -> Kemet; Manufacturers Part Number (none) -> C0603C104J3RACAUTO
- C175, C181: Characteristics (none) -> CAP CER 1UF 25V X7R 0603; Description (none) -> MLCC Capacitor
- C176, C177: footprint Capacitor_SMD:C_0603_1608Metric -> Capacitor_SMD:C_0805_2012Metric; Characteristics (none) -> CAP CER 2.2UF 25V X7R 0805; Description (none) -> MLCC Capacitor; Manufacturer (none) -> TDK; Manufacturers Part Number (none) -> CGA4J3X7R1E225K125AB; Package ID 0603in/1608mm -> 0805in/2012mm
- C178, C179: Characteristics (none) -> CAP CER 0805 1UF 25V X7R 5%; Description (none) -> MLCC Capacitor; Manufacturers Part Number C0805X105J3RACAUTO -> C0805X105J3RECAUTO
- C182, C184: Characteristics (none) -> CAP CER 10UF 25V X7R 1206; Description (none) -> MLCC Capacitor
- FB7: footprint Resistor_SMD:R_0603_1608Metric -> Inductor_SMD:L_0603_1608Metric; Description (none) -> Ferrite Bead
- R21, R22: Description (none) -> Resistor
- U18: Description (none) -> I2C Buffer / Voltage Translator; Manufacturer (none) -> Texas Instruments; Manufacturers Part Number (none) -> P82B96; Package ID (none) -> TSSOP8
- U19: Description (none) -> I2S Audio Codec; Manufacturer (none) -> Texas Instruments; Package ID (none) -> UQFN40
- U20: Description (none) -> Clickless Audio Switch; Manufacturer (none) -> Maxim Integrated; Package ID (none) -> TQFN16

Commit message: Fixed resistor footprint
Parts:
- R21, R22: footprint Resistor_SMD:R_0603_1608Metric -> Resistor_SMD:R_0402_1005Metric
Changed lines of the file:
@@
 F 0 "R22" H 1800 3950 50  0000 L CNN
 F 1 "750Ω" H 1800 3900 50  0000 L CNN
-F 2 "Resistor_SMD:R_0603_1608Metric" H 1700 3900 50  0001 C CNN
+F 2 "Resistor_SMD:R_0402_1005Metric" H 1700 3900 50  0001 C CNN
 F 3 "~" H 1700 3900 50  0001 C CNN
 F 4 "0402in/1005mm" H 0   0   50  0001 C CNN "Package ID"
@@
 F 0 "R21" H 1650 4350 50  0000 L CNN
 F 1 "750Ω" H 1650 4300 50  0000 L CNN
-F 2 "Resistor_SMD:R_0603_1608Metric" H 1550 4300 50  0001 C CNN
+F 2 "Resistor_SMD:R_0402_1005Metric" H 1550 4300 50  0001 C CNN
 F 3 "~" H 1550 4300 50  0001 C CNN
 F 4 "0402in/1005mm" H 0   0   50  0001 C CNN "Package ID"
