File: edc-mux-board-fpga/conn6.sch (KiCad schematic (older format))
At the start: 24 parts

Commit message: Finished FPGA and MCU interconnections.
Finished up interrupt wiring
Fixed a few missing connections
Annotated Schematic
Parts:
- removed C?: 1uF, Capacitor_SMD:C_0805_2012Metric, symbol Device:C_Small
- removed C? (x2): 2.2uF X7R, Capacitor_SMD:C_0603_1608Metric, symbol Device:C_Small
- removed C? (x2): 1uF, Capacitor_SMD:C_0603_1608Metric, symbol Device:C_Small
- removed C? (x8): 100nF, Capacitor_SMD:C_0603_1608Metric, symbol Device:C_Small
- removed C?: 33pF, Capacitor_SMD:C_0603_1608Metric, symbol Device:C_Small
- removed C? (x2): 10uF, Capacitor_SMD:C_1206_3216Metric, symbol Device:C_Small
- removed FB?: 220Ω/2A, Resistor_SMD:R_0603_1608Metric, symbol Device:Ferrite_Bead_Small
- removed R? (x2): 750Ω, Resistor_SMD:R_0603_1608Metric, symbol Device:R_Small_US
- removed U?: TLV320AIC3206, Package_DFN_QFN:UQFN-40-1EP_5x5mm_P0.4mm_EP3.8x3.8mm_ThermalVias, symbol SW-Texas:TLV320AIC3206
- removed U?: MAX4910, Package_DFN_QFN:TQFN-16-1EP_3x3mm_P0.5mm_EP1.23x1.23mm, symbol SW-dallas-semi-maxim:MAX4910
- removed U?: P82B96, Package_SO:TSSOP-8_3x3mm_P0.65mm, symbol Interface_Expansion:P82B96
- added C113, C130: 2.2uF X7R, Capacitor_SMD:C_0603_1608Metric, symbol Device:C_Small
- added C114, C116, C117, C120, C121, C122, C123, C128: 100nF, Capacitor_SMD:C_0603_1608Metric, symbol Device:C_Small
- added C115, C125: 10uF, Capacitor_SMD:C_1206_3216Metric, symbol Device:C_Small
- added C119: 33pF, Capacitor_SMD:C_0603_1608Metric, symbol Device:C_Small
- added C124, C129: 1uF, Capacitor_SMD:C_0603_1608Metric, symbol Device:C_Small
- added C127: 1uF, Capacitor_SMD:C_0805_2012Metric, symbol Device:C_Small
- added FB9: 220Ω/2A, Resistor_SMD:R_0603_1608Metric, symbol Device:Ferrite_Bead_Small
- added R27, R28: 750Ω, Resistor_SMD:R_0603_1608Metric, symbol Device:R_Small_US
- added U22: MAX4910, Package_DFN_QFN:TQFN-16-1EP_3x3mm_P0.5mm_EP1.23x1.23mm, symbol SW-dallas-semi-maxim:MAX4910
- added U23: TLV320AIC3206, Package_DFN_QFN:UQFN-40-1EP_5x5mm_P0.4mm_EP3.8x3.8mm_ThermalVias, symbol SW-Texas:TLV320AIC3206
- added U24: P82B96, Package_SO:TSSOP-8_3x3mm_P0.65mm, symbol Interface_Expansion:P82B96
- gave numbers to parts that had none: 2
Connections:
- net +12V: now also C128.1, R27.1, R28.1, U24.8 (VCC)
- net +1V8: now also C116.2, C120.2, U23.30 (VSYS), U23.40 (DVDD)
- net +1V8A: now also C123.2, C124.2, C125.2, U23.29 (AVDD), U23.32 (DRVDD_HP), U23.39 (DVDD_CP)
- net +3V3: now also C114.2, C115.1, C117.2, U22.14 (VCC), U23.10 (IOVDD)
- net AUD_GND: now also U22.4 (COM2)
- net BCLK: now also U23.6 (BCLK)
- net DIN: now also U23.8 (DIN)
- net DOUT: now also U23.9 (DOUT)
- net GND: now also C114.1, C115.2, C116.1, C117.1, C119.1, C120.1, C121.1, C122.1, C123.1, C124.1, C125.1, C128.2, C129.1, C130.1, FB9.2, U22.17 (PAD), U22.5 (NC2), U22.6 (GND), U23.1 (DVSS), U23.11 (IOVSS), U23.16 (SPI_SELECT), U23.2 (DVSS), U23.21 (AVSS), U23.37 (DVSS_CP), U23.41 (PAD), U24.4 (GND)
- net HP_~LINE~_SEL: now also U22.10 (CB2), U22.2 (CB1), U23.4 (INT2_OUT)
- net L_IN: now also U23.17 (IN1_L)
- net L_OUT: now also U22.16 (COM1)
- net MCLK: now also U23.5 (MCLK)
- net R_IN: now also C119.2, U23.18 (IN1_R)
- net R_OUT: now also U22.8 (COM3)
- net SCL: now also U23.13 (SCL), U24.7 (SCL)
- net SCL_HV: now also R28.2, U24.5 (TXD-SCL), U24.6 (RXD-SCL)
- net SDA: now also U23.14 (SDA), U24.1 (SDA)
- net SDA_HV: now also R27.2, U24.2 (RXD-SDA), U24.3 (TXD-SDA)
- net WCLK: now also U23.7 (WCLK)
- net ~RESET: now also U23.3 (~RESET)
- net at C126.1: now also U22.1 (NC1)
- net at C126.2: now also U23.26 (LINE_OUT_L)
- new net: C127.1, U22.9 (NC3)
- new net: C127.2, U23.27 (LINE_OUT_R)
- new net: C121.2, U23.19 (IN2_L), U23.20 (IN2_R)
- new net: C129.2, U23.22 (REF)
- new net: C122.2, U23.24 (IN3_L), U23.25 (IN3_R)
- new net: FB9.1, U22.3 (NO2), U23.28 (GND_SENSE)
- new net: U22.15 (NO1), U23.31 (HPL)
- new net: U22.7 (NO3), U23.33 (HPR)
- new net: C130.2, U23.35 (VNEG)
- new net: C113.1, U23.36 (FLY_N)
- new net: C113.2, U23.38 (FLY_P)
Changed lines of the file:
@@
 $EndDescr
 $Comp
-L SW-Texas:TLV320AIC3206 U?
-U 1 1 5CE6F2E7
+L SW-Texas:TLV320AIC3206 U23
+U 1 1 5DAC04B3
 P 5200 3400
-F 0 "U?" H 5650 2350 50  0000 C CNN
+F 0 "U23" H 5650 2350 50  0000 C CNN
 F 1 "TLV320AIC3206" H 4700 4450 50  0000 C CNN
 F 2 "Package_DFN_QFN:UQFN-40-1EP_5x5mm_P0.4mm_EP3.8x3.8mm_ThermalVias" H 5250 4800 50  0001 C CNN
@@
 $EndComp
 $Comp
-L Device:C_Small C?
-U 1 1 5CE6F309
+L Device:C_Small C113
+U 1 1 5DAC04C7
 P 5200 2150
-F 0 "C?" V 4950 2150 50  0000 C CNN
+F 0 "C113" V 4950 2150 50  0000 C CNN
 F 1 "2.2uF X7R" V 5050 2150 50  0000 C CNN
 F 2 "Capacitor_SMD:C_0603_1608Metric" H 5200 2150 50  0001 C CNN
@@
 	5300 2250 5300 2150
 $Comp
-L Device:C_Small C?
-U 1 1 5CE6F311
+L Device:C_Small C130
+U 1 1 5DAC04CF
 P 6050 4250
-F 0 "C?" V 5800 4250 50  0000 C CNN
+F 0 "C130" V 5800 4250 50  0000 C CNN
 F 1 "2.2uF X7R" V 5900 4250 50  0000 C CNN
 F 2 "Capacitor_SMD:C_0603_1608Metric" H 6050 4250 50  0001 C CNN
@@
 	6050 4100 6050 4150
 $Comp
-L power:GND #PWR?
-U 1 1 5CE6F323
+L power:GND #PWR082
+U 1 1 5DAC04E7
 P 5750 4750
-F 0 "#PWR?" H 5750 4500 50  0001 C CNN
+F 0 "#PWR082" H 5750 4500 50  0001 C CNN
 F 1 "GND" H 5750 4600 50  0000 C CNN
 F 2 "" H 5750 4750 50  0001 C CNN
@@
 	5450 4650 5750 4650
 $Comp
-L Device:C_Small C?
-U 1 1 5CE6F329
+L Device:C_Small C129
+U 1 1 5DAC04F0
 P 4400 4250
-F 0 "C?" H 4500 4200 50  0000 L CNN
+F 0 "C129" H 4500 4200 50  0000 L CNN
 F 1 "1uF" H 4500 4250 50  0000 L CNN
 F 2 "Capacitor_SMD:C_0603_1608Metric" H 4400 4250 50  0001 C CNN
@@
 Connection ~ 4950 4650
 $Comp
-L Device:C_Small C?
-U 1 1 5CE6F348
+L Device:C_Small C121
+U 1 1 5DAC0504
 P 3950 3050
-F 0 "C?" H 4050 3000 50  0000 L CNN
+F 0 "C121" H 4050 3000 50  0000 L CNN
 F 1 "100nF" H 4050 3050 50  0000 L CNN
 F 2 "Capacitor_SMD:C_0603_1608Metric" H 3950 3050 50  0001 C CNN
@@
 $EndComp
 $Comp
-L Device:C_Small C?
-U 1 1 5CE6F363
+L Device:C_Small C122
+U 1 1 5DAC0508
 P 4150 3050
-F 0 "C?" H 4050 3000 50  0000 R CNN
+F 0 "C122" H 4050 3000 50  0000 R CNN
 F 1 "100nF" H 4050 3050 50  0000 R CNN
 F 2 "Capacitor_SMD:C_0603_1608Metric" H 4150 3050 50  0001 C CNN
@@
 Connection ~ 4400 2950
 $Comp
-L power:GND #PWR?
-U 1 1 5CE6F368
+L power:GND #PWR077
+U 1 1 5DAC0524
 P 3550 3250
-F 0 "#PWR?" H 3550 3000 50  0001 C CNN
+F 0 "#PWR077" H 3550 3000 50  0001 C CNN
 F 1 "GND" H 3550 3100 50  0000 C CNN
 F 2 "" H 3550 3250 50  0001 C CNN
@@
 	8650 3300 8850 3300
 $Comp
-L SW-dallas-semi-maxim:MAX4910 U?
-U 1 1 5CE6F375
+L SW-dallas-semi-maxim:MAX4910 U22
+U 1 1 5DAC052C
 P 8300 3350
-F 0 "U?" H 8500 2800 50  0000 C CNN
+F 0 "U22" H 8500 2800 50  0000 C CNN
 F 1 "MAX4910" H 7950 3350 50  0000 C CNN
 F 2 "Package_DFN_QFN:TQFN-16-1EP_3x3mm_P0.5mm_EP1.23x1.23mm" H 9950 4500 50  0001 C CNN
@@
 	7750 3450 7750 4250
 $Comp
-L power:GND #PWR?
-U 1 1 5CE6F387
+L power:GND #PWR081
+U 1 1 5DAC053D
 P 7750 4400
-F 0 "#PWR?" H 7750 4150 50  0001 C CNN
+F 0 "#PWR081" H 7750 4150 50  0001 C CNN
 F 1 "GND" H 7750 4250 50  0000 C CNN
 F 2 "" H 7750 4400 50  0001 C CNN
@@
 	8650 3500 8850 3500
 $Comp
-L Device:Ferrite_Bead_Small FB?
-U 1 1 5CE6F39A
+L Device:Ferrite_Bead_Small FB9
+U 1 1 5DAC0549
 P 6550 4150
-F 0 "FB?" H 6625 4200 50  0000 L CNN
+F 0 "FB9" H 6625 4200 50  0000 L CNN
 F 1 "220Ω/2A" H 6625 4100 50  0000 L CNN
 F 2 "Resistor_SMD:R_0603_1608Metric" V 6480 4150 50  0001 C CNN
@@
 	3750 2600 4450 2600
 $Comp
-L Device:C_Small C?
+L Device:C_Small C118
 U 1 1 5CE6F3AC
 P 3550 2750
-F 0 "C?" H 3650 2700 50  0000 L CNN
+F 0 "C118" H 3650 2700 50  0000 L CNN
 F 1 "33pF" H 3650 2750 50  0000 L CNN
 F 2 "Capacitor_SMD:C_0603_1608Metric" H 3550 2750 50  0001 C CNN
@@
 	3200 2550 3750 2550
 $Comp
-L Device:C_Small C?
-U 1 1 5CE6F3B7
+L Device:C_Small C119
+U 1 1 5DAC0561
 P 3750 2750
-F 0 "C?" H 3650 2700 50  0000 R CNN
+F 0 "C119" H 3650 2700 50  0000 R CNN
 F 1 "33pF" H 3650 2750 50  0000 R CNN
 F 2 "Capacitor_SMD:C_0603_1608Metric" H 3750 2750 50  0001 C CNN
@@
 	5950 3000 6500 3000
 $Comp
-L SW-power:+1V8A #+1V8A?
-U 1 1 5CE6F3C8
+L SW-power:+1V8A #+1V8A08
+U 1 1 5DAC0579
 P 6750 2100
-F 0 "#+1V8A?" H 7500 1800 60  0001 C CNN
+F 0 "#+1V8A08" H 7500 1800 60  0001 C CNN
 F 1 "+1V8A" H 6750 2300 50  0000 C CNN
 F 2 "" H 6750 2100 60  0001 C CNN
@@
 $EndComp
 $Comp
-L power:+1V8 #PWR?
-U 1 1 5CE6F3D1
+L power:+1V8 #PWR075
+U 1 1 5DAC0588
 P 6500 2100
-F 0 "#PWR?" H 6500 1950 50  0001 C CNN
+F 0 "#PWR075" H 6500 1950 50  0001 C CNN
 F 1 "+1V8" H 6500 2240 50  0000 C CNN
 F 2 "" H 6500 2100 50  0001 C CNN
@@
 	6750 2800 6750 2900
 $Comp
-L power:+3V3 #PWR?
-U 1 1 5CE6F3E5
+L power:+3V3 #PWR074
+U 1 1 5DAC0590
 P 6250 2100
-F 0 "#PWR?" H 6250 1950 50  0001 C CNN
+F 0 "#PWR074" H 6250 1950 50  0001 C CNN
 F 1 "+3V3" H 6250 2240 50  0000 C CNN
 F 2 "" H 6250 2100 50  0001 C CNN
@@
 	6250 2600 6250 2350
 $Comp
-L Device:C_Small C?
-U 1 1 5CE6F3F4
+L Device:C_Small C124
+U 1 1 5DAC05AB
 P 6750 3200
-F 0 "C?" H 6850 3100 50  0000 R CNN
+F 0 "C124" H 6850 3100 50  0000 R CNN
 F 1 "1uF" H 6900 3300 50  0000 R CNN
 F 2 "Capacitor_SMD:C_0603_1608Metric" H 6750 3200 50  0001 C CNN
@@
 $EndComp
 $Comp
-L power:GND #PWR?
+L power:GND #PWR078
 U 1 1 5CE6F403
 P 6650 3400
-F 0 "#PWR?" H 6650 3150 50  0001 C CNN
+F 0 "#PWR078" H 6650 3150 50  0001 C CNN
 F 1 "GND" H 6650 3250 50  0000 C CNN
 F 2 "" H 6650 3400 50  0001 C CNN
@@
 $EndComp
 $Comp
-L Device:C_Small C?
-U 1 1 5CE6F40F
+L Device:C_Small C125
+U 1 1 5DAC05C4
 P 6900 3200
-F 0 "C?" H 6800 3150 50  0000 R CNN
+F 0 "C125" H 6800 3150 50  0000 R CNN
 F 1 "10uF" H 6800 3200 50  0000 R CNN
 F 2 "Capacitor_SMD:C_1206_3216Metric" H 6900 3200 50  0001 C CNN
@@
 $EndComp
 $Comp
-L Device:C_Small C?
-U 1 1 5CE6F425
+L Device:C_Small C123
+U 1 1 5DAC05CE
 P 6500 3200
-F 0 "C?" H 6650 3100 50  0000 R CNN
+F 0 "C123" H 6650 3100 50  0000 R CNN
 F 1 "100nF" V 6600 3400 50  0000 R CNN
 F 2 "Capacitor_SMD:C_0603_1608Metric" H 6500 3200 50  0001 C CNN
@@
 	6650 3350 6750 3350
 $Comp
-L Device:C_Small C?
-U 1 1 5CE6F42F
+L Device:C_Small C114
+U 1 1 5DAC05E2
 P 7050 2150
-F 0 "C?" H 7200 2050 50  0000 R CNN
+F 0 "C114" H 7200 2050 50  0000 R CNN
 F 1 "100nF" V 7150 2350 50  0000 R CNN
 F 2 "Capacitor_SMD:C_0603_1608Metric" H 7050 2150 50  0001 C CNN
@@
 $EndComp
 $Comp
-L Device:C_Small C?
-U 1 1 5CE6F439
+L Device:C_Small C115
+U 1 1 5DAC05EF
 P 7050 2350
-F 0 "C?" H 6950 2450 50  0000 C CNN
+F 0 "C115" H 6950 2450 50  0000 C CNN
 F 1 "10uF" V 6950 2300 50  0000 C CNN
 F 2 "Capacitor_SMD:C_1206_3216Metric" H 7050 2350 50  0001 C CNN
@@
 	6250 2150 6250 2100
 $Comp
-L Device:C_Small C?
-U 1 1 5CE6F451
+L Device:C_Small C116
+U 1 1 5DAC05FE
 P 7050 2550
-F 0 "C?" H 7200 2450 50  0000 R CNN
+F 0 "C116" H 7200 2450 50  0000 R CNN
 F 1 "100nF" V 7150 2750 50  0000 R CNN
 F 2 "Capacitor_SMD:C_0603_1608Metric" H 7050 2550 50  0001 C CNN
@@
 	6500 2550 6500 2500
 $Comp
-L Device:C_Small C?
-U 1 1 5CE6F456
+L Device:C_Small C120
+U 1 1 5DAC0614
 P 7050 2750
-F 0 "C?" H 7200 2650 50  0000 R CNN
+F 0 "C120" H 7200 2650 50  0000 R CNN
 F 1 "100nF" V 7150 2950 50  0000 R CNN
 F 2 "Capacitor_SMD:C_0603_1608Metric" H 7050 2750 50  0001 C CNN
@@
 NoConn ~ 8650 3750
 $Comp
-L Device:C_Small C?
-U 1 1 5CE6F46F
+L Device:C_Small C117
+U 1 1 5DAC0616
 P 8000 2600
-F 0 "C?" H 8150 2500 50  0000 R CNN
+F 0 "C117" H 8150 2500 50  0000 R CNN
 F 1 "100nF" V 8100 2800 50  0000 R CNN
 F 2 "Capacitor_SMD:C_0603_1608Metric" H 8000 2600 50  0001 C CNN
@@
 $EndComp
 $Comp
-L power:+3V3 #PWR?
-U 1 1 5CE6F47E
+L power:+3V3 #PWR076
+U 1 1 5DAC0632
 P 8300 2350
-F 0 "#PWR?" H 8300 2200 50  0001 C CNN
+F 0 "#PWR076" H 8300 2200 50  0001 C CNN
 F 1 "+3V3" H 8300 2490 50  0000 C CNN
 F 2 "" H 8300 2350 50  0001 C CNN
@@
 	8250 4250 8350 4250
 $Comp
-L Interface_Expansion:P82B96 U?
-U 1 1 5CE6F489
+L Interface_Expansion:P82B96 U24
+U 1 1 5DAC0636
 P 2600 4300
-F 0 "U?" H 2100 4800 50  0000 L CNN
+F 0 "U24" H 2100 4800 50  0000 L CNN
 F 1 "P82B96" H 2800 4800 50  0000 L CNN
 F 2 "Package_SO:TSSOP-8_3x3mm_P0.65mm" H 2600 4300 50  0001 C CNN
@@
 $EndComp
 $Comp
-L power:+12V #PWR?
-U 1 1 5CE6F490
+L power:+12V #PWR079
+U 1 1 5DAC0648
 P 1550 3550
-F 0 "#PWR?" H 1550 3400 50  0001 C CNN
+F 0 "#PWR079" H 1550 3400 50  0001 C CNN
 F 1 "+12V" H 1550 3690 50  0000 C CNN
 F 2 "" H 1550 3550 50  0001 C CNN
@@
 	1900 4100 1900 4200
 $Comp
-L Device:R_Small_US R?
-U 1 1 5CE6F4C1
+L Device:R_Small_US R27
+U 1 1 5DAC065B
 P 1700 3900
-F 0 "R?" H 1800 3950 50  0000 L CNN
+F 0 "R27" H 1800 3950 50  0000 L CNN
 F 1 "750Ω" H 1800 3900 50  0000 L CNN
 F 2 "Resistor_SMD:R_0603_1608Metric" H 1700 3900 50  0001 C CNN
@@
 $EndComp
 $Comp
-L Device:R_Small_US R?
-U 1 1 5CE6F4D0
+L Device:R_Small_US R28
+U 1 1 5DAC0667
 P 1550 4300
-F 0 "R?" H 1650 4350 50  0000 L CNN
+F 0 "R28" H 1650 4350 50  0000 L CNN
 F 1 "750Ω" H 1650 4300 50  0000 L CNN
 F 2 "Resistor_SMD:R_0603_1608Metric" H 1550 4300 50  0001 C CNN
@@
 	1700 4100 1900 4100
 $Comp
-L power:+12V #PWR?
-U 1 1 5CE6F4E1
+L power:+12V #PWR080
+U 1 1 5DAC0674
 P 3250 3750
-F 0 "#PWR?" H 3250 3600 50  0001 C CNN
+F 0 "#PWR080" H 3250 3600 50  0001 C CNN
 F 1 "+12V" H 3250 3890 50  0000 C CNN
 F 2 "" H 3250 3750 50  0001 C CNN
@@
 	3200 4400 3400 4400
 $Comp
-L Device:C_Small C?
-U 1 1 5CE6F4F3
+L Device:C_Small C128
+U 1 1 5DAC068A
 P 3700 4000
-F 0 "C?" V 3550 4000 50  0000 C CNN
+F 0 "C128" V 3550 4000 50  0000 C CNN
 F 1 "100nF" V 3450 4000 50  0000 C CNN
 F 2 "Capacitor_SMD:C_0603_1608Metric" H 3700 4000 50  0001 C CNN
@@
 	1450 4500 1550 4500
 $Comp
-L Device:C_Small C?
+L Device:C_Small C126
 U 1 1 5CE6F2C0
 P 6150 3600
-F 0 "C?" V 6300 3600 50  0000 C CNN
+F 0 "C126" V 6300 3600 50  0000 C CNN
 F 1 "1uF" V 6400 3600 50  0000 C CNN
 F 2 "Capacitor_SMD:C_0805_2012Metric" H 6150 3600 50  0001 C CNN
@@
 $EndComp
 $Comp
-L Device:C_Small C?
-U 1 1 5CE6F2D4
+L Device:C_Small C127
+U 1 1 5DAC049E
 P 6400 3700
-F 0 "C?" V 6550 3700 50  0000 C CNN
+F 0 "C127" V 6550 3700 50  0000 C CNN
 F 1 "1uF" V 6650 3700 50  0000 C CNN
 F 2 "Capacitor_SMD:C_0805_2012Metric" H 6400 3700 50  0001 C CNN

Commit message: assigned more footprints
Parts:
- C115, C125: value 10uF -> 10uF X7R
- C124, C129: value 1uF -> 1uF X7R
- C126, C127: value 1uF -> 1uF X7R flex
Changed lines of the file:
@@
 P 4400 4250
 F 0 "C129" H 4500 4200 50  0000 L CNN
-F 1 "1uF" H 4500 4250 50  0000 L CNN
+F 1 "1uF X7R" H 4500 4250 50  0000 L CNN
 F 2 "Capacitor_SMD:C_0603_1608Metric" H 4400 4250 50  0001 C CNN
 F 3 "~" H 4400 4250 50  0001 C CNN
@@
 P 6750 3200
 F 0 "C124" H 6850 3100 50  0000 R CNN
-F 1 "1uF" H 6900 3300 50  0000 R CNN
+F 1 "1uF X7R" H 6900 3300 50  0000 R CNN
 F 2 "Capacitor_SMD:C_0603_1608Metric" H 6750 3200 50  0001 C CNN
 F 3 "~" H 6750 3200 50  0001 C CNN
@@
 P 6900 3200
 F 0 "C125" H 6800 3150 50  0000 R CNN
-F 1 "10uF" H 6800 3200 50  0000 R CNN
+F 1 "10uF X7R" H 6800 3200 50  0000 R CNN
 F 2 "Capacitor_SMD:C_1206_3216Metric" H 6900 3200 50  0001 C CNN
 F 3 "~" H 6900 3200 50  0001 C CNN
@@
 P 7050 2350
 F 0 "C115" H 6950 2450 50  0000 C CNN
-F 1 "10uF" V 6950 2300 50  0000 C CNN
+F 1 "10uF X7R" V 6950 2300 50  0000 C CNN
 F 2 "Capacitor_SMD:C_1206_3216Metric" H 7050 2350 50  0001 C CNN
 F 3 "~" H 7050 2350 50  0001 C CNN
@@
 P 6150 3600
 F 0 "C126" V 6300 3600 50  0000 C CNN
-F 1 "1uF" V 6400 3600 50  0000 C CNN
+F 1 "1uF X7R flex" V 6400 3600 50  0000 C CNN
 F 2 "Capacitor_SMD:C_0805_2012Metric" H 6150 3600 50  0001 C CNN
 F 3 "~" H 6150 3600 50  0001 C CNN
@@
 P 6400 3700
 F 0 "C127" V 6550 3700 50  0000 C CNN
-F 1 "1uF" V 6650 3700 50  0000 C CNN
+F 1 "1uF X7R flex" V 6650 3700 50  0000 C CNN
 F 2 "Capacitor_SMD:C_0805_2012Metric" H 6400 3700 50  0001 C CNN
 F 3 "~" H 6400 3700 50  0001 C CNN

Commit message: re-annotating after adding power ICs and decoupling capacitors.
Also verified most footprints, and updated schematic field data.
Parts:
- C225: renamed from C128; value 100nF -> 100nF X7R
- C227: renamed from C121; value 100nF -> 100nF X7R
- C228: renamed from C122; value 100nF -> 100nF X7R
- C234: renamed from C123; value 100nF -> 100nF X7R
- C237: renamed from C114; value 100nF -> 100nF X7R
- C239: renamed from C116; value 100nF -> 100nF X7R
- C240: renamed from C120; value 100nF -> 100nF X7R
- C241: renamed from C117; value 100nF -> 100nF X7R
- R27: renamed from R28; Package ID (none) -> 0402in/1005mm
- R28: renamed from R27; Package ID (none) -> 0402in/1005mm
- renumbered C118 to C224, C119 to C226, C129 to C229, C113 to C230, C130 to C231, C126 to C232, C127 to C233, C124 to C235, C125 to C236, C115 to C238, FB9 to FB10, U24 to U27, U23 to U28, U22 to U29

Commit message: Reannotating and adding more fields to components
Parts:
- C224, C226: value 33pF -> 33pF NP0; footprint Capacitor_SMD:C_0603_1608Metric -> Capacitor_SMD:C_0402_1005Metric; Characteristics (none) -> CAP CER 33PF 25V NP0 0402; Description (none) -> MLCC Capacitor; Manufacturer (none) -> AVX; Manufacturers Part Number (none) -> 04023A330FAT2A; Package ID 0603in/1608mm -> 0402in/1005mm
- C225, C227, C228, C234, C237, C239, C240, C241: Characteristics (none) -> CAP CER 0.1UF 25V X7R 0603; Description (none) -> MLCC Capacitor; Manufacturer (none) -> Kemet; Manufacturers Part Number (none) -> C0603C104J3RACAUTO
- C229, C235: Characteristics (none) -> CAP CER 1UF 25V X7R 0603; Description (none) -> MLCC Capacitor
- C230, C231: footprint Capacitor_SMD:C_0603_1608Metric -> Capacitor_SMD:C_0805_2012Metric; Characteristics (none) -> CAP CER 2.2UF 25V X7R 0805; Description (none) -> MLCC Capacitor; Manufacturer (none) -> TDK; Manufacturers Part Number (none) -> CGA4J3X7R1E225K125AB; Package ID 0603in/1608mm -> 0805in/2012mm
- C232, C233: Characteristics (none) -> CAP CER 0805 1UF 25V X7R 5%; Description (none) -> MLCC Capacitor; Manufacturers Part Number C0805X105J3RACAUTO -> C0805X105J3RECAUTO
- C236, C238: Characteristics (none) -> CAP CER 10UF 25V X7R 1206; Description (none) -> MLCC Capacitor
- FB10: footprint Resistor_SMD:R_0603_1608Metric -> Inductor_SMD:L_0603_1608Metric; Description (none) -> Ferrite Bead
- R27, R28: Description (none) -> Resistor
- U27: Description (none) -> I2C Buffer / Voltage Translator; Manufacturer (none) -> Texas Instruments; Manufacturers Part Number (none) -> P82B96; Package ID (none) -> TSSOP8
- U28: Description (none) -> I2S Audio Codec; Manufacturer (none) -> Texas Instruments; Package ID (none) -> UQFN40
- U29: Description (none) -> Clickless Audio Switch; Manufacturer (none) -> Maxim Integrated; Package ID (none) -> TQFN16

Commit message: Fixed resistor footprint
Parts:
- R27, R28: footprint Resistor_SMD:R_0603_1608Metric -> Resistor_SMD:R_0402_1005Metric
Changed lines of the file:
@@
 F 0 "R28" H 1800 3950 50  0000 L CNN
 F 1 "750Ω" H 1800 3900 50  0000 L CNN
-F 2 "Resistor_SMD:R_0603_1608Metric" H 1700 3900 50  0001 C CNN
+F 2 "Resistor_SMD:R_0402_1005Metric" H 1700 3900 50  0001 C CNN
 F 3 "~" H 1700 3900 50  0001 C CNN
 F 4 "0402in/1005mm" H 0   0   50  0001 C CNN "Package ID"
@@
 F 0 "R27" H 1650 4350 50  0000 L CNN
 F 1 "750Ω" H 1650 4300 50  0000 L CNN
-F 2 "Resistor_SMD:R_0603_1608Metric" H 1550 4300 50  0001 C CNN
+F 2 "Resistor_SMD:R_0402_1005Metric" H 1550 4300 50  0001 C CNN
 F 3 "~" H 1550 4300 50  0001 C CNN
 F 4 "0402in/1005mm" H 0   0   50  0001 C CNN "Package ID"
