File: edc-mux-board-fpga/edc-mux-board-fpga.kicad_pcb (KiCad board)
At the start: 4 copper layers, 17 parts, among them J1 OSC_PRG_PWR, J2 OSC_PRG_I2C, J3 OSC_PRG_RST, J4 Conn_01x12, U1 10CL040YF484I7G, U2 CDCI6214, U3 CDCLVC1108, U4 CDCLVC1108, U5 TLV320AIC3206, U6 W5500, U7 SAMD21JXXAM, Y1 SiT1602BI-71-33E-48.000000

Commit message: annotated board
Parts:
- removed JP1, JP2, JP3: ~, Jumper:SolderJumper-2_P1.3mm_Open_RoundedPad1.0x1.5mm
- added C1: 100nF, Capacitor_SMD:C_0603_1608Metric, F.Cu at (140.0, 70.9)
- added C10: 100nF, Capacitor_SMD:C_0603_1608Metric, F.Cu at (65.6, 37.4)
- added C100: 1uF, SW-WIMA:2220_film_cap, F.Cu at (134.9, 156.9)
- added C101: 100nF, Capacitor_SMD:C_0603_1608Metric, F.Cu at (136.6, 151.6)
- added C102: 1uF, Capacitor_SMD:C_0603_1608Metric, F.Cu at (158.6, 178.2)
- added C103: 2.2uF X7R, Capacitor_SMD:C_0603_1608Metric, F.Cu at (156.1, 178.2)
- added C104: 2.2uF X7R, Capacitor_SMD:C_0603_1608Metric, F.Cu at (280.7, 151.7)
- added C105: 100nF, Capacitor_SMD:C_0603_1608Metric, F.Cu at (260.9, 159.0)
- added C106: 10uF, Capacitor_SMD:C_1206_3216Metric, F.Cu at (265.7, 155.3)
- added C107: 1uF, SW-WIMA:2220_film_cap, F.Cu at (259.5, 164.3)
- added C108: 1uF, SW-WIMA:2220_film_cap, F.Cu at (266.1, 164.3)
- added C109: 100nF, Capacitor_SMD:C_0603_1608Metric, F.Cu at (276.7, 143.2)
- added C11: 33pF, Capacitor_SMD:C_0603_1608Metric, F.Cu at (49.8, 53.2)
- added C110: 100nF, Capacitor_SMD:C_0603_1608Metric, F.Cu at (254.1, 162.7)
- added C111: 33pF, Capacitor_SMD:C_0603_1608Metric, F.Cu at (276.7, 140.6)
- added C112: 33pF, Capacitor_SMD:C_0603_1608Metric, F.Cu at (260.9, 156.4)
- added C113: 100nF, Capacitor_SMD:C_0603_1608Metric, F.Cu at (280.7, 138.1)
- added C114: 100nF, Capacitor_SMD:C_0603_1608Metric, F.Cu at (272.3, 146.1)
- added C115: 100nF, Capacitor_SMD:C_0603_1608Metric, F.Cu at (268.2, 152.4)
- added C116: 100nF, Capacitor_SMD:C_0603_1608Metric, F.Cu at (246.1, 167.2)
- added C117: 1uF, Capacitor_SMD:C_0603_1608Metric, F.Cu at (264.2, 152.4)
- added C118: 10uF, Capacitor_SMD:C_1206_3216Metric, F.Cu at (265.7, 158.6)
- added C119: 1uF, SW-WIMA:2220_film_cap, F.Cu at (272.8, 164.3)
- added C12: 33pF, Capacitor_SMD:C_0603_1608Metric, F.Cu at (45.8, 60.7)
- added C120: 1uF, SW-WIMA:2220_film_cap, F.Cu at (279.4, 164.3)
- added C121: 100nF, Capacitor_SMD:C_0603_1608Metric, F.Cu at (276.7, 138.1)
- added C122: 1uF, Capacitor_SMD:C_0603_1608Metric, F.Cu at (280.7, 135.6)
- added C123: 2.2uF X7R, Capacitor_SMD:C_0603_1608Metric, F.Cu at (280.7, 140.6)
- added C124: 2.2uF X7R, Capacitor_SMD:C_0603_1608Metric, F.Cu at (49.8, 168.6)
- added C125: 100nF, Capacitor_SMD:C_0603_1608Metric, F.Cu at (72.4, 146.6)
- added C126: 10uF, Capacitor_SMD:C_1206_3216Metric, F.Cu at (60.8, 154.0)
- added C127: 1uF, SW-WIMA:2220_film_cap, F.Cu at (67.1, 144.9)
- added C128: 1uF, SW-WIMA:2220_film_cap, F.Cu at (53.8, 144.9)
- added C129: 100nF, Capacitor_SMD:C_0603_1608Metric, F.Cu at (45.8, 173.6)
- added C13: 100nF, Capacitor_SMD:C_0603_1608Metric, F.Cu at (49.8, 55.7)
- added C130: 100nF, Capacitor_SMD:C_0603_1608Metric, F.Cu at (45.8, 171.1)
- added C131: 33pF, Capacitor_SMD:C_0603_1608Metric, F.Cu at (49.8, 171.1)
- added C132: 33pF, Capacitor_SMD:C_0603_1608Metric, F.Cu at (45.8, 168.6)
- added C133: 100nF, Capacitor_SMD:C_0603_1608Metric, F.Cu at (54.2, 163.2)
- added C134: 100nF, Capacitor_SMD:C_0603_1608Metric, F.Cu at (65.6, 152.8)
- added C135: 100nF, Capacitor_SMD:C_0603_1608Metric, F.Cu at (45.8, 166.1)
- added C136: 100nF, Capacitor_SMD:C_0603_1608Metric, F.Cu at (50.2, 163.2)
- added C137: 1uF, Capacitor_SMD:C_0603_1608Metric, F.Cu at (49.8, 166.1)
- added C138: 10uF, Capacitor_SMD:C_1206_3216Metric, F.Cu at (60.8, 150.7)
- added C139: 1uF, SW-WIMA:2220_film_cap, F.Cu at (60.4, 144.9)
- added C14: 100nF, Capacitor_SMD:C_0603_1608Metric, F.Cu at (65.6, 39.9)
- added C140: 1uF, SW-WIMA:2220_film_cap, F.Cu at (47.1, 144.9)
- added C141: 100nF, Capacitor_SMD:C_0603_1608Metric, F.Cu at (58.2, 163.2)
- added C142: 1uF, Capacitor_SMD:C_0603_1608Metric, F.Cu at (62.3, 156.9)
- added C143: 2.2uF X7R, Capacitor_SMD:C_0603_1608Metric, F.Cu at (80.5, 142.1)
- added C144: 2.2uF X7R, Capacitor_SMD:C_0603_1608Metric, F.Cu at (185.2, 178.2)
- added C145: 100nF, Capacitor_SMD:C_0603_1608Metric, F.Cu at (190.8, 173.8)
- added C146: 10uF, Capacitor_SMD:C_1206_3216Metric, F.Cu at (181.6, 163.2)
- added C147: 1uF, SW-WIMA:2220_film_cap, F.Cu at (172.6, 163.5)
- added C148: 1uF, SW-WIMA:2220_film_cap, F.Cu at (172.6, 156.9)
- added C149: 100nF, Capacitor_SMD:C_0603_1608Metric, F.Cu at (169.7, 143.5)
- added C15: 100nF, Capacitor_SMD:C_0603_1608Metric, F.Cu at (45.8, 58.2)
- added C150: 100nF, Capacitor_SMD:C_0603_1608Metric, F.Cu at (174.2, 151.6)
- added C151: 33pF, Capacitor_SMD:C_0603_1608Metric, F.Cu at (196.3, 178.2)
- added C152: 33pF, Capacitor_SMD:C_0603_1608Metric, F.Cu at (193.7, 178.2)
- added C153: 100nF, Capacitor_SMD:C_0603_1608Metric, F.Cu at (196.3, 174.2)
- added C154: 100nF, Capacitor_SMD:C_0603_1608Metric, F.Cu at (180.5, 158.4)
- added C155: 100nF, Capacitor_SMD:C_0603_1608Metric, F.Cu at (198.8, 178.2)
- added C156: 100nF, Capacitor_SMD:C_0603_1608Metric, F.Cu at (190.8, 169.7)
- added C157: 1uF, Capacitor_SMD:C_0603_1608Metric, F.Cu at (184.5, 165.7)
- added C158: 10uF, Capacitor_SMD:C_1206_3216Metric, F.Cu at (178.3, 163.2)
- added C159: 1uF, SW-WIMA:2220_film_cap, F.Cu at (172.6, 170.2)
- added C16: 100nF, Capacitor_SMD:C_0603_1608Metric, F.Cu at (54.2, 50.2)
- added C160: 1uF, SW-WIMA:2220_film_cap, F.Cu at (172.6, 176.8)
- added C161: 100nF, Capacitor_SMD:C_0603_1608Metric, F.Cu at (193.3, 170.1)
- added C162: 1uF, Capacitor_SMD:C_0603_1608Metric, F.Cu at (198.8, 174.2)
- added C163: 2.2uF X7R, Capacitor_SMD:C_0603_1608Metric, F.Cu at (201.3, 178.2)
- added C164: 2.2uF X7R, Capacitor_SMD:C_0603_1608Metric, F.Cu at (268.3, 108.5)
- added C165: 100nF, Capacitor_SMD:C_0603_1608Metric, F.Cu at (272.7, 106.0)
- added C166: 10uF, Capacitor_SMD:C_1206_3216Metric, F.Cu at (265.7, 120.9)
- added C167: 1uF, SW-WIMA:2220_film_cap, F.Cu at (272.8, 126.7)
- added C168: 1uF, SW-WIMA:2220_film_cap, F.Cu at (279.4, 126.7)
- added C169: 100nF, Capacitor_SMD:C_0603_1608Metric, F.Cu at (268.2, 114.7)
- added C17: 1uF, Capacitor_SMD:C_0603_1608Metric, F.Cu at (58.3, 44.0)
- added C170: 100nF, Capacitor_SMD:C_0603_1608Metric, F.Cu at (280.7, 100.5)
- added C171: 33pF, Capacitor_SMD:C_0603_1608Metric, F.Cu at (260.9, 118.8)
- added C172: 33pF, Capacitor_SMD:C_0603_1608Metric, F.Cu at (276.7, 103.0)
- added C173: 100nF, Capacitor_SMD:C_0603_1608Metric, F.Cu at (254.1, 125.0)
- added C174: 100nF, Capacitor_SMD:C_0603_1608Metric, F.Cu at (280.7, 114.1)
- added C175: 100nF, Capacitor_SMD:C_0603_1608Metric, F.Cu at (280.7, 103.0)
- added C176: 100nF, Capacitor_SMD:C_0603_1608Metric, F.Cu at (280.7, 105.5)
- added C177: 1uF, Capacitor_SMD:C_0603_1608Metric, F.Cu at (276.3, 108.5)
- added C178: 10uF, Capacitor_SMD:C_1206_3216Metric, F.Cu at (265.7, 117.6)
- added C179: 1uF, SW-WIMA:2220_film_cap, F.Cu at (259.5, 126.7)
- added C18: 10uF, Capacitor_SMD:C_1206_3216Metric, F.Cu at (60.8, 41.1)
- added C180: 1uF, SW-WIMA:2220_film_cap, F.Cu at (266.1, 126.7)
- added C181: 100nF, Capacitor_SMD:C_0603_1608Metric, F.Cu at (260.9, 121.3)
- added C182: 1uF, Capacitor_SMD:C_0603_1608Metric, F.Cu at (276.7, 105.5)
- added C183: 2.2uF X7R, Capacitor_SMD:C_0603_1608Metric, F.Cu at (246.1, 129.6)
- added C184: 2.2uF X7R, Capacitor_SMD:C_0603_1608Metric, F.Cu at (237.1, 35.9)
- added C185: 100nF, Capacitor_SMD:C_0603_1608Metric, F.Cu at (222.2, 13.8)
- added C186: 10uF, Capacitor_SMD:C_1206_3216Metric, F.Cu at (228.4, 16.3)
- added C187: 1uF, SW-WIMA:2220_film_cap, F.Cu at (234.2, 2.59)
- added C188: 1uF, SW-WIMA:2220_film_cap, F.Cu at (234.2, 9.24)
- added C189: 100nF, Capacitor_SMD:C_0603_1608Metric, F.Cu at (208.0, 1.27)
- added C19: 1uF, SW-WIMA:2220_film_cap, F.Cu at (53.8, 32.0)
- added C190: 100nF, Capacitor_SMD:C_0603_1608Metric, F.Cu at (226.3, 21.1)
- added C191: 33pF, Capacitor_SMD:C_0603_1608Metric, F.Cu at (210.5, 5.28)
- added C192: 33pF, Capacitor_SMD:C_0603_1608Metric, F.Cu at (232.5, 27.9)
- added C193: 100nF, Capacitor_SMD:C_0603_1608Metric, F.Cu at (228.8, 21.1)
- added C194: 100nF, Capacitor_SMD:C_0603_1608Metric, F.Cu at (221.6, 1.27)
- added C195: 100nF, Capacitor_SMD:C_0603_1608Metric, F.Cu at (205.5, 1.27)
- added C196: 100nF, Capacitor_SMD:C_0603_1608Metric, F.Cu at (210.5, 1.27)
- added C197: 1uF, Capacitor_SMD:C_0603_1608Metric, F.Cu at (213.0, 1.27)
- added C198: 10uF, Capacitor_SMD:C_1206_3216Metric, F.Cu at (225.1, 16.3)
- added C199: 1uF, SW-WIMA:2220_film_cap, F.Cu at (234.2, 15.9)
- added C2: 100nF, Capacitor_SMD:C_0603_1608Metric, F.Cu at (144.5, 65.7)
- added C20: 1uF, SW-WIMA:2220_film_cap, F.Cu at (47.1, 32.0)
- added C200: 1uF, SW-WIMA:2220_film_cap, F.Cu at (234.2, 22.5)
- added C201: 100nF, Capacitor_SMD:C_0603_1608Metric, F.Cu at (208.0, 5.28)
- added C202: 1uF, Capacitor_SMD:C_0603_1608Metric, F.Cu at (216.0, 5.68)
- added C203: 2.2uF X7R, Capacitor_SMD:C_0603_1608Metric, F.Cu at (213.4, 9.29)
- added C204: 2.2uF X7R, Capacitor_SMD:C_0603_1608Metric, F.Cu at (236.4, 174.2)
- added C205: 100nF, Capacitor_SMD:C_0603_1608Metric, F.Cu at (207.3, 143.5)
- added C206: 10uF, Capacitor_SMD:C_1206_3216Metric, F.Cu at (216.0, 163.2)
- added C207: 1uF, SW-WIMA:2220_film_cap, F.Cu at (210.2, 156.9)
- added C208: 1uF, SW-WIMA:2220_film_cap, F.Cu at (210.2, 170.2)
- added C209: 100nF, Capacitor_SMD:C_0603_1608Metric, F.Cu at (230.9, 170.1)
- added C21: 100nF, Capacitor_SMD:C_0603_1608Metric, F.Cu at (80.5, 29.1)
- added C210: 100nF, Capacitor_SMD:C_0603_1608Metric, F.Cu at (228.4, 165.7)
- added C211: 33pF, Capacitor_SMD:C_0603_1608Metric, F.Cu at (222.2, 161.7)
- added C212: 33pF, Capacitor_SMD:C_0603_1608Metric, F.Cu at (222.2, 165.7)
- added C213: 100nF, Capacitor_SMD:C_0603_1608Metric, F.Cu at (228.4, 169.7)
- added C214: 100nF, Capacitor_SMD:C_0603_1608Metric, F.Cu at (236.4, 178.2)
- added C215: 100nF, Capacitor_SMD:C_0603_1608Metric, F.Cu at (233.9, 174.2)
- added C216: 100nF, Capacitor_SMD:C_0603_1608Metric, F.Cu at (211.9, 151.6)
- added C217: 1uF, Capacitor_SMD:C_0603_1608Metric, F.Cu at (238.9, 178.2)
- added C218: 10uF, Capacitor_SMD:C_1206_3216Metric, F.Cu at (219.3, 163.2)
- added C219: 1uF, SW-WIMA:2220_film_cap, F.Cu at (210.2, 163.5)
- added C22: 1uF, Capacitor_SMD:C_0603_1608Metric, F.Cu at (62.3, 44.0)
- added C220: 1uF, SW-WIMA:2220_film_cap, F.Cu at (210.2, 176.8)
- added C221: 100nF, Capacitor_SMD:C_0603_1608Metric, F.Cu at (215.6, 158.4)
- added C222: 1uF, Capacitor_SMD:C_0603_1608Metric, F.Cu at (222.8, 178.2)
- added C223: 2.2uF X7R, Capacitor_SMD:C_0603_1608Metric, F.Cu at (233.9, 178.2)
- added C224: 2.2uF X7R, Capacitor_SMD:C_0603_1608Metric, F.Cu at (254.1, 87.4)
- added C225: 100nF, Capacitor_SMD:C_0603_1608Metric, F.Cu at (280.7, 76.4)
- added C226: 10uF, Capacitor_SMD:C_1206_3216Metric, F.Cu at (265.7, 83.3)
- added C227: 1uF, SW-WIMA:2220_film_cap, F.Cu at (266.1, 89.1)
- added C228: 1uF, SW-WIMA:2220_film_cap, F.Cu at (259.5, 89.1)
- added C229: 100nF, Capacitor_SMD:C_0603_1608Metric, F.Cu at (280.7, 65.4)
- added C23: 2.2uF X7R, Capacitor_SMD:C_0603_1608Metric, F.Cu at (49.8, 58.2)
- added C230: 100nF, Capacitor_SMD:C_0603_1608Metric, F.Cu at (268.2, 77.1)
- added C231: 33pF, Capacitor_SMD:C_0603_1608Metric, F.Cu at (276.3, 70.8)
- added C232: 33pF, Capacitor_SMD:C_0603_1608Metric, F.Cu at (246.1, 91.9)
- added C233: 100nF, Capacitor_SMD:C_0603_1608Metric, F.Cu at (264.2, 77.1)
- added C234: 100nF, Capacitor_SMD:C_0603_1608Metric, F.Cu at (268.3, 70.8)
- added C235: 100nF, Capacitor_SMD:C_0603_1608Metric, F.Cu at (272.7, 68.3)
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Connections:
- J1 pad 1: Net-(J1-Pad1) -> /Clocking/+3V3C
- J1 pad 2: GND -> Net-(J1-Pad2)
- J2 pad 1: Net-(J2-Pad1) -> /FPGA Data Interconnect Overview/Interface - Connector 0/AUD_GND
- J2 pad 2: Net-(J2-Pad2) -> Net-(D2-Pad1)
- J3 pad 1: Net-(J3-Pad1) -> /FPGA Data Interconnect Overview/Interface - Connector 1/AUD_GND
- J3 pad 2: Net-(J3-Pad2) -> Net-(D8-Pad1)
- J3 pad 3: Net-(J3-Pad3) -> Net-(D9-Pad1)
- J3 pad 4: Net-(J3-Pad4) -> Net-(D10-Pad1)
- J3 pad 5: Net-(J3-Pad5) -> Net-(D11-Pad1)
- J4 pad 1: Net-(J4-Pad1) -> /FPGA Data Interconnect Overview/Interface - Connector 2/AUD_GND
- J4 pad 11: Net-(J4-Pad11) -> /FPGA Data Interconnect Overview/Interface - Connector 2/ID_PIN
- J4 pad 6: Net-(J4-Pad6) -> GND
- J4 pad 7: Net-(J4-Pad7) -> /FPGA Data Interconnect Overview/Interface - Connector 2/SDA_HV
- J4 pad 8: Net-(J4-Pad8) -> /FPGA Data Interconnect Overview/Interface - Connector 2/SCL_HV
- R1 pad 1: Net-(J1-Pad1) -> /Clocking/+3V3C
- R1 pad 2: Net-(J2-Pad2) -> Net-(J1-Pad3)
- R2 pad 1: Net-(J1-Pad1) -> /Clocking/+3V3C
- R2 pad 2: Net-(J2-Pad1) -> Net-(J1-Pad2)
- U2 pad 10: Net-(U2-Pad10) -> Net-(J1-Pad2)
- U2 pad 11: Net-(J3-Pad3) -> Net-(R4-Pad2)
- U2 pad 12: Net-(J2-Pad1) -> Net-(R5-Pad2)
- U2 pad 13: Net-(U2-Pad13) -> GND
- U2 pad 14: Net-(U2-Pad14) -> /Clocking/+3V3C
- U2 pad 15: +3V3 -> Net-(R7-Pad2)
- U2 pad 16: +3V3 -> Net-(R8-Pad2)
- U2 pad 17: Net-(U2-Pad17) -> GND
- U2 pad 18: Net-(U2-Pad18) -> /Clocking/+3V3C
- U2 pad 19: Net-(J2-Pad2) -> Net-(R9-Pad2)
- U2 pad 20: Net-(J3-Pad4) -> Net-(R12-Pad2)
- U2 pad 3: Net-(J1-Pad1) -> /Clocking/+3V3C
- U2 pad 4: Net-(J3-Pad2) -> GND
- U2 pad 7: Net-(U2-Pad7) -> /Clocking/+3V3C
- U2 pad 8: Net-(J3-Pad5) -> GND
- U2 pad 9: Net-(U2-Pad9) -> Net-(J1-Pad3)
- U6 pad 15: Net-(U6-Pad11) -> Net-(U6-Pad15)
- U6 pad 16: Net-(U6-Pad14) -> Net-(U6-Pad16)
- U6 pad 17: Net-(U6-Pad11) -> Net-(U6-Pad17)
- U6 pad 19: Net-(U6-Pad14) -> Net-(U6-Pad19)
- U6 pad 21: Net-(U6-Pad11) -> Net-(U6-Pad21)
- U6 pad 3: Net-(U6-Pad14) -> Net-(U6-Pad3)
- U6 pad 4: Net-(U6-Pad11) -> Net-(U6-Pad4)
- U6 pad 8: Net-(U6-Pad11) -> Net-(U6-Pad8)
- U6 pad 9: Net-(U6-Pad14) -> Net-(U6-Pad9)
- U7 pad 10: Net-(U7-Pad10) -> /FPGA Data Interconnect Overview/Interface - Connector 0/HP_~LINE~_SEL
- U7 pad 14: Net-(U7-Pad14) -> +3V3
- U7 pad 16: Net-(U7-Pad16) -> /FPGA Data Interconnect Overview/Interface - Connector 0/L_OUT
- U7 pad 17: Net-(U7-Pad17) -> GND
- U7 pad 2: Net-(U7-Pad2) -> /FPGA Data Interconnect Overview/Interface - Connector 0/HP_~LINE~_SEL
- U7 pad 4: Net-(U7-Pad4) -> /FPGA Data Interconnect Overview/Interface - Connector 0/AUD_GND
- U7 pad 5: Net-(U7-Pad5) -> GND
- U7 pad 6: Net-(U7-Pad6) -> GND
- U7 pad 8: Net-(U7-Pad8) -> /FPGA Data Interconnect Overview/Interface - Connector 0/R_OUT
- Y1 pad 2: Net-(Y1-Pad2) -> GND
- Y1 pad 4: Net-(Y1-Pad4) -> /Clocking/+3V3C

Commit message: updated board
Parts:
- J10, J11, J12, J13, J14, J15, J16, J17, J2, J3, J4, J5, J6, J7, J8, J9: footprint Connector_PinHeader_2.54mm:PinHeader_1x12_P2.54mm_Vertical -> Connector_PinHeader_1.27mm:PinHeader_2x06_P1.27mm_Vertical
Connections:
- R12 pad 1: CLK5 -> (no net)
- R4 pad 1: CLK0 -> (no net)
- R5 pad 1: CLK1 -> (no net)
- R7 pad 1: CLK2 -> (no net)
- R8 pad 1: CLK3 -> (no net)
- R9 pad 1: CLK4 -> (no net)
- U1 pad A11: Net-(U1-PadA11) -> (no net)
- U1 pad A12: Net-(U1-PadA12) -> (no net)
- U1 pad AA11: Net-(U1-PadAA11) -> (no net)
- U1 pad AA12: Net-(U1-PadAA12) -> (no net)
- U1 pad AB11: Net-(U1-PadAB11) -> (no net)
- U1 pad AB12: Net-(U1-PadAB12) -> (no net)
- U1 pad B11: Net-(U1-PadB11) -> (no net)
- U1 pad B12: Net-(U1-PadB12) -> (no net)
- U1 pad G1: Net-(U1-PadG1) -> (no net)
- U1 pad G2: Net-(U1-PadG2) -> (no net)
- U1 pad G21: Net-(U1-PadG21) -> (no net)
- U1 pad G22: Net-(U1-PadG22) -> (no net)
- U1 pad T1: Net-(U1-PadT1) -> (no net)
- U1 pad T2: Net-(U1-PadT2) -> (no net)
- U1 pad T21: Net-(U1-PadT21) -> (no net)
- U1 pad T22: Net-(U1-PadT22) -> (no net)
- U10 pad 11: Net-(U10-Pad11) -> (no net)
- U10 pad 12: Net-(U10-Pad12) -> (no net)
- U10 pad 13: Net-(U10-Pad13) -> (no net)
- U11 pad 12: /FPGA Data Interconnect Overview/Interface - Connector 1/GPI -> (no net)
- U11 pad 15: /FPGA Data Interconnect Overview/Interface - Connector 1/INT1_OUT -> (no net)
- U11 pad 23: Net-(U11-Pad23) -> (no net)
- U11 pad 3: /FPGA Data Interconnect Overview/Interface - Connector 1/~RESET -> (no net)
- U11 pad 34: Net-(U11-Pad34) -> (no net)
- U11 pad 5: /FPGA Data Interconnect Overview/Interface - Connector 1/MCLK -> (no net)
- U11 pad 6: /FPGA Data Interconnect Overview/Interface - Connector 1/BCLK -> (no net)
- U11 pad 7: /FPGA Data Interconnect Overview/Interface - Connector 1/WCLK -> (no net)
- U11 pad 8: /FPGA Data Interconnect Overview/Interface - Connector 1/DIN -> (no net)
- U11 pad 9: /FPGA Data Interconnect Overview/Interface - Connector 1/DOUT -> (no net)
- U13 pad 11: Net-(U13-Pad11) -> (no net)
- U13 pad 12: Net-(U13-Pad12) -> (no net)
- U13 pad 13: Net-(U13-Pad13) -> (no net)
- U14 pad 23: Net-(U14-Pad23) -> (no net)
- U14 pad 34: Net-(U14-Pad34) -> (no net)
- U16 pad 11: Net-(U16-Pad11) -> (no net)
- U16 pad 12: Net-(U16-Pad12) -> (no net)
- U16 pad 13: Net-(U16-Pad13) -> (no net)
- U17 pad 23: Net-(U17-Pad23) -> (no net)
- U17 pad 34: Net-(U17-Pad34) -> (no net)
- U19 pad 11: Net-(U19-Pad11) -> (no net)
- U19 pad 12: Net-(U19-Pad12) -> (no net)
- U19 pad 13: Net-(U19-Pad13) -> (no net)
- U20 pad 23: Net-(U20-Pad23) -> (no net)
- U20 pad 34: Net-(U20-Pad34) -> (no net)
- U22 pad 11: Net-(U22-Pad11) -> (no net)
- U22 pad 12: Net-(U22-Pad12) -> (no net)
- U22 pad 13: Net-(U22-Pad13) -> (no net)
- U23 pad 23: Net-(U23-Pad23) -> (no net)
- U23 pad 34: Net-(U23-Pad34) -> (no net)
- U25 pad 11: Net-(U25-Pad11) -> (no net)
- U25 pad 12: Net-(U25-Pad12) -> (no net)
- U25 pad 13: Net-(U25-Pad13) -> (no net)
- U26 pad 23: Net-(U26-Pad23) -> (no net)
- U26 pad 34: Net-(U26-Pad34) -> (no net)
- U28 pad 11: Net-(U28-Pad11) -> (no net)
- U28 pad 12: Net-(U28-Pad12) -> (no net)
- U28 pad 13: Net-(U28-Pad13) -> (no net)
- U29 pad 23: Net-(U29-Pad23) -> (no net)
- U29 pad 34: Net-(U29-Pad34) -> (no net)
- U3 pad 1: Net-(U3-Pad1) -> (no net)
- U3 pad 11: Net-(U3-Pad11) -> (no net)
- U3 pad 13: Net-(U3-Pad13) -> (no net)
- U3 pad 15: Net-(U3-Pad15) -> (no net)
- U3 pad 16: Net-(U3-Pad16) -> (no net)
- U3 pad 2: Net-(U3-Pad2) -> (no net)
- U3 pad 3: Net-(U3-Pad3) -> (no net)
- U3 pad 6: Net-(U3-Pad6) -> (no net)
- U3 pad 8: Net-(U3-Pad8) -> (no net)
- U3 pad 9: Net-(U3-Pad9) -> (no net)
- U31 pad 11: Net-(U31-Pad11) -> (no net)
- U31 pad 12: Net-(U31-Pad12) -> (no net)
- U31 pad 13: Net-(U31-Pad13) -> (no net)
- U32 pad 23: Net-(U32-Pad23) -> (no net)
- U32 pad 34: Net-(U32-Pad34) -> (no net)
- U34 pad 11: Net-(U34-Pad11) -> (no net)
- U34 pad 12: Net-(U34-Pad12) -> (no net)
- U34 pad 13: Net-(U34-Pad13) -> (no net)
- U35 pad 23: Net-(U35-Pad23) -> (no net)
- U35 pad 34: Net-(U35-Pad34) -> (no net)
- U37 pad 11: Net-(U37-Pad11) -> (no net)
- U37 pad 12: Net-(U37-Pad12) -> (no net)
- U37 pad 13: Net-(U37-Pad13) -> (no net)
- U38 pad 23: Net-(U38-Pad23) -> (no net)
- U38 pad 34: Net-(U38-Pad34) -> (no net)
- U4 pad 1: Net-(U4-Pad1) -> (no net)
- U4 pad 11: Net-(U4-Pad11) -> (no net)
- U4 pad 13: Net-(U4-Pad13) -> (no net)
- U4 pad 15: Net-(U4-Pad15) -> (no net)
- U4 pad 16: Net-(U4-Pad16) -> (no net)
- U4 pad 2: Net-(U4-Pad2) -> (no net)
- U4 pad 3: Net-(U4-Pad3) -> (no net)
- U4 pad 6: Net-(U4-Pad6) -> (no net)
- U4 pad 8: Net-(U4-Pad8) -> (no net)
- U4 pad 9: Net-(U4-Pad9) -> (no net)
- U40 pad 11: Net-(U40-Pad11) -> (no net)
- U40 pad 12: Net-(U40-Pad12) -> (no net)
- U40 pad 13: Net-(U40-Pad13) -> (no net)
- U41 pad 23: Net-(U41-Pad23) -> (no net)
- U41 pad 34: Net-(U41-Pad34) -> (no net)
- U43 pad 11: Net-(U43-Pad11) -> (no net)
- U43 pad 12: Net-(U43-Pad12) -> (no net)
- U43 pad 13: Net-(U43-Pad13) -> (no net)
- U44 pad 23: Net-(U44-Pad23) -> (no net)
- U44 pad 34: Net-(U44-Pad34) -> (no net)
- U46 pad 11: Net-(U46-Pad11) -> (no net)
- U46 pad 12: Net-(U46-Pad12) -> (no net)
- U46 pad 13: Net-(U46-Pad13) -> (no net)
- U47 pad 23: Net-(U47-Pad23) -> (no net)
- U47 pad 34: Net-(U47-Pad34) -> (no net)
- U49 pad 11: Net-(U49-Pad11) -> (no net)
- U49 pad 12: Net-(U49-Pad12) -> (no net)
- U49 pad 13: Net-(U49-Pad13) -> (no net)
- U5 pad 1: Net-(U5-Pad1) -> (no net)
- U5 pad 10: Net-(U5-Pad10) -> (no net)
- U5 pad 11: Net-(U5-Pad11) -> (no net)
- U5 pad 12: Net-(U5-Pad12) -> (no net)
- U5 pad 13: Net-(U5-Pad13) -> (no net)
- U5 pad 14: Net-(U5-Pad14) -> (no net)
- U5 pad 15: Net-(U5-Pad15) -> (no net)
- U5 pad 16: Net-(U5-Pad16) -> (no net)
- U5 pad 17: Net-(U5-Pad17) -> (no net)
- U5 pad 18: Net-(U5-Pad18) -> (no net)
- U5 pad 19: Net-(U5-Pad19) -> (no net)
- U5 pad 2: Net-(U5-Pad2) -> (no net)
- U5 pad 20: Net-(U5-Pad20) -> (no net)
- U5 pad 21: Net-(U5-Pad21) -> (no net)
- U5 pad 22: Net-(U5-Pad22) -> (no net)
- U5 pad 23: Net-(U5-Pad23) -> (no net)
- U5 pad 24: Net-(U5-Pad24) -> (no net)
- U5 pad 3: Net-(U5-Pad3) -> (no net)
- U5 pad 4: Net-(U5-Pad4) -> (no net)
- U5 pad 5: Net-(U5-Pad5) -> (no net)
- U5 pad 6: Net-(U5-Pad6) -> (no net)
- U5 pad 7: Net-(U5-Pad7) -> (no net)
- U5 pad 8: Net-(U5-Pad8) -> (no net)
- U5 pad 9: Net-(U5-Pad9) -> (no net)
- U50 pad 23: Net-(U50-Pad23) -> (no net)
- U50 pad 34: Net-(U50-Pad34) -> (no net)
- U52 pad 11: Net-(U52-Pad11) -> (no net)
- U52 pad 12: Net-(U52-Pad12) -> (no net)
- U52 pad 13: Net-(U52-Pad13) -> (no net)
- U53 pad 23: Net-(U53-Pad23) -> (no net)
- U53 pad 34: Net-(U53-Pad34) -> (no net)
- U55 pad 1: Net-(U55-Pad1) -> (no net)
- U55 pad 10: Net-(U55-Pad10) -> (no net)
- U55 pad 12: Net-(U55-Pad12) -> (no net)
- U55 pad 13: Net-(U55-Pad13) -> (no net)
- U55 pad 18: Net-(U55-Pad18) -> (no net)
- U55 pad 2: Net-(U55-Pad2) -> (no net)
- U55 pad 20: Net-(U55-Pad20) -> (no net)
- U55 pad 22: Net-(U55-Pad22) -> (no net)
- U55 pad 23: Net-(U55-Pad23) -> (no net)
- U55 pad 24: Net-(U55-Pad24) -> (no net)
- U55 pad 25: Net-(U55-Pad25) -> (no net)
- U55 pad 26: Net-(U55-Pad26) -> (no net)
- U55 pad 27: Net-(U55-Pad27) -> (no net)
- U55 pad 28: Net-(U55-Pad28) -> (no net)
- U55 pad 29: Net-(U55-Pad29) -> (no net)
- U55 pad 30: Net-(U55-Pad30) -> (no net)
- U55 pad 31: Net-(U55-Pad31) -> (no net)
- U55 pad 32: Net-(U55-Pad32) -> (no net)
- U55 pad 33: Net-(U55-Pad33) -> (no net)
- U55 pad 34: Net-(U55-Pad34) -> (no net)
- U55 pad 35: Net-(U55-Pad35) -> (no net)
- U55 pad 36: Net-(U55-Pad36) -> (no net)
- U55 pad 37: Net-(U55-Pad37) -> (no net)
- U55 pad 38: Net-(U55-Pad38) -> (no net)
- U55 pad 39: Net-(U55-Pad39) -> (no net)
- U55 pad 40: Net-(U55-Pad40) -> (no net)
- U55 pad 41: Net-(U55-Pad41) -> (no net)
- U55 pad 42: Net-(U55-Pad42) -> (no net)
- U55 pad 43: Net-(U55-Pad43) -> (no net)
- U55 pad 44: Net-(U55-Pad44) -> (no net)
- U55 pad 45: Net-(U55-Pad45) -> (no net)
- U55 pad 46: Net-(U55-Pad46) -> (no net)
- U55 pad 47: Net-(U55-Pad47) -> (no net)
- U55 pad 5: Net-(U55-Pad5) -> (no net)
- U55 pad 6: Net-(U55-Pad6) -> (no net)
- U55 pad 7: Net-(U55-Pad7) -> (no net)
- U56 pad 1: Net-(U56-Pad1) -> (no net)
- U56 pad 10: Net-(U56-Pad10) -> (no net)
- U56 pad 11: Net-(U56-Pad11) -> (no net)
- U56 pad 12: Net-(U56-Pad12) -> (no net)
- U56 pad 13: Net-(U56-Pad13) -> (no net)
- U56 pad 14: Net-(U56-Pad14) -> (no net)
- U56 pad 15: Net-(U56-Pad15) -> (no net)
- U56 pad 16: Net-(U56-Pad16) -> (no net)
- U56 pad 17: Net-(U56-Pad17) -> (no net)
- U56 pad 18: Net-(U56-Pad18) -> (no net)
- U56 pad 19: Net-(U56-Pad19) -> (no net)
- U56 pad 2: Net-(U56-Pad2) -> (no net)
- U56 pad 20: Net-(U56-Pad20) -> (no net)
- U56 pad 23: Net-(U56-Pad23) -> (no net)
- U56 pad 24: Net-(U56-Pad24) -> (no net)
- U56 pad 25: Net-(U56-Pad25) -> (no net)
- U56 pad 26: Net-(U56-Pad26) -> (no net)
- U56 pad 27: Net-(U56-Pad27) -> (no net)
- U56 pad 28: Net-(U56-Pad28) -> (no net)
- U56 pad 29: Net-(U56-Pad29) -> (no net)
- U56 pad 3: Net-(U56-Pad3) -> (no net)
- U56 pad 30: Net-(U56-Pad30) -> (no net)
- U56 pad 31: Net-(U56-Pad31) -> (no net)
- U56 pad 32: Net-(U56-Pad32) -> (no net)
- U56 pad 35: Net-(U56-Pad35) -> (no net)
- U56 pad 36: Net-(U56-Pad36) -> (no net)
- U56 pad 37: Net-(U56-Pad37) -> (no net)
- U56 pad 38: Net-(U56-Pad38) -> (no net)
- U56 pad 39: Net-(U56-Pad39) -> (no net)
- U56 pad 4: Net-(U56-Pad4) -> (no net)
- U56 pad 40: Net-(U56-Pad40) -> (no net)
- U56 pad 41: Net-(U56-Pad41) -> (no net)
- U56 pad 42: Net-(U56-Pad42) -> (no net)
- U56 pad 43: Net-(U56-Pad43) -> (no net)
- U56 pad 44: Net-(U56-Pad44) -> (no net)
- U56 pad 45: Net-(U56-Pad45) -> (no net)
- U56 pad 46: Net-(U56-Pad46) -> (no net)
- U56 pad 49: Net-(U56-Pad49) -> (no net)
- U56 pad 5: Net-(U56-Pad5) -> (no net)
- U56 pad 50: Net-(U56-Pad50) -> (no net)
- U56 pad 51: Net-(U56-Pad51) -> (no net)
- U56 pad 52: Net-(U56-Pad52) -> (no net)
- U56 pad 53: Net-(U56-Pad53) -> (no net)
- U56 pad 55: Net-(U56-Pad55) -> (no net)
- U56 pad 56: Net-(U56-Pad56) -> (no net)
- U56 pad 57: Net-(U56-Pad57) -> (no net)
- U56 pad 58: Net-(U56-Pad58) -> (no net)
- U56 pad 59: Net-(U56-Pad59) -> (no net)
- U56 pad 6: Net-(U56-Pad6) -> (no net)
- U56 pad 60: Net-(U56-Pad60) -> (no net)
- U56 pad 61: Net-(U56-Pad61) -> (no net)
- U56 pad 62: Net-(U56-Pad62) -> (no net)
- U56 pad 63: Net-(U56-Pad63) -> (no net)
- U56 pad 64: Net-(U56-Pad64) -> (no net)
- U56 pad 7: Net-(U56-Pad7) -> (no net)
- U56 pad 8: Net-(U56-Pad8) -> (no net)
- U56 pad 9: Net-(U56-Pad9) -> (no net)
- U6 pad 1: Net-(U6-Pad1) -> (no net)
- U6 pad 10: Net-(U6-Pad10) -> (no net)
- U6 pad 11: Net-(U6-Pad11) -> (no net)
- U6 pad 12: Net-(U6-Pad12) -> (no net)
- U6 pad 13: Net-(U6-Pad13) -> (no net)
- U6 pad 14: Net-(U6-Pad14) -> (no net)
- U6 pad 15: Net-(U6-Pad15) -> (no net)
- U6 pad 16: Net-(U6-Pad16) -> (no net)
- U6 pad 17: Net-(U6-Pad17) -> (no net)
- U6 pad 18: Net-(U6-Pad18) -> (no net)
- U6 pad 19: Net-(U6-Pad19) -> (no net)
- U6 pad 2: Net-(U6-Pad2) -> (no net)
- U6 pad 20: Net-(U6-Pad20) -> (no net)
- U6 pad 21: Net-(U6-Pad21) -> (no net)
- U6 pad 22: Net-(U6-Pad22) -> (no net)
- U6 pad 23: Net-(U6-Pad23) -> (no net)
- U6 pad 24: Net-(U6-Pad24) -> (no net)
- U6 pad 3: Net-(U6-Pad3) -> (no net)
- U6 pad 4: Net-(U6-Pad4) -> (no net)
- U6 pad 5: Net-(U6-Pad5) -> (no net)
- U6 pad 6: Net-(U6-Pad6) -> (no net)
- U6 pad 7: Net-(U6-Pad7) -> (no net)
- U6 pad 8: Net-(U6-Pad8) -> (no net)
- U6 pad 9: Net-(U6-Pad9) -> (no net)
- U7 pad 11: Net-(U7-Pad11) -> (no net)
- U7 pad 12: Net-(U7-Pad12) -> (no net)
- U7 pad 13: Net-(U7-Pad13) -> (no net)
- U8 pad 12: /FPGA Data Interconnect Overview/Interface - Connector 0/GPI -> (no net)
- U8 pad 15: /FPGA Data Interconnect Overview/Interface - Connector 0/INT1_OUT -> (no net)
- U8 pad 23: Net-(U8-Pad23) -> (no net)
- U8 pad 3: /FPGA Data Interconnect Overview/Interface - Connector 0/~RESET -> (no net)
- U8 pad 34: Net-(U8-Pad34) -> (no net)
- U8 pad 5: /FPGA Data Interconnect Overview/Interface - Connector 0/MCLK -> (no net)
- U8 pad 6: /FPGA Data Interconnect Overview/Interface - Connector 0/BCLK -> (no net)
- U8 pad 7: /FPGA Data Interconnect Overview/Interface - Connector 0/WCLK -> (no net)
- U8 pad 8: /FPGA Data Interconnect Overview/Interface - Connector 0/DIN -> (no net)
- U8 pad 9: /FPGA Data Interconnect Overview/Interface - Connector 0/DOUT -> (no net)

Commit message: started pcb layout for real this time
Parts:
- removed F1, F10, F11, F12, F13, F14, F15, F16, F2, F3, F4, F5, F6, F7, F8, F9: 1A, Fuse:Fuse_0603_1608Metric
- added C324: 100nF X7R, Capacitor_SMD:C_0603_1608Metric, F.Cu at (272.4, 137.8)
- added C325: 1uF X7R, Capacitor_SMD:C_0603_1608Metric, F.Cu at (283.5, 140.2)
- added C326: 10uF X7R, Capacitor_SMD:C_1206_3216Metric, F.Cu at (273.5, 129.6)
- added C327: 100nF X7R, Capacitor_SMD:C_0603_1608Metric, F.Cu at (285.9, 134.7)
- added C328: 10uF X7R, Capacitor_SMD:C_1206_3216Metric, F.Cu at (266.2, 141.5)
- added C329: 100nF X7R, Capacitor_SMD:C_0603_1608Metric, F.Cu at (276.4, 137.8)
- added C330: 100nF X7R, Capacitor_SMD:C_0603_1608Metric, F.Cu at (284.4, 137.6)
- added C331: 100nF X7R, Capacitor_SMD:C_0603_1608Metric, F.Cu at (279.5, 140.3)
- added C332: 33pF NP0, Capacitor_SMD:C_0402_1005Metric, F.Cu at (286.9, 123.2)
- added C333: 100nF X7R, Capacitor_SMD:C_0603_1608Metric, F.Cu at (272.4, 121.1)
- added C334: 33pF NP0, Capacitor_SMD:C_0402_1005Metric, F.Cu at (287.9, 120.3)
- added C335: 100nF X7R, Capacitor_SMD:C_0603_1608Metric, F.Cu at (276.4, 121.1)
- added C336: 100nF X7R, Capacitor_SMD:C_0603_1608Metric, F.Cu at (287.1, 112.6)
- added C337: 1uF X7R, Capacitor_SMD:C_0603_1608Metric, F.Cu at (280.4, 121.0)
- added C338: 2.2uF X7R, Capacitor_SMD:C_0805_2012Metric, F.Cu at (278.5, 115.7)
- added C339: 2.2uF X7R, Capacitor_SMD:C_0805_2012Metric, F.Cu at (282.9, 112.8)
- added C340: 1uF X7R flex, Capacitor_SMD:C_0805_2012Metric, F.Cu at (278.5, 112.8)
- added C341: 1uF X7R flex, Capacitor_SMD:C_0805_2012Metric, F.Cu at (271.2, 124.7)
- added C342: 100nF X7R, Capacitor_SMD:C_0603_1608Metric, F.Cu at (283.5, 123.5)
- added C343: 1uF X7R, Capacitor_SMD:C_0603_1608Metric, F.Cu at (285.9, 118.0)
- added C344: 10uF X7R, Capacitor_SMD:C_1206_3216Metric, F.Cu at (273.5, 113.0)
- added C345: 100nF X7R, Capacitor_SMD:C_0603_1608Metric, F.Cu at (284.4, 121.0)
- added C346: 10uF X7R, Capacitor_SMD:C_1206_3216Metric, F.Cu at (266.2, 124.8)
- added C347: 100nF X7R, Capacitor_SMD:C_0603_1608Metric, F.Cu at (279.5, 123.6)
- added C348: 100nF X7R, Capacitor_SMD:C_0603_1608Metric, F.Cu at (286.7, 115.5)
- added C349: 100nF X7R, Capacitor_SMD:C_0603_1608Metric, F.Cu at (281.9, 118.5)
- added C350: 33pF NP0, Capacitor_SMD:C_0402_1005Metric, F.Cu at (286.9, 106.3)
- added C351: 100nF X7R, Capacitor_SMD:C_0603_1608Metric, F.Cu at (287.1, 95.7)
- added C352: 33pF NP0, Capacitor_SMD:C_0402_1005Metric, F.Cu at (287.9, 103.4)
- added C353: 100nF X7R, Capacitor_SMD:C_0603_1608Metric, F.Cu at (280.4, 104.1)
- added C354: 100nF X7R, Capacitor_SMD:C_0603_1608Metric, F.Cu at (281.9, 101.6)
- added C355: 1uF X7R, Capacitor_SMD:C_0603_1608Metric, F.Cu at (286.7, 98.6)
- added C356: 2.2uF X7R, Capacitor_SMD:C_0805_2012Metric, F.Cu at (278.5, 98.9)
- added C357: 2.2uF X7R, Capacitor_SMD:C_0805_2012Metric, F.Cu at (282.9, 95.9)
- added C358: 1uF X7R flex, Capacitor_SMD:C_0805_2012Metric, F.Cu at (271.2, 107.8)
- added C359: 1uF X7R flex, Capacitor_SMD:C_0805_2012Metric, F.Cu at (278.5, 95.9)
- added C360: 100nF X7R, Capacitor_SMD:C_0603_1608Metric, F.Cu at (279.5, 106.7)
- added C361: 1uF X7R, Capacitor_SMD:C_0603_1608Metric, F.Cu at (284.4, 104.1)
- added C362: 10uF X7R, Capacitor_SMD:C_1206_3216Metric, F.Cu at (266.2, 108.0)
- added C363: 100nF X7R, Capacitor_SMD:C_0603_1608Metric, F.Cu at (283.5, 106.6)
- added C364: 10uF X7R, Capacitor_SMD:C_1206_3216Metric, F.Cu at (273.5, 96.1)
- added C365: 100nF X7R, Capacitor_SMD:C_0603_1608Metric, F.Cu at (276.4, 104.2)
- added C366: 100nF X7R, Capacitor_SMD:C_0603_1608Metric, F.Cu at (285.9, 101.2)
- added C367: 100nF X7R, Capacitor_SMD:C_0603_1608Metric, F.Cu at (277.9, 101.6)
- added C368: 33pF NP0, Capacitor_SMD:C_0402_1005Metric, F.Cu at (287.9, 85.1)
- added C369: 100nF X7R, Capacitor_SMD:C_0603_1608Metric, F.Cu at (280.4, 85.8)
- added C370: 33pF NP0, Capacitor_SMD:C_0402_1005Metric, F.Cu at (287.0, 88.1)
- added C371: 100nF X7R, Capacitor_SMD:C_0603_1608Metric, F.Cu at (282.0, 83.3)
- added C372: 100nF X7R, Capacitor_SMD:C_0603_1608Metric, F.Cu at (286.8, 80.4)
- added C373: 1uF X7R, Capacitor_SMD:C_0603_1608Metric, F.Cu at (279.5, 88.5)
- added C374: 2.2uF X7R, Capacitor_SMD:C_0805_2012Metric, F.Cu at (278.5, 80.6)
- added C375: 2.2uF X7R, Capacitor_SMD:C_0805_2012Metric, F.Cu at (278.5, 77.6)
- added C376: 1uF X7R flex, Capacitor_SMD:C_0805_2012Metric, F.Cu at (282.9, 77.6)
- added C377: 1uF X7R flex, Capacitor_SMD:C_0805_2012Metric, F.Cu at (271.3, 89.5)
- added C378: 100nF X7R, Capacitor_SMD:C_0603_1608Metric, F.Cu at (286.0, 82.9)
- added C379: 1uF X7R, Capacitor_SMD:C_0603_1608Metric, F.Cu at (283.5, 88.3)
- added C380: 10uF X7R, Capacitor_SMD:C_1206_3216Metric, F.Cu at (273.5, 77.8)
- added C381: 100nF X7R, Capacitor_SMD:C_0603_1608Metric, F.Cu at (272.4, 86.0)
- added C382: 10uF X7R, Capacitor_SMD:C_1206_3216Metric, F.Cu at (266.3, 89.7)
- added C383: 100nF X7R, Capacitor_SMD:C_0603_1608Metric, F.Cu at (284.5, 85.8)
- added C384: 100nF X7R, Capacitor_SMD:C_0603_1608Metric, F.Cu at (287.2, 77.4)
- added C385: 100nF X7R, Capacitor_SMD:C_0603_1608Metric, F.Cu at (275.5, 88.5)
- added C386: 33pF NP0, Capacitor_SMD:C_0402_1005Metric, F.Cu at (286.9, 70.0)
- added C387: 100nF X7R, Capacitor_SMD:C_0603_1608Metric, F.Cu at (284.4, 67.8)
- added C388: 33pF NP0, Capacitor_SMD:C_0402_1005Metric, F.Cu at (287.8, 67.1)
- added C389: 100nF X7R, Capacitor_SMD:C_0603_1608Metric, F.Cu at (279.4, 70.4)
- added C390: 100nF X7R, Capacitor_SMD:C_0603_1608Metric, F.Cu at (286.7, 62.3)
- added C391: 1uF X7R, Capacitor_SMD:C_0603_1608Metric, F.Cu at (281.9, 65.3)
- added C392: 2.2uF X7R, Capacitor_SMD:C_0805_2012Metric, F.Cu at (271.2, 71.5)
- added C393: 2.2uF X7R, Capacitor_SMD:C_0805_2012Metric, F.Cu at (278.5, 62.5)
- added C394: 1uF X7R flex, Capacitor_SMD:C_0805_2012Metric, F.Cu at (278.5, 59.6)
- added C395: 1uF X7R flex, Capacitor_SMD:C_0805_2012Metric, F.Cu at (282.9, 59.6)
- added C396: 100nF X7R, Capacitor_SMD:C_0603_1608Metric, F.Cu at (285.9, 64.8)
- added C397: 1uF X7R, Capacitor_SMD:C_0603_1608Metric, F.Cu at (282.7, 62.3)
- added C398: 10uF X7R, Capacitor_SMD:C_1206_3216Metric, F.Cu at (266.2, 71.7)
- added C399: 100nF X7R, Capacitor_SMD:C_0603_1608Metric, F.Cu at (272.4, 67.9)
- added C400: 10uF X7R, Capacitor_SMD:C_1206_3216Metric, F.Cu at (273.4, 59.8)
- added C401: 100nF X7R, Capacitor_SMD:C_0603_1608Metric, F.Cu at (275.4, 70.4)
- added C402: 100nF X7R, Capacitor_SMD:C_0603_1608Metric, F.Cu at (283.4, 70.3)
- added C403: 100nF X7R, Capacitor_SMD:C_0603_1608Metric, F.Cu at (277.9, 65.3)
- added C404: 10uF X7R, Capacitor_SMD:C_1206_3216Metric, F.Cu at (286.8, 41.8)
- added C405: 1uF X7R, Capacitor_SMD:C_0603_1608Metric, F.Cu at (294.3, 38.5)
- added C406: 100nF X7R, Capacitor_SMD:C_0603_1608Metric, F.Cu at (300.6, 32.6)
- added C407: 10uF X7R, Capacitor_SMD:C_1206_3216Metric, F.Cu at (301.4, 29.7)
- added C408: 1uF X7R, Capacitor_SMD:C_0603_1608Metric, F.Cu at (312.2, 25.5)
- added C409: 100nF X7R, Capacitor_SMD:C_0603_1608Metric, F.Cu at (306.2, 29.3)
- added C410: 1uF X7R, Capacitor_SMD:C_0603_1608Metric, F.Cu at (291.6, 41.4)
- added C411: 100nF X7R, Capacitor_SMD:C_0603_1608Metric, F.Cu at (295.6, 41.0)
- added C412: 1uF X7R, Capacitor_SMD:C_0603_1608Metric, F.Cu at (316.6, 22.5)
- added C413: 100nF X7R, Capacitor_SMD:C_0603_1608Metric, F.Cu at (298.4, 38.5)
- added C414: 1uF X7R, Capacitor_SMD:C_0603_1608Metric, F.Cu at (298.8, 35.5)
- added C415: 100nF X7R, Capacitor_SMD:C_0603_1608Metric, F.Cu at (304.6, 32.6)
- added C416: 100nF X7R, Capacitor_SMD:C_0603_1608Metric, F.Cu at (183.5, 33.1)
- added C417: 100nF X7R, Capacitor_SMD:C_0603_1608Metric, F.Cu at (179.5, 33.1)
- added C418: 100nF X7R, Capacitor_SMD:C_0603_1608Metric, F.Cu at (161.9, 50.3)
- added C419: 100nF X7R, Capacitor_SMD:C_0603_1608Metric, F.Cu at (166.3, 48.0)
- added C420: 100nF X7R, Capacitor_SMD:C_0603_1608Metric, F.Cu at (179.5, 35.6)
- added C421: 100nF X7R, Capacitor_SMD:C_0603_1608Metric, F.Cu at (173.6, 44.7)
- added C422: 10uF X7R, Capacitor_SMD:C_1206_3216Metric, F.Cu at (157.1, 47.8)
- added C423: 4.7nF X7R, Capacitor_SMD:C_0402_1005Metric, F.Cu at (185.9, 37.4)
- added C424: 10uF X7R, Capacitor_SMD:C_1206_3216Metric, F.Cu at (168.8, 45.0)
- added C425: 100nF X7R, Capacitor_SMD:C_0603_1608Metric, F.Cu at (179.5, 38.1)
- added C426: 10nF X7R, Capacitor_SMD:C_0402_1005Metric, F.Cu at (185.9, 35.4)
- added C427: 6.8nF X7R, Capacitor_SMD:C_0402_1005Metric, F.Cu at (183.0, 37.4)
- added C428: 6.8nF X7R, Capacitor_SMD:C_0402_1005Metric, F.Cu at (175.9, 46.9)
- added C429: 22nF X7R, Capacitor_SMD:C_0402_1005Metric, F.Cu at (183.0, 39.3)
- added C430: 4.7nF X7R, Capacitor_SMD:C_0402_1005Metric, F.Cu at (155.7, 50.4)
- added C431: 100nF X7R, Capacitor_SMD:C_0603_1608Metric, F.Cu at (164.8, 84.9)
- added C432: 1uF X7R flex, Capacitor_SMD:C_0805_2012Metric, F.Cu at (172.6, 232.6)
- added C433: 1uF X7R flex, Capacitor_SMD:C_0805_2012Metric, F.Cu at (168.6, 229.7)
- added C434: 1uF X7R flex, Capacitor_SMD:C_0805_2012Metric, F.Cu at (185.3, 219.5)
- added C435: 1uF X7R flex, Capacitor_SMD:C_0805_2012Metric, F.Cu at (168.2, 234.0)
- added C436: 1uF X7R flex, Capacitor_SMD:C_0805_2012Metric, F.Cu at (194.2, 207.5)
- added C437: 1uF X7R flex, Capacitor_SMD:C_0805_2012Metric, F.Cu at (185.3, 216.6)
- added C438: 10uF X7R, Capacitor_SMD:C_1206_3216Metric, F.Cu at (159.7, 241.2)
- added C439: 220nF X7R, Capacitor_SMD:C_0603_1608Metric, F.Cu at (181.6, 231.2)
- added C440: 1uF X7R flex, Capacitor_SMD:C_0805_2012Metric, F.Cu at (173.0, 229.7)
- added C441: 1uF X7R flex, Capacitor_SMD:C_0805_2012Metric, F.Cu at (194.2, 210.4)
- added C442: 1uF X7R flex, Capacitor_SMD:C_0805_2012Metric, F.Cu at (-19.1, 104.5)
- added C443: 1uF X7R flex, Capacitor_SMD:C_0805_2012Metric, F.Cu at (-28.8, 115.0)
- added C444: 1uF X7R flex, Capacitor_SMD:C_0805_2012Metric, F.Cu at (-9.30, 95.5)
- added C445: 1uF X7R flex, Capacitor_SMD:C_0805_2012Metric, F.Cu at (-0.48, 86.7)
- added C446: 1uF X7R flex, Capacitor_SMD:C_0805_2012Metric, F.Cu at (-4.89, 89.6)
- added C447: 1uF X7R flex, Capacitor_SMD:C_0805_2012Metric, F.Cu at (-33.2, 113.6)
- added C448: 1uF X7R flex, Capacitor_SMD:C_0805_2012Metric, F.Cu at (-15.4, 100.1)
- added C449: 1uF X7R flex, Capacitor_SMD:C_0805_2012Metric, F.Cu at (-9.30, 92.6)
- added C450: 1uF X7R flex, Capacitor_SMD:C_0805_2012Metric, F.Cu at (-4.89, 92.6)
- added C451: 1uF X7R flex, Capacitor_SMD:C_0805_2012Metric, F.Cu at (-28.8, 112.0)
- added C452: 1uF X7R flex, Capacitor_SMD:C_0805_2012Metric, F.Cu at (-13.7, 97.1)
- added C453: 1uF X7R flex, Capacitor_SMD:C_0805_2012Metric, F.Cu at (-33.2, 116.6)
- added C454: 1uF X7R flex, Capacitor_SMD:C_0805_2012Metric, F.Cu at (379.6, 103.8)
- added C455: 1uF X7R flex, Capacitor_SMD:C_0805_2012Metric, F.Cu at (389.4, 87.4)
- added C456: 1uF X7R flex, Capacitor_SMD:C_0805_2012Metric, F.Cu at (367.1, 112.8)
- added C457: 1uF X7R flex, Capacitor_SMD:C_0805_2012Metric, F.Cu at (376.9, 100.8)
- added C458: 1uF X7R flex, Capacitor_SMD:C_0805_2012Metric, F.Cu at (361.8, 117.3)
- added C459: 1uF X7R flex, Capacitor_SMD:C_0805_2012Metric, F.Cu at (390.1, 90.4)
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Connections:
- C1 pad 1: GND -> +3V3
- C1 pad 2: /Clocking/+3V3C -> GND
- C10 pad 1: GND -> +2V5
- C10 pad 2: +3V3 -> GND
- C100 pad 1: Net-(C100-Pad1) -> +1V2
- C100 pad 2: Net-(C100-Pad2) -> GND
- C101 pad 1: +12V -> +1V2
- C102 pad 1: GND -> +1V2
- C102 pad 2: Net-(C102-Pad2) -> GND
- C103 pad 1: GND -> +1V2
- C103 pad 2: Net-(C103-Pad2) -> GND
- C104 pad 1: Net-(C104-Pad1) -> +1V2
- C104 pad 2: Net-(C104-Pad2) -> GND
- C105 pad 1: GND -> +1V2
- C105 pad 2: +3V3 -> GND
- C106 pad 1: +3V3 -> +1V2
- C107 pad 1: Net-(C107-Pad1) -> +1V2
- C107 pad 2: Net-(C107-Pad2) -> GND
- C108 pad 1: Net-(C108-Pad1) -> +1V2
- C108 pad 2: Net-(C108-Pad2) -> GND
- C109 pad 1: GND -> +1V2
- C109 pad 2: +1V8 -> GND
- C11 pad 1: GND -> +3V3
- C11 pad 2: Net-(C11-Pad2) -> GND
- C110 pad 1: GND -> +1V2
- C110 pad 2: +3V3 -> GND
- C111 pad 1: GND -> +1V2
- C111 pad 2: Net-(C107-Pad1) -> GND
- C112 pad 2: Net-(C108-Pad1) -> /Clocking/+3V3C
- C113 pad 2: +1V8 -> /Clocking/+3V3C
- C114 pad 1: GND -> Net-(C114-Pad1)
- C114 pad 2: Net-(C114-Pad2) -> GND
- C115 pad 2: Net-(C115-Pad2) -> /Clocking/+3V3C
- C116 pad 2: +1V8A -> /CODEC interconnection sheet/L_IN0
- C117 pad 1: GND -> +12V
- C117 pad 2: +1V8A -> GND
- C118 pad 2: +1V8A -> /CODEC interconnection sheet/R_IN0
- C119 pad 1: Net-(C119-Pad1) -> GND
- C12 pad 1: GND -> +1V2
- C12 pad 2: Net-(C12-Pad2) -> GND
- C120 pad 1: Net-(C120-Pad1) -> GND
- C121 pad 1: +12V -> GND
- C121 pad 2: GND -> Net-(C121-Pad2)
- C122 pad 1: GND -> Net-(C122-Pad1)
- C125 pad 1: GND -> Net-(C125-Pad1)
- C125 pad 2: +3V3 -> Net-(C125-Pad2)
- C126 pad 1: +3V3 -> GND
- C126 pad 2: GND -> +1V8A
- C127 pad 1: Net-(C127-Pad1) -> GND
- C127 pad 2: Net-(C127-Pad2) -> +1V8A
- C128 pad 1: Net-(C128-Pad1) -> GND
- C128 pad 2: Net-(C128-Pad2) -> +1V8A
- C129 pad 2: +1V8 -> +3V3
- C13 pad 1: GND -> +2V5
- C13 pad 2: +1V8 -> GND
- C130 pad 1: GND -> +3V3
- C130 pad 2: +3V3 -> GND
- C131 pad 2: Net-(C127-Pad1) -> +1V8
- C132 pad 2: Net-(C128-Pad1) -> +1V8
- C133 pad 2: +1V8 -> +3V3
- C134 pad 2: Net-(C134-Pad2) -> /CODEC interconnection sheet/L_IN1
- C135 pad 1: GND -> +12V
- C135 pad 2: Net-(C135-Pad2) -> GND
- C136 pad 2: +1V8A -> /CODEC interconnection sheet/R_IN1
- C137 pad 2: +1V8A -> Net-(C137-Pad2)
- C138 pad 2: +1V8A -> Net-(C138-Pad2)
- C139 pad 1: Net-(C139-Pad1) -> GND
- C14 pad 1: GND -> +3V3
- C14 pad 2: Net-(C14-Pad2) -> GND
- C141 pad 1: +12V -> GND
- C141 pad 2: GND -> Net-(C141-Pad2)
- C142 pad 1: GND -> Net-(C142-Pad1)
- C143 pad 1: GND -> Net-(C143-Pad1)
- C144 pad 1: Net-(C144-Pad1) -> GND
- C144 pad 2: Net-(C144-Pad2) -> +1V8A
- C145 pad 2: +3V3 -> +1V8A
- C146 pad 1: +3V3 -> GND
- C146 pad 2: GND -> +1V8A
- C147 pad 1: Net-(C147-Pad1) -> GND
- C147 pad 2: Net-(C147-Pad2) -> +3V3
- C148 pad 1: Net-(C148-Pad1) -> +3V3
- C148 pad 2: Net-(C148-Pad2) -> GND
- C15 pad 1: GND -> +1V2
- C15 pad 2: Net-(C15-Pad2) -> GND
- C150 pad 2: +3V3 -> +1V8
- C151 pad 2: Net-(C147-Pad1) -> +3V3
- C152 pad 2: Net-(C148-Pad1) -> /CODEC interconnection sheet/L_IN2
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