File: edc-mux-board-fpga/edc-mux-board-fpga.kicad_pcb (KiCad board)
At the start: 4 copper layers, 914 parts, among them J1 OSC_PRG_HDR, J10 Power In, J11 Left Mezzanine Board Connecto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, J12 Left Mezzanine Board Connecto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, J13 Device 0, J14 Device 1, J15 Device 2, J16 Device 3, J17 Device 4, J18 Device 5, J19 Left Mezzanine Board Connecto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, J2 Ethernet, J20 Left Mezzanine Board Connecto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, J21 Device 10, J22 Device 11, J23 Device 12, J24 Device 13, J25 Device 14, J26 Device 15, J27 Left Mezzanine Board Connecto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, J28 Left Mezzanine Board Connecto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, J29 PRG/SWD, J3 Left Mezzanine Board Connecto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, J30 USB PRG, J4 Left Mezzanine Board Connecto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, J5 FPGA_JTAG, J6 Device 6, J7 Device 7, J8 Device 8, J9 Device 9, Q1 CSD22206W, Q2 CSD22206W, Q3 CSD18501Q5A, Q4 CSD22206W, Q5 CSD22206W, SW1 LED_ENABLE, SW2 Power Switch, SW3 Reset (Microprocessor), U1 R-78B12-2.0, U10 TLV320AIC3206, U11 MAX4910, U12 P82B96, U13 TLV320AIC3206, U14 MAX4910, U15 P82B96, U16 TLV320AIC3206, U17 MAX4910, U18 P82B96, U19 TLV320AIC3206, U2 R-78B3.3-2.0, U20 MAX4910, U21 P82B96, U22 TLV320AIC3206, U23 MAX4910, U24 P82B96, U25 TLV320AIC3206, U26 MAX4910, U27 P82B96, U28 TLV320AIC3206, U29 MAX4910, U3 EP5358HUI, U30 P82B96, U31 TLV320AIC3206, U32 MAX4910, U33 P82B96, U34 TLV320AIC3206, U35 MAX4910, U36 P82B96, U37 TLV320AIC3206, U38 MAX4910, U39 P82B96, U4 EP5358HUI, U40 TLV320AIC3206, U41 MAX4910, U42 P82B96, U43 TLV320AIC3206, U44 MAX4910, U45 P82B96, U46 TLV320AIC3206, U47 MAX4910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

Commit message: More work on pcb
Mostly laid out FPGA and bypass caps
laid out one codec unit.
Parts:
- removed FB1: 600Ω @ 100MHz, Inductor_SMD:L_0805_2012Metric
- C10, C100, C101, C102, C103, C104, C105, C106, C11, C12, C13, C14, C15, C16, C17, C18, C19, C20, C21, C22, C23, C24, C25, C26, C27, C28, C29, C30, C31, C32, C33, C34, C35, C36, C37, C38, C39, C40, C41, C42, C43, C44, C45, C46, C47, C48, C49, C50, C51, C53, C54, C55, C56, C57, C58, C59, C60, C61, C62, C63, C64, C65, C66, C67, C68, C69, C7, C70, C71, C72, C73, C74, C75, C76, C77, C78, C79, C8, C80, C81, C82, C83, C84, C85, C86, C87, C88, C89, C9, C90, C91, C92, C93, C95, C96, C97, C98, C99, FB2: moved to B.Cu
- R15, R16, R17, R18, R19, R20, R21, R22, R23, R24, R25, R26, R27, R28, R29, R30, R31, R32, R33, R34, R35, R36, R37, R38, R39, R40, R41, R42, R43, R44, R45, R46: footprint Resistor_SMD:R_0603_1608Metric -> Resistor_SMD:R_0402_1005Metric
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Connections:
- net Net-(C121-Pad2) renamed /CODEC interconnection sheet/Interface - Connector 0/REF
- net Net-(C123-Pad2) renamed /CODEC interconnection sheet/Interface - Connector 0/VNEG
- net Net-(C124-Pad1) renamed /CODEC interconnection sheet/Interface - Connector 0/LINE_OUT_L
- net Net-(C125-Pad1) renamed /CODEC interconnection sheet/Interface - Connector 0/LINE_OUT_R
- net Net-(FB2-Pad2) renamed /Power Supplies/VCCDPLL
- net Net-(FB4-Pad1) renamed /CODEC interconnection sheet/Interface - Connector 0/GND_SENSE
- net Net-(J1-Pad2) renamed /Clocking/SCL
- net Net-(J1-Pad3) renamed /Clocking/SDA
- net Net-(R123-Pad1) renamed /FPGA Interconnects/MISO
- net Net-(R124-Pad1) renamed /FPGA Interconnects/~STATUS
- net Net-(R126-Pad1) renamed /FPGA Interconnects/~CONFIG
- net Net-(R128-Pad1) renamed /FPGA Interconnects/CONF_DONE
- net Net-(R129-Pad1) renamed /FPGA Interconnects/CRC_ERROR
- net Net-(R130-Pad1) renamed /FPGA Interconnects/INIT_DONE
- net Net-(R2-Pad1) renamed /Clocking/CLK_IN0
- net Net-(U10-Pad31) renamed /CODEC interconnection sheet/Interface - Connector 0/HPL
- net Net-(U10-Pad33) renamed /CODEC interconnection sheet/Interface - Connector 0/HPR
- net Net-(U6-PadD1) renamed /FPGA Interconnects/MOSI
- net Net-(U6-PadE2) renamed /FPGA Interconnects/~CS
- net Net-(U6-PadK2) renamed /FPGA Interconnects/SCK
- C126 pad 2: +1V8A -> +1V8
- C127 pad 2: +1V8A -> +1V8
- C128 pad 2: +1V8A -> +1V8
- C144 pad 2: +1V8A -> +1V8
- C145 pad 2: +1V8A -> +1V8
- C146 pad 2: +1V8A -> +1V8
- C162 pad 2: +1V8A -> +1V8
- C163 pad 2: +1V8A -> +1V8
- C164 pad 2: +1V8A -> +1V8
- C180 pad 2: +1V8A -> +1V8
- C181 pad 2: +1V8A -> +1V8
- C182 pad 2: +1V8A -> +1V8
- C198 pad 2: +1V8A -> +1V8
- C199 pad 2: +1V8A -> +1V8
- C200 pad 2: +1V8A -> +1V8
- C216 pad 2: +1V8A -> +1V8
- C217 pad 2: +1V8A -> +1V8
- C218 pad 2: +1V8A -> +1V8
- C234 pad 2: +1V8A -> +1V8
- C235 pad 2: +1V8A -> +1V8
- C236 pad 2: +1V8A -> +1V8
- C252 pad 2: +1V8A -> +1V8
- C253 pad 2: +1V8A -> +1V8
- C254 pad 2: +1V8A -> +1V8
- C270 pad 2: +1V8A -> +1V8
- C271 pad 2: +1V8A -> +1V8
- C272 pad 2: +1V8A -> +1V8
- C288 pad 2: +1V8A -> +1V8
- C289 pad 2: +1V8A -> +1V8
- C290 pad 2: +1V8A -> +1V8
- C306 pad 2: +1V8A -> +1V8
- C307 pad 2: +1V8A -> +1V8
- C308 pad 2: +1V8A -> +1V8
- C324 pad 2: +1V8A -> +1V8
- C325 pad 2: +1V8A -> +1V8
- C326 pad 2: +1V8A -> +1V8
- C342 pad 2: +1V8A -> +1V8
- C343 pad 2: +1V8A -> +1V8
- C344 pad 2: +1V8A -> +1V8
- C360 pad 2: +1V8A -> +1V8
- C361 pad 2: +1V8A -> +1V8
- C362 pad 2: +1V8A -> +1V8
- C378 pad 2: +1V8A -> +1V8
- C379 pad 2: +1V8A -> +1V8
- C380 pad 2: +1V8A -> +1V8
- C396 pad 2: +1V8A -> +1V8
- C397 pad 2: +1V8A -> +1V8
- C398 pad 2: +1V8A -> +1V8
- C434 pad 1: (no net) -> /Bottom Side Daughterboard Connector Interconnects/M_L_IN8
- C437 pad 1: (no net) -> /Bottom Side Daughterboard Connector Interconnects/M_R_IN8
- C440 pad 1: (no net) -> /Bottom Side Daughterboard Connector Interconnects/M_L_IN9
- C441 pad 1: (no net) -> /Bottom Side Daughterboard Connector Interconnects/M_R_IN9
- C444 pad 1: (no net) -> /Left Side Daughterboard Connector Interconnects/M_L_IN2
- C447 pad 1: (no net) -> /Left Side Daughterboard Connector Interconnects/M_R_IN2
- C448 pad 1: (no net) -> /Left Side Daughterboard Connector Interconnects/M_L_IN3
- C449 pad 1: (no net) -> /Left Side Daughterboard Connector Interconnects/M_L_IN4
- C450 pad 1: (no net) -> /Left Side Daughterboard Connector Interconnects/M_L_IN5
- C451 pad 1: (no net) -> /Left Side Daughterboard Connector Interconnects/M_R_IN3
- C452 pad 1: (no net) -> /Left Side Daughterboard Connector Interconnects/M_R_IN4
- C453 pad 1: (no net) -> /Left Side Daughterboard Connector Interconnects/M_R_IN5
- C456 pad 1: (no net) -> /Right Side Daughterboard Connector Interconnects/M_L_IN12
- C459 pad 1: (no net) -> /Right Side Daughterboard Connector Interconnects/M_R_IN12
- C460 pad 1: (no net) -> /Right Side Daughterboard Connector Interconnects/M_L_IN13
- C461 pad 1: (no net) -> /Right Side Daughterboard Connector Interconnects/M_L_IN14
- C462 pad 1: (no net) -> /Right Side Daughterboard Connector Interconnects/M_L_IN15
- C463 pad 1: (no net) -> /Right Side Daughterboard Connector Interconnects/M_R_IN13
- C464 pad 1: (no net) -> /Right Side Daughterboard Connector Interconnects/M_R_IN14
- C465 pad 1: (no net) -> /Right Side Daughterboard Connector Interconnects/M_R_IN15
- FB31 pad 1: (no net) -> /Bottom Side Daughterboard Connector Interconnects/M_L_OUT8
- FB34 pad 1: (no net) -> /Bottom Side Daughterboard Connector Interconnects/M_R_OUT8
- FB37 pad 1: (no net) -> /Bottom Side Daughterboard Connector Interconnects/M_L_OUT9
- FB38 pad 1: (no net) -> /Bottom Side Daughterboard Connector Interconnects/M_R_OUT9
- FB47 pad 1: (no net) -> /Left Side Daughterboard Connector Interconnects/M_L_OUT2
- FB50 pad 1: (no net) -> /Left Side Daughterboard Connector Interconnects/M_R_OUT2
- FB57 pad 1: (no net) -> /Left Side Daughterboard Connector Interconnects/M_L_OUT3
- FB58 pad 1: (no net) -> /Left Side Daughterboard Connector Interconnects/M_L_OUT4
- FB59 pad 1: (no net) -> /Left Side Daughterboard Connector Interconnects/M_L_OUT5
- FB60 pad 1: (no net) -> /Left Side Daughterboard Connector Interconnects/M_R_OUT3
- FB61 pad 1: (no net) -> /Left Side Daughterboard Connector Interconnects/M_R_OUT4
- FB62 pad 1: (no net) -> /Left Side Daughterboard Connector Interconnects/M_R_OUT5
- FB71 pad 1: (no net) -> /Right Side Daughterboard Connector Interconnects/M_L_OUT12
- FB74 pad 1: (no net) -> /Right Side Daughterboard Connector Interconnects/M_R_OUT12
- FB81 pad 1: (no net) -> /Right Side Daughterboard Connector Interconnects/M_L_OUT13
- FB82 pad 1: (no net) -> /Right Side Daughterboard Connector Interconnects/M_L_OUT14
- FB83 pad 1: (no net) -> /Right Side Daughterboard Connector Interconnects/M_L_OUT15
- FB84 pad 1: (no net) -> /Right Side Daughterboard Connector Interconnects/M_R_OUT13
- FB85 pad 1: (no net) -> /Right Side Daughterboard Connector Interconnects/M_R_OUT14
- FB86 pad 1: (no net) -> /Right Side Daughterboard Connector Interconnects/M_R_OUT15
- J12 pad 19: /FPGA Interconnects/DEV_ATT7 -> /FPGA Interconnects/DEV_INT7
- J12 pad 65: /FPGA Interconnects/DEV_ATT8 -> /FPGA Interconnects/DEV_INT8
- J12 pad 7: /FPGA Interconnects/DEV_ATT6 -> /FPGA Interconnects/DEV_INT6
- J12 pad 77: /FPGA Interconnects/DEV_ATT9 -> /FPGA Interconnects/DEV_INT9
- J14 pad 7: (no net) -> /Left Side Daughterboard Connector Interconnects/M_SDA_HV1
- J15 pad 1: (no net) -> /Left Side Daughterboard Connector Interconnects/M_AUD_GND2
- J15 pad 7: (no net) -> /Left Side Daughterboard Connector Interconnects/M_SDA_HV2
- J15 pad 8: (no net) -> /Left Side Daughterboard Connector Interconnects/M_SCL_HV2
- J15 pad 9: (no net) -> /Left Side Daughterboard Connector Interconnects/M_INT_2
- J16 pad 1: (no net) -> /Left Side Daughterboard Connector Interconnects/M_AUD_GND3
- J16 pad 7: (no net) -> /Left Side Daughterboard Connector Interconnects/M_SDA_HV3
- J16 pad 8: (no net) -> /Left Side Daughterboard Connector Interconnects/M_SCL_HV3
- J16 pad 9: (no net) -> /Left Side Daughterboard Connector Interconnects/M_INT_3
- J17 pad 1: (no net) -> /Left Side Daughterboard Connector Interconnects/M_AUD_GND4
- J17 pad 7: (no net) -> /Left Side Daughterboard Connector Interconnects/M_SDA_HV4
- J17 pad 8: (no net) -> /Left Side Daughterboard Connector Interconnects/M_SCL_HV4
- J17 pad 9: (no net) -> /Left Side Daughterboard Connector Interconnects/M_INT_4
- J18 pad 1: (no net) -> /Left Side Daughterboard Connector Interconnects/M_AUD_GND5
- J18 pad 7: (no net) -> /Left Side Daughterboard Connector Interconnects/M_SDA_HV5
- J18 pad 8: (no net) -> /Left Side Daughterboard Connector Interconnects/M_SCL_HV5
- J18 pad 9: (no net) -> /Left Side Daughterboard Connector Interconnects/M_INT_5
- J20 pad 19: /FPGA Interconnects/DEV_ATT1 -> /FPGA Interconnects/DEV_INT1
- J20 pad 31: /FPGA Interconnects/DEV_ATT2 -> /FPGA Interconnects/DEV_INT2
- J20 pad 53: /FPGA Interconnects/DEV_ATT3 -> /FPGA Interconnects/DEV_INT3
- J20 pad 65: /FPGA Interconnects/DEV_ATT4 -> /FPGA Interconnects/DEV_INT4
- J20 pad 7: /FPGA Interconnects/DEV_ATT0 -> /FPGA Interconnects/DEV_INT0
- J20 pad 77: /FPGA Interconnects/DEV_ATT5 -> /FPGA Interconnects/DEV_INT5
- J22 pad 7: (no net) -> /Right Side Daughterboard Connector Interconnects/M_SDA_HV11
- J23 pad 1: (no net) -> /Right Side Daughterboard Connector Interconnects/M_AUD_GND12
- J23 pad 7: (no net) -> /Right Side Daughterboard Connector Interconnects/M_SDA_HV12
- J23 pad 8: (no net) -> /Right Side Daughterboard Connector Interconnects/M_SCL_HV12
- J23 pad 9: (no net) -> /Right Side Daughterboard Connector Interconnects/M_INT_12
- J24 pad 1: (no net) -> /Right Side Daughterboard Connector Interconnects/M_AUD_GND13
- J24 pad 7: (no net) -> /Right Side Daughterboard Connector Interconnects/M_SDA_HV13
- J24 pad 8: (no net) -> /Right Side Daughterboard Connector Interconnects/M_SCL_HV13
- J24 pad 9: (no net) -> /Right Side Daughterboard Connector Interconnects/M_INT_13
- J25 pad 1: (no net) -> /Right Side Daughterboard Connector Interconnects/M_AUD_GND14
- J25 pad 7: (no net) -> /Right Side Daughterboard Connector Interconnects/M_SDA_HV14
- J25 pad 8: (no net) -> /Right Side Daughterboard Connector Interconnects/M_SCL_HV14
- J25 pad 9: (no net) -> /Right Side Daughterboard Connector Interconnects/M_INT_14
- J26 pad 1: (no net) -> /Right Side Daughterboard Connector Interconnects/M_AUD_GND15
- J26 pad 7: (no net) -> /Right Side Daughterboard Connector Interconnects/M_SDA_HV15
- J26 pad 8: (no net) -> /Right Side Daughterboard Connector Interconnects/M_SCL_HV15
- J26 pad 9: (no net) -> /Right Side Daughterboard Connector Interconnects/M_INT_15
- J28 pad 19: /FPGA Interconnects/DEV_ATT11 -> /FPGA Interconnects/DEV_INT11
- J28 pad 31: /FPGA Interconnects/DEV_ATT12 -> /FPGA Interconnects/DEV_INT12
- J28 pad 53: /FPGA Interconnects/DEV_ATT13 -> /FPGA Interconnects/DEV_INT13
- J28 pad 65: /FPGA Interconnects/DEV_ATT14 -> /FPGA Interconnects/DEV_INT14
- J28 pad 7: /FPGA Interconnects/DEV_ATT10 -> /FPGA Interconnects/DEV_INT10
- J28 pad 77: /FPGA Interconnects/DEV_ATT15 -> /FPGA Interconnects/DEV_INT15
- J7 pad 7: (no net) -> /Bottom Side Daughterboard Connector Interconnects/M_SDA_HV7
- J8 pad 1: (no net) -> /Bottom Side Daughterboard Connector Interconnects/M_AUD_GND8
- J8 pad 7: (no net) -> /Bottom Side Daughterboard Connector Interconnects/M_SDA_HV8
- J8 pad 8: (no net) -> /Bottom Side Daughterboard Connector Interconnects/M_SCL_HV8
- J8 pad 9: (no net) -> /Bottom Side Daughterboard Connector Interconnects/M_INT_8
- J9 pad 1: (no net) -> /Bottom Side Daughterboard Connector Interconnects/M_AUD_GND9
- J9 pad 7: (no net) -> /Bottom Side Daughterboard Connector Interconnects/M_SDA_HV9
- J9 pad 8: (no net) -> /Bottom Side Daughterboard Connector Interconnects/M_SCL_HV9
- J9 pad 9: (no net) -> /Bottom Side Daughterboard Connector Interconnects/M_INT_9
- U1 pad 1: (no net) -> +12P
- U10 pad 29: +1V8A -> +1V8
- U10 pad 32: +1V8A -> +1V8
- U10 pad 39: +1V8A -> +1V8
- U10 pad 9: /CODEC interconnection sheet/DIN0 -> /CODEC interconnection sheet/DOUT0
- U13 pad 29: +1V8A -> +1V8
- U13 pad 32: +1V8A -> +1V8
- U13 pad 39: +1V8A -> +1V8
- U13 pad 9: /CODEC interconnection sheet/DIN1 -> /CODEC interconnection sheet/DOUT1
- U16 pad 29: +1V8A -> +1V8
- U16 pad 32: +1V8A -> +1V8
- U16 pad 39: +1V8A -> +1V8
- U16 pad 9: /CODEC interconnection sheet/DIN2 -> /CODEC interconnection sheet/DOUT2
- U17 pad 16: (no net) -> /CODEC interconnection sheet/L_OUT2
- U17 pad 4: (no net) -> /CODEC interconnection sheet/AUD_GND2
- U17 pad 8: (no net) -> /CODEC interconnection sheet/R_OUT2
- U19 pad 29: +1V8A -> +1V8
- U19 pad 32: +1V8A -> +1V8
- U19 pad 39: +1V8A -> +1V8
- U19 pad 9: /CODEC interconnection sheet/DIN3 -> /CODEC interconnection sheet/DOUT3
- U20 pad 16: (no net) -> /CODEC interconnection sheet/L_OUT3
- U20 pad 4: (no net) -> /CODEC interconnection sheet/AUD_GND3
- U20 pad 8: (no net) -> /CODEC interconnection sheet/R_OUT3
- U22 pad 29: +1V8A -> +1V8
- U22 pad 32: +1V8A -> +1V8
- U22 pad 39: +1V8A -> +1V8
- U22 pad 9: /CODEC interconnection sheet/DIN4 -> /CODEC interconnection sheet/DOUT4
- U23 pad 16: (no net) -> /CODEC interconnection sheet/L_OUT4
- U23 pad 4: (no net) -> /CODEC interconnection sheet/AUD_GND4
- U23 pad 8: (no net) -> /CODEC interconnection sheet/R_OUT4
- U25 pad 29: +1V8A -> +1V8
- U25 pad 32: +1V8A -> +1V8
- U25 pad 39: +1V8A -> +1V8
- U25 pad 9: /CODEC interconnection sheet/DIN5 -> /CODEC interconnection sheet/DOUT5
- U26 pad 16: (no net) -> /CODEC interconnection sheet/L_OUT5
- U26 pad 4: (no net) -> /CODEC interconnection sheet/AUD_GND5
- U26 pad 8: (no net) -> /CODEC interconnection sheet/R_OUT5
- U28 pad 29: +1V8A -> +1V8
- U28 pad 32: +1V8A -> +1V8
- U28 pad 39: +1V8A -> +1V8
- U28 pad 9: /CODEC interconnection sheet/DIN6 -> /CODEC interconnection sheet/DOUT6
- U31 pad 29: +1V8A -> +1V8
- U31 pad 32: +1V8A -> +1V8
- U31 pad 39: +1V8A -> +1V8
- U31 pad 9: /CODEC interconnection sheet/DIN7 -> /CODEC interconnection sheet/DOUT7
- U34 pad 29: +1V8A -> +1V8
- U34 pad 32: +1V8A -> +1V8
- U34 pad 39: +1V8A -> +1V8
- U34 pad 9: /CODEC interconnection sheet/DIN8 -> /CODEC interconnection sheet/DOUT8
- U35 pad 16: (no net) -> /CODEC interconnection sheet/L_OUT8
- U35 pad 4: (no net) -> /Bottom Side Daughterboard Connector Interconnects/AUD_GND8
- U35 pad 8: (no net) -> /Bottom Side Daughterboard Connector Interconnects/L_OUT8
- U37 pad 29: +1V8A -> +1V8
- U37 pad 32: +1V8A -> +1V8
- U37 pad 39: +1V8A -> +1V8
- U37 pad 9: /CODEC interconnection sheet/DIN9 -> /CODEC interconnection sheet/DOUT9
- U38 pad 16: (no net) -> /CODEC interconnection sheet/L_OUT9
- U38 pad 4: (no net) -> /Bottom Side Daughterboard Connector Interconnects/AUD_GND9
- U38 pad 8: (no net) -> /Bottom Side Daughterboard Connector Interconnects/L_OUT9
- U40 pad 29: +1V8A -> +1V8
- U40 pad 32: +1V8A -> +1V8
- U40 pad 39: +1V8A -> +1V8
- U40 pad 9: /CODEC interconnection sheet/DIN10 -> /CODEC interconnection sheet/DOUT10
- U43 pad 29: +1V8A -> +1V8
- U43 pad 32: +1V8A -> +1V8
- U43 pad 39: +1V8A -> +1V8
- U43 pad 9: /CODEC interconnection sheet/DIN11 -> /CODEC interconnection sheet/DOUT11
- U46 pad 29: +1V8A -> +1V8
- U46 pad 32: +1V8A -> +1V8
- U46 pad 39: +1V8A -> +1V8
- U46 pad 9: /CODEC interconnection sheet/DIN12 -> /CODEC interconnection sheet/DOUT12
- U47 pad 16: (no net) -> /CODEC interconnection sheet/L_OUT12
- U47 pad 4: (no net) -> /CODEC interconnection sheet/AUD_GND12
- U47 pad 8: (no net) -> /CODEC interconnection sheet/R_OUT12
- U49 pad 29: +1V8A -> +1V8
- U49 pad 32: +1V8A -> +1V8
- U49 pad 39: +1V8A -> +1V8
- U49 pad 9: /CODEC interconnection sheet/DIN13 -> /CODEC interconnection sheet/DOUT13
- U50 pad 16: (no net) -> /CODEC interconnection sheet/L_OUT13
- U50 pad 4: (no net) -> /CODEC interconnection sheet/AUD_GND13
- U50 pad 8: (no net) -> /CODEC interconnection sheet/R_OUT13
- U52 pad 29: +1V8A -> +1V8
- U52 pad 32: +1V8A -> +1V8
- U52 pad 39: +1V8A -> +1V8
- U52 pad 9: /CODEC interconnection sheet/DIN14 -> /CODEC interconnection sheet/DOUT14
- U53 pad 16: (no net) -> /CODEC interconnection sheet/L_OUT14
- U53 pad 4: (no net) -> /CODEC interconnection sheet/AUD_GND14
- U53 pad 8: (no net) -> /CODEC interconnection sheet/R_OUT14
- U55 pad 29: +1V8A -> +1V8
- U55 pad 32: +1V8A -> +1V8
- U55 pad 39: +1V8A -> +1V8
- U55 pad 9: /CODEC interconnection sheet/DIN15 -> /CODEC interconnection sheet/DOUT15
- U56 pad 16: (no net) -> /CODEC interconnection sheet/L_OUT15
- U56 pad 4: (no net) -> /CODEC interconnection sheet/AUD_GND15
- U56 pad 8: (no net) -> /CODEC interconnection sheet/R_OUT15
- U6 pad A13: /CODEC interconnection sheet/DIN11 -> /CODEC interconnection sheet/DOUT11
- U6 pad A15: /CODEC interconnection sheet/DIN10 -> /CODEC interconnection sheet/DOUT10
- U6 pad A3: /CODEC interconnection sheet/DIN15 -> /CODEC interconnection sheet/DOUT15
- U6 pad A5: /CODEC interconnection sheet/DIN14 -> /CODEC interconnection sheet/DOUT14
- U6 pad A7: /CODEC interconnection sheet/DIN13 -> /CODEC interconnection sheet/DOUT13
- U6 pad A9: /CODEC interconnection sheet/DIN12 -> /CODEC interconnection sheet/DOUT12
- U6 pad AB10: /CODEC interconnection sheet/DIN2 -> /CODEC interconnection sheet/DOUT2
- U6 pad AB13: /CODEC interconnection sheet/DIN3 -> /CODEC interconnection sheet/DOUT3
- U6 pad AB16: /CODEC interconnection sheet/DIN4 -> /CODEC interconnection sheet/DOUT4
- U6 pad AB19: /CODEC interconnection sheet/DIN5 -> /CODEC interconnection sheet/DOUT5
- U6 pad AB4: /CODEC interconnection sheet/DIN0 -> /CODEC interconnection sheet/DOUT0
- U6 pad AB8: /CODEC interconnection sheet/DIN1 -> /CODEC interconnection sheet/DOUT1
- U6 pad B22: /FPGA Interconnects/DEV_ATT9 -> /FPGA Interconnects/DEV_INT9
- U6 pad C22: /CODEC interconnection sheet/DIN9 -> /CODEC interconnection sheet/DOUT9
- U6 pad E22: /FPGA Interconnects/DEV_ATT8 -> /FPGA Interconnects/DEV_INT8
- U6 pad F10: /FPGA Interconnects/DEV_ATT12 -> /FPGA Interconnects/DEV_INT12
- U6 pad F14: /FPGA Interconnects/DEV_ATT11 -> /FPGA Interconnects/DEV_INT11
- U6 pad F15: /FPGA Interconnects/DEV_ATT10 -> /FPGA Interconnects/DEV_INT10
- U6 pad F22: /CODEC interconnection sheet/DIN8 -> /CODEC interconnection sheet/DOUT8
- U6 pad F7: /FPGA Interconnects/DEV_ATT15 -> /FPGA Interconnects/DEV_INT15
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Routing:
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- added copper zone on B.Cu, net +1V2
- added copper zone on In2.Cu, net +1V2
- added copper zone on In2.Cu, net +1V8
- added copper zone on B.Cu, net +2V5
- added copper zone on In2.Cu, net +2V5
- added copper zone on In2.Cu, net +3V3
- added copper zone on In2.Cu, net /Power Supplies/VCCDPLL
- added copper zone on In1.Cu, net GND
Other:
- net class Analog Audio added: clearance 0.127, trace_width 0.127, via_dia 0.4572, via_drill 0.254
- net class Audio MCLKS added: clearance 0.127, trace_width 0.127, via_dia 0.4572, via_drill 0.254
- net class Default: clearance 0.2 -> 0.127; trace_width 0.25 -> 0.127; via_dia 0.8 -> 0.4572; via_drill 0.4 -> 0.254
- net class Digital Audio Signals added: clearance 0.127, trace_width 0.127, via_dia 0.4572, via_drill 0.254
- net class Ethernet Signaling added: clearance 0.127, trace_width 0.127, via_dia 0.4572, via_drill 0.254
- net class I2C added: clearance 0.127, trace_width 0.127, via_dia 0.4572, via_drill 0.254
- net class I2C HV added: clearance 0.127, trace_width 0.127, via_dia 0.4572, via_drill 0.254
- net class Master Clocks added: clearance 0.127, trace_width 0.127, via_dia 0.4572, via_drill 0.254
- net class Other Audio Clocks added: clearance 0.127, trace_width 0.127, via_dia 0.4572, via_drill 0.254
- net class USB Data added: clearance 0.127, trace_width 0.127, via_dia 0.4572, via_drill 0.254
- rule pad_to_mask_clearance: 0.051 -> 0.0381
- rule solder_mask_min_width: 0.25 -> 0.1016
- rule trace_clearance: 0.2 -> 0.127
- rule trace_min: 0.2 -> 0.127
- rule via_min_drill: 0.3 -> 0.254
- rule via_min_size: 0.4 -> 0.4572

Commit message: reloading pcb
Parts:
- removed D100, D101, D102: 12V_Vrso, Diode_SMD:D_SMA
- removed FB87: 600Ω @ 100MHz, Inductor_SMD:L_0805_2012Metric
- removed JP1: LED_ENABLE, Connector_PinHeader_1.27mm:PinHeader_1x02_P1.27mm_Vertical
- removed R138: 2k2Ω, Resistor_SMD:R_0402_1005Metric
- removed R139: 330Ω, Resistor_SMD:R_0402_1005Metric
- removed R140: 470kΩ, Resistor_SMD:R_0402_1005Metric
- added FB1: 600Ω @ 100MHz, Inductor_SMD:L_0805_2012Metric, F.Cu at (116.5, 66.3)
- C431: value 100nF X7R -> 1uF X7R flex; footprint Capacitor_SMD:C_0603_1608Metric -> Capacitor_SMD:C_0805_2012Metric
- C437, C465: value 1uF X7R flex -> 10uF X7R; footprint Capacitor_SMD:C_0805_2012Metric -> Capacitor_SMD:C_1206_3216Metric
- C438: value 10uF X7R -> 220nF X7R; footprint Capacitor_SMD:C_1206_3216Metric -> Capacitor_SMD:C_0603_1608Metric
- C439: value 220nF X7R -> 1uF X7R flex; footprint Capacitor_SMD:C_0603_1608Metric -> Capacitor_SMD:C_0805_2012Metric
- C466, C470: value 10uF X7R -> 100nF X7R; footprint Capacitor_SMD:C_1206_3216Metric -> Capacitor_SMD:C_0603_1608Metric
- C467, C472: value 100nF X7R -> 1uF X7R
- C468: value 1uF X7R -> 10uF X7R; footprint Capacitor_SMD:C_0603_1608Metric -> Capacitor_SMD:C_1206_3216Metric
- C473: value 1uF X7R -> 100pF C0G; footprint Capacitor_SMD:C_0603_1608Metric -> Capacitor_SMD:C_0402_1005Metric
- C474: value 100pF C0G -> 10uF X7R; footprint Capacitor_SMD:C_0402_1005Metric -> Capacitor_SMD:C_1206_3216Metric
- C475: value 10uF X7R -> 2.2uF X7R; footprint Capacitor_SMD:C_1206_3216Metric -> Capacitor_SMD:C_0805_2012Metric
- C476: value 2.2uF X7R -> 100nF X7R; footprint Capacitor_SMD:C_0805_2012Metric -> Capacitor_SMD:C_0603_1608Metric
- D19, D20, D21, D27, D43, D44, D45, D61, D62, D63, D79, D80, D81, D97, D98, D99: value 30pF 30kV -> 12V_Vrso; footprint Diode_SMD:D_0402_1005Metric -> Diode_SMD:D_SMA
- D22, D23, D24, D30, D46, D47, D48, D64, D65, D66, D82, D83, D84: value 12V_Vrso -> 30pF 30kV; footprint Diode_SMD:D_SMA -> Diode_SMD:D_0402_1005Metric
- D4: value CONF_ERR (RED) -> 30pF 30kV; footprint LED_SMD:LED_0402_1005Metric -> Diode_SMD:D_0402_1005Metric
- D5: value CONF_STATUS (GREEN) -> 30pF 30kV; footprint LED_SMD:LED_0402_1005Metric -> Diode_SMD:D_0402_1005Metric
- D6: value CRC_ERR (YLW) -> 30pF 30kV; footprint LED_SMD:LED_0402_1005Metric -> Diode_SMD:D_0402_1005Metric
- FB19: value 220Ω/2A -> 600Ω @ 100MHz; footprint Inductor_SMD:L_0603_1608Metric -> Inductor_SMD:L_0805_2012Metric
- FB3: value 600Ω @ 100MHz -> 220Ω/2A; footprint Inductor_SMD:L_0805_2012Metric -> Inductor_SMD:L_0603_1608Metric
- J10: value Power In -> Left Mezzanine Board Connector (Daughterboard); footprint SW-Switchcraft:PCL712AS -> Connector_PinSocket_2.54mm:PinSocket_2x40_P2.54mm_Horizontal
- J11, J19, J27: value Left Mezzanine Board Connector (Daughterboard) -> Left Mezzanine Board Connector (Motherboard); footprint Connector_PinSocket_2.54mm:PinSocket_2x40_P2.54mm_Horizontal -> Connector_PinHeader_2.54mm:PinHeader_2x40_P2.54mm_Vertical
- J12: value Left Mezzanine Board Connector (Motherboard) -> Device 0; footprint Connector_PinHeader_2.54mm:PinHeader_2x40_P2.54mm_Vertical -> SW-TEConn:T4141012121-000
- J13: value Device 0 -> Device 1
- J14: value Device 1 -> Device 2
- J15: value Device 2 -> Device 3
- J16: value Device 3 -> Device 4
- J17: value Device 4 -> Device 5
- J18: value Device 5 -> Left Mezzanine Board Connector (Daughterboard); footprint SW-TEConn:T4141012121-000 -> Connector_PinSocket_2.54mm:PinSocket_2x40_P2.54mm_Horizontal
- J20: value Left Mezzanine Board Connector (Motherboard) -> Device 10; footprint Connector_PinHeader_2.54mm:PinHeader_2x40_P2.54mm_Vertical -> SW-TEConn:T4141012121-000
- J21: value Device 10 -> Device 11
- J22: value Device 11 -> Device 12
- J23: value Device 12 -> Device 13
- J24: value Device 13 -> Device 14
- J25: value Device 14 -> Device 15
- J26: value Device 15 -> Left Mezzanine Board Connector (Daughterboard); footprint SW-TEConn:T4141012121-000 -> Connector_PinSocket_2.54mm:PinSocket_2x40_P2.54mm_Horizontal
- J28: value Left Mezzanine Board Connector (Motherboard) -> PRG/SWD; footprint Connector_PinHeader_2.54mm:PinHeader_2x40_P2.54mm_Vertical -> Connector_PinHeader_2.54mm:PinHeader_2x03_P2.54mm_Vertical
- J29: value PRG/SWD -> USB PRG; footprint Connector_PinHeader_2.54mm:PinHeader_2x03_P2.54mm_Vertical -> SW-CUI-INC:UJ2-BV-1-TH
- J30: value USB PRG -> FPGA_JTAG; footprint SW-CUI-INC:UJ2-BV-1-TH -> Connector_PinHeader_1.27mm:PinHeader_2x05_P1.27mm_Vertical
- J5: value FPGA_JTAG -> Device 6; footprint Connector_PinHeader_1.27mm:PinHeader_2x05_P1.27mm_Vertical -> SW-TEConn:T4141012121-000
- J6: value Device 6 -> Device 7
- J7: value Device 7 -> Device 8
- J8: value Device 8 -> Device 9
- J9: value Device 9 -> Power In; footprint SW-TEConn:T4141012121-000 -> SW-Switchcraft:PCL712AS
- R123: value 25Ω -> 10kΩ
- R124, R134: value 200Ω -> 10kΩ
- R125: value 10kΩ -> 1kΩ
- R126: value 10kΩ -> 2k2Ω
- R127: value 1kΩ -> 330Ω
- R128: value 10kΩ -> 470kΩ; moved to B.Cu
- R129: value 10kΩ -> 25Ω
- R132: value 200Ω -> 1kΩ
- R137: value 1kΩ -> 10kΩ
- U63: value S25FL128L -> LM74610-Q1; footprint Package_SON:WSON-8-1EP_6x5mm_P1.27mm_EP3.4x4mm -> Package_SO:VSSOP-8_3.0x3.0mm_P0.65mm
- U64: value LM74610-Q1 -> TPD3S014; footprint Package_SO:VSSOP-8_3.0x3.0mm_P0.65mm -> Package_TO_SOT_SMD:SOT-23-6
- U65: value TPD3S014 -> SAMD21JXXAM; footprint Package_TO_SOT_SMD:SOT-23-6 -> Package_DFN_QFN:QFN-64-1EP_9x9mm_P0.5mm_EP4.7x4.7mm_ThermalVias
- U66: value SAMD21JXXAM -> MCP1812; footprint Package_DFN_QFN:QFN-64-1EP_9x9mm_P0.5mm_EP4.7x4.7mm_ThermalVias -> Package_TO_SOT_SMD:SOT-23
- U67: value MCP1812 -> LTC4412; footprint Package_TO_SOT_SMD:SOT-23 -> Package_TO_SOT_SMD:TSOT-23-6
- U68: value LTC4412 -> S25FL128L; footprint Package_TO_SOT_SMD:TSOT-23-6 -> Package_SON:WSON-8-1EP_6x5mm_P1.27mm_EP3.4x4mm
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Connections:
- net Net-(C139-Pad2) renamed /CODEC interconnection sheet/Interface - Connector 1/REF
- net Net-(C141-Pad2) renamed /CODEC interconnection sheet/Interface - Connector 1/VNEG
- net Net-(C142-Pad1) renamed /CODEC interconnection sheet/Interface - Connector 1/LINE_OUT_L
- net Net-(C143-Pad1) renamed /CODEC interconnection sheet/Interface - Connector 1/LINE_OUT_R
- net Net-(C157-Pad2) renamed /CODEC interconnection sheet/Interface - Connector 2/REF
- net Net-(C159-Pad2) renamed /CODEC interconnection sheet/Interface - Connector 2/VNEG
- net Net-(C160-Pad1) renamed /CODEC interconnection sheet/Interface - Connector 2/LINE_OUT_L
- net Net-(C161-Pad1) renamed /CODEC interconnection sheet/Interface - Connector 2/LINE_OUT_R
- net Net-(C175-Pad2) renamed /CODEC interconnection sheet/Interface - Connector 3/REF
- net Net-(C177-Pad2) renamed /CODEC interconnection sheet/Interface - Connector 3/VNEG
- net Net-(C178-Pad1) renamed /CODEC interconnection sheet/Interface - Connector 3/LINE_OUT_L
- net Net-(C179-Pad1) renamed /CODEC interconnection sheet/Interface - Connector 3/LINE_OUT_R
- net Net-(C193-Pad2) renamed /CODEC interconnection sheet/Interface - Connector 4/REF
- net Net-(C195-Pad2) renamed /CODEC interconnection sheet/Interface - Connector 4/VNEG
- net Net-(C196-Pad1) renamed /CODEC interconnection sheet/Interface - Connector 4/LINE_OUT_L
- net Net-(C197-Pad1) renamed /CODEC interconnection sheet/Interface - Connector 4/LINE_OUT_R
- net Net-(C211-Pad2) renamed /CODEC interconnection sheet/Interface - Connector 5/REF
- net Net-(C213-Pad2) renamed /CODEC interconnection sheet/Interface - Connector 5/VNEG
- net Net-(C214-Pad1) renamed /CODEC interconnection sheet/Interface - Connector 5/LINE_OUT_L
- net Net-(C215-Pad1) renamed /CODEC interconnection sheet/Interface - Connector 5/LINE_OUT_R
- net Net-(C229-Pad2) renamed /CODEC interconnection sheet/Interface - Connector 6/REF
- net Net-(C231-Pad2) renamed /CODEC interconnection sheet/Interface - Connector 6/VNEG
- net Net-(C232-Pad1) renamed /CODEC interconnection sheet/Interface - Connector 6/LINE_OUT_L
- net Net-(C233-Pad1) renamed /CODEC interconnection sheet/Interface - Connector 6/LINE_OUT_R
- net Net-(C247-Pad2) renamed /CODEC interconnection sheet/Interface - Connector 7/REF
- net Net-(C249-Pad2) renamed /CODEC interconnection sheet/Interface - Connector 7/VNEG
- net Net-(C250-Pad1) renamed /CODEC interconnection sheet/Interface - Connector 7/LINE_OUT_L
- net Net-(C251-Pad1) renamed /CODEC interconnection sheet/Interface - Connector 7/LINE_OUT_R
- net Net-(C265-Pad2) renamed /CODEC interconnection sheet/Interface - Connector 8/REF
- net Net-(C267-Pad2) renamed /CODEC interconnection sheet/Interface - Connector 8/VNEG
- net Net-(C268-Pad1) renamed /CODEC interconnection sheet/Interface - Connector 8/LINE_OUT_L
- net Net-(C269-Pad1) renamed /CODEC interconnection sheet/Interface - Connector 8/LINE_OUT_R
- net Net-(C283-Pad2) renamed /CODEC interconnection sheet/Interface - Connector 9/REF
- net Net-(C285-Pad2) renamed /CODEC interconnection sheet/Interface - Connector 9/VNEG
- net Net-(C286-Pad1) renamed /CODEC interconnection sheet/Interface - Connector 9/LINE_OUT_L
- net Net-(C287-Pad1) renamed /CODEC interconnection sheet/Interface - Connector 9/LINE_OUT_R
- net Net-(C301-Pad2) renamed /CODEC interconnection sheet/Interface - Connector 10/REF
- net Net-(C303-Pad2) renamed /CODEC interconnection sheet/Interface - Connector 10/VNEG
- net Net-(C304-Pad1) renamed /CODEC interconnection sheet/Interface - Connector 10/LINE_OUT_L
- net Net-(C305-Pad1) renamed /CODEC interconnection sheet/Interface - Connector 10/LINE_OUT_R
- net Net-(C319-Pad2) renamed /CODEC interconnection sheet/Interface - Connector 11/REF
- net Net-(C321-Pad2) renamed /CODEC interconnection sheet/Interface - Connector 11/VNEG
- net Net-(C322-Pad1) renamed /CODEC interconnection sheet/Interface - Connector 11/LINE_OUT_L
- net Net-(C323-Pad1) renamed /CODEC interconnection sheet/Interface - Connector 11/LINE_OUT_R
- net Net-(C337-Pad2) renamed /CODEC interconnection sheet/Interface - Connector 12/REF
- net Net-(C339-Pad2) renamed /CODEC interconnection sheet/Interface - Connector 12/VNEG
- net Net-(C340-Pad1) renamed /CODEC interconnection sheet/Interface - Connector 12/LINE_OUT_L
- net Net-(C341-Pad1) renamed /CODEC interconnection sheet/Interface - Connector 12/LINE_OUT_R
- net Net-(C355-Pad2) renamed /CODEC interconnection sheet/Interface - Connector 13/REF
- net Net-(C357-Pad2) renamed /CODEC interconnection sheet/Interface - Connector 13/VNEG
- net Net-(C358-Pad1) renamed /CODEC interconnection sheet/Interface - Connector 13/LINE_OUT_L
- net Net-(C359-Pad1) renamed /CODEC interconnection sheet/Interface - Connector 13/LINE_OUT_R
- net Net-(C373-Pad2) renamed /CODEC interconnection sheet/Interface - Connector 14/REF
- net Net-(C375-Pad2) renamed /CODEC interconnection sheet/Interface - Connector 14/VNEG
- net Net-(C376-Pad1) renamed /CODEC interconnection sheet/Interface - Connector 14/LINE_OUT_L
- net Net-(C377-Pad1) renamed /CODEC interconnection sheet/Interface - Connector 14/LINE_OUT_R
- net Net-(C391-Pad2) renamed /CODEC interconnection sheet/Interface - Connector 15/REF
- net Net-(C393-Pad2) renamed /CODEC interconnection sheet/Interface - Connector 15/VNEG
- net Net-(C394-Pad1) renamed /CODEC interconnection sheet/Interface - Connector 15/LINE_OUT_L
- net Net-(C395-Pad1) renamed /CODEC interconnection sheet/Interface - Connector 15/LINE_OUT_R
- net Net-(U13-Pad31) renamed /CODEC interconnection sheet/Interface - Connector 1/HPL
- net Net-(U13-Pad33) renamed /CODEC interconnection sheet/Interface - Connector 1/HPR
- net Net-(U16-Pad31) renamed /CODEC interconnection sheet/Interface - Connector 2/HPL
- net Net-(U16-Pad33) renamed /CODEC interconnection sheet/Interface - Connector 2/HPR
- net Net-(U19-Pad31) renamed /CODEC interconnection sheet/Interface - Connector 3/HPL
- net Net-(U19-Pad33) renamed /CODEC interconnection sheet/Interface - Connector 3/HPR
- net Net-(U22-Pad31) renamed /CODEC interconnection sheet/Interface - Connector 4/HPL
- net Net-(U22-Pad33) renamed /CODEC interconnection sheet/Interface - Connector 4/HPR
- net Net-(U25-Pad31) renamed /CODEC interconnection sheet/Interface - Connector 5/HPL
- net Net-(U25-Pad33) renamed /CODEC interconnection sheet/Interface - Connector 5/HPR
- net Net-(U28-Pad31) renamed /CODEC interconnection sheet/Interface - Connector 6/HPL
- net Net-(U28-Pad33) renamed /CODEC interconnection sheet/Interface - Connector 6/HPR
- net Net-(U31-Pad31) renamed /CODEC interconnection sheet/Interface - Connector 7/HPL
- net Net-(U31-Pad33) renamed /CODEC interconnection sheet/Interface - Connector 7/HPR
- net Net-(U34-Pad31) renamed /CODEC interconnection sheet/Interface - Connector 8/HPL
- net Net-(U34-Pad33) renamed /CODEC interconnection sheet/Interface - Connector 8/HPR
- net Net-(U37-Pad31) renamed /CODEC interconnection sheet/Interface - Connector 9/HPL
- net Net-(U37-Pad33) renamed /CODEC interconnection sheet/Interface - Connector 9/HPR
- net Net-(U40-Pad31) renamed /CODEC interconnection sheet/Interface - Connector 10/HPL
- net Net-(U40-Pad33) renamed /CODEC interconnection sheet/Interface - Connector 10/HPR
- net Net-(U43-Pad31) renamed /CODEC interconnection sheet/Interface - Connector 11/HPL
- net Net-(U43-Pad33) renamed /CODEC interconnection sheet/Interface - Connector 11/HPR
- net Net-(U46-Pad31) renamed /CODEC interconnection sheet/Interface - Connector 12/HPL
- net Net-(U46-Pad33) renamed /CODEC interconnection sheet/Interface - Connector 12/HPR
- net Net-(U49-Pad31) renamed /CODEC interconnection sheet/Interface - Connector 13/HPL
- net Net-(U49-Pad33) renamed /CODEC interconnection sheet/Interface - Connector 13/HPR
- net Net-(U52-Pad31) renamed /CODEC interconnection sheet/Interface - Connector 14/HPL
- net Net-(U52-Pad33) renamed /CODEC interconnection sheet/Interface - Connector 14/HPR
- net Net-(U55-Pad31) renamed /CODEC interconnection sheet/Interface - Connector 15/HPL
- net Net-(U55-Pad33) renamed /CODEC interconnection sheet/Interface - Connector 15/HPR
- C431 pad 1: GND -> /Bottom Side Daughterboard Connector Interconnects/M_L_IN6
- C431 pad 2: +3V3 -> Net-(C431-Pad2)
- C432 pad 1: /Bottom Side Daughterboard Connector Interconnects/M_L_IN6 -> /Bottom Side Daughterboard Connector Interconnects/M_L_IN7
- C433 pad 1: /Bottom Side Daughterboard Connector Interconnects/M_L_IN7 -> /Bottom Side Daughterboard Connector Interconnects/M_L_IN8
- C434 pad 1: /Bottom Side Daughterboard Connector Interconnects/M_L_IN8 -> /Bottom Side Daughterboard Connector Interconnects/M_R_IN6
- C435 pad 1: /Bottom Side Daughterboard Connector Interconnects/M_R_IN6 -> /Bottom Side Daughterboard Connector Interconnects/M_R_IN7
- C436 pad 1: /Bottom Side Daughterboard Connector Interconnects/M_R_IN7 -> /Bottom Side Daughterboard Connector Interconnects/M_R_IN8
- C437 pad 1: /Bottom Side Daughterboard Connector Interconnects/M_R_IN8 -> /Bottom Side Daughterboard Connector Interconnects/M_GND
- C438 pad 1: /Bottom Side Daughterboard Connector Interconnects/M_GND -> Net-(C438-Pad1)
- C439 pad 1: Net-(C439-Pad1) -> /Bottom Side Daughterboard Connector Interconnects/M_L_IN9
- C440 pad 1: /Bottom Side Daughterboard Connector Interconnects/M_L_IN9 -> /Bottom Side Daughterboard Connector Interconnects/M_R_IN9
- C441 pad 1: /Bottom Side Daughterboard Connector Interconnects/M_R_IN9 -> /Left Side Daughterboard Connector Interconnects/M_L_IN0
- C442 pad 1: /Left Side Daughterboard Connector Interconnects/M_L_IN0 -> /Left Side Daughterboard Connector Interconnects/M_L_IN1
- C443 pad 1: /Left Side Daughterboard Connector Interconnects/M_L_IN1 -> /Left Side Daughterboard Connector Interconnects/M_L_IN2
- C444 pad 1: /Left Side Daughterboard Connector Interconnects/M_L_IN2 -> /Left Side Daughterboard Connector Interconnects/M_R_IN0
- C445 pad 1: /Left Side Daughterboard Connector Interconnects/M_R_IN0 -> /Left Side Daughterboard Connector Interconnects/M_R_IN1
- C446 pad 1: /Left Side Daughterboard Connector Interconnects/M_R_IN1 -> /Left Side Daughterboard Connector Interconnects/M_R_IN2
- C447 pad 1: /Left Side Daughterboard Connector Interconnects/M_R_IN2 -> /Left Side Daughterboard Connector Interconnects/M_L_IN3
- C448 pad 1: /Left Side Daughterboard Connector Interconnects/M_L_IN3 -> /Left Side Daughterboard Connector Interconnects/M_L_IN4
- C449 pad 1: /Left Side Daughterboard Connector Interconnects/M_L_IN4 -> /Left Side Daughterboard Connector Interconnects/M_L_IN5
- C450 pad 1: /Left Side Daughterboard Connector Interconnects/M_L_IN5 -> /Left Side Daughterboard Connector Interconnects/M_R_IN3
- C451 pad 1: /Left Side Daughterboard Connector Interconnects/M_R_IN3 -> /Left Side Daughterboard Connector Interconnects/M_R_IN4
- C452 pad 1: /Left Side Daughterboard Connector Interconnects/M_R_IN4 -> /Left Side Daughterboard Connector Interconnects/M_R_IN5
- C453 pad 1: /Left Side Daughterboard Connector Interconnects/M_R_IN5 -> /Right Side Daughterboard Connector Interconnects/M_L_IN10
- C454 pad 1: /Right Side Daughterboard Connector Interconnects/M_L_IN10 -> /Right Side Daughterboard Connector Interconnects/M_L_IN11
- C455 pad 1: /Right Side Daughterboard Connector Interconnects/M_L_IN11 -> /Right Side Daughterboard Connector Interconnects/M_L_IN12
- C456 pad 1: /Right Side Daughterboard Connector Interconnects/M_L_IN12 -> /Right Side Daughterboard Connector Interconnects/M_R_IN10
- C457 pad 1: /Right Side Daughterboard Connector Interconnects/M_R_IN10 -> /Right Side Daughterboard Connector Interconnects/M_R_IN11
- C458 pad 1: /Right Side Daughterboard Connector Interconnects/M_R_IN11 -> /Right Side Daughterboard Connector Interconnects/M_R_IN12
- C459 pad 1: /Right Side Daughterboard Connector Interconnects/M_R_IN12 -> /Right Side Daughterboard Connector Interconnects/M_L_IN13
- C460 pad 1: /Right Side Daughterboard Connector Interconnects/M_L_IN13 -> /Right Side Daughterboard Connector Interconnects/M_L_IN14
- C461 pad 1: /Right Side Daughterboard Connector Interconnects/M_L_IN14 -> /Right Side Daughterboard Connector Interconnects/M_L_IN15
- C462 pad 1: /Right Side Daughterboard Connector Interconnects/M_L_IN15 -> /Right Side Daughterboard Connector Interconnects/M_R_IN13
- C463 pad 1: /Right Side Daughterboard Connector Interconnects/M_R_IN13 -> /Right Side Daughterboard Connector Interconnects/M_R_IN14
- C464 pad 1: /Right Side Daughterboard Connector Interconnects/M_R_IN14 -> /Right Side Daughterboard Connector Interconnects/M_R_IN15
- C465 pad 1: /Right Side Daughterboard Connector Interconnects/M_R_IN15 -> GND
- C466 pad 2: Net-(C466-Pad2) -> Net-(C465-Pad2)
- C467 pad 2: Net-(C466-Pad2) -> /Microprocessor and Support/+5VUSB
- C469 pad 1: GND -> Net-(C469-Pad1)
- C469 pad 2: /Microprocessor and Support/+5VUSB -> GND
- C470 pad 1: Net-(C470-Pad1) -> Net-(C469-Pad1)
- C471 pad 1: Net-(C470-Pad1) -> Net-(C469-Pad1)
- C472 pad 1: Net-(C470-Pad1) -> (no net)
- C473 pad 1: Net-(C473-Pad1) -> /Microprocessor and Support/~RESET
- C473 pad 2: GND -> +3V3
- C474 pad 1: /Microprocessor and Support/~RESET -> Net-(C469-Pad1)
- C474 pad 2: +3V3 -> GND
- C475 pad 1: Net-(C470-Pad1) -> GND
- C475 pad 2: GND -> /Microprocessor and Support/+3V3USB
- C476 pad 2: /Microprocessor and Support/+3V3USB -> +3V3
- D16 pad 1: Net-(D16-Pad1) -> /Bottom Side Daughterboard Connector Interconnects/M_ID_PIN6
- D17 pad 1: Net-(D17-Pad1) -> /Bottom Side Daughterboard Connector Interconnects/M_ID_PIN7
- D18 pad 1: Net-(D18-Pad1) -> /Bottom Side Daughterboard Connector Interconnects/M_ID_PIN8
- D19 pad 1: /Bottom Side Daughterboard Connector Interconnects/M_ID_PIN6 -> /Bottom Side Daughterboard Connector Interconnects/M_+12V
- D20 pad 1: /Bottom Side Daughterboard Connector Interconnects/M_ID_PIN7 -> /Bottom Side Daughterboard Connector Interconnects/M_+12V
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Routing:
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