File: edc-mux-board-fpga/conn.sch (KiCad schematic (older format))
At the start: 24 parts, among them U12 P82B96, U13 TLV320AIC3206, U14 MAX4910

Commit message: Reannotating board
Parts:
- renumbered FB1 to FB4
Changed lines of the file:
@@
 $Descr USLetter 11000 8500
 encoding utf-8
-Sheet 5 28
+Sheet 20 28
 Title ""
 Date ""
@@
 AR Path="/5CC6CC1A/5CC6D62D/5DAC04B2" Ref="U52"  Part="1"
 AR Path="/5CC6CC1A/5CC6D64F/5DAC04B2" Ref="U55"  Part="1"
+AR Path="/5CC6CC1A/5CC6D47B/5DAC04B2" Ref="U10"  Part="1"
 F 0 "U55" H 5650 2350 50  0000 C CNN
 F 1 "TLV320AIC3206" H 4700 4450 50  0000 C CNN
@@
 AR Path="/5CC6CC1A/5CC6D62D/5DAC04C4" Ref="C374"  Part="1"
 AR Path="/5CC6CC1A/5CC6D64F/5DAC04C4" Ref="C392"  Part="1"
+AR Path="/5CC6CC1A/5CC6D47B/5DAC04C4" Ref="C122"  Part="1"
 F 0 "C392" V 4950 2150 50  0000 C CNN
 F 1 "2.2uF X7R" V 5050 2150 50  0000 C CNN
@@
 AR Path="/5CC6CC1A/5CC6D62D/5DAC04D3" Ref="C375"  Part="1"
 AR Path="/5CC6CC1A/5CC6D64F/5DAC04D3" Ref="C393"  Part="1"
+AR Path="/5CC6CC1A/5CC6D47B/5DAC04D3" Ref="C123"  Part="1"
 F 0 "C393" V 5800 4250 50  0000 C CNN
 F 1 "2.2uF X7R" V 5900 4250 50  0000 C CNN
@@
 AR Path="/5CC6CC1A/5CC6D62D/5DAC04E5" Ref="#PWR0168"  Part="1"
 AR Path="/5CC6CC1A/5CC6D64F/5DAC04E5" Ref="#PWR0177"  Part="1"
+AR Path="/5CC6CC1A/5CC6D47B/5DAC04E5" Ref="#PWR042"  Part="1"
 F 0 "#PWR0177" H 5750 4500 50  0001 C CNN
 F 1 "GND" H 5750 4600 50  0000 C CNN
@@
 AR Path="/5CC6CC1A/5CC6D62D/5D2F4C59" Ref="C373"  Part="1"
 AR Path="/5CC6CC1A/5CC6D64F/5D2F4C59" Ref="C391"  Part="1"
+AR Path="/5CC6CC1A/5CC6D47B/5D2F4C59" Ref="C121"  Part="1"
 F 0 "C391" H 4500 4200 50  0000 L CNN
 F 1 "1uF X7R" H 4500 4250 50  0000 L CNN
@@
 AR Path="/5CC6CC1A/5CC6D62D/5CE6F348" Ref="C371"  Part="1"
 AR Path="/5CC6CC1A/5CC6D64F/5CE6F348" Ref="C389"  Part="1"
+AR Path="/5CC6CC1A/5CC6D47B/5CE6F348" Ref="C119"  Part="1"
 F 0 "C389" H 4050 3000 50  0000 L CNN
 F 1 "100nF X7R" H 4050 3050 50  0000 L CNN
@@
 AR Path="/5CC6CC1A/5CC6D62D/5D2F4C5A" Ref="C372"  Part="1"
 AR Path="/5CC6CC1A/5CC6D64F/5D2F4C5A" Ref="C390"  Part="1"
+AR Path="/5CC6CC1A/5CC6D47B/5D2F4C5A" Ref="C120"  Part="1"
 F 0 "C390" H 4050 3000 50  0000 R CNN
 F 1 "100nF X7R" H 4050 3050 50  0000 R CNN
@@
 AR Path="/5CC6CC1A/5CC6D62D/5D2F4C5B" Ref="#PWR0167"  Part="1"
 AR Path="/5CC6CC1A/5CC6D64F/5D2F4C5B" Ref="#PWR0176"  Part="1"
+AR Path="/5CC6CC1A/5CC6D47B/5D2F4C5B" Ref="#PWR041"  Part="1"
 F 0 "#PWR0176" H 3550 3000 50  0001 C CNN
 F 1 "GND" H 3550 3100 50  0000 C CNN
@@
 AR Path="/5CC6CC1A/5CC6D62D/5D2F4C5C" Ref="U53"  Part="1"
 AR Path="/5CC6CC1A/5CC6D64F/5D2F4C5C" Ref="U56"  Part="1"
+AR Path="/5CC6CC1A/5CC6D47B/5D2F4C5C" Ref="U11"  Part="1"
 F 0 "U56" H 8500 2800 50  0000 C CNN
 F 1 "MAX4910" H 7950 3350 50  0000 C CNN
@@
 AR Path="/5CC6CC1A/5CC6D62D/5D2F4C5D" Ref="#PWR0172"  Part="1"
 AR Path="/5CC6CC1A/5CC6D64F/5D2F4C5D" Ref="#PWR0181"  Part="1"
+AR Path="/5CC6CC1A/5CC6D47B/5D2F4C5D" Ref="#PWR046"  Part="1"
 F 0 "#PWR0181" H 7750 4150 50  0001 C CNN
 F 1 "GND" H 7750 4250 50  0000 C CNN
@@
 	8650 3500 8850 3500
 $Comp
-L Device:Ferrite_Bead_Small FB1
+L Device:Ferrite_Bead_Small FB4
 U 1 1 5D2F4C5E
 P 6550 4150
-AR Path="/5CC6CC1A/5CC6D498/5D2F4C5E" Ref="FB1"  Part="1"
+AR Path="/5CC6CC1A/5CC6D498/5D2F4C5E" Ref="FB4"  Part="1"
 AR Path="/5CC6CC1A/5CC6D4B3/5D2F4C5E" Ref="FB5"  Part="1"
 AR Path="/5CC6CC1A/5CC6D4D3/5D2F4C5E" Ref="FB6"  Part="1"
@@
 AR Path="/5CC6CC1A/5CC6D62D/5D2F4C5E" Ref="FB17"  Part="1"
 AR Path="/5CC6CC1A/5CC6D64F/5D2F4C5E" Ref="FB18"  Part="1"
+AR Path="/5CC6CC1A/5CC6D47B/5D2F4C5E" Ref="FB3"  Part="1"
 F 0 "FB18" H 6625 4200 50  0000 L CNN
 F 1 "220Ω/2A" H 6625 4100 50  0000 L CNN
@@
 AR Path="/5CC6CC1A/5CC6D62D/5D2F4C5F" Ref="C368"  Part="1"
 AR Path="/5CC6CC1A/5CC6D64F/5D2F4C5F" Ref="C386"  Part="1"
+AR Path="/5CC6CC1A/5CC6D47B/5D2F4C5F" Ref="C116"  Part="1"
 F 0 "C386" H 3650 2700 50  0000 L CNN
 F 1 "33pF NP0" H 3650 2750 50  0000 L CNN
@@
 AR Path="/5CC6CC1A/5CC6D62D/5D2F4C52" Ref="C370"  Part="1"
 AR Path="/5CC6CC1A/5CC6D64F/5D2F4C52" Ref="C388"  Part="1"
+AR Path="/5CC6CC1A/5CC6D47B/5D2F4C52" Ref="C118"  Part="1"
 F 0 "C388" H 3650 2700 50  0000 R CNN
 F 1 "33pF NP0" H 3650 2750 50  0000 R CNN
@@
 AR Path="/5CC6CC1A/5CC6D62D/5D2F4C60" Ref="#+1V8A016"  Part="1"
 AR Path="/5CC6CC1A/5CC6D64F/5D2F4C60" Ref="#+1V8A017"  Part="1"
+AR Path="/5CC6CC1A/5CC6D47B/5D2F4C60" Ref="#+1V8A02"  Part="1"
 F 0 "#+1V8A017" H 7500 1800 60  0001 C CNN
 F 1 "+1V8A" H 6750 2300 50  0000 C CNN
@@
 AR Path="/5CC6CC1A/5CC6D62D/5DAC0585" Ref="#PWR0170"  Part="1"
 AR Path="/5CC6CC1A/5CC6D64F/5DAC0585" Ref="#PWR0179"  Part="1"
+AR Path="/5CC6CC1A/5CC6D47B/5DAC0585" Ref="#PWR044"  Part="1"
 F 0 "#PWR0179" H 6500 1950 50  0001 C CNN
 F 1 "+1V8" H 6500 2240 50  0000 C CNN
@@
 AR Path="/5CC6CC1A/5CC6D62D/5DAC0596" Ref="#PWR0169"  Part="1"
 AR Path="/5CC6CC1A/5CC6D64F/5DAC0596" Ref="#PWR0178"  Part="1"
+AR Path="/5CC6CC1A/5CC6D47B/5DAC0596" Ref="#PWR043"  Part="1"
 F 0 "#PWR0178" H 6250 1950 50  0001 C CNN
 F 1 "+3V3" H 6250 2240 50  0000 C CNN
@@
 AR Path="/5CC6CC1A/5CC6D62D/5DAC059F" Ref="C379"  Part="1"
 AR Path="/5CC6CC1A/5CC6D64F/5DAC059F" Ref="C397"  Part="1"
+AR Path="/5CC6CC1A/5CC6D47B/5DAC059F" Ref="C127"  Part="1"
 F 0 "C397" H 6850 3100 50  0000 R CNN
 F 1 "1uF X7R" H 6900 3300 50  0000 R CNN
@@
 AR Path="/5CC6CC1A/5CC6D62D/5D2F4C64" Ref="#PWR0171"  Part="1"
 AR Path="/5CC6CC1A/5CC6D64F/5D2F4C64" Ref="#PWR0180"  Part="1"
+AR Path="/5CC6CC1A/5CC6D47B/5D2F4C64" Ref="#PWR045"  Part="1"
 F 0 "#PWR0180" H 6650 3150 50  0001 C CNN
 F 1 "GND" H 6650 3250 50  0000 C CNN
@@
 AR Path="/5CC6CC1A/5CC6D62D/5D2F4C65" Ref="C380"  Part="1"
 AR Path="/5CC6CC1A/5CC6D64F/5D2F4C65" Ref="C398"  Part="1"
+AR Path="/5CC6CC1A/5CC6D47B/5D2F4C65" Ref="C128"  Part="1"
 F 0 "C398" H 6800 3150 50  0000 R CNN
 F 1 "10uF X7R" H 6800 3200 50  0000 R CNN
@@
 AR Path="/5CC6CC1A/5CC6D62D/5D2F4C66" Ref="C378"  Part="1"
 AR Path="/5CC6CC1A/5CC6D64F/5D2F4C66" Ref="C396"  Part="1"
+AR Path="/5CC6CC1A/5CC6D47B/5D2F4C66" Ref="C126"  Part="1"
 F 0 "C396" V 6450 3150 50  0000 R CNN
 F 1 "100nF X7R" V 6600 3400 50  0000 R CNN
@@
 AR Path="/5CC6CC1A/5CC6D62D/5D2F4C67" Ref="C381"  Part="1"
 AR Path="/5CC6CC1A/5CC6D64F/5D2F4C67" Ref="C399"  Part="1"
+AR Path="/5CC6CC1A/5CC6D47B/5D2F4C67" Ref="C129"  Part="1"
 F 0 "C399" V 7000 2100 50  0000 R CNN
 F 1 "100nF X7R" V 7100 2600 50  0000 R CNN
@@
 AR Path="/5CC6CC1A/5CC6D62D/5D2F4C68" Ref="C382"  Part="1"
 AR Path="/5CC6CC1A/5CC6D64F/5D2F4C68" Ref="C400"  Part="1"
+AR Path="/5CC6CC1A/5CC6D47B/5D2F4C68" Ref="C130"  Part="1"
 F 0 "C400" V 7100 2450 50  0000 C CNN
 F 1 "10uF X7R" V 7000 2150 50  0000 C CNN
@@
 AR Path="/5CC6CC1A/5CC6D62D/5D2F4C69" Ref="C383"  Part="1"
 AR Path="/5CC6CC1A/5CC6D64F/5D2F4C69" Ref="C401"  Part="1"
+AR Path="/5CC6CC1A/5CC6D47B/5D2F4C69" Ref="C131"  Part="1"
 F 0 "C401" V 7000 2500 50  0000 R CNN
 F 1 "100nF X7R" V 7100 3000 50  0000 R CNN
@@
 AR Path="/5CC6CC1A/5CC6D62D/5DAC0610" Ref="C384"  Part="1"
 AR Path="/5CC6CC1A/5CC6D64F/5DAC0610" Ref="C402"  Part="1"
+AR Path="/5CC6CC1A/5CC6D47B/5DAC0610" Ref="C132"  Part="1"
 F 0 "C402" V 7000 2700 50  0000 R CNN
 F 1 "100nF X7R" V 7100 3200 50  0000 R CNN
@@
 AR Path="/5CC6CC1A/5CC6D62D/5DAC061B" Ref="C385"  Part="1"
 AR Path="/5CC6CC1A/5CC6D64F/5DAC061B" Ref="C403"  Part="1"
+AR Path="/5CC6CC1A/5CC6D47B/5DAC061B" Ref="C133"  Part="1"
 F 0 "C403" V 7950 2850 50  0000 R CNN
 F 1 "100nF X7R" V 8100 2800 50  0000 R CNN
@@
 AR Path="/5CC6CC1A/5CC6D62D/5DAC062C" Ref="#PWR0173"  Part="1"
 AR Path="/5CC6CC1A/5CC6D64F/5DAC062C" Ref="#PWR0182"  Part="1"
+AR Path="/5CC6CC1A/5CC6D47B/5DAC062C" Ref="#PWR047"  Part="1"
 F 0 "#PWR0182" H 8300 2200 50  0001 C CNN
 F 1 "+3V3" H 8300 2490 50  0000 C CNN
@@
 AR Path="/5CC6CC1A/5CC6D62D/5D2F4C6D" Ref="U51"  Part="1"
 AR Path="/5CC6CC1A/5CC6D64F/5D2F4C6D" Ref="U54"  Part="1"
+AR Path="/5CC6CC1A/5CC6D47B/5D2F4C6D" Ref="U9"  Part="1"
 F 0 "U54" H 2100 4800 50  0000 L CNN
 F 1 "P82B96" H 2800 4800 50  0000 L CNN
@@
 AR Path="/5CC6CC1A/5CC6D62D/5D2F4C6E" Ref="#PWR0165"  Part="1"
 AR Path="/5CC6CC1A/5CC6D64F/5D2F4C6E" Ref="#PWR0174"  Part="1"
+AR Path="/5CC6CC1A/5CC6D47B/5D2F4C6E" Ref="#PWR039"  Part="1"
 F 0 "#PWR0174" H 1550 3400 50  0001 C CNN
 F 1 "+12V" H 1550 3690 50  0000 C CNN
@@
 AR Path="/5CC6CC1A/5CC6D62D/5DAC065C" Ref="R44"  Part="1"
 AR Path="/5CC6CC1A/5CC6D64F/5DAC065C" Ref="R46"  Part="1"
+AR Path="/5CC6CC1A/5CC6D47B/5DAC065C" Ref="R16"  Part="1"
 F 0 "R46" H 1800 3950 50  0000 L CNN
 F 1 "750Ω" H 1800 3900 50  0000 L CNN
@@
 AR Path="/5CC6CC1A/5CC6D62D/5DAC0662" Ref="R43"  Part="1"
 AR Path="/5CC6CC1A/5CC6D64F/5DAC0662" Ref="R45"  Part="1"
+AR Path="/5CC6CC1A/5CC6D47B/5DAC0662" Ref="R15"  Part="1"
 F 0 "R45" H 1650 4350 50  0000 L CNN
 F 1 "750Ω" H 1650 4300 50  0000 L CNN
@@
 AR Path="/5CC6CC1A/5CC6D62D/5D2F4C71" Ref="#PWR0166"  Part="1"
 AR Path="/5CC6CC1A/5CC6D64F/5D2F4C71" Ref="#PWR0175"  Part="1"
+AR Path="/5CC6CC1A/5CC6D47B/5D2F4C71" Ref="#PWR040"  Part="1"
 F 0 "#PWR0175" H 3250 3600 50  0001 C CNN
 F 1 "+12V" H 3250 3890 50  0000 C CNN
@@
 AR Path="/5CC6CC1A/5CC6D62D/5D2F4C72" Ref="C369"  Part="1"
 AR Path="/5CC6CC1A/5CC6D64F/5D2F4C72" Ref="C387"  Part="1"
+AR Path="/5CC6CC1A/5CC6D47B/5D2F4C72" Ref="C117"  Part="1"
 F 0 "C387" V 3550 4000 50  0000 C CNN
 F 1 "100nF X7R" V 3450 4000 50  0000 C CNN
@@
 AR Path="/5CC6CC1A/5CC6D62D/5DAC0492" Ref="C376"  Part="1"
 AR Path="/5CC6CC1A/5CC6D64F/5DAC0492" Ref="C394"  Part="1"
+AR Path="/5CC6CC1A/5CC6D47B/5DAC0492" Ref="C124"  Part="1"
 F 0 "C394" V 6300 3600 50  0000 C CNN
 F 1 "1uF X7R flex" V 6400 3600 50  0000 C CNN
@@
 AR Path="/5CC6CC1A/5CC6D62D/5DAC04AA" Ref="C377"  Part="1"
 AR Path="/5CC6CC1A/5CC6D64F/5DAC04AA" Ref="C395"  Part="1"
+AR Path="/5CC6CC1A/5CC6D47B/5DAC04AA" Ref="C125"  Part="1"
 F 0 "C395" V 6550 3700 50  0000 C CNN
 F 1 "1uF X7R flex" V 6650 3700 50  0000 C CNN
