File: edc-mux-board-fpga-main/microprocessor.sch (KiCad schematic (older format))
At the start: 27 parts, among them J11 PRG/SWD, J12 USB PRG, Q4 CSD22206W, Q5 CSD22206W, SW2 Reset (Microprocessor), U37 TPD3S014, U38 SAMD21JXXAM, U39 MCP1812, U40 LTC4412

Commit message: s/Manufacturers Part Number/MPN/g
for compatability with MacroFab automated processing
Parts:
- C286, C289, C290, C295: MPN (none) -> C1206C106J3RACAUTO; Manufacturers Part Number C1206C106J3RACAUTO -> (none)
- C287, C291, C292: MPN (none) -> 04023C104JAT2A; Manufacturers Part Number 04023C104JAT2A -> (none)
- C288, C293: MPN (none) -> CGA3E1X7R1E105K080AC; Manufacturers Part Number CGA3E1X7R1E105K080AC -> (none)
- C294: MPN (none) -> CGA2B2C0G1H101J050BA; Manufacturers Part Number CGA2B2C0G1H101J050BA -> (none)
- C296: MPN (none) -> CGA4J3X7R1E225K125AB; Manufacturers Part Number CGA4J3X7R1E225K125AB -> (none)
- FB44: MPN (none) -> BLM21AG601SZ1D; Manufacturers Part Number BLM21AG601SZ1D -> (none)
- J12: MPN (none) -> UJ2-BV-1-TH; Manufacturers Part Number UJ2-BV-1-TH -> (none)
- Q4, Q5: MPN (none) -> CSD22206W; Manufacturers Part Number CSD22206W -> (none)
- SW2: MPN (none) -> TL1105AF160R; Manufacturers Part Number TL1105AF160R -> (none)
- U37: MPN (none) -> TPD3S0x4; Manufacturers Part Number TPD3S0x4 -> (none)
- U38: MPN (none) -> SAMD21JXXAM; Manufacturers Part Number SAMD21JXXAM -> (none)
- U39: MPN (none) -> MCP1812AT-033/TT; Manufacturers Part Number MCP1812AT-033/TT -> (none)
- U40: MPN (none) -> LTC4412HS6#TRMPBF; Manufacturers Part Number LTC4412HS6#TRMPBF -> (none)
Changed lines of the file:
@@
 F 4 "SAMD21 ARM Cortex M0+ MCU" H 0   0   50  0001 C CNN "Description"
 F 5 "Atmel" H 0   0   50  0001 C CNN "Manufacturer"
-F 6 "SAMD21JXXAM" H 0   0   50  0001 C CNN "Manufacturers Part Number"
+F 6 "SAMD21JXXAM" H 0   0   50  0001 C CNN "MPN"
 F 7 "QFN64-EP" H 0   0   50  0001 C CNN "Package ID"
 	1    4300 4400
@@
 F 4 "Murata" H 4150 2000 50  0001 C CNN "Manufacturer"
 F 5 "0805in/2012mm" H 4150 2000 50  0001 C CNN "Package ID"
-F 6 "BLM21AG601SZ1D " H 4150 2000 50  0001 C CNN "Manufacturers Part Number"
+F 6 "BLM21AG601SZ1D " H 4150 2000 50  0001 C CNN "MPN"
 F 7 "600 Ohms @ 100MHz 1 Signal Line Ferrite Bead 0805 (2012 Metric) 700mA 210mOhm" H 0   0   50  0001 C CNN "Characteristics"
 F 8 "Ferrite Bead" H 0   0   50  0001 C CNN "Description"
@@
 F 3 "https://content.kemet.com/datasheets/KEM_C1023_X7R_AUTO_SMD.pdf" H 3900 2150 50  0001 C CNN
 F 4 "Kemet" H 0   0   50  0001 C CNN "Manufacturer"
-F 5 "C1206C106J3RACAUTO" H 0   0   50  0001 C CNN "Manufacturers Part Number"
+F 5 "C1206C106J3RACAUTO" H 0   0   50  0001 C CNN "MPN"
 F 6 "1206in/3216mm" H 0   0   50  0001 C CNN "Package ID"
 F 7 "CAP CER 10UF 25V X7R 1206" H 0   0   50  0001 C CNN "Characteristics"
@@
 F 4 "0402in/1005mm" H 0   0   50  0001 C CNN "Package ID"
 F 5 "AVX" H 0   0   50  0001 C CNN "Manufacturer"
-F 6 "04023C104JAT2A" H 0   0   50  0001 C CNN "Manufacturers Part Number"
+F 6 "04023C104JAT2A" H 0   0   50  0001 C CNN "MPN"
 F 7 "CAP CER 0.1UF 25V X7R 0402" H 0   0   50  0001 C CNN "Characteristics"
 F 8 "MLCC Capacitor" H 0   0   50  0001 C CNN "Description"
@@
 F 4 "Tactile Switch" H 0   0   50  0001 C CNN "Description"
 F 5 "Eswitch" H 0   0   50  0001 C CNN "Manufacturer"
-F 6 "TL1105AF160R" H 0   0   50  0001 C CNN "Manufacturers Part Number"
+F 6 "TL1105AF160R" H 0   0   50  0001 C CNN "MPN"
 F 7 "Through Hole" H 0   0   50  0001 C CNN "Package ID"
 	1    4800 7050
@@
 F 5 "CAP CER 100PF 50V C0G 0402" H 0   0   50  0001 C CNN "Characteristics"
 F 6 "TDK" H 0   0   50  0001 C CNN "Manufacturer"
-F 7 "CGA2B2C0G1H101J050BA" H 0   0   50  0001 C CNN "Manufacturers Part Number"
+F 7 "CGA2B2C0G1H101J050BA" H 0   0   50  0001 C CNN "MPN"
 F 8 "MLCC Capacitor" H 0   0   50  0001 C CNN "Description"
 	1    4750 6600
@@
 F 3 "https://content.kemet.com/datasheets/KEM_C1023_X7R_AUTO_SMD.pdf" H 4750 1950 50  0001 C CNN
 F 4 "Kemet" H 0   0   50  0001 C CNN "Manufacturer"
-F 5 "C1206C106J3RACAUTO" H 0   0   50  0001 C CNN "Manufacturers Part Number"
+F 5 "C1206C106J3RACAUTO" H 0   0   50  0001 C CNN "MPN"
 F 6 "1206in/3216mm" H 0   0   50  0001 C CNN "Package ID"
 F 7 "CAP CER 10UF 25V X7R 1206" H 0   0   50  0001 C CNN "Characteristics"
@@
 F 4 "0402in/1005mm" H 0   0   50  0001 C CNN "Package ID"
 F 5 "AVX" H 0   0   50  0001 C CNN "Manufacturer"
-F 6 "04023C104JAT2A" H 0   0   50  0001 C CNN "Manufacturers Part Number"
+F 6 "04023C104JAT2A" H 0   0   50  0001 C CNN "MPN"
 F 7 "CAP CER 0.1UF 25V X7R 0402" H 0   0   50  0001 C CNN "Characteristics"
 F 8 "MLCC Capacitor" H 0   0   50  0001 C CNN "Description"
@@
 F 4 "0402in/1005mm" H 0   0   50  0001 C CNN "Package ID"
 F 5 "AVX" H 0   0   50  0001 C CNN "Manufacturer"
-F 6 "04023C104JAT2A" H 0   0   50  0001 C CNN "Manufacturers Part Number"
+F 6 "04023C104JAT2A" H 0   0   50  0001 C CNN "MPN"
 F 7 "CAP CER 0.1UF 25V X7R 0402" H 0   0   50  0001 C CNN "Characteristics"
 F 8 "MLCC Capacitor" H 0   0   50  0001 C CNN "Description"
@@
 F 3 "https://product.tdk.com/info/en/catalog/datasheets/mlcc_automotive_general_en.pdf" H 4750 2500 50  0001 C CNN
 F 4 "TDK" H 0   0   50  0001 C CNN "Manufacturer"
-F 5 "CGA3E1X7R1E105K080AC" H 0   0   50  0001 C CNN "Manufacturers Part Number"
+F 5 "CGA3E1X7R1E105K080AC" H 0   0   50  0001 C CNN "MPN"
 F 6 "0603in/1608mm" H 0   0   50  0001 C CNN "Package ID"
 F 7 "CAP CER 1UF 25V X7R 0603" H 0   0   50  0001 C CNN "Characteristics"
@@
 F 4 "USB B female Vertical PBC mount connetor" H 0   0   50  0001 C CNN "Description"
 F 5 "CUI Inc" H 0   0   50  0001 C CNN "Manufacturer"
-F 6 "UJ2-BV-1-TH" H 0   0   50  0001 C CNN "Manufacturers Part Number"
+F 6 "UJ2-BV-1-TH" H 0   0   50  0001 C CNN "MPN"
 F 7 "Through Hole" H 0   0   50  0001 C CNN "Package ID"
 	1    1850 8550
@@
 F 4 "ESD protection and current limiting for USB ports" H 0   0   50  0001 C CNN "Description"
 F 5 "Texas Instruments" H 0   0   50  0001 C CNN "Manufacturer"
-F 6 "TPD3S0x4" H 0   0   50  0001 C CNN "Manufacturers Part Number"
+F 6 "TPD3S0x4" H 0   0   50  0001 C CNN "MPN"
 F 7 "SOT-23-6" H 0   0   50  0001 C CNN "Package ID"
 	1    3050 8450
@@
 F 5 "Microchip" H 4850 8350 50  0001 C CNN "Manufacturer"
 F 6 "3v3 regulator 300mA" H 4850 8350 50  0001 C CNN "Description"
-F 7 "MCP1812AT-033/TT" H 4850 8350 50  0001 C CNN "Manufacturers Part Number"
+F 7 "MCP1812AT-033/TT" H 4850 8350 50  0001 C CNN "MPN"
 	1    4850 8350
 	1    0    0    -1
@@
 F 3 "https://product.tdk.com/info/en/catalog/datasheets/mlcc_automotive_general_en.pdf" H 4100 8700 50  0001 C CNN
 F 4 "TDK" H 0   0   50  0001 C CNN "Manufacturer"
-F 5 "CGA3E1X7R1E105K080AC" H 0   0   50  0001 C CNN "Manufacturers Part Number"
+F 5 "CGA3E1X7R1E105K080AC" H 0   0   50  0001 C CNN "MPN"
 F 6 "0603in/1608mm" H 0   0   50  0001 C CNN "Package ID"
 F 7 "CAP CER 1UF 25V X7R 0603" H 0   0   50  0001 C CNN "Characteristics"
@@
 F 4 "0805in/2012mm" H 0   0   50  0001 C CNN "Package ID"
 F 5 "TDK" H 0   0   50  0001 C CNN "Manufacturer"
-F 6 "CGA4J3X7R1E225K125AB" H 0   0   50  0001 C CNN "Manufacturers Part Number"
+F 6 "CGA4J3X7R1E225K125AB" H 0   0   50  0001 C CNN "MPN"
 F 7 "CAP CER 2.2UF 25V X7R 0805" H 0   0   50  0001 C CNN "Characteristics"
 F 8 "MLCC Capacitor" H 0   0   50  0001 C CNN "Description"
@@
 F 3 "https://content.kemet.com/datasheets/KEM_C1023_X7R_AUTO_SMD.pdf" H 4300 8700 50  0001 C CNN
 F 4 "Kemet" H 0   0   50  0001 C CNN "Manufacturer"
-F 5 "C1206C106J3RACAUTO" H 0   0   50  0001 C CNN "Manufacturers Part Number"
+F 5 "C1206C106J3RACAUTO" H 0   0   50  0001 C CNN "MPN"
 F 6 "1206in/3216mm" H 0   0   50  0001 C CNN "Package ID"
 F 7 "CAP CER 10UF 25V X7R 1206" H 0   0   50  0001 C CNN "Characteristics"
@@
 F 3 "https://www.analog.com/media/en/technical-documentation/data-sheets/4412fb.pdf" H 6550 1950 50  0001 C CNN
 F 4 "Linear Technologies" H 6000 1150 50  0001 C CNN "Manufacturer"
-F 5 "LTC4412HS6#TRMPBF" H 6000 1150 50  0001 C CNN "Manufacturers Part Number"
+F 5 "LTC4412HS6#TRMPBF" H 6000 1150 50  0001 C CNN "MPN"
 F 6 "Ideal Diode Controller" H 0   0   50  0001 C CNN "Description"
 F 7 "SOT-23-6" H 0   0   50  0001 C CNN "Package ID"
@@
 F 4 "P Channel MOSFET" H 0   0   50  0001 C CNN "Description"
 F 5 "Texas Instruments" H 0   0   50  0001 C CNN "Manufacturer"
-F 6 "CSD22206W" H 0   0   50  0001 C CNN "Manufacturers Part Number"
+F 6 "CSD22206W" H 0   0   50  0001 C CNN "MPN"
 F 7 "DSBGA9" H 0   0   50  0001 C CNN "Package ID"
 	1    4650 1450
@@
 F 4 "P Channel MOSFET" H 0   0   50  0001 C CNN "Description"
 F 5 "Texas Instruments" H 0   0   50  0001 C CNN "Manufacturer"
-F 6 "CSD22206W" H 0   0   50  0001 C CNN "Manufacturers Part Number"
+F 6 "CSD22206W" H 0   0   50  0001 C CNN "MPN"
 F 7 "DSBGA9" H 0   0   50  0001 C CNN "Package ID"
 	1    5450 1600
@@
 F 3 "https://content.kemet.com/datasheets/KEM_C1023_X7R_AUTO_SMD.pdf" H 5050 1800 50  0001 C CNN
 F 4 "Kemet" H 0   0   50  0001 C CNN "Manufacturer"
-F 5 "C1206C106J3RACAUTO" H 0   0   50  0001 C CNN "Manufacturers Part Number"
+F 5 "C1206C106J3RACAUTO" H 0   0   50  0001 C CNN "MPN"
 F 6 "1206in/3216mm" H 0   0   50  0001 C CNN "Package ID"
 F 7 "CAP CER 10UF 25V X7R 1206" H 0   0   50  0001 C CNN "Characteristics"
