File: edc-mux-board-fpga-main/clocks.sch (KiCad schematic (older format))
At the start: 25 parts, among them J1 OSC_PRG_HDR, Q1 CSD22206W, Q2 CSD22206W, U7 CDCE706, U8 LTC4412, Y1 SiT1602BI-71-33E-48.000000

Commit message: Reannotate main schematic and pcb after expansion transition
Parts:
- renumbered C112 to C115, C113 to C116, C114 to C117, C115 to C118, J1 to J2, Q1 to Q2, Q2 to Q3, U7 to U8, U8 to U9
Changed lines of the file:
@@
 Do I need a separate Reset connection\nto the MCU so it can reset the clock chips\nindependantly?
 $Comp
-L power:GND #PWR035
+L power:GND #PWR036
 U 1 1 5CB6F7AE
 P 5350 4650
-F 0 "#PWR035" H 5350 4400 50  0001 C CNN
+F 0 "#PWR036" H 5350 4400 50  0001 C CNN
 F 1 "GND" H 5400 4450 50  0000 C CNN
 F 2 "" H 5350 4650 50  0001 C CNN
@@
 $EndComp
 $Comp
-L Device:C_Small C112
+L Device:C_Small C115
 U 1 1 5CB7C30C
 P 2850 3100
-F 0 "C112" V 2600 3100 50  0000 C CNN
+F 0 "C115" V 2600 3100 50  0000 C CNN
 F 1 "100nF X7R" V 2700 3100 50  0000 C CNN
 F 2 "Capacitor_SMD:C_0603_1608Metric" H 2850 3100 50  0001 C CNN
@@
 	2600 3100 2750 3100
 $Comp
-L power:GND #PWR030
+L power:GND #PWR032
 U 1 1 5CB7F01E
 P 2950 3250
-F 0 "#PWR030" H 2950 3000 50  0001 C CNN
+F 0 "#PWR032" H 2950 3000 50  0001 C CNN
 F 1 "GND" H 3000 3050 50  0000 C CNN
 F 2 "" H 2950 3250 50  0001 C CNN
@@
 $EndComp
 $Comp
-L power:GND #PWR029
+L power:GND #PWR031
 U 1 1 5CB809B1
 P 2600 4300
-F 0 "#PWR029" H 2600 4050 50  0001 C CNN
+F 0 "#PWR031" H 2600 4050 50  0001 C CNN
 F 1 "GND" H 2650 4100 50  0000 C CNN
 F 2 "" H 2600 4300 50  0001 C CNN
@@
 Y0 = 48MHz for FPGA\nY1 = 48MHz for CODECs\nY2 = 48MHz for CODECs\nY3 = for Microprocessor\nY4 = 25MHz for W5500 Ethernet
 $Comp
-L SW-Texas:CDCE706 U7
+L SW-Texas:CDCE706 U8
 U 1 1 5CB9BD83
 P 5350 3850
-F 0 "U7" H 5700 3500 50  0000 C CNN
+F 0 "U8" H 5700 3500 50  0000 C CNN
 F 1 "CDCE706" H 4950 4200 50  0000 C CNN
 F 2 "Package_SO:TSSOP-20_4.4x6.5mm_P0.65mm" H 4550 4750 50  0001 C CNN
@@
 	3450 3900 3450 4000
 $Comp
-L power:GND #PWR031
+L power:GND #PWR033
 U 1 1 5CBADCB5
 P 3450 4400
-F 0 "#PWR031" H 3450 4150 50  0001 C CNN
+F 0 "#PWR033" H 3450 4150 50  0001 C CNN
 F 1 "GND" H 3500 4200 50  0000 C CNN
 F 2 "" H 3450 4400 50  0001 C CNN
@@
 	3300 3800 4650 3800
 $Comp
-L Connector_Generic:Conn_01x04 J1
+L Connector_Generic:Conn_01x04 J2
 U 1 1 5CBAFEA0
 P 3300 3200
-F 0 "J1" H 3200 3550 50  0000 C CNN
+F 0 "J2" H 3200 3550 50  0000 C CNN
 F 1 "OSC_PRG_HDR" H 3200 3450 50  0000 C CNN
 F 2 "Connector_PinHeader_2.54mm:PinHeader_1x04_P2.54mm_Vertical" H 3300 3200 50  0001 C CNN
@@
 $EndComp
 $Comp
-L power:GND #PWR032
+L power:GND #PWR034
 U 1 1 5CBB95F3
 P 3500 3500
-F 0 "#PWR032" H 3500 3250 50  0001 C CNN
+F 0 "#PWR034" H 3500 3250 50  0001 C CNN
 F 1 "GND" H 3550 3300 50  0000 C CNN
 F 2 "" H 3500 3500 50  0001 C CNN
@@
 	6350 3600 6550 3600
 $Comp
-L Device:C_Small C115
+L Device:C_Small C118
 U 1 1 5CBDE920
 P 5850 3100
-F 0 "C115" H 5750 3050 50  0000 R CNN
+F 0 "C118" H 5750 3050 50  0000 R CNN
 F 1 "100nF X7R" H 5750 3100 50  0000 R CNN
 F 2 "Capacitor_SMD:C_0603_1608Metric" H 5850 3100 50  0001 C CNN
@@
 $EndComp
 $Comp
-L Device:C_Small C113
+L Device:C_Small C116
 U 1 1 5CBE047E
 P 5650 3100
-F 0 "C113" H 5800 3050 50  0000 R CNN
+F 0 "C116" H 5800 3050 50  0000 R CNN
 F 1 "100nF X7R" H 5900 3150 50  0000 R CNN
 F 2 "Capacitor_SMD:C_0603_1608Metric" H 5650 3100 50  0001 C CNN
@@
 Connection ~ 5650 2950
 $Comp
-L power:GND #PWR036
+L power:GND #PWR037
 U 1 1 5CBE6F18
 P 5750 3250
-F 0 "#PWR036" H 5750 3000 50  0001 C CNN
+F 0 "#PWR037" H 5750 3000 50  0001 C CNN
 F 1 "GND" H 5800 3050 50  0000 C CNN
 F 2 "" H 5750 3250 50  0001 C CNN
@@
 P 6800 1900
 AR Path="/5CAA362B/5CC5E70E" Ref="U?"  Part="1"
-AR Path="/5CC3E5DC/5CC5E70E" Ref="U8"  Part="1"
-F 0 "U8" H 7000 1700 50  0000 C CNN
+AR Path="/5CC3E5DC/5CC5E70E" Ref="U9"  Part="1"
+F 0 "U9" H 7000 1700 50  0000 C CNN
 F 1 "LTC4412" H 6750 2100 50  0000 C CNN
 F 2 "Package_TO_SOT_SMD:TSOT-23-6" H 6800 2200 50  0001 C CNN
@@
 P 5350 1900
 AR Path="/5CAA362B/5CC5E714" Ref="#PWR?"  Part="1"
-AR Path="/5CC3E5DC/5CC5E714" Ref="#PWR034"  Part="1"
-F 0 "#PWR034" H 5350 1750 50  0001 C CNN
+AR Path="/5CC3E5DC/5CC5E714" Ref="#PWR035"  Part="1"
+F 0 "#PWR035" H 5350 1750 50  0001 C CNN
 F 1 "+3.3V" H 5350 2040 50  0000 C CNN
 F 2 "" H 5350 1900 50  0001 C CNN
@@
 P 5450 2200
 AR Path="/5CAA362B/5CC5E71A" Ref="Q?"  Part="1"
-AR Path="/5CC3E5DC/5CC5E71A" Ref="Q1"  Part="1"
-F 0 "Q1" H 5650 2250 50  0000 L CNN
+AR Path="/5CC3E5DC/5CC5E71A" Ref="Q2"  Part="1"
+F 0 "Q2" H 5650 2250 50  0000 L CNN
 F 1 "CSD22206W" H 5650 2150 50  0000 L CNN
 F 2 "SW-Texas:DSBGA9" H 5650 2250 50  0001 C CNN
@@
 P 7200 1600
 AR Path="/5CAA362B/5CC5E726" Ref="#PWR?"  Part="1"
-AR Path="/5CC3E5DC/5CC5E726" Ref="#PWR037"  Part="1"
-F 0 "#PWR037" H 7200 1450 50  0001 C CNN
+AR Path="/5CC3E5DC/5CC5E726" Ref="#PWR038"  Part="1"
+F 0 "#PWR038" H 7200 1450 50  0001 C CNN
 F 1 "+3.3V" H 7200 1740 50  0000 C CNN
 F 2 "" H 7200 1600 50  0001 C CNN
@@
 P 6250 2350
 AR Path="/5CAA362B/5CC5E732" Ref="Q?"  Part="1"
-AR Path="/5CC3E5DC/5CC5E732" Ref="Q2"  Part="1"
-F 0 "Q2" V 6550 2350 50  0000 C CNN
+AR Path="/5CC3E5DC/5CC5E732" Ref="Q3"  Part="1"
+F 0 "Q3" V 6550 2350 50  0000 C CNN
 F 1 "CSD22206W" V 6650 2350 50  0000 C CNN
 F 2 "SW-Texas:DSBGA9" H 6450 2400 50  0001 C CNN
@@
 P 7400 2850
 AR Path="/5CAA362B/5CC5E749" Ref="#PWR?"  Part="1"
-AR Path="/5CC3E5DC/5CC5E749" Ref="#PWR038"  Part="1"
-F 0 "#PWR038" H 7400 2600 50  0001 C CNN
+AR Path="/5CC3E5DC/5CC5E749" Ref="#PWR039"  Part="1"
+F 0 "#PWR039" H 7400 2600 50  0001 C CNN
 F 1 "GND" H 7400 2700 50  0000 C CNN
 F 2 "" H 7400 2850 50  0001 C CNN
@@
 P 5850 2550
 AR Path="/5CAA362B/5CC5E754" Ref="C?"  Part="1"
-AR Path="/5CC3E5DC/5CC5E754" Ref="C114"  Part="1"
-F 0 "C114" H 5950 2600 50  0000 L CNN
+AR Path="/5CC3E5DC/5CC5E754" Ref="C117"  Part="1"
+F 0 "C117" H 5950 2600 50  0000 L CNN
 F 1 "10uF X7R" H 5950 2550 50  0000 L CNN
 F 2 "Capacitor_SMD:C_1206_3216Metric" H 5850 2550 50  0001 C CNN

Commit message: swapping 100nF capacitors from 0603 to 0402 size
Parts:
- C115, C116, C118: footprint Capacitor_SMD:C_0603_1608Metric -> Capacitor_SMD:C_0402_1005Metric; Characteristics CAP CER 0.1UF 25V X7R 0603 -> CAP CER 0.1UF 25V X7R 0402; Manufacturer Kemet -> AVX; Manufacturers Part Number C0603C104J3RACAUTO -> 04023C104JAT2A; Package ID 0603in/1608mm -> 0402in/1005mm
Changed lines of the file:
@@
 F 0 "C115" V 2600 3100 50  0000 C CNN
 F 1 "100nF X7R" V 2700 3100 50  0000 C CNN
-F 2 "Capacitor_SMD:C_0603_1608Metric" H 2850 3100 50  0001 C CNN
-F 3 "https://content.kemet.com/datasheets/KEM_C1023_X7R_AUTO_SMD.pdf" H 2850 3100 50  0001 C CNN
-F 4 "0603in/1608mm" H 250 850 50  0001 C CNN "Package ID"
-F 5 "Kemet" H 250 850 50  0001 C CNN "Manufacturer"
-F 6 "C0603C104J3RACAUTO" H 250 850 50  0001 C CNN "Manufacturers Part Number"
-F 7 "CAP CER 0.1UF 25V X7R 0603" H 250 850 50  0001 C CNN "Characteristics"
+F 2 "Capacitor_SMD:C_0402_1005Metric" H 2850 3100 50  0001 C CNN
+F 3 "http://datasheets.avx.com/X7RDielectric.pdf" H 2850 3100 50  0001 C CNN
+F 4 "0402in/1005mm" H 250 850 50  0001 C CNN "Package ID"
+F 5 "AVX" H 250 850 50  0001 C CNN "Manufacturer"
+F 6 "04023C104JAT2A" H 250 850 50  0001 C CNN "Manufacturers Part Number"
+F 7 "CAP CER 0.1UF 25V X7R 0402" H 250 850 50  0001 C CNN "Characteristics"
 F 8 "MLCC Capacitor" H 250 850 50  0001 C CNN "Description"
 	1    2850 3100
@@
 F 0 "C118" H 5750 3050 50  0000 R CNN
 F 1 "100nF X7R" H 5750 3100 50  0000 R CNN
-F 2 "Capacitor_SMD:C_0603_1608Metric" H 5850 3100 50  0001 C CNN
-F 3 "https://content.kemet.com/datasheets/KEM_C1023_X7R_AUTO_SMD.pdf" H 5850 3100 50  0001 C CNN
-F 4 "0603in/1608mm" H 250 850 50  0001 C CNN "Package ID"
-F 5 "Kemet" H 250 850 50  0001 C CNN "Manufacturer"
-F 6 "C0603C104J3RACAUTO" H 250 850 50  0001 C CNN "Manufacturers Part Number"
-F 7 "CAP CER 0.1UF 25V X7R 0603" H 250 850 50  0001 C CNN "Characteristics"
+F 2 "Capacitor_SMD:C_0402_1005Metric" H 5850 3100 50  0001 C CNN
+F 3 "http://datasheets.avx.com/X7RDielectric.pdf" H 5850 3100 50  0001 C CNN
+F 4 "0402in/1005mm" H 250 850 50  0001 C CNN "Package ID"
+F 5 "AVX" H 250 850 50  0001 C CNN "Manufacturer"
+F 6 "04023C104JAT2A" H 250 850 50  0001 C CNN "Manufacturers Part Number"
+F 7 "CAP CER 0.1UF 25V X7R 0402" H 250 850 50  0001 C CNN "Characteristics"
 F 8 "MLCC Capacitor" H 250 850 50  0001 C CNN "Description"
 	1    5850 3100
@@
 F 0 "C116" H 5800 3050 50  0000 R CNN
 F 1 "100nF X7R" H 5900 3150 50  0000 R CNN
-F 2 "Capacitor_SMD:C_0603_1608Metric" H 5650 3100 50  0001 C CNN
-F 3 "https://content.kemet.com/datasheets/KEM_C1023_X7R_AUTO_SMD.pdf" H 5650 3100 50  0001 C CNN
-F 4 "0603in/1608mm" H 250 850 50  0001 C CNN "Package ID"
-F 5 "Kemet" H 250 850 50  0001 C CNN "Manufacturer"
-F 6 "C0603C104J3RACAUTO" H 250 850 50  0001 C CNN "Manufacturers Part Number"
-F 7 "CAP CER 0.1UF 25V X7R 0603" H 250 850 50  0001 C CNN "Characteristics"
+F 2 "Capacitor_SMD:C_0402_1005Metric" H 5650 3100 50  0001 C CNN
+F 3 "http://datasheets.avx.com/X7RDielectric.pdf" H 5650 3100 50  0001 C CNN
+F 4 "0402in/1005mm" H 250 850 50  0001 C CNN "Package ID"
+F 5 "AVX" H 250 850 50  0001 C CNN "Manufacturer"
+F 6 "04023C104JAT2A" H 250 850 50  0001 C CNN "Manufacturers Part Number"
+F 7 "CAP CER 0.1UF 25V X7R 0402" H 250 850 50  0001 C CNN "Characteristics"
 F 8 "MLCC Capacitor" H 250 850 50  0001 C CNN "Description"
 	1    5650 3100

Commit message: Updated footprints in order to add 3d models
Parts:
- U9: footprint Package_TO_SOT_SMD:TSOT-23-6 -> SW-Package-TO-SOT-SMD:TSOT-23-6
Changed lines of the file:
@@
 F 0 "U9" H 7000 1700 50  0000 C CNN
 F 1 "LTC4412" H 6750 2100 50  0000 C CNN
-F 2 "Package_TO_SOT_SMD:TSOT-23-6" H 6800 2200 50  0001 C CNN
+F 2 "SW-Package-TO-SOT-SMD:TSOT-23-6" H 6800 2200 50  0001 C CNN
 F 3 "https://www.analog.com/media/en/technical-documentation/data-sheets/4412fb.pdf" H 7350 2700 50  0001 C CNN
 F 4 "Linear Technologies" H 6800 1900 50  0001 C CNN "Manufacturer"

Commit message: s/Manufacturers Part Number/MPN/g
for compatability with MacroFab automated processing
Parts:
- C115, C116, C118: MPN (none) -> 04023C104JAT2A; Manufacturers Part Number 04023C104JAT2A -> (none)
- C117: MPN (none) -> C1206C106J3RACAUTO; Manufacturers Part Number C1206C106J3RACAUTO -> (none)
- FB2: MPN (none) -> BLM21AG601SZ1D; Manufacturers Part Number BLM21AG601SZ1D -> (none)
- Q2, Q3: MPN (none) -> CSD22206W; Manufacturers Part Number CSD22206W -> (none)
- U8: MPN (none) -> CDCE706; Manufacturers Part Number CDCE706 -> (none)
- U9: MPN (none) -> LTC4412HS6#TRMPBF; Manufacturers Part Number LTC4412HS6#TRMPBF -> (none)
- Y1: MPN (none) -> SiT1602BI-71-33E-48.000000; Manufacturers Part Number SiT1602BI-71-33E-48.000000 -> (none)
Changed lines of the file:
@@
 F 4 "0402in/1005mm" H 250 850 50  0001 C CNN "Package ID"
 F 5 "AVX" H 250 850 50  0001 C CNN "Manufacturer"
-F 6 "04023C104JAT2A" H 250 850 50  0001 C CNN "Manufacturers Part Number"
+F 6 "04023C104JAT2A" H 250 850 50  0001 C CNN "MPN"
 F 7 "CAP CER 0.1UF 25V X7R 0402" H 250 850 50  0001 C CNN "Characteristics"
 F 8 "MLCC Capacitor" H 250 850 50  0001 C CNN "Description"
@@
 F 4 "MEMS Oscillator" H 250 850 50  0001 C CNN "Description"
 F 5 "SI-Time" H 250 850 50  0001 C CNN "Manufacturer"
-F 6 "SiT1602BI-71-33E-48.000000" H 250 850 50  0001 C CNN "Manufacturers Part Number"
+F 6 "SiT1602BI-71-33E-48.000000" H 250 850 50  0001 C CNN "MPN"
 F 7 "Crystal 2016-4pim SMD" H 250 850 50  0001 C CNN "Package ID"
 	1    2600 3800
@@
 F 4 "Programmable Clock Generator" H 250 850 50  0001 C CNN "Description"
 F 5 "Texas Instruments" H 250 850 50  0001 C CNN "Manufacturer"
-F 6 "CDCE706" H 250 850 50  0001 C CNN "Manufacturers Part Number"
+F 6 "CDCE706" H 250 850 50  0001 C CNN "MPN"
 F 7 "TSSOP20" H 250 850 50  0001 C CNN "Package ID"
 	1    5350 3850
@@
 F 4 "0402in/1005mm" H 250 850 50  0001 C CNN "Package ID"
 F 5 "AVX" H 250 850 50  0001 C CNN "Manufacturer"
-F 6 "04023C104JAT2A" H 250 850 50  0001 C CNN "Manufacturers Part Number"
+F 6 "04023C104JAT2A" H 250 850 50  0001 C CNN "MPN"
 F 7 "CAP CER 0.1UF 25V X7R 0402" H 250 850 50  0001 C CNN "Characteristics"
 F 8 "MLCC Capacitor" H 250 850 50  0001 C CNN "Description"
@@
 F 4 "0402in/1005mm" H 250 850 50  0001 C CNN "Package ID"
 F 5 "AVX" H 250 850 50  0001 C CNN "Manufacturer"
-F 6 "04023C104JAT2A" H 250 850 50  0001 C CNN "Manufacturers Part Number"
+F 6 "04023C104JAT2A" H 250 850 50  0001 C CNN "MPN"
 F 7 "CAP CER 0.1UF 25V X7R 0402" H 250 850 50  0001 C CNN "Characteristics"
 F 8 "MLCC Capacitor" H 250 850 50  0001 C CNN "Description"
@@
 F 4 "Murata" H 5350 2800 50  0001 C CNN "Manufacturer"
 F 5 "0805in/2012mm" H 5350 2800 50  0001 C CNN "Package ID"
-F 6 "BLM21AG601SZ1D " H 5350 2800 50  0001 C CNN "Manufacturers Part Number"
+F 6 "BLM21AG601SZ1D " H 5350 2800 50  0001 C CNN "MPN"
 F 7 "600 Ohms @ 100MHz 1 Signal Line Ferrite Bead 0805 (2012 Metric) 700mA 210mOhm" H 250 850 50  0001 C CNN "Characteristics"
 F 8 "Ferrite Bead" H 250 850 50  0001 C CNN "Description"
@@
 F 3 "https://www.analog.com/media/en/technical-documentation/data-sheets/4412fb.pdf" H 7350 2700 50  0001 C CNN
 F 4 "Linear Technologies" H 6800 1900 50  0001 C CNN "Manufacturer"
-F 5 "LTC4412HS6#TRMPBF" H 6800 1900 50  0001 C CNN "Manufacturers Part Number"
+F 5 "LTC4412HS6#TRMPBF" H 6800 1900 50  0001 C CNN "MPN"
 F 6 "Ideal Diode Controller" H 250 850 50  0001 C CNN "Description"
 F 7 "SOT-23-6" H 250 850 50  0001 C CNN "Package ID"
@@
 F 4 "P Channel MOSFET" H 250 850 50  0001 C CNN "Description"
 F 5 "Texas Instruments" H 250 850 50  0001 C CNN "Manufacturer"
-F 6 "CSD22206W" H 250 850 50  0001 C CNN "Manufacturers Part Number"
+F 6 "CSD22206W" H 250 850 50  0001 C CNN "MPN"
 F 7 "DSBGA9" H 250 850 50  0001 C CNN "Package ID"
 	1    5450 2200
@@
 F 4 "P Channel MOSFET" H 250 850 50  0001 C CNN "Description"
 F 5 "Texas Instruments" H 250 850 50  0001 C CNN "Manufacturer"
-F 6 "CSD22206W" H 250 850 50  0001 C CNN "Manufacturers Part Number"
+F 6 "CSD22206W" H 250 850 50  0001 C CNN "MPN"
 F 7 "DSBGA9" H 250 850 50  0001 C CNN "Package ID"
 	1    6250 2350
@@
 F 3 "https://content.kemet.com/datasheets/KEM_C1023_X7R_AUTO_SMD.pdf" H 5850 2550 50  0001 C CNN
 F 4 "Kemet" H 250 850 50  0001 C CNN "Manufacturer"
-F 5 "C1206C106J3RACAUTO" H 250 850 50  0001 C CNN "Manufacturers Part Number"
+F 5 "C1206C106J3RACAUTO" H 250 850 50  0001 C CNN "MPN"
 F 6 "1206in/3216mm" H 250 850 50  0001 C CNN "Package ID"
 F 7 "CAP CER 10UF 25V X7R 1206" H 250 850 50  0001 C CNN "Characteristics"

Commit message: Updated annotation, since it seems to have gotten out of sync
Parts:
- renumbered C115 to C114, C116 to C115, C117 to C116, C118 to C117
Changed lines of the file:
@@
 EESchema Schematic File Version 4
 LIBS:edc-mux-board-fpga-main-cache
-EELAYER 29 0
+EELAYER 30 0
 EELAYER END
 $Descr USLetter 11000 8500
@@
 Do I need a separate Reset connection\nto the MCU so it can reset the clock chips\nindependantly?
 $Comp
-L power:GND #PWR036
+L power:GND #PWR035
 U 1 1 5CB6F7AE
 P 5350 4650
-F 0 "#PWR036" H 5350 4400 50  0001 C CNN
+F 0 "#PWR035" H 5350 4400 50  0001 C CNN
 F 1 "GND" H 5400 4450 50  0000 C CNN
 F 2 "" H 5350 4650 50  0001 C CNN
@@
 $EndComp
 $Comp
-L Device:C_Small C115
+L Device:C_Small C114
 U 1 1 5CB7C30C
 P 2850 3100
-F 0 "C115" V 2600 3100 50  0000 C CNN
+F 0 "C114" V 2600 3100 50  0000 C CNN
 F 1 "100nF X7R" V 2700 3100 50  0000 C CNN
 F 2 "Capacitor_SMD:C_0402_1005Metric" H 2850 3100 50  0001 C CNN
@@
 	2600 3100 2750 3100
 $Comp
-L power:GND #PWR032
+L power:GND #PWR031
 U 1 1 5CB7F01E
 P 2950 3250
-F 0 "#PWR032" H 2950 3000 50  0001 C CNN
+F 0 "#PWR031" H 2950 3000 50  0001 C CNN
 F 1 "GND" H 3000 3050 50  0000 C CNN
 F 2 "" H 2950 3250 50  0001 C CNN
@@
 $EndComp
 $Comp
-L power:GND #PWR031
+L power:GND #PWR030
 U 1 1 5CB809B1
 P 2600 4300
-F 0 "#PWR031" H 2600 4050 50  0001 C CNN
+F 0 "#PWR030" H 2600 4050 50  0001 C CNN
 F 1 "GND" H 2650 4100 50  0000 C CNN
 F 2 "" H 2600 4300 50  0001 C CNN
@@
 	3450 3900 3450 4000
 $Comp
-L power:GND #PWR033
+L power:GND #PWR032
 U 1 1 5CBADCB5
 P 3450 4400
-F 0 "#PWR033" H 3450 4150 50  0001 C CNN
+F 0 "#PWR032" H 3450 4150 50  0001 C CNN
 F 1 "GND" H 3500 4200 50  0000 C CNN
 F 2 "" H 3450 4400 50  0001 C CNN
@@
 $EndComp
 $Comp
-L power:GND #PWR034
+L power:GND #PWR033
 U 1 1 5CBB95F3
 P 3500 3500
-F 0 "#PWR034" H 3500 3250 50  0001 C CNN
+F 0 "#PWR033" H 3500 3250 50  0001 C CNN
 F 1 "GND" H 3550 3300 50  0000 C CNN
 F 2 "" H 3500 3500 50  0001 C CNN
@@
 	6350 3600 6550 3600
 $Comp
-L Device:C_Small C118
+L Device:C_Small C117
 U 1 1 5CBDE920
 P 5850 3100
-F 0 "C118" H 5750 3050 50  0000 R CNN
+F 0 "C117" H 5750 3050 50  0000 R CNN
 F 1 "100nF X7R" H 5750 3100 50  0000 R CNN
 F 2 "Capacitor_SMD:C_0402_1005Metric" H 5850 3100 50  0001 C CNN
@@
 $EndComp
 $Comp
-L Device:C_Small C116
+L Device:C_Small C115
 U 1 1 5CBE047E
 P 5650 3100
-F 0 "C116" H 5800 3050 50  0000 R CNN
+F 0 "C115" H 5800 3050 50  0000 R CNN
 F 1 "100nF X7R" H 5900 3150 50  0000 R CNN
 F 2 "Capacitor_SMD:C_0402_1005Metric" H 5650 3100 50  0001 C CNN
@@
 Connection ~ 5650 2950
 $Comp
-L power:GND #PWR037
+L power:GND #PWR036
 U 1 1 5CBE6F18
 P 5750 3250
-F 0 "#PWR037" H 5750 3000 50  0001 C CNN
+F 0 "#PWR036" H 5750 3000 50  0001 C CNN
 F 1 "GND" H 5800 3050 50  0000 C CNN
 F 2 "" H 5750 3250 50  0001 C CNN
@@
 P 5350 1900
 AR Path="/5CAA362B/5CC5E714" Ref="#PWR?"  Part="1"
-AR Path="/5CC3E5DC/5CC5E714" Ref="#PWR035"  Part="1"
-F 0 "#PWR035" H 5350 1750 50  0001 C CNN
+AR Path="/5CC3E5DC/5CC5E714" Ref="#PWR034"  Part="1"
+F 0 "#PWR034" H 5350 1750 50  0001 C CNN
 F 1 "+3.3V" H 5350 2040 50  0000 C CNN
 F 2 "" H 5350 1900 50  0001 C CNN
@@
 P 7200 1600
 AR Path="/5CAA362B/5CC5E726" Ref="#PWR?"  Part="1"
-AR Path="/5CC3E5DC/5CC5E726" Ref="#PWR038"  Part="1"
-F 0 "#PWR038" H 7200 1450 50  0001 C CNN
+AR Path="/5CC3E5DC/5CC5E726" Ref="#PWR037"  Part="1"
+F 0 "#PWR037" H 7200 1450 50  0001 C CNN
 F 1 "+3.3V" H 7200 1740 50  0000 C CNN
 F 2 "" H 7200 1600 50  0001 C CNN
@@
 P 7400 2850
 AR Path="/5CAA362B/5CC5E749" Ref="#PWR?"  Part="1"
-AR Path="/5CC3E5DC/5CC5E749" Ref="#PWR039"  Part="1"
-F 0 "#PWR039" H 7400 2600 50  0001 C CNN
+AR Path="/5CC3E5DC/5CC5E749" Ref="#PWR038"  Part="1"
+F 0 "#PWR038" H 7400 2600 50  0001 C CNN
 F 1 "GND" H 7400 2700 50  0000 C CNN
 F 2 "" H 7400 2850 50  0001 C CNN
@@
 P 5850 2550
 AR Path="/5CAA362B/5CC5E754" Ref="C?"  Part="1"
-AR Path="/5CC3E5DC/5CC5E754" Ref="C117"  Part="1"
-F 0 "C117" H 5950 2600 50  0000 L CNN
+AR Path="/5CC3E5DC/5CC5E754" Ref="C116"  Part="1"
+F 0 "C116" H 5950 2600 50  0000 L CNN
 F 1 "10uF X7R" H 5950 2550 50  0000 L CNN
 F 2 "Capacitor_SMD:C_1206_3216Metric" H 5850 2550 50  0001 C CNN

Commit message: Some minor fixes
- swapped 5Ω resistors to 4.99Ω resistors so I could actually buy them
- swapped power switch connector over to a JST PH connector like the rest of the connectors.
Parts:
- R10, R11, R12, R13, R14, R9: value 5Ω -> 4.99Ω 0.1%; Characteristics (none) -> RES SMD 4.99 OHM 0.1% 1/16W 0402; MPN (none) -> RT0402BRE074R99L; Manufacturer (none) -> Yageo
Changed lines of the file:
@@
 P 6250 3600
 F 0 "R9" V 6200 3450 50  0000 C CNN
-F 1 "5Ω" V 6200 3750 50  0000 C CNN
+F 1 "4.99Ω 0.1%" V 6200 3750 50  0000 C CNN
 F 2 "Resistor_SMD:R_0402_1005Metric" H 6250 3600 50  0001 C CNN
-F 3 "~" H 6250 3600 50  0001 C CNN
+F 3 "http://www.yageo.com/documents/recent/PYu-RT_1-to-0.01_RoHS_L_11.pdf" H 6250 3600 50  0001 C CNN
 F 4 "0402in/1005mm" H 250 850 50  0001 C CNN "Package ID"
 F 5 "Resistor" H 250 850 50  0001 C CNN "Description"
+F 6 "RES SMD 4.99 OHM 0.1% 1/16W 0402" H 6250 3600 50  0001 C CNN "Characteristics"
+F 7 "RT0402BRE074R99L" H 6250 3600 50  0001 C CNN "MPN"
+F 8 "Yageo" H 6250 3600 50  0001 C CNN "Manufacturer"
 	1    6250 3600
 	0    1    1    0
@@
 P 6250 3700
 F 0 "R10" V 6200 3550 50  0000 C CNN
-F 1 "5Ω" V 6200 3850 50  0000 C CNN
+F 1 "4.99Ω 0.1%" V 6200 3850 50  0000 C CNN
 F 2 "Resistor_SMD:R_0402_1005Metric" H 6250 3700 50  0001 C CNN
-F 3 "~" H 6250 3700 50  0001 C CNN
+F 3 "http://www.yageo.com/documents/recent/PYu-RT_1-to-0.01_RoHS_L_11.pdf" H 6250 3700 50  0001 C CNN
 F 4 "0402in/1005mm" H 250 850 50  0001 C CNN "Package ID"
 F 5 "Resistor" H 250 850 50  0001 C CNN "Description"
+F 6 "RES SMD 4.99 OHM 0.1% 1/16W 0402" H 6250 3700 50  0001 C CNN "Characteristics"
+F 7 "RT0402BRE074R99L" H 6250 3700 50  0001 C CNN "MPN"
+F 8 "Yageo" H 6250 3700 50  0001 C CNN "Manufacturer"
 	1    6250 3700
 	0    1    1    0
@@
 P 6250 3800
 F 0 "R11" V 6200 3650 50  0000 C CNN
-F 1 "5Ω" V 6200 3950 50  0000 C CNN
+F 1 "4.99Ω 0.1%" V 6200 3950 50  0000 C CNN
 F 2 "Resistor_SMD:R_0402_1005Metric" H 6250 3800 50  0001 C CNN
-F 3 "~" H 6250 3800 50  0001 C CNN
+F 3 "http://www.yageo.com/documents/recent/PYu-RT_1-to-0.01_RoHS_L_11.pdf" H 6250 3800 50  0001 C CNN
 F 4 "0402in/1005mm" H 250 850 50  0001 C CNN "Package ID"
 F 5 "Resistor" H 250 850 50  0001 C CNN "Description"
+F 6 "RES SMD 4.99 OHM 0.1% 1/16W 0402" H 6250 3800 50  0001 C CNN "Characteristics"
+F 7 "RT0402BRE074R99L" H 6250 3800 50  0001 C CNN "MPN"
+F 8 "Yageo" H 6250 3800 50  0001 C CNN "Manufacturer"
 	1    6250 3800
 	0    1    1    0
@@
 P 6250 3900
 F 0 "R12" V 6200 3750 50  0000 C CNN
-F 1 "5Ω" V 6200 4050 50  0000 C CNN
+F 1 "4.99Ω 0.1%" V 6200 4050 50  0000 C CNN
 F 2 "Resistor_SMD:R_0402_1005Metric" H 6250 3900 50  0001 C CNN
-F 3 "~" H 6250 3900 50  0001 C CNN
+F 3 "http://www.yageo.com/documents/recent/PYu-RT_1-to-0.01_RoHS_L_11.pdf" H 6250 3900 50  0001 C CNN
 F 4 "0402in/1005mm" H 250 850 50  0001 C CNN "Package ID"
 F 5 "Resistor" H 250 850 50  0001 C CNN "Description"
+F 6 "RES SMD 4.99 OHM 0.1% 1/16W 0402" H 6250 3900 50  0001 C CNN "Characteristics"
+F 7 "RT0402BRE074R99L" H 6250 3900 50  0001 C CNN "MPN"
+F 8 "Yageo" H 6250 3900 50  0001 C CNN "Manufacturer"
 	1    6250 3900
 	0    1    1    0
@@
 P 6250 4000
 F 0 "R13" V 6200 3850 50  0000 C CNN
-F 1 "5Ω" V 6200 4150 50  0000 C CNN
+F 1 "4.99Ω 0.1%" V 6200 4150 50  0000 C CNN
 F 2 "Resistor_SMD:R_0402_1005Metric" H 6250 4000 50  0001 C CNN
-F 3 "~" H 6250 4000 50  0001 C CNN
+F 3 "http://www.yageo.com/documents/recent/PYu-RT_1-to-0.01_RoHS_L_11.pdf" H 6250 4000 50  0001 C CNN
 F 4 "0402in/1005mm" H 250 850 50  0001 C CNN "Package ID"
 F 5 "Resistor" H 250 850 50  0001 C CNN "Description"
+F 6 "RES SMD 4.99 OHM 0.1% 1/16W 0402" H 6250 4000 50  0001 C CNN "Characteristics"
+F 7 "RT0402BRE074R99L" H 6250 4000 50  0001 C CNN "MPN"
+F 8 "Yageo" H 6250 4000 50  0001 C CNN "Manufacturer"
 	1    6250 4000
 	0    1    1    0
@@
 P 6250 4100
 F 0 "R14" V 6200 3950 50  0000 C CNN
-F 1 "5Ω" V 6200 4250 50  0000 C CNN
+F 1 "4.99Ω 0.1%" V 6200 4250 50  0000 C CNN
 F 2 "Resistor_SMD:R_0402_1005Metric" H 6250 4100 50  0001 C CNN
-F 3 "~" H 6250 4100 50  0001 C CNN
+F 3 "http://www.yageo.com/documents/recent/PYu-RT_1-to-0.01_RoHS_L_11.pdf" H 6250 4100 50  0001 C CNN
 F 4 "0402in/1005mm" H 250 850 50  0001 C CNN "Package ID"
 F 5 "Resistor" H 250 850 50  0001 C CNN "Description"
+F 6 "RES SMD 4.99 OHM 0.1% 1/16W 0402" H 6250 4100 50  0001 C CNN "Characteristics"
+F 7 "RT0402BRE074R99L" H 6250 4100 50  0001 C CNN "MPN"
+F 8 "Yageo" H 6250 4100 50  0001 C CNN "Manufacturer"
 	1    6250 4100
 	0    1    1    0
