File: edc-mux-board-fpga-main/clocks.sch (KiCad schematic (older format))
At the start: 25 parts, among them J2 OSC_PRG_HDR, Q2 CSD22206W, Q3 CSD22206W, U8 CDCE706, U9 LTC4412, Y1 SiT1602BI-71-33E-48.000000

Commit message: More minor changes
fixing part numbers and adding more notes
Parts:
- Y1: value SiT1602BI-71-33E-48.000000 -> SiT1602BI-72-33E-24.000000; MPN SiT1602BI-71-33E-48.000000 -> SiT1602BI-72-33E-24.000000
Other:
- note added: "Resistors for source termination of 50Ω\ntransmission lines per TI App Note:\nSCAA080A\n4.99Ω resistors are the closest you\ncan get in 0402"
- note added: "Y0 = 48MHz for FPGA\nY1 = 48MHz for CODECs\nY2 = 48MHz for CODECs\nY3 = 48MHz for Microprocessor\nY4 = 25MHz for W5500 Ethernet\n\nfout = Fin * (N/M)/P\n\nfor 25MHz: N=25, M=24, P=1\nfor 48MHz: N=2, M=1, P=1"
- note removed: "Do I need a separate Reset connection\nto the MCU so it can reset the clock chips\nindependantly?"
- note removed: "Resistors for source termination of 50Ω\ntransmission lines per TI App Note:\nSCAA080A"
- note removed: "Y0 = 48MHz for FPGA\nY1 = 48MHz for CODECs\nY2 = 48MHz for CODECs\nY3 = for Microprocessor\nY4 = 25MHz for W5500 Ethernet"
- moved on the sheet: R10, R11, R12, R13, R14, R9
